File: Dash/Dash.kicad_pcb (KiCad board)
At the start: 2 copper layers, 95.5 x 82.5 mm, 40 parts, among them CN1 NUCLEO-L432KC, J1 40 pin ZIF FPC Connector, J2 Nanofit Connector, U1 LF33_TO220, U2 LM7805_TO220, U3 BT817Q, U5 ISO1050DUB, U6 MCP2515-I/SO

Commit message: Dash PCB revision 1
Parts:
- added C21: 100 nF, Capacitor_SMD:C_0805_2012Metric, F.Cu at (133.0, 73.5)
- added U7: ~, Package_SO:SOIC-8_3.9x4.9mm_P1.27mm, F.Cu at (138.6, 75.5)
- D1: footprint Diode_SMD:D_0201_0603Metric -> FS_3_Global_Footprint_Library:US2H_TOS
- L1: footprint Inductor_SMD:L_1008_2520Metric -> Inductor_SMD:L_TDK_SLF7045
- moved C3 13.7 mm to (104.5, 113.0)
- moved C1 10.6 mm to (89.5, 112.0)
- moved C2 8.24 mm to (80.0, 109.0), turned to -90 degrees
- moved C4 7.57 mm to (95.5, 106.9), turned to -90 degrees
- moved D1 5.22 mm to (86.0, 88.9), turned to 90 degrees
- moved C18 5.22 mm to (121.0, 68.0), turned to 90 degrees
- moved U2 3.89 mm to (104.5, 107.0)
- moved C10 1.99 mm to (74.0, 91.8)
- moved C11 1.99 mm to (74.0, 88.8)
- moved L1 1.58 mm to (80.0, 90.5)
- moved C6 0.76 mm to (118.1, 69.0)
- moved C16 0.50 mm to (121.6, 71.0), turned to 180 degrees
Routing:
- net MEM-SCLK: track 0.00 -> 37.2 mm
- net MEM-MOSI: track 0.00 -> 34.2 mm
- net MEM-IO2: track 0.00 -> 24.2 mm
- net MEM-MISO: track 0.00 -> 23.3 mm
- net MEM-IO3: track 0.00 -> 21.4 mm
- net MEM-CS: track 0.00 -> 19.4 mm
- net +5V: track 96.4 -> 108.8 mm, vias 1 -> 2
- net GND: track 113.2 -> 121.8 mm, vias 16 -> 19
- net +3.3V: track 228.0 -> 222.1 mm, vias 8 -> 19
- net +12V: track 40.3 -> 46.0 mm
- net OV: track 28.5 -> 32.8 mm
- net Host-MISO: track 64.4 -> 65.7 mm
- net BL-High: track 29.6 -> 28.4 mm
- net VCC1.2: track 32.6 -> 31.5 mm
- net PD: track 32.8 -> 33.4 mm
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
Commit message: fixed ground plane of Dash PCB
Parts:
- moved C21 4.59 mm to (128.4, 73.5)
- moved U7 4.59 mm to (134.0, 75.5)
- moved C8 0.71 mm to (114.5, 85.0), turned to 0 degrees
- moved C7 0.63 mm to (107.5, 80.0), turned to 180 degrees
- turned C9 to 0 degrees
Routing:
- net MEM-MOSI: track 34.2 -> 28.9 mm
- net MEM-CS: track 19.4 -> 14.3 mm
- net MEM-SCLK: track 37.2 -> 32.1 mm
- net MEM-IO3: track 21.4 -> 16.4 mm
- net MEM-MISO: track 23.3 -> 18.4 mm
- net MEM-IO2: track 24.2 -> 19.5 mm
- net +3.3V: track 222.1 -> 219.7 mm
- net VCC1.2: track 31.5 -> 29.9 mm
- net R7: track 18.0 -> 17.2 mm
- net R6: track 18.3 -> 17.6 mm
- net R0: track 20.5 -> 19.9 mm
- net R4: track 18.7 -> 18.1 mm
- net R2: track 19.2 -> 18.6 mm
- net R5: track 18.5 -> 17.8 mm
- net R3: track 19.0 -> 18.3 mm
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
Commit message: Fix footprint of flash chip
Parts:
- U7: footprint Package_SO:SOIC-8_3.9x4.9mm_P1.27mm -> Package_SO:SOIC-8_5.23x5.23mm_P1.27mm
- moved R6 3.94 mm to (146.6, 126.0)
- moved C20 3.64 mm to (153.0, 127.0)
- moved D2 3.64 mm to (153.5, 124.0)
- moved R7 3.64 mm to (150.5, 124.0)
Routing:
- net GND: track 121.4 -> 116.2 mm
- net +3.3V: track 219.7 -> 214.7 mm, vias 19 -> 18
- net Net-(U6-*RESET): track 7.02 -> 3.15 mm
- net MEM-MISO: track 18.4 -> 19.6 mm
- net MEM-IO2: track 19.5 -> 20.6 mm
- net MEM-MOSI: track 28.9 -> 27.9 mm
- net MEM-SCLK: track 32.1 -> 32.9 mm
- net Host-MISO: track 65.7 -> 66.4 mm

Commit message: Added 9V linear regulator for nucleo power
Parts:
- added C22: 100 nF, Capacitor_SMD:C_0805_2012Metric, F.Cu at (114.0, 123.5)
- added C23: 100 nF, Capacitor_SMD:C_0805_2012Metric, F.Cu at (98.5, 124.0)
- added U8: LM7809_TO220, Package_TO_SOT_THT:TO-220-3_Vertical, F.Cu at (104.0, 121.9)
- moved C5 5.50 mm to (149.9, 119.0), turned to 0 degrees
Connections:
- C5 pad 2: +5V -> +9V
- CN1 pad CN4_1: unconnected-(CN1A-VIN-PadCN4_1) -> +9V
- CN1 pad CN4_4: +5V -> unconnected-(CN1A-5V-PadCN4_4)
Routing:
- net +5V: track 108.8 -> 54.0 mm, vias 2 -> 0
- net +9V: track 0.00 -> 48.3 mm, vias 0 -> 2
- net GND: track 116.2 -> 132.9 mm
- net +12V: track 46.0 -> 54.7 mm
- net VCC1.2: track 29.9 -> 33.2 mm
- net +3.3V: track 214.7 -> 217.6 mm

Commit message: Updated input capacitor value for 9V linear regulator on dash pcb
Parts:
- C23: value 100 nF -> 330 nF
Routing:
- net +3.3V: track 217.6 -> 217.5 mm, vias 18 -> 17
Changed lines of the file:
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@@
 			)
 		)
-		(property "Value" "100 nF"
+		(property "Value" "330 nF"
 			(at 0 1.68 90)
 			(layer "F.Fab")
@@
 		(tags "capacitor")
 		(property "Reference" "C5"
-			(at -0.05 2 360)
+			(at -0.05 2 0)
 			(layer "F.SilkS")
 			(effects
@@
 		)
 		(property "Value" "100 nF"
-			(at 0 1.68 360)
+			(at 0 1.68 0)
 			(layer "F.Fab")
 			(hide yes)
@@
 		)
 		(fp_text user "${REFERENCE}"
-			(at 0 0 360)
+			(at 0 0 0)
 			(layer "F.Fab")
 			(effects
@@
 	)
 	(segment
-		(start 131 92.737256)
-		(end 131 93)
-		(width 0.2)
-		(layer "F.Cu")
-		(net 27)
-	)
-	(segment
 		(start 119.5 136.05)
 		(end 119.5 134.5)
@@
 	)
 	(segment
+		(start 116.823032 79.025113)
+		(end 117.060704 79.262785)
+		(width 0.2)
+		(layer "F.Cu")
+		(net 27)
+	)
+	(segment
 		(start 146.525 122.475)
 		(end 147.863971 122.475)
@@
 	)
 	(segment
+		(start 117.525529 79.262785)
+		(end 130.762744 92.5)
+		(width 0.2)
+		(layer "F.Cu")
+		(net 27)
+	)
+	(segment
 		(start 119.490258 71.4)
 		(end 119.890258 71)
@@
 	)
 	(segment
-		(start 117.525529 79.262785)
-		(end 131 92.737256)
+		(start 119.5 136.05)
+		(end 128.45 136.05)
 		(width 0.2)
 		(layer "F.Cu")
@@
 	)
 	(segment
-		(start 119.5 136.05)
-		(end 128.45 136.05)
+		(start 114.350001 81.78173)
+		(end 114.350001 85.709744)
 		(width 0.2)
 		(layer "F.Cu")
@@
 	)
 	(segment
-		(start 114.350001 81.78173)
-		(end 114.350001 85.709744)
+		(start 130.762744 92.5)
+		(end 131.303552 92.5)
 		(width 0.2)
 		(layer "F.Cu")
@@
 	)
 	(segment
-		(start 117.060704 79.262785)
-		(end 117.525529 79.262785)
-		(width 0.2)
-		(layer "F.Cu")
-		(net 27)
-	)
-	(segment
 		(start 150.5 123.0875)
 		(end 152.5 121.0875)
@@
 	)
 	(segment
-		(start 116.823032 79.025113)
-		(end 117.060704 79.262785)
-		(width 0.2)
-		(layer "F.Cu")
-		(net 27)
-	)
-	(segment
-		(start 131.803552 93)
-		(end 132.376776 93.573224)
-		(width 0.2)
-		(layer "F.Cu")
-		(net 27)
-	)
-	(segment
 		(start 149.5 122.0875)
 		(end 150.5 123.0875)
@@
 	)
 	(segment
+		(start 116.823032 78.741574)
+		(end 116.823032 79.025113)
+		(width 0.2)
+		(layer "F.Cu")
+		(net 27)
+	)
+	(segment
 		(start 117.116416 78.44819)
 		(end 117.116416 77.762863)
@@
 	)
 	(segment
+		(start 117.060704 79.262785)
+		(end 117.525529 79.262785)
+		(width 0.2)
+		(layer "F.Cu")
+		(net 27)
+	)
+	(segment
 		(start 134.0875 94.733947)
 		(end 134.0875 96.5)
@@
 	)
 	(segment
-		(start 131 93)
-		(end 131.803552 93)
+		(start 119.5 132.835)
+		(end 119.475 132.81)
 		(width 0.2)
 		(layer "F.Cu")
@@
 	)
 	(segment
-		(start 119.5 132.835)
-		(end 119.475 132.81)
+		(start 131.303552 92.5)
+		(end 132.376776 93.573224)
 		(width 0.2)
 		(layer "F.Cu")
@@
 	)
 	(segment
-		(start 116.823032 78.741574)
-		(end 116.823032 79.025113)
-		(width 0.2)
-		(layer "F.Cu")
-		(net 27)
-	)
-	(segment
 		(start 152.5 115.33)
 		(end 138.995 101.825)
@@
 		(size 0.6)
 		(drill 0.3)
-		(layers "F.Cu" "B.Cu")
-		(net 27)
-	)
-	(via
-		(at 131 93)
-		(size 0.6)
-		(drill 0.3)
