File: Dash/Dash.kicad_sch (KiCad schematic)
At the start: 16 parts, among them CN1 NUCLEO-L432KC, J1 40 pin ZIF FPC Connector, U1 LF33_TO220, U2 LM341T-12_TO220, U3 BT817Q

Commit message: Dash schematic initial revision
Parts:
- removed U2: LM341T-12_TO220, Package_TO_SOT_THT:TO-220-3_Vertical, symbol Regulator_Linear:LM341T-12_TO220
- added C12, C13: 1 µF, symbol Device:C
- added D1: 470 mV @ 2A Forward / 40V 2A Reverse, symbol Device:D_Schottky
- added JP1: Open, symbol Jumper:SolderJumper_2_Open
- added L1: 4.7 µH, symbol Device:L
- added R1: 33K ±1%, symbol Device:R_US
- added R2: 100K ±1%, symbol Device:R_US
- added R3: 4.99 ±1%, symbol Device:R_US
- added R4: 2.49 ±1%, symbol Device:R_US
- added R5: 4.7k, symbol Device:R_US
- added U2: LM7805_TO220, Package_TO_SOT_THT:TO-220-3_Vertical, symbol Regulator_Linear:LM7805_TO220
- added U4: ~, Package_TO_SOT_SMD:SOT-23-6_Handsoldering, symbol FS_3_Global_Symbol_Library:AP3032KTR-G1
- C3: value 0.33 µF -> 330 nF
- C4: value 0.1 µF -> 100 nF
Connections:
- net +12V: now also U2.1 (VI); no longer C10.1, C11.1, C4.1, C5.1, CN1.CN4_1 (VIN)
- net +3.3V: now also R5.1; no longer U3.12 (PD_N)
- net GND: now also C5.1, C9.2, C12.2, C13.2, R2.2, R3.1, R4.1, U2.2 (GND), U4.2 (GND); no longer C5.2, C9.1
- net VCC1.2: now also C9.1; no longer C9.2
- net BL-Low: now reaches J1.1 (Pin_1)
- net BL-Low: now also JP1.2 (B), R3.2, U4.3 (FB)
- net BL-High: now reaches J1.2 (Pin_2)
- net BL-High: now also C12.1, C13.1, D1.1 (K), R1.1
- net INT: now reaches U3.11 (INT_N)
- net INT: now also CN1.CN3_2 (PA10), R5.2
- net MEM-SCLK: now reaches U3.14 (SPIM_SCLK)
- net MEM-CS: now reaches U3.15 (SPIM_SS_N)
- net MEM-MOSI: now reaches U3.16 (SPIM_MOSI)
- net MEM-MISO: now reaches U3.18 (SPIM_MISO)
- net MEM-IO2: now reaches U3.19 (SPIM_IO2)
- net MEM-IO3: now reaches U3.20 (SPIM_IO3)
- net Host-SCLK: now reaches U3.3 (SCK)
- net Host-SCLK: now also CN1.CN4_15 (PB3)
- net Host-MISO: now reaches U3.4 (MISO)
- net Host-MISO: now also CN1.CN3_15 (PB4)
- net Host-MOSI: now reaches U3.5 (MOSI)
- net Host-MOSI: now also CN1.CN3_14 (PB5)
- net Host-CS: now reaches U3.6 (CS_N)
- net Host-CS: now also CN1.CN3_1 (PA9)
- net PD: now reaches CN1.CN3_6 (PB0)
- net PD: now also U3.12 (PD_N)
- net +5V: now reaches CN1.CN4_4 (5V)
- net +5V: now also C10.1, C11.1, C4.1, C5.2, L1.1, U2.3 (VO), U4.6 (VIN)
- net BL_PWM renamed BL-PWM
- net BL-PWM: now also U4.4 (CTRL)
- new net: D1.2 (A), L1.2, U4.1 (SW)
- new net: JP1.1 (A), R4.2
- new net OV: R1.2, R2.1, U4.5 (OV)
- no-connect marks 14 -> 37
Other:
- moved on the sheet: C10, C11, C5, C6, C7, C8, C9, CN1A, U3

Commit message: dash PCB work
Parts:
- added C14, C15, C16, C17, C18, C19: 100nF, Capacitor_SMD:C_0805_2012Metric, symbol Device:C
- added C20: 2 µF, Capacitor_SMD:C_0805_2012Metric, symbol Device:C
- added D2: D, Diode_SMD:D_0805_2012Metric, symbol Device:D
- added J2: Nanofit Connector, Connector_Molex:Molex_Nano-Fit_105310-xx04_2x02_P2.50mm_Vertical, symbol Connector:Conn_01x04_Pin
- added R6: 10K, Resistor_SMD:R_0805_2012Metric, symbol Device:R_US
- added R7: 1 Ω, Resistor_SMD:R_0805_2012Metric, symbol Device:R_US
- added U5: ISO1050DUB, Package_SO:SOP-8_6.62x9.15mm_P2.54mm, symbol Interface_CAN_LIN:ISO1050DUB
- added U6: MCP2515-I/SO, Package_SO:SOIC-18W_7.5x11.6mm_P1.27mm, symbol FS_3_Global_Symbol_Library:MCP2515-I_SO
- C1, C10, C11, C12, C13, C2, C3, C4, C5, C6, C7, C8, C9: footprint (none) -> Capacitor_SMD:C_0805_2012Metric
- D1: footprint (none) -> Diode_SMD:D_0201_0603Metric
- J1: footprint (none) -> Connector_FFC-FPC:TE_4-1734839-0_1x40-1MP_P0.5mm_Horizontal; symbol Connector:Conn_01x40_Pin -> Connector_Generic_MountingPin:Conn_01x40_MountingPin
- JP1: footprint (none) -> Jumper:SolderJumper-2_P1.3mm_Open_RoundedPad1.0x1.5mm
- L1: footprint (none) -> Inductor_SMD:L_1008_2520Metric
- R1, R2, R3, R4, R5: footprint (none) -> Resistor_SMD:R_0805_2012Metric
Connections:
- net +12V: now also J2.4 (Pin_4)
- net +3.3V: now also C14.2, C15.2, C16.2, C17.2, C18.2, C19.2, D2.1 (K), R7.1, U5.1 (VCC1), U5.8 (VCC2), U6.18 (VDD); no longer U3.27 (VCCA)
- net GND: now also C14.1, C15.1, C16.1, C17.1, C18.1, C19.1, C20.2, J2.3 (Pin_3), U5.4 (GND1), U5.5 (GND2), U6.9 (VSS)
- net Host-CS: now also CN1.CN3_12 (PA8); no longer CN1.CN3_1 (PA9)
- net Host-MISO: now also U6.15 (SO)
- net Host-MOSI: now also U6.14 (SI)
- net Host-SCLK: now also U6.13 (SCK)
- net INT: now also CN1.CN3_7 (PB7); no longer CN1.CN3_2 (PA10)
- net CAN-CS: now reaches CN1.CN3_13 (PA11)
- net CAN-CS: now also U6.16 (*CS)
- new net: C20.1, D2.2 (A), R6.2, R7.2
- new net: R6.1, U6.17 (*RESET)
- new net CAN-H: J2.1 (Pin_1), U5.7 (CANH)
- new net CAN-L: J2.2 (Pin_2), U5.6 (CANL)
- new net CAN-RX: U5.2 (RXD), U6.2 (RXCAN)
- new net CAN-TX: U5.3 (TXD), U6.1 (TXCAN)
- no-connect marks 37 -> 47
Other:
- moved on the sheet: C10, C11, C12, C13, C6, D1, JP1, L1, R1, R2, R3, R4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

Commit message: Dash PCB revision 1
Parts:
- added C21: 100 nF, symbol Device:C
- added U7: ~, symbol FS_3_Global_Symbol_Library:W25Q40CLSNIG_TR
- D1: footprint Diode_SMD:D_0201_0603Metric -> FS_3_Global_Footprint_Library:US2H_TOS
- L1: footprint Inductor_SMD:L_1008_2520Metric -> Inductor_SMD:L_TDK_SLF7045
Connections:
- net +3.3V: now also C21.2, U7.8 (VCC)
- net GND: now also C21.1, U7.4 (GND)
- net MEM-CS: now also U7.1 (CS)
- net MEM-IO2: now also U7.3 (WP)
- net MEM-IO3: now also U7.7 (Hold)
- net MEM-MISO: now also U7.2 (DO)
- net MEM-MOSI: now also U7.5 (DI)
- net MEM-SCLK: now also U7.6 (CLK)

Commit message: fixed footprints for Dash
Parts:
- C21: footprint (none) -> Capacitor_SMD:C_0805_2012Metric
- U7: footprint (none) -> Package_SO:SOIC-8_3.9x4.9mm_P1.27mm
Changed lines of the file:
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@@
 			)
 		)
-		(property "Footprint" ""
+		(property "Footprint" "Capacitor_SMD:C_0805_2012Metric"
 			(at 230.8352 50.8 0)
 			(effects
@@
 			)
 		)
-		(property "Footprint" ""
+		(property "Footprint" "Package_SO:SOIC-8_3.9x4.9mm_P1.27mm"
 			(at 210.82 50.8 0)
 			(effects

Commit message: Fix footprint of flash chip
Parts:
- U7: footprint Package_SO:SOIC-8_3.9x4.9mm_P1.27mm -> Package_SO:SOIC-8_5.23x5.23mm_P1.27mm
Changed lines of the file:
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@@
 			)
 		)
-		(property "Footprint" "Package_SO:SOIC-8_3.9x4.9mm_P1.27mm"
+		(property "Footprint" "Package_SO:SOIC-8_5.23x5.23mm_P1.27mm"
 			(at 210.82 50.8 0)
 			(effects

Commit message: Added 9V linear regulator for nucleo power
Parts:
- added C22, C23: 100 nF, Capacitor_SMD:C_0805_2012Metric, symbol Device:C
- added U8: LM7809_TO220, Package_TO_SOT_THT:TO-220-3_Vertical, symbol Regulator_Linear:LM7809_TO220
Connections:
- net +12V: now also C23.1, U8.1 (VI)
- net +5V: no longer C5.2, CN1.CN4_4 (5V)
- net GND: now also C22.2, C23.2, U8.2 (GND)
- net +9V: now reaches CN1.CN4_1 (VIN)
- net +9V: now also C5.2, C22.1, U8.3 (VO)
Other:
- moved on the sheet: C5

Commit message: Updated input capacitor value for 9V linear regulator on dash pcb
Parts:
- C23: value 100 nF -> 330 nF
Changed lines of the file:
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@@
 			)
 		)
-		(property "Value" "100 nF"
+		(property "Value" "330 nF"
 			(at 13.716 74.422 0)
 			(effects

Commit message: Updated ribbon cable footprint and added pcb text to Dash board
Parts:
- J1: footprint Connector_FFC-FPC:TE_4-1734839-0_1x40-1MP_P0.5mm_Horizontal -> FS_3_Global_Footprint_Library:CONN_F32D-1A7Y1-21040_AMP; symbol Connector_Generic_MountingPin:Conn_01x40_MountingPin -> Connector_Generic:Conn_01x42
Connections:
- no-connect marks 47 -> 48
