File: Telemetry Upright Hall Effect Breakout Board/Telemetry Upright Hall Effect Breakout Board.kicad_sch (KiCad schematic)
At the start: 2 parts, among them J1 Hall Effect Breakout, J2 Molex Nanofit 1x3

Commit message: Added name and stuff
Parts:
- J1: footprint (none) -> FS_3_Global_Footprint_Library:ATS668LSMTN-T
Changed lines of the file:
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@@
 			)
 		)
-		(property "Footprint" ""
+		(property "Footprint" "FS_3_Global_Footprint_Library:ATS668LSMTN-T"
 			(at 77.47 68.58 0)
 			(effects
