File: Telemetry Main Board/Telemetry Main Board.kicad_sch (KiCad schematic)
At the start: 19 parts, among them J1 776180-1, U3 CD74HC4067SM96, U4 ISO1050DUB, U5 NUCLEO-L432KC, U7 MCP2515-I/SO, U8 ISO1050DUB, U9 MCP2515-I/SO

Commit message: Added SD to SPI board and generated temp PCB
Parts:
- added C13: 100nf, Capacitor_SMD:C_0805_2012Metric_Pad1.18x1.45mm_HandSolder, symbol Device:C
- added J2: Conn_01x09_Pin, Connector_PinHeader_2.54mm:PinHeader_1x09_P2.54mm_Vertical, symbol Connector:Conn_01x09_Pin
- J1: footprint 1FS_2_Global_Footprint_Library:TE_776180-1 -> Connector_PinHeader_1.00mm:PinHeader_1x35_P1.00mm_Horizontal
- U5: footprint 1FS_2_Global_Footprint_Library:MODULE_NUCLEO-L432KC -> FS_3_Global_Footprint_Library:NUCLEO-L432KC
Connections:
- net +3.3V is gone; now on net +3V3: C11.1, C12.1, U7.18 (VDD), U9.18 (VDD)
- net +3V3: now also C13.1, J2.1 (Pin_1)
- net GND: now also C13.2, J2.2 (Pin_2)
- net SPI3_MISO: now also J2.4 (Pin_4)
- net SPI3_MOSI: now also J2.5 (Pin_5)
- net SPI3_SCLK: now also J2.3 (Pin_3)
- net SPI3_SSEL1: now also U5.CN4_6 (PA7); no longer U5.CN3_1 (PA9)
- net SPI3_SSEL2: now also U5.CN4_7 (PA6); no longer U5.CN3_2 (PA10)
- net SPI3_SSEL3: now reaches U5.CN4_8 (PA5)
- net SPI3_SSEL3: now also J2.6 (Pin_6)
- net SD Card Detect T/F: now reaches U3.2 (I7)
- net SD Card Detect T/F: now also J2.9 (Pin_9)
- no-connect marks 18 -> 17

Commit message: Update Telemetry Main Board.kicad_sch
Parts:
- removed J1: 776180-1, Connector_PinHeader_1.00mm:PinHeader_1x35_P1.00mm_Horizontal, symbol 1FS_2_Global_Symbol_Library:776180-1
- added J3: Conn_01x23_Pin, FS_3_Global_Footprint_Library:CONN23_776087_TEC, symbol Connector:Conn_01x23_Pin
Connections:
- net +12V: now also J3.2 (Pin_2)
- net +3V3: now also J3.12 (Pin_12)
- net Acc Exhaust Temp: now also J3.17 (Pin_17)
- net Acc Intake Flow Rate: now also J3.19 (Pin_19)
- net Acc Intake Pressure: now also J3.18 (Pin_18)
- net Acc Intake Temp: now also J3.16 (Pin_16)
- net Brake Sensor B: now also J3.15 (Pin_15)
- net Brake Sensor F: now also J3.14 (Pin_14)
- net CAN1_H: now also J3.3 (Pin_3), J3.4 (Pin_4)
- net CAN1_L: now also J3.7 (Pin_7), J3.8 (Pin_8)
- net CAN2_H: now also J3.5 (Pin_5), J3.6 (Pin_6)
- net CAN2_L: now also J3.10 (Pin_10), J3.9 (Pin_9)
- net GND: now also J3.1 (Pin_1), J3.11 (Pin_11)
- net Steering Sensor: now also J3.13 (Pin_13)
- no-connect marks 17 -> 21
Other:
- note added: "23 pin connector"
- note removed: "35 pin connector"

Commit message: put SD card on molex, split 23 pin connector into 2 ATM connectors (8 pin and 12 pin)
Parts:
- removed J2: Conn_01x09_Pin, Connector_PinHeader_2.54mm:PinHeader_1x09_P2.54mm_Vertical, symbol Connector:Conn_01x09_Pin
- removed J3: Conn_01x23_Pin, FS_3_Global_Footprint_Library:CONN23_776087_TEC, symbol Connector:Conn_01x23_Pin
- added J1: 8 pin ATM connector, symbol Connector:Conn_01x08_Pin
- added J3: 12 pin ATM connector, symbol Connector:Conn_01x12_Pin
- added J4: SD to SPI (Molex nanofit), Connector_Molex:Molex_Nano-Fit_105310-xx10_2x05_P2.50mm_Vertical, symbol Connector_Generic:Conn_2Rows-09Pins
Connections:
- net +12V: now also J3.2 (Pin_2)
- net +3V3: now also J3.3 (Pin_3), J4.1 (Pin_1)
- net Acc Exhaust Temp: now also J3.8 (Pin_8)
- net Acc Intake Flow Rate: now also J3.10 (Pin_10)
- net Acc Intake Pressure: now also J3.9 (Pin_9)
- net Acc Intake Temp: now also J3.7 (Pin_7)
- net Brake Sensor B: now also J3.6 (Pin_6)
- net Brake Sensor F: now also J3.5 (Pin_5)
- net CAN1_H: now also J1.1 (Pin_1), J1.2 (Pin_2)
- net CAN1_L: now also J1.5 (Pin_5), J1.6 (Pin_6)
- net CAN2_H: now also J1.3 (Pin_3), J1.4 (Pin_4)
- net CAN2_L: now also J1.7 (Pin_7), J1.8 (Pin_8)
- net GND: now also J3.1 (Pin_1), J4.2 (Pin_2)
- net SD Card Detect T/F: now also J4.9 (Pin_9)
- net SPI3_MISO: now also J4.4 (Pin_4)
- net SPI3_MOSI: now also J4.5 (Pin_5)
- net SPI3_SCLK: now also J4.3 (Pin_3)
- net SPI3_SSEL3: now also J4.6 (Pin_6)
- net Steering Sensor: now also J3.4 (Pin_4)
- no-connect marks 21 -> 17
Other:
- note removed: "23 pin connector"

Commit message: Added changes after 11/10 meeting
Parts:
- removed R1, R3: 10k, Resistor_SMD:R_0805_2012Metric_Pad1.20x1.40mm_HandSolder, symbol Device:R_US
- removed R2, R4: 20k, Resistor_SMD:R_0805_2012Metric_Pad1.20x1.40mm_HandSolder, symbol Device:R_US
- added C14: 100nf, Capacitor_SMD:C_0805_2012Metric_Pad1.18x1.45mm_HandSolder, symbol Device:C
- added R5, R7: 10k, Resistor_SMD:R_0805_2012Metric_Pad1.20x1.40mm_HandSolder, symbol Device:R_US
- added R6, R8: 20k, Resistor_SMD:R_0805_2012Metric_Pad1.20x1.40mm_HandSolder, symbol Device:R_US
- added U6: MCP6004, symbol Amplifier_Operational:MCP6004
Connections:
- net +5V: now also C14.1, U6.4 (V+)
- net Brake Sensor B: now also U6.5 (+)
- net Brake Sensor F: now also U6.3 (+)
- net Brake Sensor F 3V3: now also R7.2, R8.2
- net Brake Sensor R 3V3: now also R5.2, R6.2
- net GND: now also C14.2, R6.1, R8.1, U6.11 (V-)
- new net: R5.1, U6.6 (-), U6.7
- new net: R7.1, U6.1, U6.2 (-)
- no-connect marks 17 -> 54

Commit message: Added changes from during and after 11-10-24 work meeting
Parts:
- removed U3: CD74HC4067SM96, Package_SO:SSOP-24_5.3x8.2mm_P0.65mm, symbol 1FS_2_Global_Symbol_Library:CD74HC4067SM96
- removed U7: MCP2515-I/SO, Package_SO:SOIC-18W_7.5x11.6mm_P1.27mm, symbol FS_3_Global_Symbol_Library:MCP2515-I_SO
- added C15, C16: 100nf, Capacitor_SMD:C_0805_2012Metric_Pad1.18x1.45mm_HandSolder, symbol Device:C
- added D1, D2: CD4148W, Diode_SMD:D_0805_2012Metric, symbol Diode:CD4148W
- added R10, R3, R4, R9: 10k, Resistor_SMD:R_0805_2012Metric_Pad1.20x1.40mm_HandSolder, symbol Device:R_US
- added U10: MCP2515-I/SO, Package_SO:SOIC-18W_7.5x11.6mm_P1.27mm, symbol FS_3_Global_Symbol_Library:MCP2515-I_SO
- added U7: ~, Package_SO:SSOP-24_5.3x8.2mm_P0.65mm, symbol FS_3_Global_Symbol_Library:CD74HC4067SM96
Connections:
- net +3V3: now also C15.1, D1.1 (K), D2.1 (K), R10.2, R4.2, U10.18 (VDD); no longer C11.1
- net +5V: now also C11.1, U7.24 (Vcc); no longer C5.1
- net ADC: now also U7.1 (Common)
- net Acc Exhaust Temp: now also U7.5 (I4)
- net Acc Intake Flow Rate: now also U7.3 (I6)
- net Acc Intake Pressure: now also U7.4 (I5)
- net Acc Intake Temp: now also U7.6 (I3)
- net Brake Sensor F 3V3: now also U7.7 (I2)
- net Brake Sensor R 3V3: now also U7.8 (I1)
- net CAN1_RX: now also U10.2 (RXCAN); no longer U9.2 (RXCAN)
- net CAN1_TX: now also U10.1 (TXCAN); no longer U9.1 (TXCAN)
- net CAN2_RX: now also U9.2 (RXCAN)
- net CAN2_TX: now also U9.1 (TXCAN)
- net GND: now also C15.2, C16.2, U10.9 (VSS), U7.12 (GND), U7.15 (E)
- net S1: now also U7.10 (S0)
- net S2: now also U7.11 (S1)
- net S3: now also U7.14 (S2)
- net S4: now also U7.13 (S3)
- net SD Card Detect T/F: now also U7.2 (I7)
- net SPI3_MISO: now also U10.15 (SO)
- net SPI3_MOSI: now also U10.14 (SI)
- net SPI3_SCLK: now also U10.13 (SCK)
- net SPI3_SSEL1: now also U10.16 (*CS); no longer U9.16 (*CS)
- net SPI3_SSEL2: now also U9.16 (*CS)
- net Steering Sensor: now also U6.10 (+)
- net at U9.17 (*RESET): now also R3.1
- net Steering Sensor 3V3: now reaches U6.8
- net Steering Sensor 3V3: now also U6.9 (-), U7.9 (I0)
- new net: C5.1, D1.2 (A), R3.2, R4.1
- new net: R9.1, U10.17 (*RESET)
- new net: C16.1, D2.2 (A), R10.1, R9.2
- no-connect marks 54 -> 49
Other:
- moved on the sheet: C14, R5, R6, R7, R8, U6A, U6B, U6C, U6D, U6E

Commit message: Updated main PCB board
Updated PCB board to 1.8. Made it more compact
Parts:
- U6: footprint (none) -> FS_3_Global_Footprint_Library:PDIP14_300MC_MCH
Changed lines of the file:
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@@
 			)
 		)
-		(property "Footprint" ""
+		(property "Footprint" "FS_3_Global_Footprint_Library:PDIP14_300MC_MCH"
 			(at 41.91 147.32 0)
 			(effects
@@
 			)
 		)
-		(property "Footprint" ""
+		(property "Footprint" "FS_3_Global_Footprint_Library:PDIP14_300MC_MCH"
 			(at 41.91 170.18 0)
 			(effects
@@
 			)
 		)
-		(property "Footprint" ""
+		(property "Footprint" "FS_3_Global_Footprint_Library:PDIP14_300MC_MCH"
 			(at 73.66 187.96 0)
 			(effects
@@
 			)
 		)
-		(property "Footprint" ""
+		(property "Footprint" "FS_3_Global_Footprint_Library:PDIP14_300MC_MCH"
 			(at 41.91 123.19 0)
 			(effects
@@
 			)
 		)
-		(property "Footprint" ""
+		(property "Footprint" "FS_3_Global_Footprint_Library:PDIP14_300MC_MCH"
 			(at 35.56 195.58 0)
 			(effects

Commit message: Updated resistor values for CAN over SPI reset circuit
Parts:
- C16, C5: value 100nf -> 2 μf
- R10, R4: value 10k -> 1 Ω
Changed lines of the file:
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@@
 	)
 	(junction
+		(at 259.08 139.7)
+		(diameter 0)
+		(color 0 0 0 0)
+	)
+	(junction
 		(at 50.8 125.73)
 		(diameter 0)
@@
 	)
 	(junction
+		(at 260.35 96.52)
+		(diameter 0)
+		(color 0 0 0 0)
+	)
+	(junction
 		(at 58.42 149.86)
 		(diameter 0)
@@
 	(wire
 		(pts
+			(xy 246.38 88.9) (xy 246.38 86.36)
+		)
+		(stroke
+			(width 0)
+			(type default)
+		)
+	)
+	(wire
+		(pts
 			(xy 116.84 50.8) (xy 120.65 50.8)
 		)
@@
 	(wire
 		(pts
+			(xy 260.35 86.36) (xy 260.35 96.52)
+		)
+		(stroke
+			(width 0)
+			(type default)
+		)
+	)
+	(wire
+		(pts
 			(xy 114.3 88.9) (xy 119.38 88.9)
 		)
@@
 	(wire
 		(pts
+			(xy 259.08 129.54) (xy 259.08 139.7)
+		)
+		(stroke
+			(width 0)
+			(type default)
+		)
+	)
+	(wire
+		(pts
 			(xy 90.17 93.98) (xy 93.98 93.98)
 		)
@@
 	(wire
 		(pts
+			(xy 246.38 86.36) (xy 260.35 86.36)
+		)
+		(stroke
+			(width 0)
+			(type default)
+		)
+	)
+	(wire
+		(pts
 			(xy 116.84 100.33) (xy 120.65 100.33)
 		)
@@
 	(wire
 		(pts
+			(xy 260.35 96.52) (xy 259.08 96.52)
+		)
+		(stroke
+			(width 0)
+			(type default)
+		)
+	)
+	(wire
+		(pts
 			(xy 114.3 91.44) (xy 116.84 91.44)
 		)
@@
 	(wire
 		(pts
+			(xy 259.08 139.7) (xy 257.81 139.7)
+		)
+		(stroke
+			(width 0)
+			(type default)
+		)
+	)
+	(wire
+		(pts
+			(xy 245.11 129.54) (xy 259.08 129.54)
+		)
+		(stroke
+			(width 0)
+			(type default)
+		)
+	)
+	(wire
+		(pts
 			(xy 114.3 55.88) (xy 116.84 55.88)
 		)
@@
 	(wire
 		(pts
+			(xy 260.35 139.7) (xy 259.08 139.7)
+		)
+		(stroke
+			(width 0)
+			(type default)
+		)
+	)
+	(wire
+		(pts
 			(xy 83.82 77.47) (xy 83.82 82.55)
 		)
@@
 	(wire
 		(pts
+			(xy 245.11 132.08) (xy 245.11 129.54)
+		)
+		(stroke
+			(width 0)
+			(type default)
+		)
+	)
+	(wire
+		(pts
 			(xy 76.2 77.47) (xy 76.2 99.06)
 		)
@@
 	(wire
 		(pts
+			(xy 261.62 96.52) (xy 260.35 96.52)
+		)
+		(stroke
+			(width 0)
+			(type default)
+		)
+	)
+	(wire
+		(pts
 			(xy 64.77 149.86) (xy 58.42 149.86)
 		)
@@
 			)
 		)
-		(property "Value" "10k"
+		(property "Value" "1 Ω"
 			(at 248.412 134.874 0)
 			(effects
@@
 	(symbol
 		(lib_id "power:+5V")
-		(at 259.08 96.52 270)
+		(at 261.62 96.52 270)
 		(unit 1)
 		(exclude_from_sim no)
@@
 		(fields_autoplaced yes)
 		(property "Reference" "#PWR054"
-			(at 255.27 96.52 0)
+			(at 257.81 96.52 0)
 			(effects
 				(font
@@
 		)
 		(property "Value" "+3V3"
-			(at 262.89 96.5199 90)
+			(at 265.43 96.5199 90)
 			(effects
 				(font
@@
 		)
 		(property "Footprint" ""
-			(at 259.08 96.52 0)
+			(at 261.62 96.52 0)
 			(effects
 				(font
@@
 		)
 		(property "Datasheet" ""
-			(at 259.08 96.52 0)
+			(at 261.62 96.52 0)
 			(effects
 				(font
@@
 		)
 		(property "Description" ""
-			(at 259.08 96.52 0)
+			(at 261.62 96.52 0)
 			(effects
 				(font
@@
 			)
 		)
-		(property "Value" "100nf"
+		(property "Value" "2 μf"
 			(at 240.03 145.542 0)
 			(effects
@@
 	)
 	(symbol
-		(lib_id "power:+5V")
-		(at 245.11 132.08 0)
-		(unit 1)
-		(exclude_from_sim no)
-		(in_bom yes)
-		(on_board yes)
-		(dnp no)
-		(fields_autoplaced yes)
-		(property "Reference" "#PWR022"
-			(at 245.11 135.89 0)
-			(effects
-				(font
-					(size 1.27 1.27)
-				)
-				(hide yes)
-			)
-		)
-		(property "Value" "+3V3"
-			(at 245.11 127 0)
-			(effects
-				(font
-					(size 1.27 1.27)
-				)
-			)
-		)
-		(property "Footprint" ""
-			(at 245.11 132.08 0)
-			(effects
-				(font
-					(size 1.27 1.27)
-				)
-				(hide yes)
-			)
-		)
-		(property "Datasheet" ""
-			(at 245.11 132.08 0)
-			(effects
-				(font
-					(size 1.27 1.27)
-				)
-				(hide yes)
-			)
-		)
-		(property "Description" ""
-			(at 245.11 132.08 0)
-			(effects
-				(font
-					(size 1.27 1.27)
-				)
-				(hide yes)
-			)
-		)
-		(pin "1"
-		)
-		(instances
-			(project "Telemetry Main Board"
-				(path "/dde73ecd-f7ea-407a-a1ab-cf1927044ecb"
-					(reference "#PWR022")
-					(unit 1)
-				)
-			)
-		)
-	)
-	(symbol
 		(lib_id "power:GND")
 		(at 71.12 17.78 270)
@@
 			)
 		)
-		(property "Value" "10k"
+		(property "Value" "1 Ω"
 			(at 249.682 91.694 0)
 			(effects
@@
 	(symbol
 		(lib_id "power:+5V")
-		(at 257.81 139.7 270)
+		(at 260.35 139.7 270)
 		(unit 1)
 		(exclude_from_sim no)
@@
 		(fields_autoplaced yes)
 		(property "Reference" "#PWR032"
-			(at 254 139.7 0)
+			(at 256.54 139.7 0)
 			(effects
 				(font
@@
 		)
 		(property "Value" "+3V3"
-			(at 261.62 139.6999 90)
+			(at 264.16 139.6999 90)
 			(effects
 				(font
@@
 		)
 		(property "Footprint" ""
-			(at 257.81 139.7 0)
+			(at 260.35 139.7 0)
 			(effects
 				(font
@@
 		)
 		(property "Datasheet" ""
-			(at 257.81 139.7 0)
+			(at 260.35 139.7 0)
 			(effects
 				(font
@@
 		)
 		(property "Description" ""
-			(at 257.81 139.7 0)
+			(at 260.35 139.7 0)
 			(effects
 				(font
@@
 	)
 	(symbol
-		(lib_id "power:+5V")
-		(at 246.38 88.9 0)
-		(unit 1)
-		(exclude_from_sim no)
-		(in_bom yes)
-		(on_board yes)
-		(dnp no)
-		(fields_autoplaced yes)
-		(property "Reference" "#PWR052"
-			(at 246.38 92.71 0)
-			(effects
-				(font
-					(size 1.27 1.27)
-				)
-				(hide yes)
-			)
-		)
-		(property "Value" "+3V3"
-			(at 246.38 83.82 0)
-			(effects
-				(font
-					(size 1.27 1.27)
-				)
-			)
-		)
-		(property "Footprint" ""
-			(at 246.38 88.9 0)
-			(effects
-				(font
-					(size 1.27 1.27)
-				)
-				(hide yes)
-			)
-		)
-		(property "Datasheet" ""
-			(at 246.38 88.9 0)
-			(effects
-				(font
-					(size 1.27 1.27)
-				)
-				(hide yes)
-			)
-		)
-		(property "Description" ""
-			(at 246.38 88.9 0)
-			(effects
-				(font
-					(size 1.27 1.27)
-				)
-				(hide yes)
-			)
-		)
-		(pin "1"
-		)
-		(instances
-			(project "Telemetry Main Board"
-				(path "/dde73ecd-f7ea-407a-a1ab-cf1927044ecb"
-					(reference "#PWR052")
-					(unit 1)
-				)
-			)
-		)
-	)
-	(symbol
 		(lib_id "power:+9V")
 		(at 71.12 22.86 90)
@@
 			)
 		)
-		(property "Value" "100nf"
+		(property "Value" "2 μf"
 			(at 241.3 102.362 0)
 			(effects

Commit message: saving midway through pcb work
Parts:
- U6: footprint FS_3_Global_Footprint_Library:PDIP14_300MC_MCH -> Package_SO:SOIC-14_3.9x8.7mm_P1.27mm
Connections:
- net SPI3_SSEL2: now also U5.CN3_2 (PA10); no longer U5.CN4_7 (PA6)
- net SPI3_SSEL3: now also U5.CN3_1 (PA9); no longer U5.CN4_8 (PA5)
Changed lines of the file:
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@@
 	)
 	(no_connect
-		(at 163.83 35.56)
+		(at 194.31 50.8)
 	)
 	(no_connect
@@
 	)
 	(no_connect
-		(at 163.83 38.1)
+		(at 194.31 53.34)
 	)
 	(no_connect
@@
 		)
 	)
-	(global_label "SPI3_SSEL3"
-		(shape output)
-		(at 194.31 53.34 0)
-		(fields_autoplaced yes)
-		(effects
-			(font
-				(size 1.27 1.27)
-			)
-			(justify left)
-		)
-		(property "Intersheetrefs" "${INTERSHEET_REFS}"
-			(at 208.3622 53.34 0)
-			(effects
-				(font
-					(size 1.27 1.27)
-				)
-				(justify left)
-				(hide yes)
-			)
-		)
-	)
 	(global_label "SD Card Detect T{slash}F"
 		(shape input)
@@
 		)
 	)
+	(global_label "SPI3_SSEL2"
+		(shape output)
+		(at 163.83 38.1 180)
+		(fields_autoplaced yes)
+		(effects
+			(font
+				(size 1.27 1.27)
+			)
+			(justify right)
+		)
+		(property "Intersheetrefs" "${INTERSHEET_REFS}"
+			(at 149.7778 38.1 0)
+			(effects
+				(font
+					(size 1.27 1.27)
+				)
+				(justify right)
+				(hide yes)
+			)
+		)
+	)
 	(global_label "ADC"
 		(shape input)
@@
 		)
 	)
+	(global_label "SPI3_SSEL3"
+		(shape output)
+		(at 163.83 35.56 180)
+		(fields_autoplaced yes)
+		(effects
+			(font
+				(size 1.27 1.27)
+			)
+			(justify right)
+		)
+		(property "Intersheetrefs" "${INTERSHEET_REFS}"
+			(at 149.7778 35.56 0)
+			(effects
+				(font
+					(size 1.27 1.27)
+				)
+				(justify right)
+				(hide yes)
+			)
+		)
+	)
 	(global_label "CAN2_H"
 		(shape bidirectional)
@@
 		)
 	)
-	(global_label "SPI3_SSEL2"
-		(shape output)
-		(at 194.31 50.8 0)
-		(fields_autoplaced yes)
-		(effects
-			(font
-				(size 1.27 1.27)
-			)
-			(justify left)
-		)
-		(property "Intersheetrefs" "${INTERSHEET_REFS}"
-			(at 208.3622 50.8 0)
-			(effects
-				(font
-					(size 1.27 1.27)
-				)
-				(justify left)
-				(hide yes)
-			)
-		)
-	)
 	(global_label "SD Card Detect T{slash}F"
 		(shape output)
@@
 			)
 		)
-		(property "Footprint" "FS_3_Global_Footprint_Library:PDIP14_300MC_MCH"
+		(property "Footprint" "Package_SO:SOIC-14_3.9x8.7mm_P1.27mm"
 			(at 41.91 147.32 0)
 			(effects
@@
 			)
 		)
-		(property "Footprint" "FS_3_Global_Footprint_Library:PDIP14_300MC_MCH"
+		(property "Footprint" "Package_SO:SOIC-14_3.9x8.7mm_P1.27mm"
 			(at 41.91 170.18 0)
 			(effects
@@
 			)
 		)
-		(property "Footprint" "FS_3_Global_Footprint_Library:PDIP14_300MC_MCH"
+		(property "Footprint" "Package_SO:SOIC-14_3.9x8.7mm_P1.27mm"
 			(at 73.66 187.96 0)
 			(effects
@@
 			)
 		)
-		(property "Footprint" "FS_3_Global_Footprint_Library:PDIP14_300MC_MCH"
+		(property "Footprint" "Package_SO:SOIC-14_3.9x8.7mm_P1.27mm"
 			(at 41.91 123.19 0)
 			(effects
@@
 			)
 		)
-		(property "Footprint" "FS_3_Global_Footprint_Library:PDIP14_300MC_MCH"
+		(property "Footprint" "Package_SO:SOIC-14_3.9x8.7mm_P1.27mm"
 			(at 35.56 195.58 0)
 			(effects
