File: Telemetry Main Board/Telemetry Main Board.kicad_pcb (KiCad board)
At the start: 2 copper layers, 107 x 73 mm, 42 parts, among them J1 8 pin ATM connector, J3 12 pin ATM connector, J4 SD to SPI (Molex nanofit), U1 LM7805_TO220, U10 MCP2515-I/SO, U2 LM7809_TO220, U4 ISO1050DUB, U5 NUCLEO-L432KC, U6 MCP6004, U8 ISO1050DUB, U9 MCP2515-I/SO

Commit message: added gerbers
Routing:
- net SD Card Detect T/F: track 19.8 -> 14.4 mm
Changed lines of the file:
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@@
-	)
-	(segment
-		(start 153.9625 74.0375)
-		(end 153.9625 76.5)
-		(width 0.2)
-		(layer "F.Cu")
-		(net 3)
 	)
 	(segment
@@
 	)
 	(segment
-		(start 154 74)
-		(end 153.9625 74.0375)
-		(width 0.2)
-		(layer "F.Cu")
-		(net 3)
-	)
-	(segment
 		(start 127.5 58.43)
 		(end 134.226321 58.43)
@@
 	)
 	(segment
+		(start 153.988908 63.711092)
+		(end 153.9625 63.7375)
+		(width 0.2)
+		(layer "F.Cu")
+		(net 3)
+	)
+	(segment
 		(start 134.226321 58.43)
 		(end 135.105 59.308679)
@@
 	)
 	(segment
+		(start 153.9625 63.7375)
+		(end 153.9625 76.5)
+		(width 0.2)
+		(layer "F.Cu")
+		(net 3)
+	)
+	(segment
 		(start 135.105 61.895)
 		(end 131.46 65.54)
@@
 	)
 	(via
-		(at 154 74)
+		(at 153.988908 63.711092)
 		(size 0.6)
 		(drill 0.3)
@@
 	)
 	(segment
-		(start 138 68.5)
+		(start 154 63.5)
 		(end 143 63.5)
 		(width 0.2)
@@
 	)
 	(segment
-		(start 154 63.5)
-		(end 154 74)
+		(start 154 63.7)
+		(end 154 63.5)
 		(width 0.2)
 		(layer "B.Cu")
@@
 	(segment
 		(start 143 63.5)
-		(end 154 63.5)
+		(end 138 68.5)
 		(width 0.2)
 		(layer "B.Cu")
@@
 	)
 	(segment
+		(start 153.988908 63.711092)
+		(end 154 63.7)
+		(width 0.2)
+		(layer "B.Cu")
+		(net 3)
+	)
+	(segment
 		(start 169.5 62)
 		(end 169.5 106.5)
@@
 	)
 	(segment
-		(start 152.25 67)
-		(end 150.925 68.325)
-		(width 0.2)
-		(layer "F.Cu")
-		(net 38)
-	)
-	(segment
 		(start 160.5 73.5)
 		(end 159.5 74.5)
@@
 	)
 	(segment
-		(start 150.925 68.325)
+		(start 153.25 74.75)
+		(end 150.925 72.425)
+		(width 0.2)
+		(layer "F.Cu")
+		(net 38)
+	)
+	(segment
+		(start 150.925 72.425)
 		(end 150.925 69.4)
-		(width 0.2)
-		(layer "F.Cu")
-		(net 38)
-	)
-	(segment
-		(start 153.25 67)
-		(end 152.25 67)
 		(width 0.2)
 		(layer "F.Cu")
@@
 	)
 	(via
-		(at 153.25 67)
+		(at 153.25 74.75)
 		(size 0.6)
 		(drill 0.3)
@@
 	)
 	(segment
-		(start 158 74.5)
+		(start 153.25 75)
 		(end 157.5 75)
 		(width 0.2)
@@
 	)
 	(segment
-		(start 153.25 75)
-		(end 153.25 67)
+		(start 153.25 74.75)
+		(end 153.25 75)
 		(width 0.2)
 		(layer "B.Cu")
@@
 	(segment
 		(start 157.5 75)
-		(end 153.25 75)
-		(width 0.2)
-		(layer "B.Cu")
+		(end 158 74.5)
+		(width 0.2)
+		(layer "B.Cu")

Commit message: revised gerbers
Other:
- board text added: "FS-3 Main Telemetry Board Formula Slug Designed by Shaunak Lal and Slav Miroshnichenko V 1.8"
- board text removed: "FS-3 Main Telemetry Board Formula Slug Designed by Shaunak Lal and Slav Miroshnichenko Rev 2.3"
Changed lines of the file:
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@@
 		)
 	)
-	(gr_text "FS-3 Main Telemetry Board\nFormula Slug\nDesigned by Shaunak Lal and Slav Miroshnichenko\nRev 2.3"
+	(gr_text "FS-3 Main Telemetry Board\nFormula Slug\nDesigned by Shaunak Lal and Slav Miroshnichenko\nV 1.8"
 		(at 179 115.5 90)
 		(layer "F.SilkS")
@@
 	)
 	(segment
-		(start 101.27 104.02)
-		(end 101.5 104.25)
+		(start 101.27 104.23)
+		(end 101.25 104.25)
 		(width 0.2)
 		(layer "F.Cu")
@@
 	)
 	(segment
-		(start 101.27 101.18)
-		(end 101.27 104.02)
+		(start 101.27 101.05)
+		(end 101.27 104.23)
 		(width 0.2)
 		(layer "F.Cu")
@@
 	)
 	(via
+		(at 101.25 104.25)
+		(size 0.6)
+		(drill 0.3)
+		(layers "F.Cu" "B.Cu")
+		(net 39)
+	)
+	(via
 		(at 87.5 103.75)
 		(size 0.6)
 		(drill 0.3)
-		(layers "F.Cu" "B.Cu")
-		(net 39)
-	)
-	(via
-		(at 101.5 104.25)
-		(size 0.6)
-		(drill 0.3)

Commit message: finished pcb for updated micro
Parts:
- removed C12, C15, C9: 100nf, Capacitor_SMD:C_0805_2012Metric_Pad1.18x1.45mm_HandSolder
- removed C16: 100 μf, Capacitor_SMD:C_0805_2012Metric_Pad1.18x1.45mm_HandSolder
- removed D1, D2: CD4148W, Diode_SMD:D_0805_2012Metric
- removed the G*** at (76.3, 42.8)
- removed the G*** at (178.1, 42.8)
- removed the G*** at (76.3, 111.3)
- removed R10, R4: 100Ω, Resistor_SMD:R_0805_2012Metric_Pad1.20x1.40mm_HandSolder
- removed R3, R9: 10k, Resistor_SMD:R_0805_2012Metric_Pad1.20x1.40mm_HandSolder
- removed U10, U9: MCP2515-I/SO, Package_SO:SOIC-18W_7.5x11.6mm_P1.27mm
- removed U5: NUCLEO-L432KC, FS_3_Global_Footprint_Library:NUCLEO-L432KC
- removed U7: ~, Package_SO:SSOP-24_5.3x8.2mm_P0.65mm
- added U3: NUCLEO-F446RE, FS_3_Global_Footprint_Library:NUCLEO-F446RE, F.Cu at (127.8, 126.8)
- C5: value 100 μf -> 100nf
- moved C5 72.7 mm to (171.8, 85.5), turned to 180 degrees
- moved G*** 2.51 mm to (117.5, 74.5), turned to 0 degrees
Connections:
- C5 pad 1: Net-(D1-A) -> +9V
- J4 pad 3: SPI3_SCLK -> SPI2_SCK
- J4 pad 4: SPI3_MISO -> SPI2_MISO
- J4 pad 5: SPI3_MOSI -> SPI2_MOSI
- J4 pad 6: SPI3_SSEL3 -> SPI2_CS
Routing:
- net SPI3_SCLK: track 110.0 -> 0.00 mm, vias 2 -> 0
- net SPI3_MOSI: track 101.7 -> 0.00 mm, vias 4 -> 0
- net SPI3_MISO: track 98.8 -> 0.00 mm, vias 3 -> 0
- net SPI2_MISO: track 0.00 -> 90.9 mm
- net Steering Sensor 3V3: track 22.6 -> 113.5 mm
- net SPI2_SCK: track 0.00 -> 87.2 mm
- net SPI2_CS: track 0.00 -> 80.9 mm
- net GND: track 153.6 -> 87.7 mm, vias 10 -> 8
- net SD Card Detect T/F: track 14.4 -> 78.9 mm, vias 2 -> 0
- net +5V: track 130.2 -> 194.3 mm, vias 8 -> 9
- net Brake Sensor F 3V3: track 13.5 -> 72.7 mm, vias 2 -> 0
- net SPI3_SSEL1: track 58.1 -> 0.00 mm, vias 2 -> 0
- net SPI3_SSEL2: track 54.6 -> 0.00 mm, vias 1 -> 0
- net ADC: track 53.5 -> 0.00 mm, vias 1 -> 0
- net CAN1_RX: track 17.2 -> 65.6 mm, vias 2 -> 1
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Other:
- board size 107 x 73 mm -> 107 x 144.2 mm
- board text removed: "100Ω"

Commit message: Update Telemetry Main Board.kicad_pcb
Routing:
- net Brake Sensor R 3V3: track 67.3 -> 69.8 mm
Changed lines of the file:
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@@
 		(at 117.5 74.5)
 		(property "Reference" "G***"
-			(at 0 0 360)
+			(at 0 0 0)
 			(layer "F.SilkS")
 			(hide yes)
@@
 		)
 		(property "Value" "LOGO"
-			(at 0.75 0 360)
+			(at 0.75 0 0)
 			(layer "F.SilkS")
 			(hide yes)
@@
 		)
 		(property "Footprint" ""
-			(at 0 0 360)
+			(at 0 0 0)
 			(layer "F.Fab")
 			(hide yes)
@@
 		)
 		(property "Datasheet" ""
-			(at 0 0 360)
+			(at 0 0 0)
 			(layer "F.Fab")
 			(hide yes)
@@
 		)
 		(property "Description" ""
-			(at 0 0 360)
+			(at 0 0 0)
 			(layer "F.Fab")
 			(hide yes)
@@
 		(at 127.79 126.85 180)
 		(property "Reference" "U3"
-			(at 30.8 -16.4 360)
+			(at 30.8 -16.4 0)
 			(layer "F.SilkS")
 			(hide yes)
@@
 		)
 		(property "Value" "NUCLEO-F446RE"
-			(at 30.6 -13.8 360)
+			(at 30.6 -13.8 0)
 			(layer "F.Fab")
 			(hide yes)
@@
 		)
 		(property "Footprint" "FS_3_Global_Footprint_Library:NUCLEO-F446RE"
-			(at 0 0 360)
+			(at 0 0 0)
 			(layer "F.Fab")
 			(hide yes)
@@
 		)
 		(property "Datasheet" ""
-			(at 0 0 360)
+			(at 0 0 0)
 			(layer "F.Fab")
 			(hide yes)
@@
 		)
 		(property "Description" "NUCLEO with 2 can busses and an STM 32 MCU"
-			(at 0 0 360)
+			(at 0 0 0)
 			(layer "F.Fab")
 			(hide yes)
@@
 		(tags "capacitor handsolder")
 		(property "Reference" "C5"
-			(at 0 -1.68 360)
+			(at 0 -1.68 0)
 			(layer "F.SilkS")
 			(effects
@@
 		)
 		(property "Value" "100nf"
-			(at 0 1.68 360)
+			(at 0 1.68 0)
 			(layer "F.Fab")
 			(effects
@@
 		)
 		(fp_text user "${REFERENCE}"
-			(at 0 0 360)
+			(at 0 0 0)
 			(layer "F.Fab")
 			(effects
@@
 	)
 	(gr_text "FS-3 Main Telemetry Board\nFormula Slug\nDesigned by Shaunak Lal and Slav Miroshnichenko\nV 1.8"
-		(at 203.25 112 90)
+		(at 84.5 120.75 90)
 		(layer "F.SilkS")
 		(effects
@@
 	)
 	(segment
-		(start 148.93 59.319034)
-		(end 148.93 87.65)
-		(width 0.15)
-		(layer "F.Cu")
-		(net 7)
-	)
-	(segment
-		(start 149 55.25)
-		(end 149 59.249034)
+		(start 146.205 53.58)
+		(end 147.33 53.58)
 		(width 0.15)
 		(layer "F.Cu")
@@
 	)
 	(segment
-		(start 149 59.249034)
-		(end 148.93 59.319034)
+		(start 148.93 55.18)
+		(end 148.93 87.65)
 		(width 0.15)
 		(layer "F.Cu")
@@
 	)
 	(segment
-		(start 146.205 53.58)
-		(end 147.33 53.58)
+		(start 148.93 87.65)
+		(end 157 95.72)
 		(width 0.15)
 		(layer "F.Cu")
@@
 	(segment
 		(start 147.33 53.58)
-		(end 149 55.25)
-		(width 0.15)
-		(layer "F.Cu")
-		(net 7)
-	)
-	(segment
-		(start 148.93 87.65)
-		(end 157 95.72)
+		(end 148.93 55.18)
 		(width 0.15)
 		(layer "F.Cu")
@@
 	)
 	(segment
-		(start 97.515 118.138862)
-		(end 97.515 120.055)
+		(start 98.138862 117.515)
+		(end 97.515 118.138862)
 		(width 0.2)
 		(layer "F.Cu")
@@
 	)
 	(segment
-		(start 98.138862 117.515)
-		(end 97.515 118.138862)
+		(start 99.021138 117.515)
+		(end 98.138862 117.515)
 		(width 0.2)
 		(layer "F.Cu")
@@
 	(segment
 		(start 122.25 67)
-		(end 124.25 67)
+		(end 125.25 70)
 		(width 0.2)
 		(layer "F.Cu")
@@
 	)
 	(segment
-		(start 122.25 94.286138)
-		(end 99.021138 117.515)
+		(start 122.25 67)
+		(end 124.25 67)
 		(width 0.2)
 		(layer "F.Cu")
@@
 	)
 	(segment
-		(start 99.021138 117.515)
-		(end 98.138862 117.515)
+		(start 125.25 70)
+		(end 125.25 91.286138)
 		(width 0.2)
 		(layer "F.Cu")
@@
 	)
 	(segment
-		(start 122.25 67)
-		(end 122.25 94.286138)
+		(start 125.25 91.286138)
+		(end 99.021138 117.515)
 		(width 0.2)
 		(layer "F.Cu")
@@
 	)
 	(segment
+		(start 97.515 118.138862)
+		(end 97.515 120.055)
+		(width 0.2)
+		(layer "F.Cu")
+		(net 18)
+	)
+	(segment
 		(start 127.055 106.945)
 		(end 97.515 106.945)
@@
 	)
 	(segment
-		(start 97.105 99.735)
-		(end 96.04 100.8)
+		(start 110.265 99.735)
+		(end 97.105 99.735)
 		(width 0.2)
 		(layer "B.Cu")
@@
 	)
 	(segment
-		(start 164.15 74.85)
-		(end 164.15 70.523654)
+		(start 163.376346 69.75)
+		(end 145.5 69.75)
 		(width 0.2)
 		(layer "B.Cu")
@@
 	)
 	(segment
-		(start 164.15 70.523654)
-		(end 163.376346 69.75)
+		(start 164.15 74.85)
+		(end 164.15 70.523654)
 		(width 0.2)
 		(layer "B.Cu")
@@
 	)
 	(segment
-		(start 136.5 78.75)
-		(end 130.75 78.75)
+		(start 97.105 99.735)
+		(end 96.04 100.8)
 		(width 0.2)
 		(layer "B.Cu")
@@
 	)
 	(segment
-		(start 163 76)
-		(end 164.15 74.85)
+		(start 131.25 78.75)
+		(end 110.265 99.735)
 		(width 0.2)
 		(layer "B.Cu")
@@
 	)
 	(segment
-		(start 130.75 78.75)
-		(end 109.765 99.735)
+		(start 145.5 69.75)
+		(end 136.5 78.75)
 		(width 0.2)
 		(layer "B.Cu")
@@
 	)
 	(segment
-		(start 145.5 69.75)
-		(end 136.5 78.75)
+		(start 163 76)
+		(end 164.15 74.85)
 		(width 0.2)
 		(layer "B.Cu")
@@
 	)
 	(segment
-		(start 109.765 99.735)
-		(end 97.105 99.735)
+		(start 136.5 78.75)
+		(end 131.25 78.75)
 		(width 0.2)
 		(layer "B.Cu")
@@
 	)
 	(segment
-		(start 163.376346 69.75)
-		(end 145.5 69.75)
+		(start 164.15 70.523654)
+		(end 163.376346 69.75)
 		(width 0.2)
 		(layer "B.Cu")

Commit message: fixed telemetry main pcb
Parts:
- removed C11: 100nf, Capacitor_SMD:C_0805_2012Metric_Pad1.18x1.45mm_HandSolder
- added G1: FS Logo, 1FS_2_Global_Footprint_Library:FS Logo Big, F.Cu at (132.0, 112.2)
- moved C5 77.6 mm to (105.2, 125.5), turned to 90 degrees
- moved C8 69.5 mm to (157.5, 80.2)
- moved C7 69.0 mm to (157.5, 64.5)
- moved J1 66.6 mm to (148.3, 61.0)
- moved U4 66.0 mm to (154.7, 72.0)
- moved C10 64.8 mm to (168.3, 80.2)
- moved C6 64.2 mm to (168.2, 64.5)
- moved U8 61.9 mm to (165.5, 72.0)
- moved G*** 58.5 mm to (176.0, 73.5), turned to 90 degrees
- moved J4 54.9 mm to (171.2, 135.2)
- moved C13 53.0 mm to (174.8, 135.5)
- moved C4 34.0 mm to (134.5, 62.0)
- moved J3 33.7 mm to (89.9, 42.6)
- moved U1 33.7 mm to (85.6, 58.6)
- moved U2 33.7 mm to (129.9, 58.3)
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Connections:
- J1 pad 3: CAN2_H -> CAN1_L
- J1 pad 4: CAN2_H -> CAN1_L
- J1 pad 5: CAN1_L -> CAN2_H
- J1 pad 6: CAN1_L -> CAN2_H
- U3 pad CN10_7: +3V3 -> unconnected-(U3B-AVDD-PadCN10_7)
- U3 pad CN10_8: +5V -> unconnected-(U3B-U5V-PadCN10_8)
- U3 pad CN7_12: +3V3 -> unconnected-(U3A-CN7_IOREF-PadCN7_12)
- U3 pad CN7_28: Acc Intake Temp -> Acc Intake Flow Rate
- U3 pad CN7_30: Acc Exhaust Temp -> Acc Intake Pressure
- U3 pad CN7_32: Acc Intake Pressure -> Acc Exhaust Temp
- U3 pad CN7_34: Acc Intake Flow Rate -> Acc Intake Temp
Routing:
- net SPI2_MISO: track 90.9 -> 13.8 mm
- net SPI2_SCK: track 87.2 -> 13.8 mm
- net SD Card Detect T/F: track 78.9 -> 9.75 mm
- net +5V: track 194.3 -> 126.4 mm, vias 9 -> 2
- net SPI2_CS: track 80.9 -> 22.7 mm, vias 0 -> 1
- net Steering Sensor 3V3: track 113.5 -> 59.2 mm, vias 0 -> 1
- net Acc Intake Flow Rate: track 47.3 -> 94.4 mm
- net CAN1_RX: track 65.6 -> 23.9 mm
- net Acc Intake Pressure: track 53.7 -> 95.1 mm
- net GND: track 87.7 -> 48.5 mm, vias 8 -> 7
- net Acc Exhaust Temp: track 60.1 -> 94.0 mm
- net CAN1_TX: track 62.6 -> 29.5 mm
- net CAN2_RX: track 33.1 -> 66.0 mm, vias 2 -> 1
- net Acc Intake Temp: track 66.4 -> 93.0 mm
- net +9V: track 61.8 -> 88.1 mm, vias 1 -> 2
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Other:
- board size 107 x 144.2 mm -> 106 x 108.5 mm

Commit message: Update Telemetry Main Board.kicad_pcb
Other:
- board text added: "100μF"
- board text added: "20μF"
- board text added: "330μF"
Changed lines of the file:
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@@
 		(tags "capacitor handsolder")
 		(property "Reference" "C7"
-			(at 0 -1.68 360)
+			(at -0.4625 2.5 0)
 			(layer "F.SilkS")
 			(effects
@@
 		)
 		(property "Value" "100nf"
-			(at 0 1.68 360)
+			(at 0 1.68 0)
 			(layer "F.Fab")
 			(effects
@@
 		)
 		(fp_text user "${REFERENCE}"
-			(at 0 0 360)
+			(at 0 0 0)
 			(layer "F.Fab")
 			(effects
@@
 		(tags "capacitor handsolder")
 		(property "Reference" "C4"
-			(at 0 -1.68 360)
+			(at 0.4625 1.75 0)
 			(layer "F.SilkS")
 			(effects
@@
 		)
 		(property "Value" "100nf"
-			(at 0 1.68 360)
+			(at 0 1.68 0)
 			(layer "F.Fab")
 			(effects
@@
 		)
 		(fp_text user "${REFERENCE}"
-			(at -2.25 -0.26 360)
+			(at -2.25 -0.26 0)
 			(layer "F.Fab")
 			(effects
@@
 		(tags "capacitor handsolder")
 		(property "Reference" "C8"
-			(at 0 -1.68 360)
+			(at 0 -1.68 0)
 			(layer "F.SilkS")
 			(effects
@@
 		)
 		(property "Value" "100nf"
-			(at 0 1.68 360)
+			(at 0 1.68 0)
 			(layer "F.Fab")
 			(effects
@@
 		)
 		(fp_text user "${REFERENCE}"
-			(at 0 0 360)
+			(at 0 0 0)
 			(layer "F.Fab")
 			(effects
@@
 		(tags "capacitor handsolder")
 		(property "Reference" "C6"
-			(at 0 -1.68 360)
+			(at -0.5 2.5 0)
 			(layer "F.SilkS")
 			(effects
@@
 		)
 		(property "Value" "100nf"
-			(at 0 1.68 360)
+			(at 0 1.68 0)
 			(layer "F.Fab")
 			(effects
@@
 		)
 		(fp_text user "${REFERENCE}"
-			(at 0 0 360)
+			(at 0 0 0)
 			(layer "F.Fab")
 			(effects
@@
 		(tags "capacitor handsolder")
 		(property "Reference" "C10"
-			(at 0 -1.68 360)
+			(at 0 -1.68 0)
 			(layer "F.SilkS")
 			(effects
@@
 		)
 		(property "Value" "100nf"
-			(at 0 1.68 360)
+			(at 0 1.68 0)
 			(layer "F.Fab")
 			(effects
@@
 		)
 		(fp_text user "${REFERENCE}"
-			(at 0 0 360)
+			(at 0 0 0)
 			(layer "F.Fab")
 			(effects
@@
 		(tags "capacitor handsolder")
 		(property "Reference" "C2"
-			(at 0 -1.68 360)
+			(at 0 -1.68 0)
 			(layer "F.SilkS")
 			(effects
@@
 		)
 		(property "Value" "330nf"
-			(at 0 1.68 360)
+			(at 0 1.68 0)
 			(layer "F.Fab")
 			(effects
@@
 		)
 		(fp_text user "${REFERENCE}"
-			(at 0 0 360)
+			(at 0 0 0)
 			(layer "F.Fab")
 			(effects
@@
 		(tags "connector Molex Nano-Fit side entry")
 		(property "Reference" "J4"
-			(at 1.25 -2.92 360)
+			(at 1.25 -2.92 0)
 			(layer "F.SilkS")
 			(effects
@@
 		)
 		(property "Value" "SD to SPI (Molex nanofit)"
-			(at 1.25 12.92 360)
+			(at 1.25 12.92 0)
 			(layer "F.Fab")
 			(effects
@@
 		)
 	)
+	(gr_text "100μF"
+		(at 156.5 63.25 0)
+		(layer "F.SilkS")
+		(effects
+			(font
+				(size 0.5 0.5)
+				(thickness 0.1)
+				(bold yes)
+			)
+			(justify left bottom)
+		)
+	)
+	(gr_text "10KΩ"
+		(at 135.75 68.25 0)
+		(layer "F.SilkS")
+		(effects
+			(font
+				(size 0.5 0.5)
+				(thickness 0.1)
+				(bold yes)
+			)
+			(justify left bottom)
+		)
+	)
 	(gr_text "10KΩ"
 		(at 124.25 70 0)
@@
 		)
 	)
-	(gr_text "100 μF"
+	(gr_text "20μF"
+		(at 169.75 82.5 0)
+		(layer "F.SilkS")
+		(effects
+			(font
+				(size 0.5 0.5)
+				(thickness 0.1)
+				(bold yes)
+			)
+			(justify left bottom)
+		)
+	)
+	(gr_text "100μF"
+		(at 107.25 127.75 90)
+		(layer "F.SilkS")
+		(effects
+			(font
+				(size 0.5 0.5)
+				(thickness 0.1)
+				(bold yes)
+			)
+			(justify left bottom)
+		)
+	)
+	(gr_text "100μF"
 		(at 141 74 90)
 		(layer "F.SilkS")
@@
 				(bold yes)
 			)
+			(justify left bottom)
+		)
+	)
+	(gr_text "330μF"
+		(at 129.25 63.75 0)
+		(layer "F.SilkS")
+		(effects
+			(font
+				(size 0.5 0.5)
+				(thickness 0.1)
+				(bold yes)
+			)
+			(justify left bottom)
+		)
+	)
+	(gr_text "20μF"
+		(at 158.5 82.5 0)
+		(layer "F.SilkS")
+		(effects
+			(font
+				(size 0.5 0.5)
+				(thickness 0.1)
+				(bold yes)
+			)
+			(justify left bottom)
+		)
+	)
+	(gr_text "100μF"
+		(at 167.25 63.25 0)
+		(layer "F.SilkS")
+		(effects
+			(font
+				(size 0.5 0.5)
+				(thickness 0.1)
+				(bold yes)
+			)
+			(justify left bottom)
+		)
+	)
+	(gr_text "100μF"
+		(at 136.75 62.25 0)
+		(layer "F.SilkS")
+		(effects
+			(font
+				(size 0.5 0.5)
+				(thickness 0.1)
+				(bold yes)
+			)

Commit message: Update Telemetry Main Board.kicad_pcb
Other:
- board text added: "FS-3 Main Telemetry Board Formula Slug Designed by Shaunak Lal and Slav Miroshnichenko Rev 1.0"
- board text removed: "FS-3 Main Telemetry Board Formula Slug Designed by Shaunak Lal and Slav Miroshnichenko V 1.8"
Changed lines of the file:
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@@
 		)
 	)
-	(gr_text "FS-3 Main Telemetry Board\nFormula Slug\nDesigned by Shaunak Lal and Slav Miroshnichenko\nV 1.8"
+	(gr_text "FS-3 Main Telemetry Board\nFormula Slug\nDesigned by Shaunak Lal and Slav Miroshnichenko\nRev 1.0"
 		(at 89.5 147.25 90)
 		(layer "F.SilkS")

Commit message: added mounting holes and specified diode
Parts:
- added REF**: MountingHole_2.2mm_M2, MountingHole:MountingHole_2.2mm_M2, F.Cu at (72.0, 48.2)
- added REF**: MountingHole_2.2mm_M2, MountingHole:MountingHole_2.2mm_M2, F.Cu at (71.8, 146.0)
- added REF**: MountingHole_2.2mm_M2, MountingHole:MountingHole_2.2mm_M2, F.Cu at (187.0, 146.0)
- added REF**: MountingHole_2.2mm_M2, MountingHole:MountingHole_2.2mm_M2, F.Cu at (187.0, 48.2)
- moved G1 4.92 mm to (129.6, 107.9)
Other:
- board size 106 x 108.5 mm -> 125 x 107.8 mm
