File: Acc_Board_Christian/FS_3_Accumulator_Board/FS_3_Accumulator_Board.kicad_sch (KiCad schematic)
At the start: 13 parts, among them CN1 NUCLEO-L432KC, J1 Conn_01x04_Pin, U1 MCP6004, U3 ISO1050DUB

Commit message: updates: voltage regulators added to schematic
Parts:
- added C4, C7: 10uF, symbol Device:C
- added C5, C6: 100nF, symbol Device:C
- added C8, C9: 330nF, symbol Device:C
- added D2: D_Zener, symbol Device:D_Zener
- added J2: Conn_01x23, symbol Connector_Generic:Conn_01x23
- added U2: R-78B5.0-2.0, Converter_DCDC:Converter_DCDC_RECOM_R-78B-2.0_THT, symbol Regulator_Switching:R-78B5.0-2.0
- added U4: LM7809_TO220, Package_TO_SOT_THT:TO-220-3_Vertical, symbol Regulator_Linear:LM7809_TO220
Connections:
- net +5V: now also C6.1, C7.1, U2.3 (OUT)
- net +9V: now also C9.1, U4.3 (VO)
- net GND: now also C4.2, C5.2, C6.2, C7.2, C8.2, C9.2, D2.2 (A), U2.2 (GND), U4.2 (GND)
- new net +12V: C4.1, C5.1, C8.1, D2.1 (K), U2.1 (IN), U4.1 (VI)
Other:
- note added: "Power Block"

Commit message: Mistake
Connections:
- net +12V: now also J2.2 (Pin_2)
- net CAN_H: now also J2.6 (Pin_6)
- net GND: now also J2.1 (Pin_1)
- net AIRS+_GND: now reaches J2.3 (Pin_3)
- net CAN_L _RES: now reaches J2.5 (Pin_5)
- no-connect marks 10 -> 11
Other:
- moved on the sheet: U1B

Commit message: Working on acc fs2 remake
Parts:
- removed J1: Conn_01x04_Pin, symbol Connector:Conn_01x04_Pin
- added C10: 1uf, Capacitor_SMD:C_0805_2012Metric_Pad1.18x1.45mm_HandSolder, symbol Device:C
- added C11: 100nF, Capacitor_SMD:C_0805_2012Metric_Pad1.18x1.45mm_HandSolder, symbol Device:C
- added C12: 1uF, symbol Device:C
- added C13: 10µF, Capacitor_SMD:C_0805_2012Metric_Pad1.18x1.45mm_HandSolder, symbol Device:C
- added C14: 100nF, symbol Device:C
- added D3, D4, D5, D6: D, symbol Device:D
- added D7: 1N47xxA, Diode_THT:D_DO-41_SOD81_P10.16mm_Horizontal, symbol Diode:1N47xxA
- added D8: D, Diode_SMD:D_2010_5025Metric_Pad1.52x2.65mm_HandSolder, symbol Device:D
- added J1: Current Sensor, 1FS_2_Global_Footprint_Library:MOLEX_1053091204, symbol 1FS_2_Global_Symbol_Library:1053091204
- added J10: Fans, 1FS_2_Global_Footprint_Library:MOLEX_1053091206, symbol 1FS_2_Global_Symbol_Library:1053091206
- added J11: Conn_01x04_Pin, symbol Connector:Conn_01x04_Pin
- added J3: IMD, symbol Connector:Conn_01x03_Pin
- added J4: Shutdown IL, 1FS_2_Global_Footprint_Library:MOLEX_1053091202, symbol molex_1053091202:1053091202
- added J5: IMD BAT, 1FS_2_Global_Footprint_Library:MOLEX_1053091202, symbol 1FS_2_Global_Symbol_Library:1053091202
- added J6: HV Power, 1FS_2_Global_Footprint_Library:MOLEX_1053091204, symbol 1FS_2_Global_Symbol_Library:1053091204
- added J7: HVIL, 1FS_2_Global_Footprint_Library:MOLEX_1053091204, symbol 1FS_2_Global_Symbol_Library:1053091204
- added J8: Precharge Resistor, 1FS_2_Global_Footprint_Library:MOLEX_1053091202, symbol 1FS_2_Global_Symbol_Library:1053091202
- added J9: AIRs Power, 1FS_2_Global_Footprint_Library:MOLEX_1053091204, symbol 1FS_2_Global_Symbol_Library:1053091204
- added K1, K2: DK1A1B-12V, 1FS_2_Global_Footprint_Library:RELAY_DK2A_PAN, symbol 2FS-1_Symbol Library:DK1A1B-12V
- added K3: G6BK-1114P-US, 1FS_2_Global_Footprint_Library:Omron G6BK-1114P-US, symbol 1FS_2_Global_Symbol_Library:G6BK-1114P-US
- added K4: G5PZ-1A-X DC12, 1FS_2_Global_Footprint_Library:G5PZ-1A-X DC12, symbol Relay:Relay_SPST-NO
- added Q1, Q2, Q3, Q4, Q5: NMOS, symbol Simulation_SPICE:NMOS
- added Q6, Q7, Q8: STS6NF20V, 1FS_2_Global_Footprint_Library:SO-8_STM, symbol 1_ACC_BOARD:STS6NF20V
- added R10, R11, R12, R8, R9: R, symbol Device:R
- added R13: 2.4M, symbol Device:R
- added R14: 120, 1FS_2_Global_Footprint_Library:THS15120RJ, symbol Device:R
- added R15, R16: 1k, symbol Device:R
- added R17: 2k, symbol Device:R
- added R18: 22k, Resistor_SMD:R_0805_2012Metric_Pad1.20x1.40mm_HandSolder, symbol Device:R
- added R19: 6.8K, Resistor_SMD:R_0805_2012Metric_Pad1.20x1.40mm_HandSolder, symbol Device:R
- added R20: 3.9k, Resistor_SMD:R_0805_2012Metric_Pad1.20x1.40mm_HandSolder, symbol Device:R
- added R21: 18k, Resistor_SMD:R_0805_2012Metric_Pad1.20x1.40mm_HandSolder, symbol Device:R
- added R6: 1.6k, Resistor_SMD:R_0805_2012Metric_Pad1.20x1.40mm_HandSolder, symbol Device:R
- added R7: 560, Resistor_SMD:R_0805_2012Metric_Pad1.20x1.40mm_HandSolder, symbol Device:R
- added TP1, TP2: GND, TestPoint:TestPoint_Loop_D2.50mm_Drill1.0mm, symbol Connector:TestPoint
- added TP10: Shutdown_Acc_IL, TestPoint:TestPoint_Loop_D2.50mm_Drill1.0mm, symbol Connector:TestPoint
- added TP11: Shutdown_Acc_Out, TestPoint:TestPoint_Loop_D2.50mm_Drill1.0mm, symbol Connector:TestPoint
- added TP12: AIRS_Final, TestPoint:TestPoint_Loop_D2.50mm_Drill1.0mm, symbol Connector:TestPoint
- added TP13: CAN_H, TestPoint:TestPoint_Loop_D2.50mm_Drill1.0mm, symbol Connector:TestPoint
- added TP14: CAN_L, TestPoint:TestPoint_Loop_D2.50mm_Drill1.0mm, symbol Connector:TestPoint
- added TP15: BMS_FAULT_5V, TestPoint:TestPoint_Loop_D2.50mm_Drill1.0mm, symbol Connector:TestPoint
- added TP16: IMD_FAULT_5V, TestPoint:TestPoint_Loop_D2.50mm_Drill1.0mm, symbol Connector:TestPoint
- added TP17: AIRS+_GND, TestPoint:TestPoint_Loop_D2.50mm_Drill1.0mm, symbol Connector:TestPoint
- added TP3, TP4: GLV, TestPoint:TestPoint_Loop_D2.50mm_Drill1.0mm, symbol Connector:TestPoint
- added TP5: 5V, TestPoint:TestPoint_Loop_D2.50mm_Drill1.0mm, symbol Connector:TestPoint
- added TP6: 9V, TestPoint:TestPoint_Loop_D2.50mm_Drill1.0mm, symbol Connector:TestPoint
- added TP7: Shutdown_Acc_In, TestPoint:TestPoint_Loop_D2.50mm_Drill1.0mm, symbol Connector:TestPoint
- added TP8: Shutdown_Acc_BMS, TestPoint:TestPoint_Loop_D2.50mm_Drill1.0mm, symbol Connector:TestPoint
- added TP9: Shutdown_Acc_IMD, TestPoint:TestPoint_Loop_D2.50mm_Drill1.0mm, symbol Connector:TestPoint
- added unit 5 of U1
- added U5: HEF4093B, Package_SO:SOIC-14_3.9x8.7mm_P1.27mm, symbol 4xxx:HEF4093B
- added U6: LM555N, Package_DIP:DIP-8_W7.62mm, symbol 2FS-1_Symbol Library:LM555N
- added U7: PQDE6W-Q110-S5-H-D, 1FS_2_Global_Footprint_Library:PQDE6W-Q110-S5-H-D_CUI, symbol 1_ACC_BOARD:PQDE6W-Q110-S5-H-D
Connections:
- net CAN_1RD is gone; now on net +3.3V: CN1.CN3_13 (PA11), U3.2 (RXD)
- net CAN_H is gone; now on net +5V: J2.6 (Pin_6), R1.2, U3.6 (CANL), U3.7 (CANH)
- net +12V: now also D3.1 (K), D4.1 (K), D6.1 (K), J10.2, J10.4, J10.6, J3.2 (Pin_2), K1.8 (+), K2.8 (+), K3.5, Q3.1 (D), Q4.1 (D), Q5.1 (D), R21.2, TP3.1, TP4.1
- net +5V: now also J2.16 (Pin_16), J2.17 (Pin_17), J2.7 (Pin_7), J2.8 (Pin_8), C10.1, C11.1, J1.2, Q1.1 (D), Q2.1 (D), Q3.2 (G), Q4.2 (G), R10.1, R11.1, TP13.1, TP14.1, TP15.1, TP16.1, TP5.1, U1.4 (V+), U5.1, U5.14 (VCC), U5.2, U6.4 (R)
- net +9V: now also TP6.1
- net AIRS+_GND: now also J9.1, Q7.5 (D), Q7.6 (D), Q7.7 (D), Q7.8 (D), TP17.1
- net BMS_FAULT: now also Q2.2 (G), R9.1
- net Charge_State: now also J2.11 (Pin_11)
- net Fan_Control: now also Q8.4 (G)
- net GND: now also C11.2, C13.2, C14.1, D3.2 (A), D4.2 (A), D5.2 (A), D8.2 (A), J1.1, J3.3 (Pin_3), J7.1, J7.3, J9.3, K1.1 (-), K2.1 (-), K3.1, K4.4, Q1.3 (S), Q2.3 (S), Q3.3 (S), Q4.3 (S), Q5.3 (S), Q6.1 (S), Q6.2 (S), Q6.3 (S), Q7.1 (S), Q7.2 (S), Q7.3 (S), Q8.1 (S), Q8.2 (S), Q8.3 (S), R10.2, R11.2, R12.1, R13.2, R15.1, R17.1, R19.2, R20.1, R7.1, R8.2, R9.2, TP1.1, TP2.1, U1.11 (V-), U5.7 (GND), U6.1 (GND), U7.6
- net IMD_Status: now also R6.2, R7.2
- net Precharge_Control: now also Q7.4 (G)
- net Charge_Enable: now reaches J2.12 (Pin_12)
- net Shutdown_ACC_IN: now reaches J2.18 (Pin_18)
- net Shutdown_ACC_IN: now also K1.3, TP7.1
- net Shutdown_ACC_Out: now reaches J2.19 (Pin_19)
- net AIRS+_12V: now reaches J2.20 (Pin_20)
- net AIRS+_12V: now also D8.1 (K), J9.2, J9.4, K4.1, R18.1, TP12.1
- net Current_Output: now reaches J2.21 (Pin_21)
- net Current_Output: now also U1.5 (+), J1.3, R15.2
- net Current_Vref: now reaches J2.22 (Pin_22)
- net Current_Vref: now also U1.3 (+), J1.4
- net SH_Reset: now reaches J2.23 (Pin_23)
- net at U1.6 (-), U1.7: now also R16.2; no longer U1.5 (+)
- net at CN1.CN3_14 (PB5): now also J11.1 (Pin_1)
- net at CN1.CN3_15 (PB4): now also J11.2 (Pin_2)
- net Buffered_C_Out: now reaches CN1.CN4_11 (PA1)
- net Buffered_C_Out: now also C14.2, R16.1, R17.2
- net at CN1.CN4_15 (PB3): now also J11.3 (Pin_3)
- net at CN1.CN4_9 (PA4): now also J11.4 (Pin_4)
- new net: Q5.2 (G), R12.2, U5.3
- new net: D6.2 (A), K3.2, Q6.5 (D), Q6.6 (D), Q6.7 (D), Q6.8 (D)
- new net: J8.2, K4.3, R14.1
- new net: C10.2, R13.1, U6.2 (TR), U6.6 (THR)
- new net: C12.1, D7.2 (A), U7.3
- new net: J10.1, J10.3, J10.5, Q8.5 (D), Q8.6 (D), Q8.7 (D), Q8.8 (D)
- new net BAT+: J5.2, J6.3, K4.2
- new net BAT-: J5.1, J6.4
- new net GLV Voltage: R20.2, R21.1
- new net HVIL+: C13.1, J7.2, J7.4, U7.4
- new net IMD_FAULT: J3.1 (Pin_1), Q1.2 (G), R6.1, R8.1
- new net IMD_Latch_Delay: Q6.4 (G), U6.3 (Q)
- new net SH_RESET: D5.1 (K), K3.6
- new net Shutdown_ACC_BMS: K1.4, K2.3, TP8.1
- new net Shutdown_ACC_IL: J4.2, K3.4, TP10.1
- new net Shutdown_ACC_IMD: J4.1, K2.4, TP9.1
- new net Shutdown_ACC_OUT: K3.3, TP11.1
- new net Shutdown_Measure: R18.2, R19.1
- new net TS+: D7.1 (K), J6.1, J8.1, R14.2
- new net TS-: C12.2, J6.2, U7.2
- no-connect marks 11 -> 23
Other:
- note added: "+Vo"
- note added: "0V or 2-3.1V"
- note added: "0V or 8-12V"
- note added: "12V"
- note added: "3.7V"
- note added: "ACC Shutdown"
- note added: "AIR power from shutdown circuit; inside acc"
- note added: "Charge_Enable out from micro when charging allowed Charge_State into micro when charging"
- note added: "Current Sensor Inside ACC"
- note added: "Current Sensor Module"
- note added: "DCDC converter (110V ~ 5V)"
- note added: "Fans"
- note added: "GLV"
- note added: "GND"
- note added: "Goes to IMD; inside ACC"
- note added: "HV power in"
- note added: "HVIL"
- note added: "High Voltage"
- note added: "IMD BAT+ and BAT-"
- note added: "Latch Delay logic"
- note added: "Main shutdown logic"
- note added: "Micro drives Gate"
- note added: "Microcontroller Module"
- note added: "Outside_Connector"
- note added: "Precharge Circuit"
- note added: "Regulating FAULTS to 5V"
- note added: "STM_MISO"
- note added: "STM_MOSI"
- note added: "STM_NSS"
- note added: "STM_SCK"
- note added: "Shutdown interlock (BFC), inside ACC"
- note added: "TS"
- note added: "Test Points"
- note added: "Test point --> Micro"
- note added: "Using HV to power IMD?"
- moved on the sheet: C1, C2, C3, C4, C5, C6, C7, C8, C9, CN1A, D1, D2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

Commit message: Connector Added. Need to add CAN-SPI
Parts:
- added J12, J13: Molex Nanofit 12pin, symbol Connector:Conn_01x12_Pin
- added P1: DTM1312PC12PDR008, TE_DTM1312PC12PDR008, symbol FS_3_Global_Symbol_Library:DTM1312PC12PDR008
Connections:
- net +12V: now also J13.1 (Pin_1)
- net +5V: now also J12.8 (Pin_8), J12.9 (Pin_9)
- net Charge_State: now also J12.3 (Pin_3)
- net Current_Output: now also J12.5 (Pin_5)
- net Current_Vref: now also J12.4 (Pin_4)
- net GND: now also J13.2 (Pin_2)
- net SH_Reset: now also J12.1 (Pin_1)
- net Shutdown_ACC_IN: now also J12.12 (Pin_12)
- net Shutdown_ACC_Out: now also J12.11 (Pin_11)
- net at R16.2, U1.6 (-), U1.7: now also P1.D10
- net at R5.2, U1.1, U1.2 (-): now also P1.C7, P1.C8, P1.C9
- net Charge_Enable: no longer names the net of J2.12 (Pin_12)
- net Charge_Enable : no longer names the net of CN1.CN3_1 (PA9)
- new net CAN1_H: J13.7 (Pin_7)
- new net CAN1_H_RES: J13.5 (Pin_5)
- new net CAN1_L: J13.6 (Pin_6)
- new net CAN1_L _RES: J13.4 (Pin_4)
- new net CAN2_H: J13.12 (Pin_12)
- new net CAN2_H_RES: J13.10 (Pin_10)
- new net CAN2_L: J13.11 (Pin_11)
- new net CAN2_L _RES: J13.9 (Pin_9)
- new net IR+_GND: J13.3 (Pin_3)
- new net Shutdown_IRS_IN: J12.2 (Pin_2)
- no-connect marks 23 -> 27
Other:
- moved on the sheet: J2

Commit message: Implementing SPI -CAN. WIP
Parts:
- removed J11: Conn_01x04_Pin, symbol Connector:Conn_01x04_Pin
- removed J2: Conn_01x23, symbol Connector_Generic:Conn_01x23
- removed P1: DTM1312PC12PDR008, TE_DTM1312PC12PDR008, symbol FS_3_Global_Symbol_Library:DTM1312PC12PDR008
- added C15, C17, C20, C21, C26, C27: 100nF, symbol Device:C
- added C16: 10uF, symbol Device:C
- added C18, C19: 22pF, symbol Device:C
- added R29: 120, symbol Device:R
- added U10, U12: ISO1050DUB, Package_SO:SOP-8_6.62x9.15mm_P2.54mm, symbol Interface_CAN_LIN:ISO1050DUB
- added U8: MCP2518FD-xQBB, Package_DFN_QFN:DFN-14-1EP_3x4.5mm_P0.65mm_EP1.65x4.25mm, symbol Interface_CAN_LIN:MCP2518FD-xQBB
- added U9: LD1117S33TR_SOT223, Package_TO_SOT_SMD:SOT-223-3_TabPin2, symbol Regulator_Linear:LD1117S33TR_SOT223
- added Y1: Crystal, symbol Device:Crystal
Connections:
- net +12V: now also C15.1, U9.3 (VI)
- net +3.3V: now also C16.1, C17.1, C20.2, C26.2, U10.1 (VCC1), U12.1 (VCC1), U8.14 (VDD), U9.2 (VO); no longer CN1.CN3_13 (PA11)
- net +5V: now also J12.6 (Pin_6), J12.7 (Pin_7), C21.2, C27.2, U10.8 (VCC2), U12.8 (VCC2); no longer J12.8 (Pin_8), J12.9 (Pin_9)
- net CAN1_TD: now also U12.3 (TXD); no longer CN1.CN3_5 (PA12), U3.3 (TXD)
- net GND: now also C15.2, C16.2, C17.2, C18.2, C19.1, C20.1, C21.1, C26.1, C27.1, U10.4 (GND1), U10.5 (GND2), U12.4 (GND1), U12.5 (GND2), U8.15 (VSS), U8.7 (VSS), U9.1 (GND)
- net CAN1_RD: now reaches CN1.CN3_14 (PB5)
- net CAN1_RD: now also U12.2 (RXD)
- new net: U10.2 (RXD), U8.2 (RXCAN)
- new net: U10.3 (TXD), U8.1 (TXCAN)
- new net: C19.2, U8.6 (OSC1), Y1.1
- new net: C18.1, U8.5 (OSC2), Y1.2
- new net: R29.1, U12.6 (CANL)
- new net: R29.2, U12.7 (CANH)
- no-connect marks 27 -> 21
Other:
- added sheet Iso SPI (isoSPI.kicad_sch)
- note removed: "3.7V"
- note removed: "STM_MISO"
- note removed: "STM_MOSI"
- note removed: "STM_NSS"
- note removed: "STM_SCK"
- moved on the sheet: C1, C10, C11, C12, C13, C14, C2, C3, C4, C5, C6, C7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

Commit message: SPI-CAN added. Current Sensor updated too
Parts:
- removed C1, C14, C2, C3: 100nF, symbol Device:C
- removed unit 2 of U1
- removed unit 5 of U1
- removed U3: ISO1050DUB, Package_SO:SOP-8_6.62x9.15mm_P2.54mm, symbol Interface_CAN_LIN:ISO1050DUB
- added R30: 120, symbol Device:R
- added U13, U3: MCP6004, 1FS_2_Global_Footprint_Library:TSSOP14_MC_MCH, symbol Amplifier_Operational:MCP6004
- R1: value 120 -> R
- R15, R16, R5: value 1k -> R
- R17, R4: value 2k -> R
- U1: footprint (none) -> 1FS_2_Global_Footprint_Library:TSSOP14_MC_MCH
Connections:
- net CAN1_H_RES is gone; now on net CAN1_H: J13.5 (Pin_5)
- net CAN1_L _RES is gone; now on net CAN1_L: J13.4 (Pin_4)
- net CAN2_H_RES is gone; now on net CAN2_H: J13.10 (Pin_10)
- net CAN2_L _RES is gone; now on net CAN2_L: J13.9 (Pin_9)
- net +3.3V: no longer CN1.CN4_14 (3V3)
- net +5V: now also C27.1, J1.1; no longer C27.2, J1.2, R1.2, TP13.1, TP14.1
- net BMS_FAULT: now also CN1.CN3_6 (PB0); no longer CN1.CN3_7 (PB7)
- net CAN1_H: now also R29.2, U12.7 (CANH)
- net CAN1_L: now also R29.1, U12.6 (CANL)
- net CAN1_RD: now also CN1.CN3_13 (PA11); no longer CN1.CN3_14 (PB5)
- net CAN1_TD: now also CN1.CN3_5 (PA12)
- net CAN2_H: now also U10.7 (CANH), R30.2
- net CAN2_L: now also U10.6 (CANL), R30.1
- net Current_Output: no longer J1.3, R15.2
- net Current_Vref: no longer J1.4, U1.3 (+)
- net GND: now also C27.2, J1.2, R1.2, R17.2; no longer C27.1, J1.1, R15.1, R17.1, R4.1
- net IMD_Status: now also CN1.CN3_1 (PA9); no longer CN1.CN3_6 (PB0)
- net at R16.2: now also CN1.CN4_11 (PA1), R17.1
- net ST_MISO: now reaches CN1.CN3_15 (PB4)
- net SPI_Tx: now reaches CN1.CN3_8 (PB6)
- net STM_SCK: now reaches CN1.CN4_15 (PB3)
- net STM_SCK: now also U8.10 (SCK)
- net STM_NSS: now reaches CN1.CN4_9 (PA4)
- net STM_NSS: now also U8.13 (~{CS})
- net at U1.1, U1.2 (-): now also R4.1; no longer R5.2
- net STM_MOSI: now reaches U8.11 (SDI)
- net STM_MOSI: now also CN1.CN3_14 (PB5)
- net STM_MISO: now reaches U8.12 (SDO)
- removed net Buffered_C_Out: CN1.CN4_11 (PA1), R16.1, R17.2
- removed net Buffered_C_Vref: CN1.CN4_10 (PA3), R4.2, R5.1
- net CAN_L_RES: no longer names the net of R1.1
- net CAN_L_RES: now also R4.2, U13.3 (+)
- new net: J1.3, U1.3 (+)
- new net: J1.4, U3.3 (+)
- new net: R15.1, R5.2, U13.2 (-)
- new net: R15.2, R16.1, U13.1
- new net: R5.1, U3.1, U3.2 (-)
- new net CAN_H: TP13.1
- new net CAN_L: TP14.1
- new net SPI_Rx: CN1.CN3_7 (PB7)
Other:
- note removed: "3.3V"
- note removed: "CAN Transciever"
- note removed: "Charge_Enable out from micro when charging allowed Charge_State into micro when charging"
- note removed: "Current Sensor Inside ACC"
- note removed: "Current Sensor Module"
- moved on the sheet: C17, C18, C19, C20, C21, C26, C27, CN1A, D1, R18, R19, R2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
