File: Acc_Board_Christian/FS_3_Accumulator_Board/isoSPI.kicad_sch (KiCad schematic)
At the start: 16 parts, among them J2 IsoSPI, U11 LTC6820

Commit message: New Micro added to acc board
Parts:
- renumbered C22 to C34, C23 to C35, C24 to C36, C25 to C37, J2 to J17, L1 to L2, R22 to R35, R23 to R36, R24 to R37, R25 to R38, R26 to R39, R27 to R40, R28 to R41, TP18 to TP20, TP19 to TP21, U11 to U22
