File: Precharge/Precharge.kicad_sch (KiCad schematic)
At the start: 5 parts, among them K1 Relay_SPST-NO

Commit message: precharge pcb (still wip)
edited schematics to have connectors, connected pcb together
Parts:
- removed R1, R2: 57.692/2, Library:HSA1030RJ, symbol Device:R
- added J1: Conn_01x02, Connector_Molex:Molex_Nano-Fit_105309-xx02_1x02_P2.50mm_Vertical, symbol Connector_Generic:Conn_01x02
- added J2: Conn_01x04, Connector_Molex:Molex_Nano-Fit_105309-xx04_1x04_P2.50mm_Vertical, symbol Connector_Generic:Conn_01x04
- added J3: Conn_01x01, Connector_Molex:Molex_Nano-Fit_105309-xx02_1x02_P2.50mm_Vertical, symbol Connector_Generic:Conn_01x01
- CR1: footprint Library:SO-8_STM -> Package_SO:SOIC-8_3.9x4.9mm_P1.27mm
- K1: footprint Library:G5PZ-1A-X DC12 -> FS_3_Global_Footprint_Library:G5PZ-1A-X DC12
Connections:
- net AIRS+: now also J2.1 (Pin_1), J2.2 (Pin_2), J2.3 (Pin_3), J2.4 (Pin_4)
- net GND: now also K1.4; no longer K1.A2
- net Precharge Control: now also J3.1 (Pin_1)
- net Shutdown: now also K1.1; no longer K1.A1
- new net BAT+_RES: J1.2 (Pin_2), K1.3
- new net TS+_RES: J1.1 (Pin_1), K1.2

Commit message: changes to connections
changed connector pin for airs+ from 1x4 to 1x2, increased width of airs+ traces, moved connectors around
Parts:
- removed J2: Conn_01x04, Connector_Molex:Molex_Nano-Fit_105309-xx04_1x04_P2.50mm_Vertical, symbol Connector_Generic:Conn_01x04
- added J4: Conn_01x01, Connector_Molex:Molex_Nano-Fit_105309-xx02_1x02_P2.50mm_Vertical, symbol Connector_Generic:Conn_01x01
Connections:
- net AIRS+: now also J4.1 (Pin_1)
Changed lines of the file:
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@@
-	)
-	(junction
-		(at 160.02 118.11)
-		(diameter 0)
-		(color 0 0 0 0)
 	)
 	(junction
@@
 	(wire
 		(pts
-			(xy 160.02 123.19) (xy 162.56 123.19)
-		)
-		(stroke
-			(width 0)
-			(type default)
-		)
-	)
-	(wire
-		(pts
 			(xy 118.11 120.65) (xy 118.11 123.19)
 		)
@@
 	(wire
 		(pts
-			(xy 160.02 118.11) (xy 162.56 118.11)
-		)
-		(stroke
-			(width 0)
-			(type default)
-		)
-	)
-	(wire
-		(pts
 			(xy 127 71.12) (xy 127 78.74)
 		)
@@
 	(wire
 		(pts
-			(xy 160.02 125.73) (xy 162.56 125.73)
-		)
-		(stroke
-			(width 0)
-			(type default)
-		)
-	)
-	(wire
-		(pts
 			(xy 160.02 123.19) (xy 160.02 125.73)
-		)
-		(stroke
-			(width 0)
-			(type default)
-		)
-	)
-	(wire
-		(pts
-			(xy 160.02 120.65) (xy 162.56 120.65)
 		)
 		(stroke
@@
 				(justify right)
 				(hide yes)
+			)
+		)
+	)
+	(symbol
+		(lib_id "Connector_Generic:Conn_01x01")
+		(at 165.1 128.27 0)
+		(unit 1)
+		(exclude_from_sim no)
+		(in_bom yes)
+		(on_board yes)
+		(dnp no)
+		(fields_autoplaced yes)
+		(property "Reference" "J4"
+			(at 167.64 126.9999 0)
+			(effects
+				(font
+					(size 1.27 1.27)
+				)
+				(justify left)
+			)
+		)
+		(property "Value" "Conn_01x01"
+			(at 167.64 129.5399 0)
+			(effects
+				(font
+					(size 1.27 1.27)
+				)
+				(justify left)
+			)
+		)
+		(property "Footprint" "Connector_Molex:Molex_Nano-Fit_105309-xx02_1x02_P2.50mm_Vertical"
+			(at 165.1 128.27 0)
+			(effects
+				(font
+					(size 1.27 1.27)
+				)
+				(hide yes)
+			)
+		)
+		(property "Datasheet" "~"
+			(at 165.1 128.27 0)
+			(effects
+				(font
+					(size 1.27 1.27)
+				)
+				(hide yes)
+			)
+		)
+		(property "Description" "Generic connector, single row, 01x01, script generated (kicad-library-utils/schlib/autogen/connector/)"
+			(at 165.1 128.27 0)
+			(effects
+				(font
+					(size 1.27 1.27)
+				)
+				(hide yes)
+			)
+		)
+		(pin "1"
+		)
+		(instances
+			(project "Precharge"
+				(path "/f73cc31d-1bab-4ab9-be2f-0e022f0be386"
+					(reference "J4")
+					(unit 1)
+				)
 			)
 		)
@@
 					(unit 1)
 				)
-			)
-		)
-	)
-	(symbol
-		(lib_id "Connector_Generic:Conn_01x04")
-		(at 167.64 120.65 0)
-		(unit 1)
-		(exclude_from_sim no)
-		(in_bom yes)
-		(on_board yes)
-		(dnp no)
-		(property "Reference" "J2"
-			(at 170.18 120.6499 0)
-			(effects
-				(font
-					(size 1.27 1.27)
-				)
-				(justify left)
-			)
-		)
-		(property "Value" "Conn_01x04"
-			(at 170.18 123.1899 0)
-			(effects
-				(font
-					(size 1.27 1.27)
-				)
-				(justify left)
-			)
-		)
-		(property "Footprint" "Connector_Molex:Molex_Nano-Fit_105309-xx04_1x04_P2.50mm_Vertical"
-			(at 167.64 120.65 0)
-			(effects
-				(font
-					(size 1.27 1.27)
-				)
-				(hide yes)
-			)
-		)
-		(property "Datasheet" "~"
-			(at 167.64 120.65 0)
-			(effects
-				(font
-					(size 1.27 1.27)
-				)
-				(hide yes)
-			)
-		)
-		(property "Description" "Generic connector, single row, 01x04, script generated (kicad-library-utils/schlib/autogen/connector/)"
-			(at 167.64 120.65 0)
-			(effects
-				(font
-					(size 1.27 1.27)
-				)
-				(hide yes)
-			)
-		)
-		(pin "3"
-		)
-		(pin "2"
-		)
-		(pin "1"
-		)
-		(pin "4"
-		)
-		(instances
-			(project ""
-				(path "/f73cc31d-1bab-4ab9-be2f-0e022f0be386"
-					(reference "J2")
-					(unit 1)
-				)

Commit message: Inverter Added
Changed schematics and PCB by including new inverter
Parts:
- removed J3, J4: Conn_01x01, Connector_Molex:Molex_Nano-Fit_105309-xx02_1x02_P2.50mm_Vertical, symbol Connector_Generic:Conn_01x01
- added CR2: STS6NF20V, Package_SO:SO-8_3.9x4.9mm_P1.27mm, symbol 1FS_2_Global_Symbol_Library:STS6NF20V
- added U1: 74AHC1G04, Package_TO_SOT_SMD:SOT-23-5, symbol 74xGxx:74AHC1G04
- CR1: footprint Package_SO:SOIC-8_3.9x4.9mm_P1.27mm -> Package_SO:SO-8_3.9x4.9mm_P1.27mm
Connections:
- net GND: now also CR2.1 (S), CR2.2 (S), CR2.3 (S), U1.3 (GND); no longer D1.2 (A), K1.4
- net Precharge Control: now also U1.2
- net AIRS+ renamed IR+
- net BAT+_RES renamed BAT+
- net TS+_RES renamed TS+
- new net: CR2.4 (G), U1.4
- new net: CR2.5 (D), CR2.6 (D), CR2.7 (D), CR2.8 (D), D1.2 (A), K1.4
Other:
- moved on the sheet: CR1
