File: ACC Board Shutdown/ACC Board Shutdown.kicad_sch (KiCad schematic)
At the start: 33 parts, among them J1 IMD, J2 Shutdown IL, K1 DK1A1B-5V, K2 DK1A1B-5V, K3 DK1A1B-5V, K4 G6BK-1114P-US, U1 74AHC1G04, U1 HEF4093B, U1 LM555xN, U2 74AHC1GU04, U3 74AHC1GU04, U4 74AHC1GU04

Commit message: Update ACC Board Shutdown.kicad_sch
Parts:
- removed C2: 1uf, symbol Device:C
- removed C3, C4, C5, C7, C8: 100uF, symbol Device:C
- removed R3: 1.8M, symbol Device:R
- removed U1: LM555xN, Package_DIP:DIP-8_W7.62mm, symbol Timer:LM555xN
- removed U2, U3, U4: 74AHC1GU04, symbol 74xGxx:74AHC1GU04
- added C10: 1uf, symbol Device:C
- added C11, C9: 100uF, symbol Device:C
- added R4: 10k, symbol Device:R
- added U5: LM555xN, Package_DIP:DIP-8_W7.62mm, symbol Timer:LM555xN
Connections:
- net GND is gone; now on net +5V: C1.1, CR1.1 (S), CR1.3 (S), CR2.1 (S), CR2.2 (S), CR2.3 (S), CR3.1 (S), CR3.2 (S), CR3.3 (S), CR4.1 (S), CR4.2 (S), CR4.3 (S), J1.3, R2.1, U1.5 (VCC), U1.7 (GND)
- net +5V: now also C6.1, U1.3 (GND), C11.1, C9.1, R4.2, U5.1 (GND)
- net IMD_DELAY: now also U1.1, U1.11
- net IMD_FAULT: now also U1.8; no longer U1.1
- net at U1.13: now also U1.10, U1.12
- net at U1.9: now also U5.3 (Q)
- new net: C10.2, C9.2, U5.4 (R)
- new net: C10.1, R4.1, U5.2 (TR), U5.6 (THR)
- new net: C11.2, U5.8 (VCC)
Other:
- note added: "On fault condition triggers TSSI light"
- note added: "Upstream delay of ~2sec durring power on"
- note removed: "Light goes off board to trigger TSSI"
- note removed: "Upstream delay of ~6sec durring power on"
- moved on the sheet: C1, C6, CR4, U1, U1A, U1B, U1E

Commit message: Update to Pinouts
Connections:
- net BSPD_FAULT is gone; now on net BSPD_FAULT_5V: CR3.4 (G)
Other:
- note added: "--> BMS Relay"
- note added: "--> BSPD Relay"
- note added: "--> IMD Relay"
Changed lines of the file:
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@@
 		(title "Accumulator Shutdown Logic")
 		(date "2024-10-27")
-		(rev "1")
+		(rev "3")
 		(company "Ethan James - Formula Slug")
 	)
@@
 	(wire
 		(pts
+			(xy 185.42 124.46) (xy 181.61 124.46)
+		)
+		(stroke
+			(width 0)
+			(type default)
+		)
+	)
+	(wire
+		(pts
 			(xy 133.35 119.38) (xy 140.97 119.38)
 		)
@@
 	(wire
 		(pts
+			(xy 74.93 124.46) (xy 69.85 124.46)
+		)
+		(stroke
+			(width 0)
+			(type default)
+		)
+	)
+	(wire
+		(pts
 			(xy 175.26 72.39) (xy 181.61 72.39)
 		)
@@
 	(wire
 		(pts
+			(xy 185.42 127) (xy 185.42 124.46)
+		)
+		(stroke
+			(width 0)
+			(type default)
+		)
+	)
+	(wire
+		(pts
 			(xy 68.58 88.9) (xy 68.58 91.44)
 		)
@@
 	(wire
 		(pts
+			(xy 128.27 124.46) (xy 124.46 124.46)
+		)
+		(stroke
+			(width 0)
+			(type default)
+		)
+	)
+	(wire
+		(pts
 			(xy 100.33 91.44) (xy 109.22 91.44)
 		)
@@
 	(wire
 		(pts
+			(xy 128.27 125.73) (xy 128.27 124.46)
+		)
+		(stroke
+			(width 0)
+			(type default)
+		)
+	)
+	(wire
+		(pts
 			(xy 163.83 72.39) (xy 163.83 78.74)
 		)
@@
 	(wire
 		(pts
-			(xy 181.61 124.46) (xy 196.85 124.46)
-		)
-		(stroke
-			(width 0)
-			(type default)
-		)
-	)
-	(wire
-		(pts
 			(xy 83.82 127) (xy 83.82 129.54)
 		)
@@
 	(wire
 		(pts
+			(xy 74.93 135.89) (xy 74.93 124.46)
+		)
+		(stroke
+			(width 0)
+			(type default)
+		)
+	)
+	(wire
+		(pts
 			(xy 134.62 91.44) (xy 138.43 91.44)
 		)
@@
 	(wire
 		(pts
-			(xy 124.46 124.46) (xy 137.16 124.46)
-		)
-		(stroke
-			(width 0)
-			(type default)
-		)
-	)
-	(wire
-		(pts
 			(xy 83.82 129.54) (xy 83.82 132.08)
 		)
@@
 		(pts
 			(xy 41.91 63.5) (xy 45.72 63.5)
-		)
-		(stroke
-			(width 0)
-			(type default)
-		)
-	)
-	(wire
-		(pts
-			(xy 69.85 124.46) (xy 81.28 124.46)
 		)
 		(stroke
@@
 		)
 	)
+	(text "--> IMD Relay"
+		(exclude_from_sim no)
+		(at 30.48 115.824 0)
+		(effects
+			(font
+				(size 1.27 1.27)
+			)
+		)
+	)
 	(text "SMD NAND GATE"
 		(exclude_from_sim no)
@@
 		)
 	)
+	(text "--> BSPD Relay"
+		(exclude_from_sim no)
+		(at 78.74 115.824 0)
+		(effects
+			(font
+				(size 1.27 1.27)
+			)
+		)
+	)
 	(text "BMS Fault Low --> 5V Relay"
 		(exclude_from_sim no)
@@
 		)
 	)
+	(text "--> BMS Relay"
+		(exclude_from_sim no)
+		(at 137.668 115.57 0)
+		(effects
+			(font
+				(size 1.27 1.27)
+			)
+		)
+	)
 	(text "On fault condition triggers TSSI light"
 		(exclude_from_sim no)
@@
 	)
 	(label "IMD_DELAY"
-		(at 81.28 124.46 180)
-		(fields_autoplaced yes)
-		(effects
-			(font
-				(size 1.27 1.27)
-			)
-			(justify right bottom)
+		(at 74.93 135.89 90)
+		(fields_autoplaced yes)
+		(effects
+			(font
+				(size 1.27 1.27)
+			)
+			(justify left bottom)
 		)
 	)
@@
 		)
 	)
-	(label "BSPD_FAULT"
-		(at 137.16 124.46 180)
-		(fields_autoplaced yes)
-		(effects
-			(font
-				(size 1.27 1.27)
-			)
-			(justify right bottom)
-		)
-	)
 	(label "BSPD_RL"
 		(at 74.93 119.38 0)
@@
 		)
 	)
-	(label "BMS_FAULT_5V"
-		(at 196.85 124.46 180)
-		(fields_autoplaced yes)
-		(effects
-			(font
-				(size 1.27 1.27)
-			)
-			(justify right bottom)
-		)
-	)
 	(label "IMD_DELAY"
 		(at 273.05 82.55 180)
@@
 			)
 			(justify right bottom)
+		)
+	)
+	(hierarchical_label "BSPD_FAULT_5V"
+		(shape input)
+		(at 128.27 125.73 270)
+		(fields_autoplaced yes)
+		(effects
+			(font
+				(size 1.27 1.27)
+			)
+			(justify right)
 		)
 	)
@@
 		)
 	)
+	(hierarchical_label "BMS_FAULT_5V"
+		(shape input)
+		(at 185.42 127 270)
+		(fields_autoplaced yes)
+		(effects
+			(font
+				(size 1.27 1.27)
+			)
+			(justify right)
+		)
+	)

Commit message: Update components and layout
Resistor updated to 10MOhms on 555, remove decoupling capacitor from 5V to reset pin on 555, Add NOT gate between NAND and MOSFET to fix logic.
Parts:
- removed C11, C9: 100uF, symbol Device:C
- added C2, C3: 100uF, symbol Device:C
- added U2: 74AHC1G04, symbol 74xGxx:74AHC1G04
- R4: value 10k -> 10M
Connections:
- net +5V: now also C10.2, U5.4 (R), U5.8 (VCC), C2.1, C3.1, U2.5 (VCC); no longer C1.1, C6.2, CR1.1 (S), CR1.3 (S), CR2.1 (S), CR2.2 (S), CR2.3 (S), CR3.1 (S), CR3.2 (S), CR3.3 (S), CR4.1 (S), CR4.2 (S), CR4.3 (S), J1.3, R2.1, R4.2, U1.3 (GND), U1.7 (GND), U5.1 (GND)
- net at CR4.4 (G): now also U2.4; no longer U1.4
- new net: U1.4, U2.2
- new net GND: C1.1, C2.2, C3.2, C6.2, CR1.1 (S), CR1.3 (S), CR2.1 (S), CR2.2 (S), CR2.3 (S), CR3.1 (S), CR3.2 (S), CR3.3 (S), CR4.1 (S), CR4.2 (S), CR4.3 (S), J1.3, R2.1, R4.2, U1.3 (GND), U1.7 (GND), U2.3 (GND), U5.1 (GND)
Other:
- note added: "555 Timer ~10 sec on 5V Power"
- note removed: "555 Timer ~2 sec on 5V Power"
- moved on the sheet: C6, U1, U1A, U1B

Commit message: Update 555 Logic
Parts:
- removed C10: 1uf, symbol Device:C
- removed C3: 100uF, symbol Device:C
- removed CR3: STS6NF20V, SO-8_STM, symbol FS_2_Global_Symbol_Library:STS6NF20V
- removed D5: D, Diode_SMD:D_2010_5025Metric_Pad1.52x2.65mm_HandSolder, symbol Device:D
- removed K2: DK1A1B-5V, FS_3_Global_Footprint_Library:DK1A1B, symbol 2FS-1_Symbol Library:DK1A1B-12V
- removed unit 3 of U1
- removed unit 4 of U1
- added C3: 1uF, symbol Device:C_Polarized
- added C4, C5: 100uF, symbol Device:C
- added R3: 10k, symbol Device:R
- added R5: 7.2k, symbol Device:R
- added U3: 74AHC1G32, symbol 74xGxx:74AHC1G32
Connections:
- net Shutdown_ACC_BSPD is gone; now on net Shutdown_ACC_BMS: K3.3
- net +5V: now also R4.2, C4.1, C5.2, U3.5 (VCC)
- net GND: now also C3.2, C4.2, C5.1, R3.2, U3.3 (GND); no longer R4.2
- net IMD_DELAY: now also U3.4
- net at R4.1, U5.2 (TR), U5.6 (THR): now also C3.1
- net at U5.3 (Q): now also U3.2
- net IMD_FAULT renamed IMD_FAULT_12V
- net IMD_FAULT_12V: now also R5.1
- new net: R3.1, R5.2, U3.1
- no-connect marks 8 -> 6
Other:
- note added: "12V --> ~5V Input to LV Logic at 5V"
- note added: "555 Timer ~11 sec on 5V Power"
- note added: "Upstream delay of ~11sec durring power on"
- note removed: "--> BSPD Relay"
- note removed: "555 Timer ~10 sec on 5V Power"
- note removed: "BSPD Fault Low --> 5V Relay"
- note removed: "BSPD Relay"
- note removed: "Upstream delay of ~2sec durring power on"
- moved on the sheet: C1, CR2, U1E, U5
