File: Power Distrobution Board/Power DIstrobution Board.kicad_pcb (KiCad board)
At the start: 2 copper layers, 158.5 x 73.7 mm, 43 parts, among them CN2 NUCLEO-L432KC, J2 Conn_01x10_Pin, J3 0768250004, J4 Conn_01x04_Pin, K3 AZ2150-1A-12DEF, U1 3.3v linear reg, U10 ACS71240LLCBTR-025B3, U11 ACS71240LLCBTR-025B3, U12 ACS71240LLCBTR-025B3, U13 CD74HC4067M, U14 MC7809CTG 9v linear reg, U15 MC7809CTG 9v linear reg, U16 ACS71240LLCBTR-025B3, U17 ACS71240LLCBTR-025B3, U18 ISO1050DUB, U2 ACS71240LLCBTR-025B3, U3 ACS71240LLCBTR-025B3, U4 ACS71240LLCBTR-025B3, U5 ACS71240LLCBTR-025B3, U7 ACS71240LLCBTR-025B3, U8 ACS71240LLCBTR-025B3, U9 ACS71240LLCBTR-025B3

Commit message: version 1.1
Parts:
- added C10: C_Small, Capacitor_SMD:C_0805_2012Metric_Pad1.18x1.45mm_HandSolder, F.Cu at (208.0, 47.0)
- added C11: C_Small, Capacitor_SMD:C_0805_2012Metric_Pad1.18x1.45mm_HandSolder, F.Cu at (129.5, 81.0)
- added C12: C_Small, Capacitor_SMD:C_0805_2012Metric_Pad1.18x1.45mm_HandSolder, F.Cu at (125.0, 58.2)
- added C13: C_Small, Capacitor_SMD:C_0805_2012Metric_Pad1.18x1.45mm_HandSolder, F.Cu at (207.8, 42.5)
- added C14: C_Small, Capacitor_SMD:C_0805_2012Metric_Pad1.18x1.45mm_HandSolder, F.Cu at (140.5, 55.0)
- added C15: C_Small, Capacitor_SMD:C_0805_2012Metric_Pad1.18x1.45mm_HandSolder, F.Cu at (143.5, 71.8)
- added C16: C_Small, Capacitor_SMD:C_0805_2012Metric_Pad1.18x1.45mm_HandSolder, F.Cu at (118.0, 80.5)
- added C17: C_Small, Capacitor_SMD:C_0805_2012Metric_Pad1.18x1.45mm_HandSolder, F.Cu at (173.8, 54.5)
- added C18: C_Small, Capacitor_SMD:C_0805_2012Metric_Pad1.18x1.45mm_HandSolder, F.Cu at (152.0, 53.0)
- added C19: C_Small, Capacitor_SMD:C_0805_2012Metric_Pad1.18x1.45mm_HandSolder, F.Cu at (141.2, 81.2)
- added C20: C_Small, Capacitor_SMD:C_0805_2012Metric_Pad1.18x1.45mm_HandSolder, F.Cu at (152.8, 81.0)
- added C21: C_Small, Capacitor_SMD:C_0805_2012Metric_Pad1.18x1.45mm_HandSolder, F.Cu at (163.5, 80.0)
- added C22: C_Small, Capacitor_SMD:C_0805_2012Metric_Pad1.18x1.45mm_HandSolder, F.Cu at (162.8, 54.5)
- added C4: C_Small, Capacitor_SMD:C_0805_2012Metric_Pad1.18x1.45mm_HandSolder, F.Cu at (223.0, 34.5)
- added C6: C_Small, Capacitor_SMD:C_0805_2012Metric_Pad1.18x1.45mm_HandSolder, F.Cu at (184.8, 51.0)
- added C9: C_Small, Capacitor_SMD:C_0805_2012Metric_Pad1.18x1.45mm_HandSolder, F.Cu at (174.8, 78.8)
- moved U18 48.0 mm to (215.8, 38.5), turned to 0 degrees
- moved C1 42.7 mm to (172.8, 68.2)
- moved C3 42.7 mm to (172.8, 65.2)
- moved U1 42.7 mm to (178.0, 66.8)
Connections:
- J2 pad 8: unconnected-(J2-Pin_8-Pad8) -> brake_pressure_sensor_9v
Routing:
- net GND: track 71.1 -> 116.0 mm, vias 19 -> 21
- net +3.3V: track 234.1 -> 278.2 mm, vias 17 -> 25
- net Net-(CN2A-PA11): track 13.5 -> 55.3 mm, vias 0 -> 4
- net CAN H: track 57.6 -> 39.5 mm, vias 4 -> 0
- net Net-(CN2A-PA12): track 13.4 -> 31.1 mm, vias 2 -> 1
- net CAN L: track 58.2 -> 40.6 mm, vias 2 -> 0
- net Net-(J3-Pin_4): track 0.00 -> 17.6 mm
- net Net-(D1-K): track 81.8 -> 66.6 mm
- net shutdown_viout: track 17.4 -> 12.5 mm
- net accumulator_viout: track 28.9 -> 24.1 mm
- net +5V: track 50.0 -> 45.4 mm, vias 4 -> 0
- net brake_pressure_sensor_9v: track 12.0 -> 16.3 mm
- net +9V: track 12.5 -> 16.1 mm
- net dash_viout: track 39.0 -> 35.5 mm
- net pd_board_out: track 98.7 -> 96.0 mm, vias 8 -> 7
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
Commit message: v1.3
changed footprint of linear regulators
Parts:
- U1: value 3.3v linear reg -> LD1117V33C 3.3v linear reg; footprint Package_TO_SOT_SMD:SOT-89-3 -> Package_TO_SOT_THT:TO-220-3_Horizontal_TabDown
- U14, U15: footprint Package_TO_SOT_SMD:SOT-89-3 -> Package_TO_SOT_THT:TO-220-3_Horizontal_TabDown
- moved C2 44.3 mm to (216.8, 96.7), turned to 180 degrees
- moved C5 42.1 mm to (220.9, 96.8)
- moved U14 40.0 mm to (215.8, 94.2)
- moved C8 20.5 mm to (211.6, 97.5), turned to -90 degrees
- moved U15 19.9 mm to (209.0, 96.9), turned to 90 degrees
- moved C7 13.0 mm to (211.8, 93.0), turned to 90 degrees
- moved C1 9.45 mm to (181.4, 64.5), turned to 90 degrees
- moved C3 9.21 mm to (181.4, 68.5), turned to -90 degrees
- moved U1 2.34 mm to (178.7, 69.0), turned to 90 degrees
Routing:
- net +9V: track 16.1 -> 78.7 mm, vias 0 -> 2
- net brake_pressure_sensor_9v: track 16.3 -> 39.5 mm
- net pd_board_out: track 96.0 -> 112.7 mm
- net GND: track 116.0 -> 108.7 mm, vias 21 -> 18
- net extra1_viout: track 50.7 -> 43.6 mm, vias 0 -> 2
- net brake_pressure_sensor_out: track 47.1 -> 51.5 mm
- net +3.3V: track 278.2 -> 276.3 mm, vias 25 -> 26
- net Net-(CN2A-PB0): track 78.2 -> 76.5 mm
- net extra1_out: track 51.1 -> 49.5 mm
- net Net-(CN2A-PB6): track 59.0 -> 59.9 mm
- net Net-(CN2A-PB7): track 55.7 -> 56.6 mm
- net Net-(CN2A-PA9): track 61.8 -> 61.0 mm
- net Net-(CN2A-PA10): track 59.5 -> 58.8 mm
Other:
- board text added: "FS-3 Power Distrobution Board V1.3 Formula Slug PCB Designed By: Aaron Gondo Schematic Designed By: Niwa Babista, Jaelyn Flores, Aaron Gondo, Nataniel Jayaseelan,Shreyas J Kiran, Francesco Menegoli,Dylan Ortiz , Atul Pethe, Muneeb Syed"
- board text removed: "Power Distrobution Board V1.1"

Commit message: changes after cdr
Parts:
- added J1: 768250002, Connector_Molex:Molex_Mega-Fit_76825-0002_2x01_P5.70mm_Horizontal, F.Cu at (108.2, 83.8)
- C1: value C_Small -> .33nF
- C10: value C_Small -> 904.7nF?
- C11, C12, C13, C14, C15, C16, C17, C18, C19, C20, C21, C22, C9: value C_Small -> 0.1nF
- C2, C4, C6: value C_Small -> .01nF
- C3: value C_Small -> 10nF
- C5: value C_Small -> 100nF
- C7: value C_Small -> 0.33nF
- C8: value C_Small -> 0.01nF
- D1: value D -> ACGRAT105L-HF
- moved F1 21.2 mm to (113.6, 66.6), turned to -90 degrees
- moved K3 9.10 mm to (82.0, 58.1)
- moved C16 6.53 mm to (121.0, 74.7)
- moved J3 2.85 mm to (87.2, 96.0)
Connections:
- F1 pad 1: +12V -> Net-(J1-Pin_2)
Routing:
- net Net-(D1-K): track 66.6 -> 85.6 mm
- net dcdc_ctrl: track 30.3 -> 43.5 mm
- net Net-(J1-Pin_2): track 0.00 -> 9.97 mm
- net +3.3V: track 276.3 -> 286.0 mm
- net +12V: track 206.6 -> 214.3 mm
- net Net-(J3-Pin_4): track 17.6 -> 22.4 mm
- net GND: track 108.7 -> 110.9 mm
- net CAN L: track 40.6 -> 39.2 mm
- net CAN H: track 39.5 -> 38.2 mm
- net Net-(CN2A-PB6): vias 2 -> 0

Commit message: even newer changes
Parts:
- moved CR1 2.97 mm to (119.6, 63.9)
Connections:
- C4 pad 1: +5V -> GND
- C4 pad 2: GND -> +5V
- CN2 pad CN3_14: Net-(CN2A-PB5) -> dcdc_ctrl
- CR1 pad 4: Net-(CN2A-PB5) -> dcdc_ctrl
- CR1 pad 5: dcdc_ctrl -> Net-(D1-A)
- CR1 pad 6: dcdc_ctrl -> Net-(D1-A)
- CR1 pad 7: dcdc_ctrl -> Net-(D1-A)
- CR1 pad 8: dcdc_ctrl -> Net-(D1-A)
- D1 pad 2: dcdc_ctrl -> Net-(D1-A)
- J3 pad 2: GND -> Net-(J3-Pin_2)
- J3 pad 4: Net-(J3-Pin_4) -> GND
- K3 pad 2: Net-(J3-Pin_4) -> Net-(J3-Pin_2)
- K3 pad 5: dcdc_ctrl -> Net-(D1-A)
Routing:
- net Net-(CN2A-PB5): track 83.4 -> 0.00 mm, vias 6 -> 0
- net Net-(D1-A): track 0.00 -> 43.6 mm
- net dcdc_ctrl: track 43.5 -> 80.3 mm, vias 0 -> 6
- net Net-(J3-Pin_4): track 22.4 -> 0.00 mm
- net Net-(J3-Pin_2): track 0.00 -> 20.8 mm
- net GND: track 110.9 -> 113.4 mm, vias 18 -> 16
- net +5V: track 45.4 -> 47.0 mm, vias 0 -> 1

Commit message: fixed backwards cap
Parts:
- moved C4 0.10 mm to (223.0, 34.4), turned to 90 degrees
- renumbered J1 to CON_GLVMS
Routing:
- net GND: track 113.4 -> 115.0 mm, vias 16 -> 17
- net +5V: track 47.0 -> 45.4 mm, vias 1 -> 0
Changed lines of the file:
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@@
 	(footprint "Capacitor_SMD:C_0805_2012Metric_Pad1.18x1.45mm_HandSolder"
 		(layer "F.Cu")
-		(at 223 34.4625 -90)
+		(at 222.99 34.36 90)
 		(descr "Capacitor SMD 0805 (2012 Metric), square (rectangular) end terminal, IPC_7351 nominal with elongated pad for handsoldering. (Body size source: IPC-SM-782 page 76, https://www.pcb-3d.com/wordpress/wp-content/uploads/ipc-sm-782a_amendment_1_and_2.pdf, https://docs.google.com/spreadsheets/d/1BsfQQcO9C6DZCsRaXUlFlo91Tg2WpOkGARC1WS5S8t0/edit?usp=sharing), generated with kicad-footprint-generator")
 		(tags "capacitor handsolder")
 		(property "Reference" "C4"
-			(at -2.5825 -0.03 180)
+			(at -2.5825 -0.03 360)
 			(layer "F.SilkS")
 			(effects
@@
 		)
 		(property "Footprint" "Capacitor_SMD:C_0805_2012Metric_Pad1.18x1.45mm_HandSolder"
-			(at 0 0 -90)
+			(at 0 0 90)
 			(unlocked yes)
 			(layer "F.Fab")
@@
 		)
 		(property "Datasheet" "https://www.yageo.com/upload/media/product/productsearch/datasheet/mlcc/UPY-GPHC_X7R_6.3V-to-250V_24.pdf"
-			(at 0 0 -90)
+			(at 0 0 90)
 			(unlocked yes)
 			(layer "F.Fab")
@@
 		)
 		(property "Description" "Unpolarized capacitor, small symbol"
-			(at 0 0 -90)
+			(at 0 0 90)
 			(unlocked yes)
 			(layer "F.Fab")
@@
 		(attr smd)
 		(fp_line
-			(start -0.261252 0.735)
-			(end 0.261252 0.735)
+			(start -0.261252 -0.735)
+			(end 0.261252 -0.735)
 			(stroke
 				(width 0.12)
@@
 		)
 		(fp_line
-			(start -0.261252 -0.735)
-			(end 0.261252 -0.735)
+			(start -0.261252 0.735)
+			(end 0.261252 0.735)
 			(stroke
 				(width 0.12)
@@
 		)
 		(fp_line
-			(start -1.88 0.98)
-			(end -1.88 -0.98)
+			(start 1.88 -0.98)
+			(end 1.88 0.98)
 			(stroke
 				(width 0.05)
@@
 		)
 		(fp_line
-			(start 1.88 0.98)
-			(end -1.88 0.98)
+			(start -1.88 -0.98)
+			(end 1.88 -0.98)
 			(stroke
 				(width 0.05)
@@
 		)
 		(fp_line
-			(start -1.88 -0.98)
-			(end 1.88 -0.98)
+			(start 1.88 0.98)
+			(end -1.88 0.98)
 			(stroke
 				(width 0.05)
@@
 		)
 		(fp_line
-			(start 1.88 -0.98)
-			(end 1.88 0.98)
+			(start -1.88 0.98)
+			(end -1.88 -0.98)
 			(stroke
 				(width 0.05)
@@
 		)
 		(fp_line
-			(start -1 0.625)
-			(end -1 -0.625)
+			(start 1 -0.625)
+			(end 1 0.625)
 			(stroke
 				(width 0.1)
@@
 		)
 		(fp_line
-			(start 1 0.625)
-			(end -1 0.625)
+			(start -1 -0.625)
+			(end 1 -0.625)
 			(stroke
 				(width 0.1)
@@
 		)
 		(fp_line
-			(start -1 -0.625)
-			(end 1 -0.625)
+			(start 1 0.625)
+			(end -1 0.625)
 			(stroke
 				(width 0.1)
@@
 		)
 		(fp_line
-			(start 1 -0.625)
-			(end 1 0.625)
+			(start -1 0.625)
+			(end -1 -0.625)
 			(stroke
 				(width 0.1)
@@
 		)
 		(pad "1" smd roundrect
-			(at -1.0375 0 270)
+			(at -1.0375 0 90)
 			(size 1.175 1.45)
 			(layers "F.Cu" "F.Paste" "F.Mask")
@@
 		)
 		(pad "2" smd roundrect
-			(at 1.0375 0 270)
+			(at 1.0375 0 90)
 			(size 1.175 1.45)
 			(layers "F.Cu" "F.Paste" "F.Mask")
@@
 		(descr "Molex Mega-Fit Power Connectors, 76825-0002 (compatible alternatives: 172064-0002, 172064-1002), 1 Pins per row (http://www.molex.com/pdm_docs/sd/1720640002_sd.pdf), generated with kicad-footprint-generator")
 		(tags "connector Molex Mega-Fit top entry")
-		(property "Reference" "J1"
-			(at 0 -17.1 360)
+		(property "Reference" "CON_GLVMS"
+			(at -5.84 -9.58 90)
 			(layer "F.SilkS")
 			(effects
@@
 	)
 	(segment
+		(start 223 36.75)
+		(end 223.25 37)
+		(width 0.2)
+		(layer "F.Cu")
+		(net 1)
+	)
+	(segment
 		(start 218.7825 96.282984)
 		(end 219.8525 96.282984)
@@
 	)
 	(segment
+		(start 223 35.5)
+		(end 223 36.75)
+		(width 0.2)
+		(layer "F.Cu")
+		(net 1)
+	)
+	(segment
 		(start 184.75 52.0375)
 		(end 183.7245 53.063)
@@
 	)
 	(via
+		(at 223.25 37)
+		(size 0.6)
+		(drill 0.3)
+		(layers "F.Cu" "B.Cu")
+		(net 1)
+	)
+	(via
 		(at 142 69.75)
 		(size 0.6)
@@
 	)
 	(segment
-		(start 223 36.75)
-		(end 223.25 37)
-		(width 0.2)
-		(layer "F.Cu")
-		(net 21)
-	)
-	(segment
 		(start 202.75 52.285)
 		(end 204.62 54.155)
@@
 	)
 	(segment
-		(start 223 35.5)
-		(end 223 36.75)
-		(width 0.2)
-		(layer "F.Cu")
-		(net 21)
-	)
-	(segment
 		(start 202.75 47.057492)
 		(end 202.75 52.285)
@@
 		(net 21)
 	)
-	(via
-		(at 223.25 37)
-		(size 0.6)
-		(drill 0.3)
-		(layers "F.Cu" "B.Cu")
-		(net 21)
-	)

Commit message: silkscreen updates
Other:
- board text added: "10A"
- board text added: "1A"
- board text added: "3A"
- board text added: "CAN TRANSCEVER"
- board text added: "DC/DC LV BATT CON"
- board text added: "FS-3 PD Board V1.3 PCB Designed By: Aaron Gondo Schematic By: Hardware Integration"
- board text added: "HIGHER CURRENT OUTPUT"
- board text added: "LOWER CURRENT OUT +CAN"
- board text removed: "FS-3 Power Distrobution Board V1.3 Formula Slug PCB Designed By: Aaron Gondo Schematic Designed By: Niwa Babista, Jaelyn Flores, Aaron Gondo, Nataniel Jayaseelan,Shreyas J Kiran, Francesco Menegoli,Dylan Ortiz , Atul Pethe, Muneeb Syed"

Commit message: updated cap values
Parts:
- C1: value .33nF -> 0.33uF
- C10: value 904.7nF? -> 0.1uF
- C11, C12, C13, C14, C15, C16, C17, C18, C19, C20, C21, C22, C9: value 0.1nF -> 0.1uF
- C2, C4, C6: value .01nF -> 0.1uF
- C3: value 10nF -> 10uF
- C5: value 100nF -> 0.1uF
- C7: value 0.33nF -> 0.33uF
- C8: value 0.01nF -> 0.1uF
- renumbered CON_GLVMS to J1
Changed lines of the file:
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@@
 			)
 		)
-		(property "Value" "0.1nF"
+		(property "Value" "0.1uF"
 			(at 0 1.68 90)
 			(layer "F.Fab")
@@
 			)
 		)
-		(property "Value" "0.01nF"
+		(property "Value" "0.1uF"
 			(at 0 1.68 90)
 			(layer "F.Fab")
@@
 			)
 		)
-		(property "Value" "0.1nF"
+		(property "Value" "0.1uF"
 			(at 0 1.68 90)
 			(layer "F.Fab")
@@
 			)
 		)
-		(property "Value" "0.33nF"
+		(property "Value" "0.33uF"
 			(at 0 1.68 90)
 			(layer "F.Fab")
@@
 			)
 		)
-		(property "Value" "0.1nF"
+		(property "Value" "0.1uF"
 			(at 0 1.68 0)
 			(layer "F.Fab")
@@
 			)
 		)
-		(property "Value" ".01nF"
+		(property "Value" "0.1uF"
 			(at 0 1.68 90)
 			(layer "F.Fab")
@@
 			)
 		)
-		(property "Value" "0.1nF"
+		(property "Value" "0.1uF"
 			(at 0 1.68 90)
 			(layer "F.Fab")
@@
 			)
 		)
-		(property "Value" "0.1nF"
+		(property "Value" "0.1uF"
 			(at 0 1.68 90)
 			(layer "F.Fab")
@@
 			)
 		)
-		(property "Value" ".01nF"
+		(property "Value" "0.1uF"
 			(at 0 1.68 0)
 			(layer "F.Fab")
@@
 			)
 		)
-		(property "Value" "904.7nF?"
+		(property "Value" "0.1uF"
 			(at 0 1.68 90)
 			(layer "F.Fab")
@@
 			)
 		)
-		(property "Value" "0.1nF"
+		(property "Value" "0.1uF"
 			(at 0 1.68 90)
 			(layer "F.Fab")
@@
 			)
 		)
-		(property "Value" ".33nF"
+		(property "Value" "0.33uF"
 			(at 0 1.68 90)
 			(layer "F.Fab")
@@
 			)
 		)
-		(property "Value" "0.1nF"
+		(property "Value" "0.1uF"
 			(at 0 1.68 90)
 			(layer "F.Fab")
@@
 			)
 		)
-		(property "Value" "0.1nF"
+		(property "Value" "0.1uF"
 			(at 0 1.68 90)
 			(layer "F.Fab")
@@
 			)
 		)
-		(property "Value" "10nF"
+		(property "Value" "10uF"
 			(at 0 1.68 90)
 			(layer "F.Fab")
@@
 			)
 		)
-		(property "Value" "0.1nF"
+		(property "Value" "0.1uF"
 			(at 0 1.68 90)
 			(layer "F.Fab")
@@
 			)
 		)
-		(property "Value" "100nF"
+		(property "Value" "0.1uF"
 			(at 0 1.68 0)
 			(layer "F.Fab")
@@
 			)
 		)
-		(property "Value" ".01nF"
+		(property "Value" "0.1uF"
 			(at 0 1.68 90)
 			(layer "F.Fab")
@@
 		(descr "Molex Mega-Fit Power Connectors, 76825-0002 (compatible alternatives: 172064-0002, 172064-1002), 1 Pins per row (http://www.molex.com/pdm_docs/sd/1720640002_sd.pdf), generated with kicad-footprint-generator")
 		(tags "connector Molex Mega-Fit top entry")
-		(property "Reference" "CON_GLVMS"
+		(property "Reference" "J1"
 			(at -5.84 -9.58 90)
 			(layer "F.SilkS")
@@
 			)
 		)
-		(property "Value" "0.1nF"
+		(property "Value" "0.1uF"
 			(at 0 1.68 0)
 			(layer "F.Fab")
@@
 			)
 		)
-		(property "Value" "0.1nF"
+		(property "Value" "0.1uF"
 			(at 0 1.68 90)
 			(layer "F.Fab")
@@
 			)
 		)
-		(property "Value" "0.1nF"
+		(property "Value" "0.1uF"
 			(at 0 1.68 90)
 			(layer "F.Fab")
@@
 			)
 		)
-		(property "Value" "0.1nF"
+		(property "Value" "0.1uF"
 			(at 0 1.68 90)
 			(layer "F.Fab")

Commit message: made changes per nathaniel
Parts:
- added R1: 10k, Resistor_SMD:R_0805_2012Metric_Pad1.20x1.40mm_HandSolder, F.Cu at (123.1, 70.4)
- added R10: 10k, Resistor_SMD:R_0805_2012Metric_Pad1.20x1.40mm_HandSolder, F.Cu at (152.1, 88.6)
- added R11: 10k, Resistor_SMD:R_0805_2012Metric_Pad1.20x1.40mm_HandSolder, F.Cu at (163.7, 87.2)
- added R12: 10k, Resistor_SMD:R_0805_2012Metric_Pad1.20x1.40mm_HandSolder, F.Cu at (124.0, 62.8)
- added R13: 10k, Resistor_SMD:R_0805_2012Metric_Pad1.20x1.40mm_HandSolder, F.Cu at (140.5, 89.2)
- added R2: 10k, Resistor_SMD:R_0805_2012Metric_Pad1.20x1.40mm_HandSolder, F.Cu at (118.9, 80.6)
- added R3: 10k, Resistor_SMD:R_0805_2012Metric_Pad1.20x1.40mm_HandSolder, F.Cu at (185.0, 45.3)
- added R4: 10k, Resistor_SMD:R_0805_2012Metric_Pad1.20x1.40mm_HandSolder, F.Cu at (174.3, 47.5)
- added R5: 10k, Resistor_SMD:R_0805_2012Metric_Pad1.20x1.40mm_HandSolder, F.Cu at (140.2, 49.0)
- added R6: 10k, Resistor_SMD:R_0805_2012Metric_Pad1.20x1.40mm_HandSolder, F.Cu at (152.1, 47.7)
- added R7: 10k, Resistor_SMD:R_0805_2012Metric_Pad1.20x1.40mm_HandSolder, F.Cu at (175.0, 87.7)
- added R8: 10k, Resistor_SMD:R_0805_2012Metric_Pad1.20x1.40mm_HandSolder, F.Cu at (129.6, 83.3)
- added R9: 10k, Resistor_SMD:R_0805_2012Metric_Pad1.20x1.40mm_HandSolder, F.Cu at (162.6, 49.7)
- moved C16 8.12 mm to (115.4, 80.6)
- moved C11 1.93 mm to (128.7, 79.2)
Connections:
- U10 pad 6: unconnected-(U10-FAULT-Pad6) -> Net-(U10-FAULT)
- U11 pad 6: unconnected-(U11-FAULT-Pad6) -> Net-(U11-FAULT)
- U12 pad 6: unconnected-(U12-FAULT-Pad6) -> Net-(U12-FAULT)
- U13 pad 15: unconnected-(U13-~{E}-Pad15) -> Net-(U13-~{E})
- U16 pad 6: unconnected-(U16-FAULT-Pad6) -> Net-(U16-FAULT)
- U17 pad 6: unconnected-(U17-FAULT-Pad6) -> Net-(U17-FAULT)
- U2 pad 6: unconnected-(U2-FAULT-Pad6) -> Net-(U2-FAULT)
- U3 pad 6: unconnected-(U3-FAULT-Pad6) -> Net-(U3-FAULT)
- U4 pad 6: unconnected-(U4-FAULT-Pad6) -> Net-(U4-FAULT)
- U5 pad 6: unconnected-(U5-FAULT-Pad6) -> Net-(U5-FAULT)
- U7 pad 6: unconnected-(U7-FAULT-Pad6) -> Net-(U7-FAULT)
- U8 pad 6: unconnected-(U8-FAULT-Pad6) -> Net-(U8-FAULT)
- U9 pad 6: unconnected-(U9-FAULT-Pad6) -> Net-(U9-FAULT)
Routing:
- net +3.3V: track 286.0 -> 343.9 mm
- net Net-(U13-~{E}): track 0.00 -> 19.9 mm, vias 0 -> 4
- net Net-(U17-FAULT): track 0.00 -> 12.7 mm, vias 0 -> 2
- net Net-(U9-FAULT): track 0.00 -> 12.6 mm, vias 0 -> 2
- net Net-(U7-FAULT): track 0.00 -> 12.1 mm, vias 0 -> 2
- net Net-(U4-FAULT): track 0.00 -> 11.1 mm, vias 0 -> 2
- net Net-(U8-FAULT): track 0.00 -> 10.7 mm, vias 0 -> 2
- net Net-(U12-FAULT): track 0.00 -> 10.6 mm, vias 0 -> 2
- net Net-(U10-FAULT): track 0.00 -> 10.5 mm, vias 0 -> 2
- net Net-(U5-FAULT): track 0.00 -> 10.2 mm, vias 0 -> 2
- net Net-(U11-FAULT): track 0.00 -> 10.0 mm, vias 0 -> 2
- net Net-(U16-FAULT): track 0.00 -> 8.47 mm, vias 0 -> 2
- net Net-(CN2A-PB0): track 76.5 -> 68.9 mm
- net GND: track 115.0 -> 122.5 mm
- net Net-(U3-FAULT): track 0.00 -> 4.09 mm
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