File: Power Distrobution Board/micro.kicad_sch (KiCad schematic)
At the start: 4 parts, among them CN2 NUCLEO-L432KC, U13 CD74HC4067M, U18 ISO1050DUB

Commit message: version 1.1
Parts:
- added C10, C4, C6, C9: C_Small, Capacitor_SMD:C_0805_2012Metric_Pad1.18x1.45mm_HandSolder, symbol Device:C_Small
Connections:
- net +3.3V: now also C6.1, C9.1
- net +5V: now also C4.1
- net +9V: now also C10.2
- net GND: now also C10.1, C4.2, C6.2, C9.2
- no-connect marks 8 -> 23
Other:
- title: (none) -> PD Micro

Commit message: changes after cdr
Parts:
- C10: value C_Small -> 904.7nF?
- C4, C6: value C_Small -> .01nF
- C9: value C_Small -> 0.1nF
Changed lines of the file:
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@@
 			)
 		)
-		(property "Value" "C_Small"
+		(property "Value" "904.7nF?"
 			(at 138.43 60.9535 0)
 			(effects
@@
 			)
 		)
-		(property "Value" "C_Small"
+		(property "Value" ".01nF"
 			(at 36.8363 115.57 90)
 			(effects
@@
 			)
 		)
-		(property "Value" "C_Small"
+		(property "Value" "0.1nF"
 			(at 66.0463 86.36 90)
 			(effects
@@
 			)
 		)
-		(property "Value" "C_Small"
+		(property "Value" ".01nF"
 			(at 76.2063 115.57 90)
 			(effects

Commit message: even newer changes
Parts:
- removed CR1: STS6NF20V, Package_SO:SOIC-8_3.9x4.9mm_P1.27mm, symbol FS_3_Global_Symbol_Library:STS6NF20V
Connections:
- net +5V: now also C4.2; no longer C4.1
- net GND: now also C4.1; no longer C4.2
- net dcdc_ctrl: now also CN2.CN3_14 (PB5)
Other:
- moved on the sheet: C4

Commit message: updated cap values
Parts:
- C10: value 904.7nF? -> 0.1uF
- C4, C6: value .01nF -> 0.1uF
- C9: value 0.1nF -> 0.1uF
Changed lines of the file:
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@@
 			)
 		)
-		(property "Value" "904.7nF?"
+		(property "Value" "0.1uF"
 			(at 138.43 60.9535 0)
 			(effects
@@
 			)
 		)
-		(property "Value" ".01nF"
+		(property "Value" "0.1uF"
 			(at 30.4863 115.57 90)
 			(effects
@@
 			)
 		)
-		(property "Value" "0.1nF"
+		(property "Value" "0.1uF"
 			(at 66.0463 86.36 90)
 			(effects
@@
 			)
 		)
-		(property "Value" ".01nF"
+		(property "Value" "0.1uF"
 			(at 76.2063 115.57 90)
 			(effects

Commit message: made changes per nathaniel
Parts:
- added R1: 10k, Resistor_SMD:R_0805_2012Metric_Pad1.20x1.40mm_HandSolder, symbol Device:R_Small_US
Connections:
- net GND: now also R1.2
- net at U13.15 (~{E}): now also R1.1
- no-connect marks 23 -> 22
Changed lines of the file:
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@@
-	)
-	(no_connect
-		(at 68.58 48.26)
 	)
 	(no_connect
@@
 		(pts
 			(xy 85.09 113.03) (xy 71.12 113.03)
+		)
+		(stroke
+			(width 0)
+			(type default)
+		)
+	)
+	(wire
+		(pts
+			(xy 73.66 48.26) (xy 73.66 49.53)
 		)
 		(stroke
@@
 	(symbol
 		(lib_id "power:GND")
+		(at 73.66 49.53 0)
+		(unit 1)
+		(exclude_from_sim no)
+		(in_bom yes)
+		(on_board yes)
+		(dnp no)
+		(fields_autoplaced yes)
+		(property "Reference" "#PWR058"
+			(at 73.66 55.88 0)
+			(effects
+				(font
+					(size 1.27 1.27)
+				)
+				(hide yes)
+			)
+		)
+		(property "Value" "GND"
+			(at 73.66 54.61 0)
+			(effects
+				(font
+					(size 1.27 1.27)
+				)
+			)
+		)
+		(property "Footprint" ""
+			(at 73.66 49.53 0)
+			(effects
+				(font
+					(size 1.27 1.27)
+				)
+				(hide yes)
+			)
+		)
+		(property "Datasheet" ""
+			(at 73.66 49.53 0)
+			(effects
+				(font
+					(size 1.27 1.27)
+				)
+				(hide yes)
+			)
+		)
+		(property "Description" "Power symbol creates a global label with name \"GND\" , ground"
+			(at 73.66 49.53 0)
+			(effects
+				(font
+					(size 1.27 1.27)
+				)
+				(hide yes)
+			)
+		)
+		(pin "1"
+		)
+		(instances
+			(project ""
+				(path "/cd827802-ab32-49ad-ad84-bccf81c569e7/ea797ac0-04c8-4aab-978e-f3f6d7333a50"
+					(reference "#PWR058")
+					(unit 1)
+				)
+			)
+		)
+	)
+	(symbol
+		(lib_id "power:GND")
 		(at 27.94 121.92 0)
 		(unit 1)
@@
 					(unit 1)
 				)
+			)
+		)
+	)
+	(symbol
+		(lib_id "Device:R_Small_US")
+		(at 71.12 48.26 90)
+		(unit 1)
+		(exclude_from_sim no)
+		(in_bom yes)
+		(on_board yes)
+		(dnp no)
+		(fields_autoplaced yes)
+		(property "Reference" "R1"
+			(at 71.12 41.91 90)
+			(effects
+				(font
+					(size 1.27 1.27)
+				)
+			)
+		)
+		(property "Value" "10k"
+			(at 71.12 44.45 90)
+			(effects
+				(font
+					(size 1.27 1.27)
+				)
+			)
+		)
+		(property "Footprint" "Resistor_SMD:R_0805_2012Metric_Pad1.20x1.40mm_HandSolder"
+			(at 71.12 48.26 0)
+			(effects
+				(font
+					(size 1.27 1.27)
+				)
+				(hide yes)
+			)
+		)
+		(property "Datasheet" "https://www.yageo.com/upload/media/product/products/datasheet/rchip/PYu-RC_Group_51_RoHS_L_12.pdf"
+			(at 71.12 48.26 0)
+			(effects
+				(font
+					(size 1.27 1.27)
+				)
+				(hide yes)
+			)
+		)
+		(property "Description" "Resistor, small US symbol"
+			(at 71.12 48.26 0)
+			(effects
+				(font
+					(size 1.27 1.27)
+				)
+				(hide yes)
+			)
+		)
+		(pin "2"
+		)
+		(pin "1"
+		)
+		(instances
+			(project ""
+				(path "/cd827802-ab32-49ad-ad84-bccf81c569e7/ea797ac0-04c8-4aab-978e-f3f6d7333a50"
+					(reference "R1")
+					(unit 1)
+				)

Commit message: commit 1 of v2
pd board v2 work first commit
Connections:
- net reset_ctrl: now reaches CN2.CN4_11 (PA1)
- net lv_sense: now reaches CN2.CN4_12 (PA0)
- no-connect marks 22 -> 20
Changed lines of the file:
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@@
-	)
-	(no_connect
-		(at 128.27 86.36)
 	)
 	(no_connect
@@
 	)
 	(no_connect
-		(at 128.27 83.82)
-	)
-	(no_connect
 		(at 97.79 83.82)
 	)
@@
 		)
 	)
+	(global_label "lv_sense"
+		(shape input)
+		(at 128.27 86.36 0)
+		(fields_autoplaced yes)
+		(effects
+			(font
+				(size 1.27 1.27)
+			)
+			(justify left)
+		)
+		(property "Intersheetrefs" "${INTERSHEET_REFS}"
+			(at 139.238 86.36 0)
+			(effects
+				(font
+					(size 1.27 1.27)
+				)
+				(justify left)
+				(hide yes)
+			)
+		)
+	)
 	(global_label "ready_to_move_viout"
 		(shape input)
@@
 				(hide yes)
 			)
+		)
+	)
+	(global_label "reset_ctrl"
+		(shape output)
+		(at 128.27 83.82 0)
+		(fields_autoplaced yes)
+		(effects
+			(font
+				(size 1.27 1.27)
+			)
+			(justify left)
+		)
+		(property "Intersheetrefs" "${INTERSHEET_REFS}"
+			(at 140.2057 83.82 0)
+			(effects
+				(font
+					(size 1.27 1.27)
+				)
+				(justify left)
+				(hide yes)
+			)
