File: Power Distrobution Board/brake_pressure_sensor_power.kicad_sch (KiCad schematic)
At the start: 3 parts, among them U15 MC7809CTG 9v linear reg

Commit message: v1.3
changed footprint of linear regulators
Parts:
- U15: footprint Package_TO_SOT_SMD:SOT-89-3 -> Package_TO_SOT_THT:TO-220-3_Horizontal_TabDown
Changed lines of the file:
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@@
 			)
 		)
-		(property "Footprint" "Package_TO_SOT_SMD:SOT-89-3"
+		(property "Footprint" "Package_TO_SOT_THT:TO-220-3_Horizontal_TabDown"
 			(at 73.66 99.06 0)
 			(effects

Commit message: changes after cdr
Parts:
- C7: value C_Small -> 0.33nF
- C8: value C_Small -> 0.01nF
Changed lines of the file:
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@@
 			)
 		)
-		(property "Value" "C_Small"
+		(property "Value" "0.33nF"
 			(at 58.4263 86.36 90)
 			(effects
@@
 			)
 		)
-		(property "Value" "C_Small"
+		(property "Value" "0.01nF"
 			(at 58.4263 104.14 90)
 			(effects

Commit message: even newer changes
Other:
- moved on the sheet: C7, C8
Changed lines of the file:
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@@
 	(paper "A4")
 	(junction
-		(at 53.34 107.95)
+		(at 53.34 113.03)
 		(diameter 0)
 		(color 0 0 0 0)
@@
 		(color 0 0 0 0)
 	)
-	(junction
-		(at 68.58 90.17)
-		(diameter 0)
-		(color 0 0 0 0)
-	)
-	(wire
-		(pts
-			(xy 68.58 107.95) (xy 60.96 107.95)
-		)
-		(stroke
-			(width 0)
-			(type default)
-		)
-	)
-	(wire
-		(pts
-			(xy 53.34 107.95) (xy 53.34 109.22)
-		)
-		(stroke
-			(width 0)
-			(type default)
-		)
-	)
-	(wire
-		(pts
-			(xy 68.58 90.17) (xy 68.58 91.44)
-		)
-		(stroke
-			(width 0)
-			(type default)
-		)
-	)
-	(wire
-		(pts
-			(xy 53.34 107.95) (xy 53.34 99.06)
-		)
-		(stroke
-			(width 0)
-			(type default)
-		)
-	)
-	(wire
-		(pts
-			(xy 55.88 107.95) (xy 53.34 107.95)
-		)
-		(stroke
-			(width 0)
-			(type default)
-		)
-	)
-	(wire
-		(pts
-			(xy 68.58 106.68) (xy 68.58 107.95)
-		)
-		(stroke
-			(width 0)
-			(type default)
-		)
-	)
-	(wire
-		(pts
-			(xy 53.34 90.17) (xy 55.88 90.17)
+	(wire
+		(pts
+			(xy 53.34 113.03) (xy 53.34 114.3)
+		)
+		(stroke
+			(width 0)
+			(type default)
+		)
+	)
+	(wire
+		(pts
+			(xy 68.58 82.55) (xy 68.58 91.44)
+		)
+		(stroke
+			(width 0)
+			(type default)
+		)
+	)
+	(wire
+		(pts
+			(xy 53.34 113.03) (xy 53.34 99.06)
+		)
+		(stroke
+			(width 0)
+			(type default)
+		)
+	)
+	(wire
+		(pts
+			(xy 55.88 113.03) (xy 53.34 113.03)
+		)
+		(stroke
+			(width 0)
+			(type default)
+		)
+	)
+	(wire
+		(pts
+			(xy 68.58 106.68) (xy 68.58 113.03)
+		)
+		(stroke
+			(width 0)
+			(type default)
+		)
+	)
+	(wire
+		(pts
+			(xy 60.96 113.03) (xy 68.58 113.03)
+		)
+		(stroke
+			(width 0)
+			(type default)
+		)
+	)
+	(wire
+		(pts
+			(xy 53.34 82.55) (xy 55.88 82.55)
 		)
 		(stroke
@@
 	(wire
 		(pts
-			(xy 68.58 90.17) (xy 68.58 87.63)
-		)
-		(stroke
-			(width 0)
-			(type default)
-		)
-	)
-	(wire
-		(pts
-			(xy 53.34 99.06) (xy 53.34 90.17)
-		)
-		(stroke
-			(width 0)
-			(type default)
-		)
-	)
-	(wire
-		(pts
-			(xy 68.58 90.17) (xy 60.96 90.17)
+			(xy 53.34 99.06) (xy 53.34 82.55)
+		)
+		(stroke
+			(width 0)
+			(type default)
+		)
+	)
+	(wire
+		(pts
+			(xy 68.58 82.55) (xy 60.96 82.55)
 		)
 		(stroke
@@
 	(global_label "brake_pressure_sensor_out"
 		(shape input)
-		(at 68.58 87.63 90)
+		(at 68.58 82.55 0)
 		(fields_autoplaced yes)
 		(effects
@@
 		)
 		(property "Intersheetrefs" "${INTERSHEET_REFS}"
-			(at 68.58 59.1846 90)
+			(at 97.0254 82.55 0)
 			(effects
 				(font
@@
 	(global_label "brake_pressure_sensor_9v"
 		(shape input)
-		(at 68.58 107.95 270)
+		(at 68.58 113.03 0)
 		(fields_autoplaced yes)
 		(effects
@@
 				(size 1.27 1.27)
 			)
-			(justify right)
+			(justify left)
 		)
 		(property "Intersheetrefs" "${INTERSHEET_REFS}"
-			(at 68.58 135.5488 90)
-			(effects
-				(font
-					(size 1.27 1.27)
-				)
-				(justify right)
+			(at 96.1788 113.03 0)
+			(effects
+				(font
+					(size 1.27 1.27)
+				)
+				(justify left)
 				(hide yes)
 			)
@@
 	(symbol
 		(lib_id "Device:C_Small")
-		(at 58.42 90.17 90)
+		(at 58.42 82.55 90)
 		(unit 1)
 		(exclude_from_sim no)
@@
 		(fields_autoplaced yes)
 		(property "Reference" "C7"
-			(at 58.4263 83.82 90)
+			(at 58.4263 76.2 90)
 			(effects
 				(font
@@
 		)
 		(property "Value" "0.33nF"
-			(at 58.4263 86.36 90)
+			(at 58.4263 78.74 90)
 			(effects
 				(font
@@
 		)
 		(property "Footprint" "Capacitor_SMD:C_0805_2012Metric_Pad1.18x1.45mm_HandSolder"
-			(at 58.42 90.17 0)
+			(at 58.42 82.55 0)
 			(effects
 				(font
@@
 		)
 		(property "Datasheet" "https://www.yageo.com/upload/media/product/productsearch/datasheet/mlcc/UPY-GPHC_X7R_6.3V-to-250V_24.pdf"
-			(at 58.42 90.17 0)
+			(at 58.42 82.55 0)
 			(effects
 				(font
@@
 		)
 		(property "Description" "Unpolarized capacitor, small symbol"
-			(at 58.42 90.17 0)
+			(at 58.42 82.55 0)
 			(effects
 				(font
@@
 	(symbol
 		(lib_id "Device:C_Small")
-		(at 58.42 107.95 90)
+		(at 58.42 113.03 90)
 		(unit 1)
 		(exclude_from_sim no)
@@
 		(fields_autoplaced yes)
 		(property "Reference" "C8"
-			(at 58.4263 101.6 90)
+			(at 58.4263 106.68 90)
 			(effects
 				(font
@@
 		)
 		(property "Value" "0.01nF"
-			(at 58.4263 104.14 90)
+			(at 58.4263 109.22 90)
 			(effects
 				(font
@@
 		)
 		(property "Footprint" "Capacitor_SMD:C_0805_2012Metric_Pad1.18x1.45mm_HandSolder"
-			(at 58.42 107.95 0)
+			(at 58.42 113.03 0)
 			(effects
 				(font
@@
 		)
 		(property "Datasheet" "https://www.yageo.com/upload/media/product/productsearch/datasheet/mlcc/UPY-GPHC_X7R_6.3V-to-250V_24.pdf"
-			(at 58.42 107.95 0)
+			(at 58.42 113.03 0)
 			(effects
 				(font
@@
 		)
 		(property "Description" "Unpolarized capacitor, small symbol"
-			(at 58.42 107.95 0)
+			(at 58.42 113.03 0)
 			(effects
 				(font
@@
 	(symbol
 		(lib_id "power:GND")
-		(at 53.34 109.22 0)
+		(at 53.34 114.3 0)
 		(unit 1)
 		(exclude_from_sim no)
@@
 		(fields_autoplaced yes)
 		(property "Reference" "#PWR031"
-			(at 53.34 115.57 0)
+			(at 53.34 120.65 0)
 			(effects
 				(font
@@
 		)
 		(property "Value" "GND"
+			(at 53.34 119.38 0)
+			(effects
+				(font
+					(size 1.27 1.27)
+				)
+			)
+		)
+		(property "Footprint" ""
 			(at 53.34 114.3 0)
 			(effects
@@
 					(size 1.27 1.27)
 				)
-			)
-		)
-		(property "Footprint" ""
-			(at 53.34 109.22 0)
-			(effects
-				(font
-					(size 1.27 1.27)
-				)
 				(hide yes)
 			)
 		)
 		(property "Datasheet" ""
-			(at 53.34 109.22 0)
+			(at 53.34 114.3 0)
 			(effects
 				(font
@@
 		)
 		(property "Description" "Power symbol creates a global label with name \"GND\" , ground"
-			(at 53.34 109.22 0)
-			(effects
-				(font
+			(at 53.34 114.3 0)
+			(effects
+				(font

Commit message: updated cap values
Parts:
- C7: value 0.33nF -> 0.33uF
- C8: value 0.01nF -> 0.1uF
Changed lines of the file:
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@@
 			)
 		)
-		(property "Value" "0.33nF"
+		(property "Value" "0.33uF"
 			(at 58.4263 78.74 90)
 			(effects
@@
 			)
 		)
-		(property "Value" "0.01nF"
+		(property "Value" "0.1uF"
 			(at 58.4263 109.22 90)
 			(effects

Commit message: commit 1 of v2
pd board v2 work first commit
Other:
- note added: "backwards 1 in 2 gnd 3 out"
Changed lines of the file:
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@@
+		)
+	)
+	(text "backwards 1 in 2 gnd 3 out "
+		(exclude_from_sim no)
+		(at 96.266 98.552 0)
+		(effects
+			(font
+				(size 1.27 1.27)
+			)
 		)
 	)

Commit message: v2 3/29
almost done need to add mounting holes text, clean up screen printing, and get linear regs re speced
Connections:
- net brake_pressure_sensor_9v: now also U15.3 (OUT); no longer U15.1 (OUT)
- net brake_pressure_sensor_out: now also U15.1 (IN); no longer U15.3 (IN)
