File: Power Distrobution Board/pd_board_power.kicad_sch (KiCad schematic)
At the start: 6 parts, among them U1 3.3v linear reg, U14 MC7809CTG 9v linear reg

Commit message: v1.3
changed footprint of linear regulators
Parts:
- U1: value 3.3v linear reg -> LD1117V33C 3.3v linear reg; footprint Package_TO_SOT_SMD:SOT-89-3 -> Package_TO_SOT_THT:TO-220-3_Horizontal_TabDown
- U14: footprint Package_TO_SOT_SMD:SOT-89-3 -> Package_TO_SOT_THT:TO-220-3_Horizontal_TabDown
Changed lines of the file:
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@@
 			)
 		)
-		(property "Footprint" "Package_TO_SOT_SMD:SOT-89-3"
+		(property "Footprint" "Package_TO_SOT_THT:TO-220-3_Horizontal_TabDown"
 			(at 64.77 74.93 0)
 			(effects
@@
 			)
 		)
-		(property "Value" "3.3v linear reg"
+		(property "Value" "LD1117V33C 3.3v linear reg"
 			(at 82.55 74.93 0)
 			(effects
@@
 			)
 		)
-		(property "Footprint" "Package_TO_SOT_SMD:SOT-89-3"
+		(property "Footprint" "Package_TO_SOT_THT:TO-220-3_Horizontal_TabDown"
 			(at 83.82 74.93 0)
 			(effects

Commit message: changes after cdr
Parts:
- C1: value C_Small -> .33nF
- C2: value C_Small -> .01nF
- C3: value C_Small -> 10nF
- C5: value C_Small -> 100nF
Changed lines of the file:
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@@
 			)
 		)
-		(property "Value" "C_Small"
+		(property "Value" ".01nF"
 			(at 49.5363 80.01 90)
 			(effects
@@
 			)
 		)
-		(property "Value" "C_Small"
+		(property "Value" "10nF"
 			(at 70.104 79.756 90)
 			(effects
@@
 			)
 		)
-		(property "Value" "C_Small"
+		(property "Value" ".33nF"
 			(at 49.5363 62.23 90)
 			(effects
@@
 			)
 		)
-		(property "Value" "C_Small"
+		(property "Value" "100nF"
 			(at 69.8563 62.23 90)
 			(effects

Commit message: updated cap values
Parts:
- C1: value .33nF -> 0.33uF
- C2: value .01nF -> 0.1uF
- C3: value 10nF -> 10uF
- C5: value 100nF -> 0.1uF
Changed lines of the file:
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@@
 			)
 		)
-		(property "Value" ".01nF"
+		(property "Value" "0.1uF"
 			(at 49.5363 80.01 90)
 			(effects
@@
 			)
 		)
-		(property "Value" "10nF"
+		(property "Value" "10uF"
 			(at 70.104 79.756 90)
 			(effects
@@
 			)
 		)
-		(property "Value" ".33nF"
+		(property "Value" "0.33uF"
 			(at 49.5363 62.23 90)
 			(effects
@@
 			)
 		)
-		(property "Value" "100nF"
+		(property "Value" "0.1uF"
 			(at 69.8563 62.23 90)
 			(effects

Commit message: commit 1 of v2
pd board v2 work first commit
Other:
- note added: "backwards 1 in 2 gnd 3 out"
- note added: "fucked. 1 gnd 2 out 3 in"
Changed lines of the file:
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@@
+		)
+	)
+	(text "backwards 1 in 2 gnd 3 out "
+		(exclude_from_sim no)
+		(at 29.464 75.184 0)
+		(effects
+			(font
+				(size 1.27 1.27)
+			)
+		)
+	)
+	(text "fucked. 1 gnd 2 out 3 in"
+		(exclude_from_sim no)
+		(at 96.266 77.216 0)
+		(effects
+			(font
+				(size 1.27 1.27)
+			)
 		)
 	)

Commit message: v2 3/29
almost done need to add mounting holes text, clean up screen printing, and get linear regs re speced
Connections:
- net +3.3V: now also U1.2 (OUT); no longer U1.1 (OUT)
- net +9V: now also U14.3 (OUT); no longer U14.1 (OUT)
- net GND: now also U1.1 (GND); no longer U1.2 (GND)
- net pd_board_out: now also U14.1 (IN); no longer U14.3 (IN)
Other:
- note removed: "backwards 1 in 2 gnd 3 out"
- note removed: "fucked. 1 gnd 2 out 3 in"
Changed lines of the file:
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@@
+	)
+	(junction
+		(at 77.47 66.04)
+		(diameter 0)
+		(color 0 0 0 0)
+	)
+	(junction
+		(at 66.04 74.93)
+		(diameter 0)
+		(color 0 0 0 0)
+	)
+	(junction
+		(at 44.45 74.93)
+		(diameter 0)
+		(color 0 0 0 0)
+	)
+	(junction
+		(at 66.04 83.82)
+		(diameter 0)
+		(color 0 0 0 0)
 	)
 	(junction
@@
 	)
 	(junction
-		(at 77.47 66.04)
-		(diameter 0)
-		(color 0 0 0 0)
-	)
-	(junction
-		(at 66.04 74.93)
-		(diameter 0)
-		(color 0 0 0 0)
-	)
-	(junction
-		(at 44.45 74.93)
-		(diameter 0)
-		(color 0 0 0 0)
-	)
-	(junction
 		(at 59.69 66.04)
 		(diameter 0)
@@
 	)
 	(junction
-		(at 66.04 83.82)
-		(diameter 0)
-		(color 0 0 0 0)
-	)
-	(junction
 		(at 44.45 83.82)
 		(diameter 0)
@@
 	(wire
 		(pts
-			(xy 59.69 66.04) (xy 52.07 66.04)
-		)
-		(stroke
-			(width 0)
-			(type default)
-		)
-	)
-	(wire
-		(pts
 			(xy 44.45 66.04) (xy 46.99 66.04)
 		)
@@
 	(wire
 		(pts
-			(xy 59.69 83.82) (xy 52.07 83.82)
-		)
-		(stroke
-			(width 0)
-			(type default)
-		)
-	)
-	(wire
-		(pts
 			(xy 66.04 66.04) (xy 66.04 74.93)
 		)
@@
 	(wire
 		(pts
+			(xy 52.07 66.04) (xy 59.69 66.04)
+		)
+		(stroke
+			(width 0)
+			(type default)
+		)
+	)
+	(wire
+		(pts
 			(xy 66.04 74.93) (xy 66.04 83.82)
 		)
@@
 	(wire
 		(pts
+			(xy 52.07 83.82) (xy 59.69 83.82)
+		)
+		(stroke
+			(width 0)
+			(type default)
+		)
+	)
+	(wire
+		(pts
 			(xy 66.04 85.09) (xy 66.04 83.82)
 		)
@@
 			(width 0)
 			(type default)
-		)
-	)
-	(text "backwards 1 in 2 gnd 3 out "
-		(exclude_from_sim no)
-		(at 29.464 75.184 0)
-		(effects
-			(font
-				(size 1.27 1.27)
-			)
-		)
-	)
-	(text "fucked. 1 gnd 2 out 3 in"
-		(exclude_from_sim no)
-		(at 96.266 77.216 0)
-		(effects
-			(font
-				(size 1.27 1.27)
-			)
 		)
 	)
@@
 	)
 	(symbol
+		(lib_name "L78L09_SOT89_1")
 		(lib_id "Regulator_Linear:L78L09_SOT89")
 		(at 59.69 74.93 270)

Commit message: flipped cons
Parts:
- U1: value LD1117V33C 3.3v linear reg -> LF33CV 3.3v linear reg
Connections:
- net +3.3V: now also U1.3 (OUT); no longer U1.2 (OUT)
- net GND: now also U1.2 (GND); no longer U1.1 (GND)
- net pd_board_out: now also U1.1 (IN); no longer U1.3 (IN)
Changed lines of the file:
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@@
 			)
 		)
-		(property "Value" "LD1117V33C 3.3v linear reg"
-			(at 82.55 74.93 0)
+		(property "Value" "LF33CV 3.3v linear reg"
+			(at 82.55 74.9299 90)
 			(effects
 				(font
 					(size 1.27 1.27)
 				)
+				(justify left)
 			)
 		)
