File: Power Distrobution Board/current_sensors.kicad_sch (KiCad schematic)
At the start: 48 parts, among them U10 ACS71240LLCBTR-025B3, U11 ACS71240LLCBTR-025B3, U12 ACS71240LLCBTR-025B3, U16 ACS71240LLCBTR-025B3, U17 ACS71240LLCBTR-025B3, U2 ACS71240LLCBTR-025B3, U3 ACS71240LLCBTR-025B3, U4 ACS71240LLCBTR-025B3, U5 ACS71240LLCBTR-025B3, U7 ACS71240LLCBTR-025B3, U8 ACS71240LLCBTR-025B3, U9 ACS71240LLCBTR-025B3

Commit message: v2 3/29
almost done need to add mounting holes text, clean up screen printing, and get linear regs re speced
Parts:
- F10, F11, F12, F13, F2, F3, F4, F5, F6, F7, F8, F9: value Fuse -> 01530008LXN; footprint project lib:CNM-03-BT mini blade fuse holder -> FS_3_Global_Footprint_Library:01530008LXN
Other:
- moved on the sheet: F12
Changed lines of the file:
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@@
 	(wire
 		(pts
-			(xy 215.9 101.6) (xy 218.44 101.6)
+			(xy 214.63 101.6) (xy 218.44 101.6)
 		)
 		(stroke
@@
 	(wire
 		(pts
+			(xy 238.76 101.6) (xy 242.57 101.6)
+		)
+		(stroke
+			(width 0)
+			(type default)
+		)
+	)
+	(wire
+		(pts
 			(xy 266.7 22.86) (xy 228.6 22.86)
 		)
@@
 	(wire
 		(pts
-			(xy 205.74 101.6) (xy 208.28 101.6)
+			(xy 205.74 101.6) (xy 207.01 101.6)
 		)
 		(stroke
@@
 	(wire
 		(pts
-			(xy 238.76 101.6) (xy 240.03 101.6)
-		)
-		(stroke
-			(width 0)
-			(type default)
-		)
-	)
-	(wire
-		(pts
 			(xy 92.71 76.2) (xy 93.98 76.2)
 		)
@@
 	(global_label "tractive_out"
 		(shape output)
-		(at 240.03 101.6 0)
+		(at 242.57 101.6 0)
 		(fields_autoplaced yes)
 		(effects
@@
 		)
 		(property "Intersheetrefs" "${INTERSHEET_REFS}"
-			(at 254.1427 101.6 0)
+			(at 256.6827 101.6 0)
 			(effects
 				(font
@@
 		(length 2.54)
 		(shape round)
-		(at 238.76 101.6 0)
-		(fields_autoplaced yes)
-		(effects
-			(font
-				(size 1.27 1.27)
-			)
-			(justify left bottom)
-		)
-		(property "Netclass" "10A"
-			(at 239.4585 99.06 0)
-			(effects
-				(font
-					(size 1.27 1.27)
-					(italic yes)
-				)
-				(justify left)
-			)
-		)
-	)
-	(netclass_flag ""
-		(length 2.54)
-		(shape round)
 		(at 69.85 102.87 0)
 		(fields_autoplaced yes)
@@
 		(length 2.54)
 		(shape round)
+		(at 238.76 101.6 0)
+		(fields_autoplaced yes)
+		(effects
+			(font
+				(size 1.27 1.27)
+			)
+			(justify left bottom)
+		)
+		(property "Netclass" "10a"
+			(at 239.4585 99.06 0)
+			(effects
+				(font
+					(size 1.27 1.27)
+					(italic yes)
+				)
+				(justify left)
+			)
+		)
+	)
+	(netclass_flag ""
+		(length 2.54)
+		(shape round)
 		(at 167.64 66.04 0)
 		(fields_autoplaced yes)
@@
 			)
 		)
-		(property "Value" "Fuse"
+		(property "Value" "01530008LXN"
 			(at 212.09 134.62 90)
 			(effects
@@
 			)
 		)
-		(property "Footprint" "project lib:CNM-03-BT mini blade fuse holder"
+		(property "Footprint" "FS_3_Global_Footprint_Library:01530008LXN"
 			(at 212.09 140.208 90)
 			(effects
@@
 			)
 		)
-		(property "Datasheet" "https://www.optifuse.com/optifuse_ecommerce_tools/datasheets/CNM-03.pdf"
+		(property "Datasheet" "https://www.digikey.com/en/products/detail/littelfuse-commercial-vehicle-products/01530008LXN/3425426?s=N4IgTCBcDaIAwEYCsBmO6AcAZAGgORAF0BfIA"
 			(at 212.09 138.43 0)
 			(effects
@@
 			)
 		)
-		(property "Value" "Fuse"
+		(property "Value" "01530008LXN"
 			(at 66.04 99.06 90)
 			(effects
@@
 			)
 		)
-		(property "Footprint" "project lib:CNM-03-BT mini blade fuse holder"
+		(property "Footprint" "FS_3_Global_Footprint_Library:01530008LXN"
 			(at 66.04 104.648 90)
 			(effects
@@
 			)
 		)
-		(property "Datasheet" "https://www.optifuse.com/optifuse_ecommerce_tools/datasheets/CNM-03.pdf"
+		(property "Datasheet" "https://www.digikey.com/en/products/detail/littelfuse-commercial-vehicle-products/01530008LXN/3425426?s=N4IgTCBcDaIAwEYCsBmO6AcAZAGgORAF0BfIA"
 			(at 66.04 102.87 0)
 			(effects
@@
 			)
 		)
-		(property "Value" "Fuse"
+		(property "Value" "01530008LXN"
 			(at 212.09 60.96 90)
 			(effects
@@
 			)
 		)
-		(property "Footprint" "project lib:CNM-03-BT mini blade fuse holder"
+		(property "Footprint" "FS_3_Global_Footprint_Library:01530008LXN"
 			(at 212.09 66.548 90)
 			(effects
@@
 			)
 		)
-		(property "Datasheet" "https://www.optifuse.com/optifuse_ecommerce_tools/datasheets/CNM-03.pdf"
+		(property "Datasheet" "https://www.digikey.com/en/products/detail/littelfuse-commercial-vehicle-products/01530008LXN/3425426?s=N4IgTCBcDaIAwEYCsBmO6AcAZAGgORAF0BfIA"
 			(at 212.09 64.77 0)
 			(effects
@@
 			)
 		)
-		(property "Value" "Fuse"
+		(property "Value" "01530008LXN"
 			(at 212.09 24.13 90)
 			(effects
@@
 			)
 		)
-		(property "Footprint" "project lib:CNM-03-BT mini blade fuse holder"
+		(property "Footprint" "FS_3_Global_Footprint_Library:01530008LXN"
 			(at 212.09 29.718 90)
 			(effects
@@
 			)
 		)
-		(property "Datasheet" "https://www.optifuse.com/optifuse_ecommerce_tools/datasheets/CNM-03.pdf"
+		(property "Datasheet" "https://www.digikey.com/en/products/detail/littelfuse-commercial-vehicle-products/01530008LXN/3425426?s=N4IgTCBcDaIAwEYCsBmO6AcAZAGgORAF0BfIA"
 			(at 212.09 27.94 0)
 			(effects
@@
 			)
 		)
-		(property "Value" "Fuse"
+		(property "Value" "01530008LXN"
 			(at 66.04 135.89 90)
 			(effects
@@
 			)
 		)
-		(property "Footprint" "project lib:CNM-03-BT mini blade fuse holder"
+		(property "Footprint" "FS_3_Global_Footprint_Library:01530008LXN"
 			(at 66.04 141.478 90)
 			(effects
@@
 			)
 		)
-		(property "Datasheet" "https://www.optifuse.com/optifuse_ecommerce_tools/datasheets/CNM-03.pdf"
+		(property "Datasheet" "https://www.digikey.com/en/products/detail/littelfuse-commercial-vehicle-products/01530008LXN/3425426?s=N4IgTCBcDaIAwEYCsBmO6AcAZAGgORAF0BfIA"
 			(at 66.04 139.7 0)
 			(effects
@@
 			)
 		)
-		(property "Value" "Fuse"
+		(property "Value" "01530008LXN"
 			(at 140.97 62.23 90)
 			(effects
@@
 			)
 		)
-		(property "Footprint" "project lib:CNM-03-BT mini blade fuse holder"
+		(property "Footprint" "FS_3_Global_Footprint_Library:01530008LXN"
 			(at 140.97 67.818 90)
 			(effects
@@
 			)
 		)
-		(property "Datasheet" "https://www.optifuse.com/optifuse_ecommerce_tools/datasheets/CNM-03.pdf"
+		(property "Datasheet" "https://www.digikey.com/en/products/detail/littelfuse-commercial-vehicle-products/01530008LXN/3425426?s=N4IgTCBcDaIAwEYCsBmO6AcAZAGgORAF0BfIA"
 			(at 140.97 66.04 0)
 			(effects
@@
 			)
 		)
-		(property "Value" "Fuse"
+		(property "Value" "01530008LXN"
 			(at 140.97 99.06 90)
 			(effects
@@
 			)
 		)
-		(property "Footprint" "project lib:CNM-03-BT mini blade fuse holder"
+		(property "Footprint" "FS_3_Global_Footprint_Library:01530008LXN"
 			(at 140.97 104.648 90)
 			(effects
@@
 			)
 		)
-		(property "Datasheet" "https://www.optifuse.com/optifuse_ecommerce_tools/datasheets/CNM-03.pdf"
+		(property "Datasheet" "https://www.digikey.com/en/products/detail/littelfuse-commercial-vehicle-products/01530008LXN/3425426?s=N4IgTCBcDaIAwEYCsBmO6AcAZAGgORAF0BfIA"
 			(at 140.97 102.87 0)
 			(effects
@@
 			)
 		)
-		(property "Value" "Fuse"
+		(property "Value" "01530008LXN"
 			(at 140.97 135.89 90)
 			(effects
@@
 			)
 		)
-		(property "Footprint" "project lib:CNM-03-BT mini blade fuse holder"
+		(property "Footprint" "FS_3_Global_Footprint_Library:01530008LXN"
 			(at 140.97 141.478 90)
 			(effects
@@
 			)
 		)
-		(property "Datasheet" "https://www.optifuse.com/optifuse_ecommerce_tools/datasheets/CNM-03.pdf"
+		(property "Datasheet" "https://www.digikey.com/en/products/detail/littelfuse-commercial-vehicle-products/01530008LXN/3425426?s=N4IgTCBcDaIAwEYCsBmO6AcAZAGgORAF0BfIA"
 			(at 140.97 139.7 0)
 			(effects
@@
 			)
 		)
-		(property "Value" "Fuse"
+		(property "Value" "01530008LXN"
 			(at 140.97 25.4 90)
 			(effects
@@
 			)
 		)
-		(property "Footprint" "project lib:CNM-03-BT mini blade fuse holder"
+		(property "Footprint" "FS_3_Global_Footprint_Library:01530008LXN"
 			(at 140.97 30.988 90)
 			(effects
@@
 			)
 		)
-		(property "Datasheet" "https://www.optifuse.com/optifuse_ecommerce_tools/datasheets/CNM-03.pdf"
+		(property "Datasheet" "https://www.digikey.com/en/products/detail/littelfuse-commercial-vehicle-products/01530008LXN/3425426?s=N4IgTCBcDaIAwEYCsBmO6AcAZAGgORAF0BfIA"
 			(at 140.97 29.21 0)
 			(effects
@@
 			)
 		)
-		(property "Value" "Fuse"
+		(property "Value" "01530008LXN"
 			(at 66.04 62.23 90)
 			(effects
@@
 			)
 		)
-		(property "Footprint" "project lib:CNM-03-BT mini blade fuse holder"
+		(property "Footprint" "FS_3_Global_Footprint_Library:01530008LXN"
 			(at 66.04 67.818 90)
 			(effects
@@
 			)
 		)
-		(property "Datasheet" "https://www.optifuse.com/optifuse_ecommerce_tools/datasheets/CNM-03.pdf"
+		(property "Datasheet" "https://www.digikey.com/en/products/detail/littelfuse-commercial-vehicle-products/01530008LXN/3425426?s=N4IgTCBcDaIAwEYCsBmO6AcAZAGgORAF0BfIA"
 			(at 66.04 66.04 0)
 			(effects
@@
 	(symbol
 		(lib_id "Device:Fuse")
-		(at 212.09 101.6 90)
+		(at 210.82 101.6 90)
 		(unit 1)
 		(exclude_from_sim no)
@@
 		(fields_autoplaced yes)
 		(property "Reference" "F12"
-			(at 212.09 95.25 90)
+			(at 210.82 95.25 90)
 			(effects
 				(font
@@
 			)
 		)
-		(property "Value" "Fuse"
-			(at 212.09 97.79 90)
+		(property "Value" "01530008LXN"
+			(at 210.82 97.79 90)
 			(effects
 				(font
@@
 			)
 		)
-		(property "Footprint" "project lib:CNM-03-BT mini blade fuse holder"
-			(at 212.09 103.378 90)
+		(property "Footprint" "FS_3_Global_Footprint_Library:01530008LXN"
+			(at 210.82 103.378 90)
 			(effects
 				(font
@@
 			)
 		)
-		(property "Datasheet" "https://www.optifuse.com/optifuse_ecommerce_tools/datasheets/CNM-03.pdf"
-			(at 212.09 101.6 0)
+		(property "Datasheet" "https://www.digikey.com/en/products/detail/littelfuse-commercial-vehicle-products/01530008LXN/3425426?s=N4IgTCBcDaIAwEYCsBmO6AcAZAGgORAF0BfIA"
+			(at 210.82 101.6 0)
 			(effects
 				(font
@@
 		)
 		(property "Description" "Fuse"
-			(at 212.09 101.6 0)
+			(at 210.82 101.6 0)
 			(effects
 				(font
@@
 			)
 		)
-		(property "Value" "Fuse"
+		(property "Value" "01530008LXN"
 			(at 66.04 25.4 90)
 			(effects
@@
 			)
 		)
-		(property "Footprint" "project lib:CNM-03-BT mini blade fuse holder"
+		(property "Footprint" "FS_3_Global_Footprint_Library:01530008LXN"
 			(at 66.04 30.988 90)
 			(effects
@@
 			)
 		)
-		(property "Datasheet" "https://www.optifuse.com/optifuse_ecommerce_tools/datasheets/CNM-03.pdf"
+		(property "Datasheet" "https://www.digikey.com/en/products/detail/littelfuse-commercial-vehicle-products/01530008LXN/3425426?s=N4IgTCBcDaIAwEYCsBmO6AcAZAGgORAF0BfIA"
 			(at 66.04 29.21 0)
 			(effects
