File: LT_MainBoard_TestingV1/LT_MainBoard_V1.kicad_sch (KiCad schematic)
At the start: 24 parts, among them CN1 NUCLEO-L432KC, J1 Molar Nanofit Connectors, U1 ISO1050DUB, U2 MCP2515-I/SO, U3 317990687, U4 LM7809_TO220, U5 LM7805_TO220, U6 LM3480-3.3

Commit message: Adapter V1
Made adapter board, modified lt mainboard
Connections:
- net +3V3: now also CN1.CN4_14 (3V3)
- net +9V: now also CN1.CN4_1 (VIN); no longer CN1.CN3_1 (PA9)
- net GND: now also CN1.CN4_2 (GND)
- net SPI3-MISO: now also CN1.CN3_15 (PB4); no longer CN1.CN4_15 (PB3)
- net SPI3-MOSI: now also CN1.CN3_14 (PB5); no longer CN1.CN4_14 (3V3)
- net SPI3-SCLK: now also CN1.CN4_15 (PB3); no longer CN1.CN3_15 (PB4)
- net SPI3_SSELI1: now also CN1.CN4_6 (PA7); no longer CN1.CN3_6 (PB0)
- net at CN1.CN3_2 (PA10): now also R2.2
- net at R1.1: now also CN1.CN3_1 (PA9); no longer CN1.CN4_1 (VIN)
- net NRST: now reaches CN1.CN4_12 (PA0)
- net NRST: now also U3.17 (RST)
Other:
- title: (none) -> Live Telemetry Testing Board
- moved on the sheet: C1, C2, C3, C4, C5, C6, C7, CN1A, J1, L1, R1, R2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

Commit message: Updating name
Parts:
- removed C13: 100nf, Capacitor_SMD:C_0805_2012Metric_Pad1.18x1.45mm_HandSolder, symbol Device:C
- removed L1: L, symbol Device:L
- removed R1, R2: R, symbol Device:R
- removed U3: 317990687, FS_3_Global_Footprint_Library:SEEED-317990687, symbol FS_3_Global_Symbol_Library:SEEED317990687
- added U3: XBP9B-DPST-001, FS_3_Global_Footprint_Library:XBP9B-DPST-001, symbol FS_3_Global_Symbol_Library:XBP9B-DPST-001
- C12: value 330nf -> 100nf
- C5: value 4.7 uF -> 1.0 uF; footprint (none) -> Capacitor_SMD:C_0805_2012Metric_Pad1.18x1.45mm_HandSolder
- C6: value C -> 47 pF; footprint (none) -> Capacitor_SMD:C_0805_2012Metric_Pad1.18x1.45mm_HandSolder
- C7: value C -> 330nf; footprint (none) -> Capacitor_SMD:C_0805_2012Metric_Pad1.18x1.45mm_HandSolder
Connections:
- net +12V: now also C7.1; no longer C12.1
- net GND: now also U3.10 (GND)
- net RADIO_IN: now reaches CN1.CN3_1 (PA9)
- net RADIO_IN: now also U3.3 (DIN/NCONFIG/DIO14)
- net RADIO_RESET: now reaches CN1.CN3_12 (PA8)
- net RADIO_RESET: now also U3.5 (~{RESET})
- net RADIO_OUT: now reaches CN1.CN3_2 (PA10)
- net RADIO_OUT: now also U3.2 (DOUT/DIO13)
- net at C6.1: now also C12.1, C3.2, C5.1, U1.1 (VCC1), U6.1 (VO), U3.1 (VCC)
- removed net +3V3: C3.2, C4.1, C5.1, CN1.CN4_14 (3V3), U1.1 (VCC1), U2.18 (VDD), U6.1 (VO)
- net NRST: no longer names the net of CN1.CN4_12 (PA0)
- new net: C4.1, CN1.CN4_14 (3V3), U2.18 (VDD)

Commit message: Update Live Telemetry Board (11/19)
Parts:
- added C13: 2 µF, Capacitor_SMD:C_0805_2012Metric, symbol Device:C
- added D1: D, Diode_SMD:D_0805_2012Metric, symbol Device:D
- added R1: 10K, Resistor_SMD:R_0805_2012Metric, symbol Device:R_US
- added R2: 1 Ω, Resistor_SMD:R_0805_2012Metric, symbol Device:R_US
Connections:
- net GND: now also C13.2
- net SPI3_SSEL1: no longer U2.16 (*CS)
- net at C12.1, C3.2, C5.1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: now also D1.1 (K), R2.1
- net at U2.17 (*RESET): now also R1.1
- new net: C13.1, D1.2 (A), R1.2, R2.2

Commit message: Updated schematic (11/19)
Parts:
- removed U6: LM3480-3.3, Package_TO_SOT_SMD:SOT-23, symbol Regulator_Linear:LM3480-3.3
- added U6: LF33_TO220, Package_TO_SOT_THT:TO-220-3_Vertical, symbol Regulator_Linear:LF33_TO220
- C12: value 100nf -> 2.2 µF; footprint Capacitor_SMD:C_0805_2012Metric_Pad1.18x1.45mm_HandSolder -> Capacitor_SMD:C_0805_2012Metric
- C13: value 2 µF -> 10 µF
- C7: value 330nf -> 0.1 µF; footprint Capacitor_SMD:C_0805_2012Metric_Pad1.18x1.45mm_HandSolder -> Capacitor_SMD:C_0805_2012Metric
- R2: value 1 Ω -> 100 Ω
Connections:
- net +12V: now also U6.1 (VI)
- net GND: now also U6.2 (GND)
- net at C12.1, C3.2, C5.1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: now also U6.3 (VO)

Commit message: d
Connections:
- net SPI3_SSEL1: now also U2.16 (*CS)
- net +3V3: now reaches C12.1, C3.2, C5.1, C6.1, U1.1 (VCC1), U3.1 (VCC), U6.3 (VO)
- net +3V3: no longer D1.1 (K), R2.1
- net at C4.1, CN1.CN4_14 (3V3), U2.18 (VDD): now also D1.1 (K), R2.1
- no-connect marks 0 -> 43

Commit message: update LT board to F446RE
Parts:
- removed C13: 10 µF, Capacitor_SMD:C_0805_2012Metric, symbol Device:C
- removed C4: 100nf, Capacitor_SMD:C_0805_2012Metric_Pad1.18x1.45mm_HandSolder, symbol Device:C
- removed CN1: NUCLEO-L432KC, FS_3_Global_Footprint_Library:NUCLEO-L432KC, symbol FS_3_Global_Symbol_Library:NUCLEO-L432KC
- removed D1: D, Diode_SMD:D_0805_2012Metric, symbol Device:D
- removed R1: 10K, Resistor_SMD:R_0805_2012Metric, symbol Device:R_US
- removed R2: 100 Ω, Resistor_SMD:R_0805_2012Metric, symbol Device:R_US
- removed U2: MCP2515-I/SO, Package_SO:SOIC-18W_7.5x11.6mm_P1.27mm, symbol FS_3_Global_Symbol_Library:MCP2515-I_SO
- added U2: NUCLEO-F446RE, FS_3_Global_Footprint_Library:NUCLEO-F446RE, symbol FS_3_Global_Symbol_Library:NUCLEO-F446RE
- C1: footprint Capacitor_SMD:C_0805_2012Metric_Pad1.18x1.45mm_HandSolder -> Capacitor_SMD:C_0805_2012Metric
Connections:
- net +5V: now also U2.CN10_8 (U5V)
- net +9V: now also U2.CN7_24 (CN7_VIN)
- net CAN1_RX: now also U2.CN10_3 (PB8)
- net CAN1_TX: now also U2.CN10_5 (PB9)
- net GND: now also U2.CN10_20 (CN10_GND__1), U2.CN10_32 (AGND), U2.CN10_9 (CN10_GND), U2.CN7_19 (CN7_GND__1)
- new net +3.3V: U2.CN10_24 (PB1), U2.CN10_7 (AVDD), U2.CN7_12 (CN7_IOREF), U2.CN7_16 (CN7_+3V3), U2.CN7_5 (VDD)
- no-connect marks 43 -> 78
Other:
- moved on the sheet: C12, C2, C3, C5, C6, C7, U1, U3, U6
