File: Live_Telemetry_Reciever_Board/Live_Telemetry_Reciever_Board.kicad_pcb (KiCad board)
At the start: 2 copper layers, 48.9 x 56.1 mm, 4 parts, among them CN1 NUCLEO-L432KC, U1 XBP9B-DPST-001

Commit message: rename LT boards (LT_MainBoard_TestingV1 -> Live_Telemetry_Board)
Other:
- board text added: "FS-3 LT Reciever Board Formula Slug Designed by Nathan Pham Verison 1"
- board text removed: "FS-3 Adaptor Board Formula Slug Designed by Nathan Pham Verison 1"
Changed lines of the file:
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@@
 		(layer "Edge.Cuts")
 	)
-	(gr_text "FS-3 Adaptor Board\nFormula Slug\nDesigned by \nNathan Pham\nVerison 1\n"
-		(at 136.65 92.45 0)
+	(gr_text "FS-3 LT Reciever \nBoard\nFormula Slug\nDesigned by \nNathan Pham\nVerison 1\n"
+		(at 137 94.5 0)
 		(layer "F.SilkS")
 		(effects
