File: ByronTam-AccBoard/ByronTam-AccBoard.kicad_sch (KiCad schematic)
At the start: 11 parts, among them CN1 NUCLEO-L432KC, J3 Fans, J4 776087-1, Q2 STS6NF20V, U1 ISO1050DUB, U2 MCP2515-I/SO, U3 ISO1050DUB

Commit message: Finished Pins
Parts:
- removed C7, C8: 100nF, Capacitor_SMD:C_0805_2012Metric_Pad1.18x1.45mm_HandSolder, symbol Device:C
- removed J3: Fans, 1FS_2_Global_Footprint_Library:MOLEX_1053091206, symbol 1FS_2_Global_Symbol_Library:1053091206
- removed J4: 776087-1, 1FS_2_Global_Footprint_Library:TE_776087-1, symbol 1FS_2_Global_Symbol_Library:776087-1
- removed Q2: STS6NF20V, 1FS_2_Global_Footprint_Library:SO-8_STM, symbol 1_ACC_BOARD:STS6NF20V
- removed U3: ISO1050DUB, Package_SO:SOP-8_6.62x9.15mm_P2.54mm, symbol Interface_CAN_LIN:ISO1050DUB
- added C1, C2: 100nF, Capacitor_SMD:C_0805_2012Metric_Pad1.18x1.45mm_HandSolder, symbol Device:C
- added J1: Fans, 1FS_2_Global_Footprint_Library:MOLEX_1053091206, symbol 1FS_2_Global_Symbol_Library:1053091206
- added J2, J3: Molex Nanofit 12pin, Connector_Molex:Molex_Nano-Fit_105310-xx12_2x06_P2.50mm_Vertical, symbol Connector:Conn_01x12_Pin
- added J6: Current Sensor, 1FS_2_Global_Footprint_Library:MOLEX_1053091204, symbol 1FS_2_Global_Symbol_Library:1053091204
- added Q1: STS6NF20V, 1FS_2_Global_Footprint_Library:SO-8_STM, symbol 1_ACC_BOARD:STS6NF20V
- added R10, R9: 120, Resistor_SMD:R_0805_2012Metric_Pad1.20x1.40mm_HandSolder, symbol Device:R
- added R11, R13: R1, symbol Device:R
- added R12, R8: R2, symbol Device:R
- added R14: 1M, symbol Device:R
- added R15: 2M, symbol Device:R
- added R16: 10K, symbol Device:R
- added U3, U7, U8: MCP6004, 1FS_2_Global_Footprint_Library:TSSOP14_MC_MCH, symbol Amplifier_Operational:MCP6004
- added U5: ISO1050DUB, Package_SO:SOP-8_6.62x9.15mm_P2.54mm, symbol Interface_CAN_LIN:ISO1050DUB
- added U6: MCP2515-I/SO, Package_SO:SOIC-18W_7.5x11.6mm_P1.27mm, symbol FS_3_Global_Symbol_Library:MCP2515-I_SO
- U2: footprint SOIC18-W_MC_MCH -> Package_SO:SOIC-18W_7.5x11.6mm_P1.27mm
Connections:
- net +12V: now also J1.2, J1.4, J1.6, J3.1 (Pin_1)
- net +3.3V: now also C10.2, CN1.CN4_14 (3V3), U1.1 (VCC1), U2.18 (VDD), C2.2, U5.1 (VCC1), U6.18 (VDD)
- net Fan_Control: now also CN1.CN4_6 (PA7), Q1.4 (G)
- net GND: now also C10.1, C9.1, CN1.CN3_4 (GND), CN1.CN4_2 (GND), U1.4 (GND1), U1.5 (GND2), U2.9 (VSS), C1.1, C2.1, J3.2 (Pin_2), J6.2, Q1.1 (S), Q1.2 (S), Q1.3 (S), R11.1, R15.2, R16.2, U5.4 (GND1), U5.5 (GND2), U6.9 (VSS)
- net at U1.2 (RXD): now also U2.2 (RXCAN)
- net at U1.3 (TXD): now also U2.1 (TXCAN)
- net CAN_L2: now reaches U1.6 (CANL)
- net CAN_L2: now also J3.8 (Pin_8), R9.2
- net CAN_H2: now reaches U1.7 (CANH)
- net CAN_H2: now also J3.7 (Pin_7), J3.9 (Pin_9)
- net +5V: now reaches C9.2, U1.8 (VCC2)
- net +5V: now also CN1.CN4_4 (5V), C1.2, J6.1, U5.8 (VCC2)
- net MOSI: now reaches CN1.CN3_14 (PB5)
- net MOSI: now also U2.14 (SI), U6.14 (SI)
- net MISO: now reaches CN1.CN3_15 (PB4)
- net MISO: now also U2.15 (SO), U6.15 (SO)
- net +9V: now reaches CN1.CN4_1 (VIN)
- net at CN1.CN4_12 (PA0): now also R14.1, R15.1
- net CLK: now reaches CN1.CN4_15 (PB3)
- net CLK: now also U2.13 (SCK), U6.13 (SCK)
- new net: U5.3 (TXD), U6.1 (TXCAN)
- new net: U5.2 (RXD), U6.2 (RXCAN)
- new net: R11.2, R8.1, U3.3 (+)
- new net: R12.1, R13.2, U3.2 (-)
- new net: R13.1, R14.2, U3.1
- new net: J1.1, J1.3, J1.5, Q1.5 (D), Q1.6 (D), Q1.7 (D), Q1.8 (D)
- new net: J6.3, R16.1, U8.3 (+)
- new net: J6.4, U7.3 (+)
- new net BMS_Fault: J2.1 (Pin_1)
- new net CAN_H1: J3.3 (Pin_3), J3.5 (Pin_5), U5.7 (CANH)
- new net CAN_L1: J3.4 (Pin_4), R10.2, U5.6 (CANL)
- new net CAN_L_RES1: J3.6 (Pin_6), R10.1
- new net CAN_L_RES2: J3.10 (Pin_10), R9.1
- new net Charge_State: J3.12 (Pin_12)
- new net Current_Vout: J2.7 (Pin_7), R8.2, U8.1, U8.2 (-)
- new net Current_Vref: J2.6 (Pin_6), R12.2, U7.1, U7.2 (-)
- new net IMD_Fault: J2.2 (Pin_2)
- new net IR_GND: J3.11 (Pin_11)
- new net Shut_Final: J2.5 (Pin_5)
- new net Shut_In: J2.3 (Pin_3)
- new net Shut_Out: J2.4 (Pin_4)
- new net Shut_Reset: J2.8 (Pin_8)
- no-connect marks 0 -> 20
Other:
- note added: "Connector"
- note removed: "Fans"
- moved on the sheet: C10, C9, CN1A, U1

Commit message: Pins on Microcontroller Added
Parts:
- removed C1, C10, C2, C9: 100nF, Capacitor_SMD:C_0805_2012Metric_Pad1.18x1.45mm_HandSolder, symbol Device:C
- removed CN1: NUCLEO-L432KC, FS_3_Global_Footprint_Library:NUCLEO-L432KC, symbol FS_3_Global_Symbol_Library:NUCLEO-L432KC
- removed J1: Fans, 1FS_2_Global_Footprint_Library:MOLEX_1053091206, symbol 1FS_2_Global_Symbol_Library:1053091206
- removed J2, J3: Molex Nanofit 12pin, Connector_Molex:Molex_Nano-Fit_105310-xx12_2x06_P2.50mm_Vertical, symbol Connector:Conn_01x12_Pin
- removed J6: Current Sensor, 1FS_2_Global_Footprint_Library:MOLEX_1053091204, symbol 1FS_2_Global_Symbol_Library:1053091204
- removed Q1: STS6NF20V, 1FS_2_Global_Footprint_Library:SO-8_STM, symbol 1_ACC_BOARD:STS6NF20V
- removed R10, R9: 120, Resistor_SMD:R_0805_2012Metric_Pad1.20x1.40mm_HandSolder, symbol Device:R
- removed R11, R13: R1, symbol Device:R
- removed R12: R2, symbol Device:R
- removed R14: 1M, symbol Device:R
- removed R15: 2M, symbol Device:R
- removed R16: 10K, symbol Device:R
- removed U1, U5: ISO1050DUB, Package_SO:SOP-8_6.62x9.15mm_P2.54mm, symbol Interface_CAN_LIN:ISO1050DUB
- removed U2, U6: MCP2515-I/SO, Package_SO:SOIC-18W_7.5x11.6mm_P1.27mm, symbol FS_3_Global_Symbol_Library:MCP2515-I_SO
- removed U7, U8: MCP6004, 1FS_2_Global_Footprint_Library:TSSOP14_MC_MCH, symbol Amplifier_Operational:MCP6004
- added C15, C16, C28, C7, C8: 100nF, Capacitor_SMD:C_0805_2012Metric_Pad1.18x1.45mm_HandSolder, symbol Device:C
- added C17, C22, C23, C24: 100uF, Capacitor_SMD:C_0805_2012Metric_Pad1.18x1.45mm_HandSolder, symbol Device:C
- added C20: 1uF, Capacitor_SMD:C_0805_2012Metric_Pad1.18x1.45mm_HandSolder, symbol Device:C_Polarized
- added C21: 100nf, Capacitor_SMD:C_0805_2012Metric_Pad1.18x1.45mm_HandSolder, symbol Device:C
- added C25: 1uF, Capacitor_SMD:C_0805_2012Metric_Pad1.18x1.45mm_HandSolder, symbol Device:C
- added C26: 10uF, Capacitor_SMD:C_0805_2012Metric_Pad1.18x1.45mm_HandSolder, symbol Device:C
- added C27: 0.33uF, Capacitor_SMD:C_0805_2012Metric_Pad1.18x1.45mm_HandSolder, symbol Device:C
- added C29, C30: 330nF, Capacitor_SMD:C_0805_2012Metric_Pad1.18x1.45mm_HandSolder, symbol Device:C
- added C31: 10µF, Capacitor_SMD:C_0805_2012Metric_Pad1.18x1.45mm_HandSolder, symbol Device:C
- added C32: 0.1uF, Capacitor_SMD:C_0805_2012Metric_Pad1.18x1.45mm_HandSolder, symbol Device:C
- added CN2: NUCLEO-L432KC, FS_3_Global_Footprint_Library:NUCLEO-L432KC, symbol FS_3_Global_Symbol_Library:NUCLEO-L432KC
- added CR1, CR2, CR3: STS6NF20V, SO-8_STM, symbol FS_2_Global_Symbol_Library:STS6NF20V
- added D1, D2, D3, D4, D7: D, Diode_SMD:D_2010_5025Metric_Pad1.52x2.65mm_HandSolder, symbol Device:D
- added D8: 50V, symbol Device:D_Zener
- added J1: Current Sensor, 1FS_2_Global_Footprint_Library:MOLEX_1053091204, symbol 1FS_2_Global_Symbol_Library:1053091204
- added J10, J9: Molex Nanofit 12pin, Connector_Molex:Molex_Nano-Fit_105310-xx12_2x06_P2.50mm_Vertical, symbol Connector:Conn_01x12_Pin
- added J11: Precharge Resistor, 1FS_2_Global_Footprint_Library:MOLEX_1053091202, symbol 1FS_2_Global_Symbol_Library:1053091202
- added J12: AIRs Power, 1FS_2_Global_Footprint_Library:MOLEX_1053091204, symbol 1FS_2_Global_Symbol_Library:1053091204
- added J4: IMD, 1FS_2_Global_Footprint_Library:MOLEX_1053091203, symbol 1FS_2_Global_Symbol_Library:1053091203
- added J7: Shutdown IL, 1FS_2_Global_Footprint_Library:MOLEX_1053091202, symbol molex_1053091202:1053091202
- added K1, K2: DK1A1B-5V, FS_3_Global_Footprint_Library:DK1A1B, symbol 2FS-1_Symbol Library:DK1A1B-12V
- added K3: G6BK-1114P-US, 1FS_2_Global_Footprint_Library:Omron G6BK-1114P-US, symbol 1FS_2_Global_Symbol_Library:G6BK-1114P-US
- added K4: G5PZ-1A-X DC12, 1FS_2_Global_Footprint_Library:G5PZ-1A-X DC12, symbol Relay:Relay_SPST-NO
- added Q2, Q3: STS6NF20V, 1FS_2_Global_Footprint_Library:SO-8_STM, symbol 1_ACC_BOARD:STS6NF20V
- added R1: 120k, Resistor_SMD:R_0805_2012Metric_Pad1.20x1.40mm_HandSolder, symbol Device:R
- added R17, R28, R5, R6: 100k, Resistor_SMD:R_0805_2012Metric_Pad1.20x1.40mm_HandSolder, symbol Device:R
- added R18, R19: 120, Resistor_SMD:R_0805_2012Metric_Pad1.20x1.40mm_HandSolder, symbol Device:R
- added R2: 200k, Resistor_SMD:R_0805_2012Metric_Pad1.20x1.40mm_HandSolder, symbol Device:R
- added R20: 1.6k, Resistor_SMD:R_0805_2012Metric_Pad1.20x1.40mm_HandSolder, symbol Device:R
- added R21: 560, Resistor_SMD:R_0805_2012Metric_Pad1.20x1.40mm_HandSolder, symbol Device:R
- added R3, R4: 400k, Resistor_SMD:R_0805_2012Metric_Pad1.20x1.40mm_HandSolder, symbol Device:R
- added R34: 10M, Resistor_SMD:R_0805_2012Metric_Pad1.20x1.40mm_HandSolder, symbol Device:R
- added R35: 7.2k, Resistor_SMD:R_0805_2012Metric_Pad1.20x1.40mm_HandSolder, symbol Device:R
- added R36: 10k, Resistor_SMD:R_0805_2012Metric_Pad1.20x1.40mm_HandSolder, symbol Device:R
- added R7: 10K, Resistor_SMD:R_0805_2012Metric_Pad1.20x1.40mm_HandSolder, symbol Device:R
- added U10, U9: ISO1050DUB, Package_SO:SOP-8_6.62x9.15mm_P2.54mm, symbol Interface_CAN_LIN:ISO1050DUB
- added U13: MCP6004, symbol Amplifier_Operational:MCP6004
- added U14, U16, U18: 74AHC1G04, symbol 74xGxx:74AHC1G04
- added U15: HEF4093B, symbol 4xxx:HEF4093B
- added U17: LM555xN, Package_DIP:DIP-8_W7.62mm, symbol Timer:LM555xN
- added U19: 74AHC1G32, symbol 74xGxx:74AHC1G32
- added U2: NUCLEO-F446RE, NUCLEO-F446RE:MODULE_NUCLEO-F446RE, symbol FS_3_Global_Symbol_Library:NUCLEO-F446RE
- added U20: ZXTR2005ZQ-13, Package_TO_SOT_THT:TO-220-3_Vertical, symbol Regulator_Linear:LM7809_TO220
- added U21: L7805CV, Converter_DCDC:Converter_DCDC_RECOM_R-78B-2.0_THT, symbol Regulator_Switching:R-78B5.0-2.0
- added U22, U23: MC7809CTG, Package_TO_SOT_THT:TO-220-3_Vertical, symbol Regulator_Linear:LM7809_TO220
- added unit 3 of U3
- added unit 2 of U3
- R8: value R2 -> 10k; footprint (none) -> Resistor_SMD:R_0805_2012Metric_Pad1.20x1.40mm_HandSolder
- U3: footprint 1FS_2_Global_Footprint_Library:TSSOP14_MC_MCH -> Package_SO:SOIC-14_3.9x8.7mm_P1.27mm
Connections:
- net +12V: now also C27.1, C28.1, C29.1, J10.1 (Pin_1), J4.2, R28.1, U21.1 (IN), U22.1 (VI), U23.1 (VI)
- net +3.3V: now also C15.2, C16.2, C31.1, CN2.CN4_13 (AREF), U10.1 (VCC1), U2.CN7_16 (CN7_+3V3), U23.3 (VO), U9.1 (VCC1)
- net +5V: now also C17.1, C21.2, C22.1, C23.1, C24.2, C32.1, C7.2, C8.2, D1.1 (K), D2.1 (K), J1.1, K1.8 (+), K2.8 (+), R34.2, U10.8 (VCC2), U13.4 (V+), U14.5 (VCC), U15.14 (VCC), U16.5 (VCC), U17.4 (R), U17.8 (VCC), U19.5 (VCC), U2.CN10_8 (U5V), U21.3 (OUT), U9.8 (VCC2)
- net +9V: now also C30.1, CN2.CN4_1 (VIN), U2.CN7_24 (CN7_VIN), U22.3 (VO)
- net CAN_H1: now also J10.3 (Pin_3), J10.5 (Pin_5), U9.7 (CANH)
- net CAN_H2: now also J10.7 (Pin_7), J10.9 (Pin_9), U10.7 (CANH)
- net CAN_L1: now also J10.4 (Pin_4), R18.2, U9.6 (CANL)
- net CAN_L2: now also J10.8 (Pin_8), R19.2, U10.6 (CANL)
- net CAN_L_RES1: now also J10.6 (Pin_6), R18.1
- net CAN_L_RES2: now also J10.10 (Pin_10), R19.1
- net CLK: now also CN2.CN4_15 (PB3)
- net Charge_State: now also R8.1, CN2.CN3_2 (PA10), J10.12 (Pin_12), R17.1, U2.CN10_33 (PA10)
- net Current_Vout: now also J9.8 (Pin_8), R5.2, U3.8, U3.9 (-); no longer R8.2
- net Current_Vref: now also J9.7 (Pin_7), R6.2, U3.6 (-), U3.7
- net GND: now also R8.2, C15.1, C16.1, C17.2, C20.2, C21.1, C22.2, C23.2, C24.1, C27.2, C28.2, C29.2, C30.2, C31.2, C32.2, C7.1, C8.1, CN2.CN3_4 (GND), CN2.CN4_2 (GND), CR1.1 (S), CR1.2 (S), CR1.3 (S), CR2.1 (S), CR2.2 (S), CR2.3 (S), CR3.1 (S), CR3.2 (S), CR3.3 (S), J1.2, J10.2 (Pin_2), J12.3, J4.3, Q2.1 (S), Q2.2 (S), Q2.3 (S), Q3.1 (S), Q3.2 (S), Q3.3 (S), R1.2, R17.2, R21.1, R36.2, R4.1, R7.2, U10.4 (GND1), U10.5 (GND2), U13.11 (V-), U14.3 (GND), U15.7 (GND), U16.3 (GND), U17.1 (GND), U18.3 (GND), U19.3 (GND), U2.CN10_20 (CN10_GND__1), U2.CN10_32 (AGND), U2.CN10_9 (CN10_GND), U2.CN7_19 (CN7_GND__1), U2.CN7_20 (CN7_GND__2), U2.CN7_22 (CN7_GND__3), U2.CN7_8 (CN7_GND), U21.2 (GND), U22.2 (GND), U23.2 (GND), U9.4 (GND1), U9.5 (GND2)
- net IR_GND: now also J10.11 (Pin_11)
- net MISO: now also CN2.CN3_15 (PB4), U2.CN10_28 (PB14)
- net MOSI: now also CN2.CN3_14 (PB5), U2.CN10_26 (PB15)
- net Shut_Reset: now also J9.9 (Pin_9)
- net at U3.3 (+): now also R4.2, R5.1; no longer R8.1
- net at U3.2 (-): now also R3.2, R6.1
- net at U3.1: now also R2.2, R3.1
- new net: Q2.4 (G), U18.4
- new net: D7.2 (A), K4.4, Q3.5 (D), Q3.6 (D), Q3.7 (D), Q3.8 (D)
- new net: D3.1 (K), K3.5, R28.2
- new net: J11.1, K4.2
- new net: J11.2, K4.3
- new net: C25.1, D8.2 (A), U20.1 (VI)
- new net: R35.2, R36.1, U19.1
- new net: U14.2, U15.4
- new net: CR2.4 (G), U14.4
- new net: D4.2 (A), K3.1
- new net: C20.1, R34.1, U17.2 (TR), U17.6 (THR)
- new net: U15.3, U16.2
- new net: U17.3 (Q), U19.2
- new net Amp_Curr_Sensor: CN2.CN4_11 (PA1), R1.1, R2.1, U2.CN7_30 (PA1)
- new net BMS_CS: CN2.CN3_13 (PA11), U2.CN10_16 (PB12)
- new net BMS_FAULT_3.3V: CN2.CN3_6 (PB0), CR1.4 (G), U2.CN10_15 (PA7)
- new net BMS_FAULT_5V: J9.1 (Pin_1), U15.2
- new net BMS_RL: CR1.5 (D), CR1.6 (D), CR1.7 (D), CR1.8 (D), D1.2 (A), K1.1 (-)
- new net BSPD_FAULT_5V: J9.3 (Pin_3), U15.5
- new net CAN1_RD: U2.CN10_3 (PB8), U9.2 (RXD)
- new net CAN1_TD: U2.CN10_5 (PB9), U9.3 (TXD)
- new net CAN2_RD: U10.2 (RXD), U2.CN10_29 (PB5)
- new net CAN2_TD: U10.3 (TXD), U2.CN10_30 (PB13)
- new net CAN_CS: CN2.CN3_8 (PB6)
- new net GLV Voltage: CN2.CN4_12 (PA0), U2.CN7_28 (PA0)
- new net IMD_DELAY: CR3.4 (G), U15.1, U19.4
- new net IMD_FAULT_12V: J4.1, R20.2, R35.1
- new net IMD_FAULT_5V: J9.2 (Pin_2)
- new net IMD_RL: CR3.5 (D), CR3.6 (D), CR3.7 (D), CR3.8 (D), D2.2 (A), K2.1 (-)
- new net IMD_Status: CN2.CN3_5 (PA12), R20.1, R21.2, U2.CN10_13 (PA6)
- new net IR+_12V: J12.2, J12.4
- new net IR+_GND: J12.1, Q2.5 (D), Q2.6 (D), Q2.7 (D), Q2.8 (D)
- new net IRs_Final: J9.6 (Pin_6)
- new net LATCH_RL: CR2.5 (D), CR2.6 (D), CR2.7 (D), CR2.8 (D), D3.2 (A), K3.2
- new net MC_CAN_CS: CN2.CN3_7 (PB7)
- new net Precharge_Control: CN2.CN3_9 (PB1), Q3.4 (G), U18.2, U2.CN10_21 (PA9)
- new net Raw_Curr_Out: J1.3, R7.1, U3.10 (+)
- new net Raw_Curr_VRef: J1.4, U3.5 (+)
- new net SCK: U2.CN10_19 (PC7)
- new net SH_RESET: D4.1 (K), K3.6
- new net Shutdown_ACC_BMS: K1.4, K2.3
- new net Shutdown_ACC_IL: J7.2, K3.4
- new net Shutdown_ACC_IMD: J7.1, K2.4
- new net Shutdown_ACC_IN: J9.4 (Pin_4), K1.3
- new net Shutdown_ACC_OUT: J9.5 (Pin_5), K3.3
- new net Shutdown_AIRS_IN: D7.1 (K), K4.1
- new net TS+: D8.1 (K)
- new net TS-: C25.2, C26.2, U20.2 (GND)
- new net TSSI: U15.6, U16.4
- new net Voltage Indicator: C26.1, U20.3 (VO)
- no-connect marks 20 -> 67
Other:
- removed sheet Iso SPI
- added sheet Iso SPI1 (isoSPI.kicad_sch)
- note added: "--> BMS Relay"
- note added: "--> IMD Relay"
- note added: "0V or 2-3.3V"
- note added: "0V or 8-12V"
- note added: "12V --> ~5V Input to LV Logic at 5V"
- note added: "3.3V"
- note added: "555 Timer ~11 sec on 5V Power"
- note added: "ACC Onboard Shutdown"
- note added: "AIR power from shutdown circuit; inside acc"
- note added: "Auxillary Connector"
- note added: "BMS Fault Low --> 5V Relay"
- note added: "BMS Relay"
- note added: "CAN"
- note added: "Check polarity and annotate"
- note added: "Current Sensor"
- note added: "Double check where the Voltage Indicator will go out to"
- note added: "GLV"
- note added: "Goes to IMD; inside ACC"
- note added: "IMD Fault Low 3.3V --> 5V Relay"
- note added: "IMS Relay"
- note added: "IsoSPI"
- note added: "Latch Trigger MOSFET"
- note added: "Move these Pins"
- note added: "Need to power GATE. What voltage?"
- note added: "On fault condition triggers TSSI light"
- note added: "Power Block"
- note added: "Precharge Circuit"
- note added: "SMD NAND GATE"
- note added: "SPST Latching Relay"
- note added: "Shutdown interlock (BFC), inside ACC"
- note added: "TS"
- note added: "Upstream delay of ~11sec durring power on"
- note added: "Voltage Indicator"
- note removed: "Connector"
- note removed: "Iso SPI"
