File: Accumulator_Board/isoSPI.kicad_sch (KiCad schematic)
At the start: 16 parts, among them J5 IsoSPI, U8 LTC6820

Commit message: footprints
Parts:
- L1: footprint 1FS_2_Global_Footprint_Library:HM2113ZNL -> FS_3_Global_Footprint_Library:HM2113ZNLT
Changed lines of the file:
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@@
 			)
 		)
-		(property "Footprint" "1FS_2_Global_Footprint_Library:HM2113ZNL"
+		(property "Footprint" "FS_3_Global_Footprint_Library:HM2113ZNLT"
 			(at 132.08 26.67 0)
 			(effects
