File: Accumulator_Board/Accumulator_Board.kicad_pcb (KiCad board)
At the start: 2 copper layers, 125.7 x 89.5 mm, 97 parts, among them J1 IMD, J10 HVIL, J11 Molex Nanofit 16pin, J2 Molex Nanofit 12pin, J4 Current Sensor, J5 IsoSPI, J6 Shutdown IL, J7 AIRs Power, J8 Precharge Resistor, J9 TS+/TS-, K1 DK1A1B-12V, K2 G5PZ-1A-X DC12, K3 DK1A1B-12V, K4 G6BK-1114P-US, Q1 STS6NF20V, Q2 STS6NF20V, U1 ISO1050DUB, U10 MC7809CTG, U12 LM555xN, U15 ZXTR2005ZQ-13, U16 4069, U2 NUCLEO-L432KC, U4 SN74HCS32DR, U5 MCP6004, U6 DS18B20U, U7 HEF4093B, U8 LTC6820, U9 L7805CV

Commit message: Fixed dk1a1b relays and CAN transceiver
Parts:
- R26: value 7.2k -> 10k
- R27: value 10k -> 7.2k
- moved R36 25.8 mm to (38.1, 64.0), turned to 90 degrees
- moved C2 18.9 mm to (52.3, 87.4)
- moved R1 16.0 mm to (32.3, 85.6), turned to 90 degrees
- moved C1 15.6 mm to (35.1, 88.6), turned to -90 degrees
- moved C14 7.68 mm to (49.0, 97.8), turned to -90 degrees
- moved C13 6.70 mm to (32.3, 97.8), turned to -90 degrees
- moved G*** 6.56 mm to (77.4, 103.2)
- moved U1 3.89 mm to (44.5, 85.9), turned to 180 degrees
- moved C11 0.78 mm to (37.1, 105.9)
- moved C10 0.65 mm to (44.5, 105.9)
Connections:
- D2 pad 1: +5V -> +12V
- D4 pad 1: +5V -> +12V
- K1 pad 8: +5V -> +12V
- K3 pad 8: +5V -> +12V
- U16 pad 3: Net-(U16-Pad3) -> (no net)
- U16 pad 4: Net-(CR2-G) -> (no net)
- U2 pad CN3_12: unconnected-(U2A-PA8-PadCN3_12) -> /Fan_PWM
- U2 pad CN4_11: /Fan_PWM -> unconnected-(U2A-PA1-PadCN4_11)
- U7 pad 4: Net-(U16-Pad3) -> Net-(CR2-G)
Routing:
- net +12V: track 251.3 -> 287.5 mm
- net GND: track 180.3 -> 149.6 mm, vias 30 -> 29
- net Net-(U16-Pad3): track 29.0 -> 0.00 mm
- net /GLV Voltage: track 31.9 -> 5.24 mm
- net +5V: track 259.9 -> 238.4 mm, vias 15 -> 12
- net /CAN_L_RES1: track 24.3 -> 4.34 mm
- net /CAN1_RD: track 24.2 -> 42.5 mm, vias 0 -> 2
- net /CAN1_TD: track 48.5 -> 63.3 mm, vias 0 -> 2
- net /IMD_Status: track 88.3 -> 78.8 mm
- net /Fan_PWM: track 30.2 -> 22.3 mm
- net Net-(CR2-G): track 16.8 -> 10.9 mm, vias 0 -> 2
- net /IMD_LED_Control: track 44.0 -> 38.3 mm
- net /CAN_H1: track 26.5 -> 20.8 mm
- net /CAN_L1: track 25.1 -> 19.4 mm
- net +3.3V: track 136.0 -> 139.7 mm, vias 4 -> 0
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Other:
- board text added: "Accumulator Board V3.1 FS-3 Designed By: Andrew She"
- board text removed: "Accumulator Board V2"
- board text removed: "Designed by: Andrew She"

Commit message: Minor cleanup and moved precharge relay
Parts:
- moved K2 0.66 mm to (94.2, 24.2)
Routing:
- net GND: track 149.6 -> 146.4 mm
- net +5V: track 238.4 -> 235.8 mm
- net +12V: track 287.5 -> 285.8 mm
- net /TS-: track 31.4 -> 29.9 mm
- net /IMD_RL: track 20.8 -> 19.8 mm
- net /IMD_DELAY: track 61.3 -> 60.3 mm
- net Net-(L1-Pad1): track 12.7 -> 11.8 mm
- net /BMS_RL: track 28.9 -> 28.0 mm
- net /MISO: track 135.1 -> 134.3 mm
- net +3.3V: track 139.7 -> 138.9 mm
- net Net-(CR1-G): track 3.14 -> 2.44 mm
- net Net-(U16-Pad1): track 19.4 -> 18.7 mm
- net /GLV Voltage: track 5.24 -> 4.60 mm
- net Net-(J8-Pad1): track 16.6 -> 16.0 mm
- net +9V: track 68.5 -> 67.9 mm
Other:
- board text added: "HV"
- board text added: "LV"

Commit message: silkscreen change
Parts:
- J9: value TS+/TS- -> TS-/TS+
Changed lines of the file:
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@@
 			)
 		)
-		(property "Value" "TS+/TS-"
+		(property "Value" "TS-/TS+"
 			(at 3.015 0.615 0)
 			(layer "F.SilkS")

Commit message: Linear Regulator Fix
Parts:
- added U3: 4069, Package_SO:SOIC-14_3.9x8.7mm_P1.27mm, F.Cu at (157.5, 49.5)
- J9: value TS-/TS+ -> TS+/TS-
- moved U15 26.4 mm to (158.1, 36.8)
Connections:
- Q1 pad 4: Net-(Q1-G) -> /Precharge_Control
- Q2 pad 4: /Precharge_Control -> Net-(Q2-G)
- U15 pad 1: Net-(D8-A) -> /TS-
- U15 pad 2: /TS- -> Net-(D8-A)
- U16 pad 5: /Precharge_Control -> (no net)
- U16 pad 6: Net-(Q1-G) -> (no net)
Routing:
- net Net-(Q1-G): track 6.00 -> 0.00 mm
- net /Precharge_Control: track 93.1 -> 99.1 mm

Commit message: Main Push
Parts:
- moved U15 26.4 mm to (132.1, 41.3)
Routing:
- net /HVIL: track 25.6 -> 17.9 mm
- net /TS-: track 29.9 -> 24.7 mm
- net Net-(D8-A): track 10.9 -> 6.29 mm
Changed lines of the file:
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@@
 	(footprint "FS_3_Global_Footprint_Library:SOT-89_4P5X2P45_DIO"
 		(layer "F.Cu")
-		(at 158.115 36.83 180)
+		(at 132.08 41.275 180)
 		(descr "5V Linear Regulator")
 		(tags "ZXTR2005ZQ-13 ")
@@
 		)
 		(property "Footprint" "FS_3_Global_Footprint_Library:SOT-89_4P5X2P45_DIO"
-			(at 0 0 360)
+			(at 0 0 0)
 			(layer "F.Fab")
 			(hide yes)
@@
 		)
 		(property "Datasheet" "https://www.diodes.com/assets/Datasheets/ZXTR2005ZQ.pdf"
-			(at 0 0 360)
+			(at 0 0 0)
 			(layer "F.Fab")
 			(hide yes)
@@
 		)
 		(property "Description" "High Voltage 5V Linear Regulator"
-			(at 0 0 360)
+			(at 0 0 0)
 			(layer "F.Fab")
 			(hide yes)
@@
 	)
 	(gr_rect
-		(start 112.04 41.275)
-		(end 147.04 71.275)
+		(start 111.405 41.275)
+		(end 146.405 71.275)
 		(stroke
 			(width 0.2)
@@
 	)
 	(segment
-		(start 125.095 34.1644)
-		(end 130.58 39.6494)
-		(width 0.5)
-		(layer "F.Cu")
-		(net 17)
-	)
-	(segment
 		(start 55.245 92.656)
 		(end 55.245 98.425)
@@
 	)
 	(segment
-		(start 134.2106 39.6494)
-		(end 133.58 39.6494)
-		(width 0.5)
-		(layer "F.Cu")
-		(net 61)
-	)
-	(segment
-		(start 137.03 36.83)
-		(end 134.2106 39.6494)
-		(width 0.5)
-		(layer "F.Cu")
-		(net 61)
-	)
-	(segment
-		(start 132.08 33.825)
-		(end 132.08 39.6494)
-		(width 0.3)
+		(start 138.43 25.4)
+		(end 138.27 25.24)
+		(width 0.2)
 		(layer "F.Cu")
 		(net 62)
 	)
 	(segment
-		(start 138.43 25.4)
-		(end 138.27 25.24)
-		(width 0.2)
+		(start 134.2106 39.6494)
+		(end 133.58 39.6494)
+		(width 0.5)
 		(layer "F.Cu")
 		(net 62)

Commit message: Accumulator_Board-V4
Parts:
- removed G***: LOGO, FS_3_Global_Footprint_Library:FORMULA SLUG
- removed the REF** at (27.3, 107.3)
- removed the REF** at (144.1, 106.0)
- removed the REF** at (144.8, 25.4)
- removed the REF** at (26.7, 26.0)
- added REF**: MountingHole_3.2mm_M3, MountingHole:MountingHole_3.2mm_M3, F.Cu at (142.5, 24.5)
- added REF**: MountingHole_3.2mm_M3, MountingHole:MountingHole_3.2mm_M3, F.Cu at (142.5, 106.0)
- added REF**: MountingHole_3.2mm_M3, MountingHole:MountingHole_3.2mm_M3, F.Cu at (23.5, 106.0)
- added REF**: MountingHole_3.2mm_M3, MountingHole:MountingHole_3.2mm_M3, F.Cu at (23.5, 24.5)
- J9: value TS+/TS- -> TS-/TS+
- moved U3 93.2 mm to (69.8, 81.0), turned to -90 degrees
- moved R18 76.3 mm to (56.0, 106.5), turned to 0 degrees
- moved R17 74.2 mm to (22.0, 88.0), turned to -90 degrees
- moved Q1 69.6 mm to (37.0, 33.0), turned to 0 degrees
- moved R35 64.4 mm to (97.5, 43.0)
- moved R36 60.2 mm to (94.5, 43.0), turned to -90 degrees
- moved C9 55.3 mm to (52.0, 27.5), turned to 0 degrees
- moved D2 55.1 mm to (40.5, 48.0), turned to -90 degrees
- moved C10 52.3 mm to (38.0, 54.0), turned to -90 degrees
- moved C11 51.9 mm to (35.5, 54.0), turned to -90 degrees
- moved J11 51.5 mm to (25.7, 49.2)
- moved R29 50.9 mm to (73.5, 33.0), turned to 0 degrees
- moved R27 50.1 mm to (47.5, 32.0), turned to -90 degrees
- moved R26 49.6 mm to (45.5, 32.0), turned to 90 degrees
- moved C22 49.4 mm to (52.2, 31.5), turned to 0 degrees
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Connections:
- J8 pad 1: Net-(J8-Pad1) -> Net-(J8-Pad2)
- K2 pad 2: Net-(J8-Pad1) -> Net-(J8-Pad2)
Routing:
- net /IR+_GND: track 192.7 -> 24.8 mm, vias 0 -> 2
- net +12V: track 285.8 -> 147.5 mm, vias 5 -> 1
- net /BMS_CS: track 127.6 -> 0.00 mm, vias 1 -> 0
- net /GLV Voltage: track 4.60 -> 125.9 mm
- net /IMD_LED_Control: track 38.3 -> 154.8 mm, vias 0 -> 3
- net /Current_Vref: track 70.2 -> 157.3 mm, vias 6 -> 3
- net /SH_RESET: track 34.7 -> 114.1 mm, vias 0 -> 3
- net /Amp_Curr_Sensor: track 34.4 -> 108.7 mm
- net /BMS_LED_Control: track 49.8 -> 115.3 mm, vias 0 -> 5
- net GND: track 146.4 -> 84.4 mm
- net +5V: track 235.8 -> 175.0 mm, vias 12 -> 2
- net /IR+_12V: track 138.6 -> 190.2 mm, vias 2 -> 6
- net +3.3V: track 138.9 -> 188.2 mm
- net Net-(D7-A): track 14.5 -> 63.1 mm, vias 0 -> 1
- net Net-(D5-K): track 12.6 -> 56.0 mm, vias 0 -> 2
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Other:
- board size 125.7 x 89.5 mm -> 127 x 89.5 mm
- board text added: "Accumulator Board V4"
- board text added: "Designed By: Eric Zhang"
- board text added: "FS-3"
- board text removed: "Accumulator Board V3.1 FS-3 Designed By: Andrew She"

Commit message: V4.1
Parts:
- moved D6 62.3 mm to (94.0, 59.5), turned to -90 degrees
- moved R18 36.0 mm to (24.5, 89.0)
- moved D7 5.75 mm to (69.3, 64.5)
- moved R17 2.69 mm to (24.5, 87.0), turned to 180 degrees
- moved C7 2.17 mm to (120.7, 97.0)
- moved C8 2.17 mm to (117.2, 97.0)
- moved R13 2.17 mm to (113.7, 97.0)
- moved REF** 2.00 mm to (142.5, 22.5)
- moved REF** 2.00 mm to (23.5, 22.5)
- moved L1 1.94 mm to (117.2, 85.9)
- moved K2 0.44 mm to (93.4, 23.7)
Routing:
- net /Shutdown_ACC_Out: track 85.8 -> 0.00 mm, vias 3 -> 0
- net /SH_RESET: track 114.1 -> 91.9 mm
- net +3.3V: track 188.2 -> 176.6 mm
- net /CAN_L_RES1: track 34.8 -> 27.4 mm
- net /GLV Voltage: track 125.9 -> 133.2 mm
- net /Charge_State: track 93.2 -> 86.2 mm
- net Net-(D7-A): track 63.1 -> 69.0 mm
- net /BMS_LED_Control: track 115.3 -> 118.7 mm
- net /Shutdown_Measure: track 52.4 -> 49.2 mm, vias 1 -> 0
- net /IMD_LED_Control: track 154.8 -> 151.7 mm, vias 3 -> 2
- net /BMS_FAULT_3.3V: track 67.6 -> 64.7 mm
- net /Iso SPI/isoSPI_+: track 16.3 -> 14.0 mm
- net /Iso SPI/isoSPI_-: track 10.3 -> 12.1 mm
- net /Current_Vout: track 107.8 -> 106.3 mm
- net /Current_Vref: track 157.3 -> 155.8 mm
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Other:
- board size 127 x 89.5 mm -> 127 x 91.5 mm
- board text added: "+5V/GND/Out/VRef"
- board text added: "ACC_IMD+TP/ACC_IL_IP"
- board text added: "Accumulator Board V4.1"
- board text added: "HVIL/TS-"
- board text added: "IMD_FAULT_12V/+12V/GND"
- board text added: "IR+_GND/IR+_12V/GND/12+_12V"
- board text added: "Net-(J8-Pad2)"
- board text removed: "Accumulator Board V4"
