File: Accumulator_Board/Accumulator_Board.kicad_sch (KiCad schematic)
At the start: 76 parts, among them J1 IMD, J10 HVIL, J11 Molex Nanofit 16pin, J2 Molex Nanofit 12pin, J4 Current Sensor, J6 Shutdown IL, J7 AIRs Power, J8 Precharge Resistor, J9 TS+/TS-, K1 DK1A1B-12V, K2 G5PZ-1A-X DC12, K3 DK1A1B-12V, K4 G6BK-1114P-US, Q1 STS6NF20V, Q2 STS6NF20V, U1 ISO1050DUB, U10 MC7809CTG, U12 LM555xN, U15 ZXTR2005ZQ-13, U16 4069, U2 NUCLEO-L432KC, U4 SN74HCS32DR, U5 MCP6004, U6 DS18B20U, U7 HEF4093B, U9 L7805CV

Commit message: PCB Drc Needed
Connections:
- net Charge_State: no longer J11.12 (Pin_12)
- net Fan_PWM: no longer J11.10 (Pin_10)
- net IR+_GND: no longer J11.11 (Pin_11)
- no-connect marks 22 -> 25
Changed lines of the file:
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@@
 	)
 	(no_connect
+		(at 234.95 46.99)
+	)
+	(no_connect
 		(at 52.07 279.4)
 	)
@@
 	)
 	(no_connect
+		(at 234.95 49.53)
+	)
+	(no_connect
 		(at 63.5 49.53)
 	)
@@
 	)
 	(no_connect
+		(at 234.95 44.45)
+	)
+	(no_connect
 		(at 116.84 279.4)
 	)
@@
 	(wire
 		(pts
-			(xy 234.95 49.53) (xy 248.92 49.53)
-		)
-		(stroke
-			(width 0)
-			(type default)
-		)
-	)
-	(wire
-		(pts
 			(xy 306.07 33.02) (xy 306.07 31.75)
 		)
@@
 	(wire
 		(pts
-			(xy 234.95 46.99) (xy 248.92 46.99)
-		)
-		(stroke
-			(width 0)
-			(type default)
-		)
-	)
-	(wire
-		(pts
 			(xy 198.12 25.4) (xy 215.9 25.4)
 		)
@@
 	(wire
 		(pts
-			(xy 234.95 44.45) (xy 248.92 44.45)
-		)
-		(stroke
-			(width 0)
-			(type default)
-		)
-	)
-	(wire
-		(pts
 			(xy 93.98 41.91) (xy 113.03 41.91)
 		)
@@
 		)
 	)
-	(label "IR+_GND"
-		(at 248.92 46.99 180)
-		(fields_autoplaced yes)
-		(effects
-			(font
-				(size 1.27 1.27)
-			)
-			(justify right bottom)
-		)
-	)
 	(label "LATCH_RL"
 		(at 189.23 266.7 180)
@@
 		)
 	)
-	(label "Fan_PWM"
-		(at 248.92 44.45 180)
-		(fields_autoplaced yes)
-		(effects
-			(font
-				(size 1.27 1.27)
-			)
-			(justify right bottom)
-		)
-	)
 	(label "TS-"
 		(at 316.23 259.08 90)
@@
 		(fields_autoplaced yes)
 		(effects
-			(font
-				(size 1.27 1.27)
-			)
-			(justify right bottom)
-		)
-	)
-	(label "Charge_State"
-		(at 248.92 49.53 180)
-		(fields_autoplaced yes)
-		(effects

Commit message: Fault logic fixes
Parts:
- removed unit 2 of U16
- R26: value 7.2k -> 10k
- R27: value 10k -> 7.2k
Connections:
- net +12V: now also D2.1 (K), D4.1 (K), K1.8 (+), K3.8 (+)
- net +5V: no longer D2.1 (K), D4.1 (K), K1.8 (+), K3.8 (+)
- net at CR2.4 (G): now also U7.4
Changed lines of the file:
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@@
 	(wire
 		(pts
-			(xy 138.43 234.95) (xy 157.48 234.95)
-		)
-		(stroke
-			(width 0)
-			(type default)
-		)
-	)
-	(wire
-		(pts
 			(xy 236.22 303.53) (xy 236.22 318.77)
 		)
@@
 	(wire
 		(pts
-			(xy 111.76 234.95) (xy 123.19 234.95)
+			(xy 111.76 234.95) (xy 157.48 234.95)
 		)
 		(stroke
@@
 			)
 		)
-		(property "Value" "10k"
+		(property "Value" "7.2k"
 			(at 251.968 318.77 90)
 			(effects
@@
 			)
 		)
-		(property "Value" "7.2k"
+		(property "Value" "10k"
 			(at 244.602 318.77 90)
 			(effects
@@
 			)
 		)
-		(property "Value" "+5V"
+		(property "Value" "+12V"
 			(at 105.41 255.27 0)
 			(effects
@@
 	)
 	(symbol
-		(lib_id "4xxx:4069")
-		(at 130.81 234.95 180)
-		(unit 2)
-		(exclude_from_sim no)
-		(in_bom yes)
-		(on_board yes)
-		(dnp no)
-		(fields_autoplaced yes)
-		(property "Reference" "U16"
-			(at 130.81 243.84 0)
-			(effects
-				(font
-					(size 1.27 1.27)
-				)
-			)
-		)
-		(property "Value" "4069"
-			(at 130.81 241.3 0)
-			(effects
-				(font
-					(size 1.27 1.27)
-				)
-			)
-		)
-		(property "Footprint" "Package_SO:SOIC-14_3.9x8.7mm_P1.27mm"
-			(at 130.81 234.95 0)
-			(effects
-				(font
-					(size 1.27 1.27)
-				)
-				(hide yes)
-			)
-		)
-		(property "Datasheet" "http://www.intersil.com/content/dam/Intersil/documents/cd40/cd4069ubms.pdf"
-			(at 130.81 234.95 0)
-			(effects
-				(font
-					(size 1.27 1.27)
-				)
-				(hide yes)
-			)
-		)
-		(property "Description" "Hex inverter"
-			(at 130.81 234.95 0)
-			(effects
-				(font
-					(size 1.27 1.27)
-				)
-				(hide yes)
-			)
-		)
-		(pin "9"
-		)
-		(pin "7"
-		)
-		(pin "12"
-		)
-		(pin "4"
-		)
-		(pin "2"
-		)
-		(pin "8"
-		)
-		(pin "5"
-		)
-		(pin "10"
-		)
-		(pin "14"
-		)
-		(pin "1"
-		)
-		(pin "6"
-		)
-		(pin "11"
-		)
-		(pin "3"
-		)
-		(pin "13"
-		)
-		(instances
-			(project ""
-				(path "/ac087927-92f1-4fcc-b2b7-d2d4010e5b25"
-					(reference "U16")
-					(unit 2)
-				)
-			)
-		)
-	)
-	(symbol
 		(lib_name "+5V_4")
 		(lib_id "power:+5V")
@@
 			)
 		)
-		(property "Value" "+5V"
+		(property "Value" "+12V"
 			(at 40.64 256.54 0)
 			(effects

Commit message: Fixed dk1a1b relays and CAN transceiver
Connections:
- net Fan_PWM: now also U2.CN3_12 (PA8); no longer U2.CN4_11 (PA1)
Changed lines of the file:
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@@
 	)
 	(no_connect
+		(at 93.98 57.15)
+	)
+	(no_connect
 		(at 116.84 279.4)
 	)
@@
 	)
 	(no_connect
-		(at 63.5 59.69)
-	)
-	(no_connect
 		(at 234.95 59.69)
 	)
@@
 	(wire
 		(pts
-			(xy 93.98 57.15) (xy 113.03 57.15)
-		)
-		(stroke
-			(width 0)
-			(type default)
-		)
-	)
-	(wire
-		(pts
 			(xy 252.73 111.76) (xy 242.57 111.76)
 		)
@@
 	(wire
 		(pts
+			(xy 45.72 59.69) (xy 63.5 59.69)
+		)
+		(stroke
+			(width 0)
+			(type default)
+		)
+	)
+	(wire
+		(pts
 			(xy 195.58 288.29) (xy 195.58 312.42)
 		)
@@
 		)
 	)
+	(label "Fan_PWM"
+		(at 45.72 59.69 0)
+		(fields_autoplaced yes)
+		(effects
+			(font
+				(size 1.27 1.27)
+			)
+			(justify left bottom)
+		)
+	)
 	(label "Current_Vref"
 		(at 81.28 97.79 270)
@@
 		)
 	)
-	(label "Fan_PWM"
-		(at 113.03 57.15 180)
-		(fields_autoplaced yes)
-		(effects
-			(font
-				(size 1.27 1.27)
-			)
-			(justify right bottom)
-		)
-	)

Commit message: Precharge logic fixed
Parts:
- removed unit 3 of U16
- added U3: 4069, Package_SO:SOIC-14_3.9x8.7mm_P1.27mm, symbol 4xxx:4069
Connections:
- net Precharge_Control: now also Q1.4 (G), U3.5; no longer Q2.4 (G)
- new net: Q2.4 (G), U3.6
Other:
- moved on the sheet: J7, Q1

Commit message: Linear Regulator Fix
Parts:
- removed U15: ZXTR2005ZQ-13, FS_3_Global_Footprint_Library:SOT-89_4P5X2P45_DIO, symbol Regulator_Linear:LM7809_TO220
- added U15: ZXTR2005ZQ-13, FS_3_Global_Footprint_Library:SOT-89_4P5X2P45_DIO, symbol FS_3_Global_Symbol_Library:ZXTR2005ZQ-13
Connections:
- net HVIL: now also U15.3 (Vout)
- net TS-: now also U15.1 (GND)
- net at C23.1, D8.2 (A): now also U15.2 (Vin)
Changed lines of the file:
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@@
 	)
 	(junction
-		(at 297.18 48.26)
+		(at 330.2 242.57)
 		(diameter 0)
 		(color 0 0 0 0)
 	)
 	(junction
-		(at 227.33 135.89)
+		(at 297.18 48.26)
 		(diameter 0)
 		(color 0 0 0 0)
 	)
 	(junction
-		(at 330.2 242.57)
+		(at 227.33 135.89)
 		(diameter 0)
 		(color 0 0 0 0)
@@
 	(wire
 		(pts
-			(xy 280.67 166.37) (xy 280.67 165.1)
+			(xy 325.12 242.57) (xy 330.2 242.57)
 		)
 		(stroke
@@
 	(wire
 		(pts
-			(xy 280.67 166.37) (xy 281.94 166.37)
-		)
-		(stroke
-			(width 0)
-			(type default)
-		)
-	)
-	(wire
-		(pts
 			(xy 415.29 26.67) (xy 417.83 26.67)
 		)
@@
 	(wire
 		(pts
-			(xy 280.67 165.1) (xy 260.35 165.1)
+			(xy 260.35 166.37) (xy 281.94 166.37)
 		)
 		(stroke
@@
 	(wire
 		(pts
-			(xy 316.23 250.19) (xy 316.23 254)
+			(xy 316.23 248.92) (xy 316.23 254)
 		)
 		(stroke
@@
 	(wire
 		(pts
-			(xy 323.85 242.57) (xy 330.2 242.57)
-		)
-		(stroke
-			(width 0)
-			(type default)
-		)
-	)
-	(wire
-		(pts
 			(xy 118.11 121.92) (xy 113.03 121.92)
 		)
@@
 	(wire
 		(pts
-			(xy 302.26 242.57) (xy 308.61 242.57)
+			(xy 302.26 242.57) (xy 307.34 242.57)
 		)
 		(stroke
@@
 	)
 	(label "Precharge_Control"
-		(at 260.35 165.1 0)
+		(at 260.35 166.37 0)
 		(fields_autoplaced yes)
 		(effects
@@
 	)
 	(symbol
+		(lib_id "FS_3_Global_Symbol_Library:ZXTR2005ZQ-13")
+		(at 316.23 242.57 0)
+		(unit 1)
+		(exclude_from_sim no)
+		(in_bom yes)
+		(on_board yes)
+		(dnp no)
+		(fields_autoplaced yes)
+		(property "Reference" "U15"
+			(at 316.23 234.95 0)
+			(effects
+				(font
+					(size 1.524 1.524)
+				)
+			)
+		)
+		(property "Value" "ZXTR2005ZQ-13"
+			(at 316.23 237.49 0)
+			(effects
+				(font
+					(size 1.524 1.524)
+				)
+			)
+		)
+		(property "Footprint" "FS_3_Global_Footprint_Library:SOT-89_4P5X2P45_DIO"
+			(at 294.132 220.98 0)
+			(effects
+				(font
+					(size 1.27 1.27)
+					(italic yes)
+				)
+				(hide yes)
+			)
+		)
+		(property "Datasheet" "https://www.diodes.com/assets/Datasheets/ZXTR2005ZQ.pdf"
+			(at 297.942 224.028 0)
+			(effects
+				(font
+					(size 1.27 1.27)
+					(italic yes)
+				)
+				(hide yes)
+			)
+		)
+		(property "Description" "High Voltage 5V Linear Regulator"
+			(at 284.734 227.33 0)
+			(effects
+				(font
+					(size 1.27 1.27)
+				)
+				(hide yes)
+			)
+		)
+		(pin "1"
+		)
+		(pin "2"
+		)
+		(pin "3"
+		)
+		(instances
+			(project ""
+				(path "/ac087927-92f1-4fcc-b2b7-d2d4010e5b25"
+					(reference "U15")
+					(unit 1)
+				)
+			)
+		)
+	)
+	(symbol
 		(lib_id "Timer:LM555xN")
 		(at 210.82 307.34 0)
@@
 					(unit 1)
 				)
-			)
-		)
-	)
-	(symbol
-		(lib_id "Regulator_Linear:LM7809_TO220")
-		(at 316.23 242.57 0)
-		(unit 1)
-		(exclude_from_sim no)
-		(in_bom yes)
-		(on_board yes)
-		(dnp no)
-		(fields_autoplaced yes)
-		(property "Reference" "U15"
-			(at 316.23 236.22 0)
-			(effects
-				(font
-					(size 1.27 1.27)
-				)
-			)
-		)
-		(property "Value" "ZXTR2005ZQ-13"
-			(at 316.23 238.76 0)
-			(effects
-				(font
-					(size 1.27 1.27)
-				)
-			)
-		)
-		(property "Footprint" "FS_3_Global_Footprint_Library:SOT-89_4P5X2P45_DIO"
-			(at 316.23 236.855 0)
-			(effects
-				(font
-					(size 1.27 1.27)
-					(italic yes)
-				)
-				(hide yes)
-			)
-		)
-		(property "Datasheet" "https://www.diodes.com/assets/Datasheets/ZXTR2005ZQ.pdf"
-			(at 316.23 243.84 0)
-			(effects
-				(font
-					(size 1.27 1.27)
-				)
-				(hide yes)
-			)
-		)
-		(property "Description" ""
-			(at 316.23 242.57 0)
-			(effects
-				(font
-					(size 1.27 1.27)
-				)
-				(hide yes)
-			)
-		)
-		(pin "1"
-		)
-		(pin "2"
-		)
-		(pin "3"
-		)
-		(instances
-			(project "Accumulator_Board"
-				(path "/ac087927-92f1-4fcc-b2b7-d2d4010e5b25"
-					(reference "U15")
-					(unit 1)
-				)

Commit message: Main Push
Changed lines of the file:
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@@
 	(wire
 		(pts
+			(xy 280.67 166.37) (xy 280.67 165.1)
+		)
+		(stroke
+			(width 0)
+			(type default)
+		)
+	)
+	(wire
+		(pts
 			(xy 191.77 289.56) (xy 210.82 289.56)
 		)
@@
 	(wire
 		(pts
+			(xy 280.67 166.37) (xy 281.94 166.37)
+		)
+		(stroke
+			(width 0)
+			(type default)
+		)
+	)
+	(wire
+		(pts
 			(xy 415.29 26.67) (xy 417.83 26.67)
 		)
@@
 	(wire
 		(pts
-			(xy 260.35 166.37) (xy 281.94 166.37)
+			(xy 280.67 165.1) (xy 260.35 165.1)
 		)
 		(stroke
@@
 	)
 	(label "Precharge_Control"
-		(at 260.35 166.37 0)
+		(at 260.35 165.1 0)
 		(fields_autoplaced yes)
 		(effects
@@
 		(on_board yes)
 		(dnp no)
-		(fields_autoplaced yes)
 		(property "Reference" "CR4"
 			(at 392.43 30.48 0)

Commit message: Added temp sensor, cleaned up tracks and vias
Parts:
- added J3: Temp Sensor, Connector_Molex:Molex_Nano-Fit_105309-xx03_1x03_P2.50mm_Vertical, symbol Connector:Conn_01x03_Pin
- added R24: 4.7k, Resistor_SMD:R_0805_2012Metric_Pad1.20x1.40mm_HandSolder, symbol Device:R
Connections:
- net +3.3V: now also R24.1
- net +5V: now also J3.3 (Pin_3)
- net GND: now also J3.1 (Pin_1)
- net ACC_Temp_Sense: now reaches U2.CN3_8 (PB6)
- net ACC_Temp_Sense: now also J3.2 (Pin_2), R24.2
- no-connect marks 25 -> 24
Other:
- note added: "For DS18B20 one wire temp sensors For acc air temperature sensing"

Commit message: TSSI and DASH Light logic adjustment
Parts:
- added CR6: STS6NF20V, Package_SO:SOIC-8_3.9x4.9mm_P1.27mm, symbol FS_2_Global_Symbol_Library:STS6NF20V
- added R25: 1k, Resistor_SMD:R_0805_2012Metric_Pad1.20x1.40mm_HandSolder, symbol Device:R
- added R34: 10k, Resistor_SMD:R_0805_2012Metric_Pad1.20x1.40mm_HandSolder, symbol Device:R
- added unit 2 of U16
- R22: value 100k -> 1k
- R29, R33: value 100k -> 10k
- renumbered U3 to U16
Connections:
- net +12V: now also D5.1 (K), K4.5, R33.1, R34.1; no longer R22.1
- net +5V: no longer R29.1, R33.1
- net BMS_FAULT_3.3V: now also R25.1; no longer U7.2
- net BMS_RL: no longer R28.2
- net GND: now also CR6.1 (S), CR6.2 (S), CR6.3 (S), R25.2
- net IMD_DELAY: now also J11.11 (Pin_11), U16.3
- net IMD_RL: no longer R32.2
- net BMS_Dash_LED_Control: now reaches J11.10 (Pin_10)
- net BMS_Dash_LED_Control: now also CR6.5 (D), CR6.6 (D), CR6.7 (D), CR6.8 (D), R34.2
- net BMS_Fault_Inverted: now reaches U2.CN4_6 (PA7)
- net BMS_Fault_Inverted: now also R22.2, R28.2
- net BMS_LED_Control renamed BMS_FAULT_5V
- net BMS_FAULT_5V: now also U7.2
- net IMD_LED_Control renamed IMD_Dash_LED_Control
- net Shutdown_ACC_IL_TP: no longer names the net of J6.2, K4.4
- new net: CR6.4 (G), R22.1
- new net: R32.2, U16.4
- new net 5V: R29.1
- no-connect marks 24 -> 21
Other:
- note added: "IMD_Delay and BMS Fault_5V to be used to drive TSSI logic"
- note added: "When BMS Fault 3.3V is low BMS_Fault_5V is low"
- moved on the sheet: C1, C2, C23, C24, C9, CR1, CR4, CR5, D5, D8, J10, J4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
