File: Live_Telemetry_Board/Live_Telemetry_Board.kicad_pcb (KiCad board)
At the start: 2 copper layers, 108.8 x 73.1 mm, 18 parts, among them J1 Molar Nanofit Connectors, U1 ISO1050DUB, U2 NUCLEO-F446RE, U3 XBP9B-DPST-001, U4 LM7809_TO220, U5 LM7805_TO220, U6 LF33_TO220

Commit message: update
Other:
- board text added: "Live Telemetry Board FS-3 Design by Nathan Pham"
Changed lines of the file:
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@@
 		(layer "Edge.Cuts")
+	)
+	(gr_text "Live Telemetry Board\nFS-3\nDesign by Nathan Pham\n"
+		(at 52.55 63.7 0)
+		(layer "F.SilkS")
+		(effects
+			(font
+				(size 1 1)
+				(thickness 0.1)
+			)
+			(justify left bottom)
+		)
 	)
 	(segment

Commit message: lol
Parts:
- U4: moved to F.Cu
- moved U4 1.75 mm to (55.1, 94.8)
Routing:
- net +12V: track 142.7 -> 144.5 mm
- net GND: track 42.2 -> 44.0 mm
- net +9V: track 14.1 -> 15.8 mm

Commit message: mounting holes
Parts:
- added REF**: MountingHole_3.5mm, MountingHole:MountingHole_3.5mm, F.Cu at (55.8, 63.0)
- added REF**: MountingHole_3.5mm, MountingHole:MountingHole_3.5mm, F.Cu at (55.5, 126.3)
- added REF**: MountingHole_3.5mm, MountingHole:MountingHole_3.5mm, F.Cu at (153.9, 63.1)
- added REF**: MountingHole_3.5mm, MountingHole:MountingHole_3.5mm, F.Cu at (154.8, 126.6)
Other:
- board text added: "Live Telemetry Board FS-3 Design by Nathan Pham Version 1"
- board text removed: "Live Telemetry Board FS-3 Design by Nathan Pham"
