File: Live_Telemetry_Receiver_Board/Live_Telemetry_Receiver_Board.kicad_pcb (KiCad board)
At the start: 2 copper layers, 48.9 x 56.1 mm, 4 parts, among them CN1 NUCLEO-L432KC, U1 XBP9B-DPST-001

Commit message: mounting holes
Parts:
- added REF**: MountingHole_3.5mm, MountingHole:MountingHole_3.5mm, F.Cu at (160.1, 94.2)
- added REF**: MountingHole_3.5mm, MountingHole:MountingHole_3.5mm, F.Cu at (111.2, 47.8)
- added REF**: MountingHole_3.5mm, MountingHole:MountingHole_3.5mm, F.Cu at (111.2, 94.2)
- added REF**: MountingHole_3.5mm, MountingHole:MountingHole_3.5mm, F.Cu at (160.1, 47.8)
Routing:
- net /RADIO_RESET: track 0.00 -> 4.89 mm, vias 0 -> 1
Other:
- board size 48.9 x 56.1 mm -> 58.5 x 56.1 mm
