File: Telemetry peripheral boards/F3 peripheral boards.kicad_sch (KiCad schematic)
At the start: 37 parts, among them J1 ATS668LSM, J2 1053131108, J3 Potentiometer, J4 Strain Gauge, U1 LM2907M/NOPB, U2 INA125U, U3 MCP2515-I/SO, U4 ISO1050DUB, U5 ATTINY1616-SNR

Commit message: Peripheral
Parts:
- U5: value ATTINY1616-SNR -> ATTINY1616-MNR; footprint Package_SO:SOIC-20W_7.5x12.8mm_P1.27mm -> New Library:VQFN20_3X3_MCH
Other:
- moved on the sheet: U5
Changed lines of the file:
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@@
 	(symbol
 		(lib_id "New_Library:ATTINY1616-MNR")
-		(at 189.23 80.01 0)
+		(at 184.15 88.9 0)
 		(unit 1)
 		(exclude_from_sim no)
@@
 		(fields_autoplaced yes)
 		(property "Reference" "U5"
-			(at 227.33 69.85 0)
+			(at 222.25 78.74 0)
 			(effects
 				(font
@@
 			)
 		)
-		(property "Value" "ATTINY1616-SNR"
-			(at 227.33 72.39 0)
+		(property "Value" "ATTINY1616-MNR"
+			(at 222.25 81.28 0)
 			(effects
 				(font
@@
 			)
 		)
-		(property "Footprint" "Package_SO:SOIC-20W_7.5x12.8mm_P1.27mm"
-			(at 188.976 69.85 0)
+		(property "Footprint" "New Library:VQFN20_3X3_MCH"
+			(at 183.896 78.74 0)
 			(effects
 				(font
@@
 		)
 		(property "Datasheet" "ATTINY1616-MNR"
-			(at 193.548 61.468 0)
+			(at 188.468 70.358 0)
 			(effects
 				(font
@@
 		)
 		(property "Description" ""
-			(at 189.23 80.01 0)
+			(at 184.15 88.9 0)
 			(effects
 				(font

Commit message: Updated peripheral Board
Parts:
- removed +3V3, TP6, TP7, TP8: TestPoint, TestPoint:TestPoint_Loop_D3.80mm_Drill2.0mm, symbol Connector:TestPoint
- removed J2: 1053131108, New Library:CON_1053131108, symbol New_Library:1053131108
- removed TP5: ~, TestPoint:TestPoint_Loop_D3.80mm_Drill2.0mm, symbol Connector:TestPoint
- added C10: 100nF, symbol Device:C
- added C11: 330nf, Capacitor_SMD:C_0805_2012Metric_Pad1.18x1.45mm_HandSolder, symbol Device:C
- added C12: 100nf, Capacitor_SMD:C_0805_2012Metric_Pad1.18x1.45mm_HandSolder, symbol Device:C
- added C13: 100nF, Capacitor_SMD:C_0805_2012Metric_Pad1.18x1.45mm_HandSolder, symbol Device:C
- added C14: 10uF, Capacitor_SMD:C_0805_2012Metric_Pad1.18x1.45mm_HandSolder, symbol Device:C
- added H1, H2: Conn_01x10_MountingPin, symbol Connector_Generic_MountingPin:Conn_01x10_MountingPin
- added J2: Conn_01x04_MountingPin, symbol Connector_Generic_MountingPin:Conn_01x04_MountingPin
- added R12: 430, symbol Device:R_US
- added U6: LM7805_TO220, Package_TO_SOT_THT:TO-220-3_Vertical, symbol Regulator_Linear:LM7805_TO220
- added U7: LD1117V33C, Package_TO_SOT_THT:TO-220-3_Vertical, symbol Regulator_Linear:LM7805_TO220
Connections:
- net SPI3_MISO is gone; now on net PA2: U3.15 (SO)
- net SPI3_MOSI is gone; now on net PA1: U3.14 (SI)
- net SPI3_SCLK is gone; now on net PA3/SCK: U3.13 (SCK)
- net SPI3_SSEL is gone; now on net PC3: U3.16 (*CS)
- net +3V3: now also C14.1, U7.3 (VO)
- net +5V: now also U5.4 (VDD), C10.2, C12.1, H1.2 (Pin_2), U6.3 (VO)
- net GND: now also U5.21 (EPAD), U5.3 (GND), C10.1, C11.2, C12.2, C13.2, C14.2, H1.3 (Pin_3), J2.4 (Pin_4), U6.2 (GND), U7.2 (GND)
- net PA2: now reaches U5.1 (PA2)
- net PA2: now also H1.5 (Pin_5)
- net PB4: now reaches U5.10 (PB4)
- net PB4: now also H2.6 (Pin_6)
- net at U5.11 (PB3/TOSC1): now also H2.5 (Pin_5)
- net at U5.12 (PB2/): now also H2.4 (Pin_4)
- net PB1: now reaches U5.13 (PB1)
- net PB1: now also H2.3 (Pin_3)
- net PB0: now reaches U5.14 (PB0)
- net PB0: now also H2.2 (Pin_2)
- net PC0: now reaches U5.15 (PC0)
- net PC0: now also H2.1 (Pin_1)
- net PC1: now reaches U5.16 (PC1)
- net PC1: now also H1.8 (Pin_8)
- net PC2: now reaches U5.17 (PC2)
- net PC2: now also H1.9 (Pin_9)
- net PC3: now reaches U5.18 (PC3)
- net PC3: now also H1.10 (Pin_10)
- net at U5.19 (PA0/*RESET/UP): now also R12.1
- net PA3/SCK: now reaches U5.2 (EXTCLK_/PA3)
- net PA3/SCK: now also H1.4 (Pin_4)
- net PA1: now reaches U5.20 (PA1)
- net PA1: now also H1.6 (Pin_6)
- net PA4/SS: now reaches U5.5 (PA4)
- net PA4/SS: now also H1.1 (Pin_1)
- net PA5: now reaches U5.6 (PA5)
- net PA5: now also H2.10 (Pin_10)
- net PA6: now reaches U5.7 (PA6)
- net PA6: now also H2.9 (Pin_9)
- net PA7: now reaches U5.8 (PA7)
- net PA7: now also H2.8 (Pin_8)
- net PB5: now reaches U5.9 (PB5)
- net PB5: now also H2.7 (Pin_7)
- net CANL: now reaches U4.6 (CANL)
- net CANL: now also J2.2 (Pin_2)
- net CANH: now reaches U4.7 (CANH)
- net CANH: now also J2.3 (Pin_3)
- new net +12V: C11.1, C13.1, J2.1 (Pin_1), U6.1 (VI), U7.1 (VI)
- new net UP: H1.7 (Pin_7), R12.2
Other:
- moved on the sheet: C7, C8, C9, U3, U4

Commit message: Updates
Parts:
- removed TP1: ~, TestPoint:TestPoint_Loop_D3.80mm_Drill2.0mm, symbol Connector:TestPoint
- removed TP9: VrefBG, TestPoint:TestPoint_Loop_D3.80mm_Drill2.0mm, symbol Connector:TestPoint
- removed TP@1: Offset, TestPoint:TestPoint_Loop_D3.80mm_Drill2.0mm, symbol Connector:TestPoint
- C10, C8, C9: footprint (none) -> Capacitor_SMD:C_0805_2012Metric_Pad1.18x1.45mm_HandSolder
- H2: footprint (none) -> Connector_PinHeader_1.00mm:PinHeader_1x10_P1.00mm_Vertical
- J2: footprint (none) -> Connector_PinHeader_1.00mm:PinHeader_1x04_P1.00mm_Vertical
- R12: footprint (none) -> Resistor_SMD:R_0805_2012Metric_Pad1.20x1.40mm_HandSolder
Connections:
- net Wheel Speed: now also C2.1, R4.2
Other:
- moved on the sheet: C7, U3

Commit message: updated can controller
Parts:
- added C15: 100 nF, Capacitor_SMD:C_0805_2012Metric_Pad1.18x1.45mm_HandSolder, symbol Device:C
- added D1: D, Diode_SMD:D_0805_2012Metric, symbol Device:D
- added R13: 10K, Resistor_SMD:R_0805_2012Metric_Pad1.20x1.40mm_HandSolder, symbol Device:R_US
- added R14: 100 Ω, Resistor_SMD:R_0805_2012Metric_Pad1.20x1.40mm_HandSolder, symbol Device:R_US
Connections:
- net GND: now also C15.2
- net at U3.17 (*RESET): now also R13.1
- new net: C15.1, D1.2 (A), R13.2, R14.2
- new net +3.3V: D1.1 (K), R14.1
Other:
- moved on the sheet: C7, U3

Commit message: PCB for peripheral boards
Parts:
- added C16, C17: 27 pF, Capacitor_SMD:C_0805_2012Metric_Pad1.18x1.45mm_HandSolder, symbol Device:C
- added Y1: Crystal, Crystal:Crystal_SMD_5032-2Pin_5.0x3.2mm_HandSoldering, symbol Device:Crystal
- H1: footprint (none) -> Connector_PinHeader_1.00mm:PinHeader_1x10_P1.00mm_Vertical
- J1: footprint (none) -> Connector_PinHeader_2.00mm:PinHeader_1x03_P2.00mm_Vertical
Connections:
- net GND: now also C16.2, C17.2
- net PA1: now also H2.10 (Pin_10); no longer H1.6 (Pin_6)
- net PA2: now also H1.4 (Pin_4); no longer H1.5 (Pin_5)
- net PA3/SCK: now also H1.1 (Pin_1); no longer H1.4 (Pin_4)
- net PA5: now also H1.6 (Pin_6); no longer H2.10 (Pin_10)
- net PA6: now also H1.7 (Pin_7); no longer H2.9 (Pin_9)
- net PA7: now also H1.8 (Pin_8); no longer H2.8 (Pin_8)
- net PB0: now also H2.4 (Pin_4); no longer H2.2 (Pin_2)
- net PB4: now also H1.10 (Pin_10); no longer H2.6 (Pin_6)
- net PB5: now also H1.9 (Pin_9); no longer H2.7 (Pin_7)
- net PC0: now also H2.5 (Pin_5); no longer H2.1 (Pin_1)
- net PC1: now also H2.6 (Pin_6); no longer H1.8 (Pin_8)
- net PC2: now also H2.7 (Pin_7); no longer H1.9 (Pin_9)
- net PC3: now also H2.8 (Pin_8); no longer H1.10 (Pin_10)
- net UP: now also H2.9 (Pin_9); no longer H1.7 (Pin_7)
- net at U5.11 (PB3/TOSC1): now also H2.1 (Pin_1); no longer H2.5 (Pin_5)
- net at U5.12 (PB2/): now also H2.2 (Pin_2); no longer H2.4 (Pin_4)
- net at U3.7 (OSC2): now also C16.1, Y1.1
- net at U3.8 (OSC1): now also C17.1, Y1.2
- net PA4/SS renamed PA4
- net PA4: now also H1.5 (Pin_5); no longer H1.1 (Pin_1)

Commit message: Peripheral boards
Changed lines of the file:
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@@
+	)
+	(junction
+		(at 60.96 97.79)
+		(diameter 0)
+		(color 0 0 0 0)
 	)
 	(junction
@@
 	(wire
 		(pts
-			(xy 60.96 95.25) (xy 60.96 100.33)
+			(xy 60.96 95.25) (xy 60.96 97.79)
 		)
 		(stroke
@@
 	(wire
 		(pts
+			(xy 60.96 97.79) (xy 53.34 97.79)
+		)
+		(stroke
+			(width 0)
+			(type default)
+		)
+	)
+	(wire
+		(pts
 			(xy 158.75 132.08) (xy 163.83 132.08)
 		)
@@
 	(wire
 		(pts
+			(xy 73.66 97.79) (xy 80.01 97.79)
+		)
+		(stroke
+			(width 0)
+			(type default)
+		)
+	)
+	(wire
+		(pts
 			(xy 172.72 81.28) (xy 166.37 81.28)
 		)
@@
 	(wire
 		(pts
+			(xy 60.96 97.79) (xy 60.96 100.33)
+		)
+		(stroke
+			(width 0)
+			(type default)
+		)
+	)
+	(wire
+		(pts
 			(xy 30.48 38.1) (xy 30.48 40.64)
 		)
@@
 	(wire
 		(pts
-			(xy 66.04 97.79) (xy 53.34 97.79)
-		)
-		(stroke
-			(width 0)
-			(type default)
-		)
-	)
-	(wire
-		(pts
 			(xy 158.75 129.54) (xy 161.29 129.54)
 		)
@@
 	(wire
 		(pts
+			(xy 66.04 97.79) (xy 60.96 97.79)
+		)
+		(stroke
+			(width 0)
+			(type default)
+		)
+	)
+	(wire
+		(pts
 			(xy 176.53 93.98) (xy 176.53 88.9)
 		)
@@
 		(pts
 			(xy 80.01 107.95) (xy 80.01 110.49)
-		)
-		(stroke
-			(width 0)
-			(type default)
-		)
-	)
-	(wire
-		(pts
-			(xy 73.66 97.79) (xy 80.01 97.79)
 		)
 		(stroke
@@
 	)
 	(label "Vin-"
-		(at 60.96 97.79 0)
+		(at 66.04 97.79 180)
 		(fields_autoplaced yes)
 		(effects
@@
 				(size 1.27 1.27)
 			)
-			(justify left bottom)
+			(justify right bottom)
 		)
 	)
@@
 	)
 	(label "Vin+"
-		(at 74.93 97.79 0)
+		(at 73.66 97.79 180)
 		(fields_autoplaced yes)
 		(effects
@@
 				(size 1.27 1.27)
 			)
-			(justify left bottom)
-		)
-	)
+			(justify right bottom)
+		)
+	)

Commit message: Update With Tire Temp Sensor
Update With Tire Temp Sensor
Parts:
- added J5: Tire temp, Connector_PinHeader_1.00mm:PinHeader_1x04_P1.00mm_Vertical, symbol Connector_Generic_MountingPin:Conn_01x04_MountingPin
Connections:
- net Shock position is gone; now on net PA6: J3.2
- net Strain is gone; now on net PA7: U2.10 (VO), U2.11 (SENSE)
- net Wheel Speed is gone; now on net PA4: C2.1, R4.2
- net +5V: now also J5.1 (Pin_1)
- net CANH: now also J5.3 (Pin_3)
- net CANL: now also J5.2 (Pin_2)
- net GND: now also J5.4 (Pin_4)

Commit message: Updated Peripheral Board(Compact)
Parts:
- J5: value Tire temp -> Tire temp Sensor
Connections:
- net +3.3V is gone; now on net +3V3: D1.1 (K), R14.1
- net VIN+ is gone; now on net Vin+: U2.6 (VIN+)
- net VIN- is gone; now on net Vin-: U2.7 (VIN-)
Changed lines of the file:
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@@
 			(width 0)
 			(type default)
+			(color 0 132 0 1)
 		)
 	)
@@
 		)
 	)
-	(label "VIN+"
+	(label "Vin+"
 		(at 27.94 134.62 0)
 		(fields_autoplaced yes)
@@
 		)
 	)
-	(label "VIN-"
+	(label "Vin-"
 		(at 27.94 132.08 0)
 		(fields_autoplaced yes)
@@
 			)
 		)
-		(property "Value" "+3.3V"
+		(property "Value" "+3V3"
 			(at 176.53 146.05 0)
 			(effects
@@
 			)
 		)
-		(property "Value" "Tire temp"
+		(property "Value" "Tire temp Sensor"
 			(at 212.09 66.3955 0)
 			(effects
