File: Telemetry peripheral boards/F3 peripheral boards.kicad_pcb (KiCad board)
At the start: 2 copper layers, 46 parts, among them J1 ATS668LSM, J2 Conn_01x04_MountingPin, J3 Potentiometer, J4 Strain Gauge, U1 LM2907M/NOPB, U2 INA125U, U3 MCP2515-I/SO, U4 ISO1050DUB, U5 ATTINY1616-MNR, U6 LM7805_TO220, U7 LD1117V33C, Y1 Crystal

Commit message: Logo added
Parts:
- added G***: LOGO, 1FS_2_Global_Footprint_Library:FS_Logo_4LinesTall, F.Cu at (88.0, 45.5)
Other:
- board text added: "Designed by Ruandy Salazar"
- board text added: "FS-3 Telemetry Peripheral Board"
- board text added: "Formula Slug"
- board text added: "V 1.0"

Commit message: Peripheral boards
Routing:
- net GND: track 396.4 -> 425.8 mm, vias 8 -> 12
- net +5V: track 382.4 -> 388.0 mm
Changed lines of the file:
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@@
+	)
+	(segment
+		(start 150.0776 65.4224)
+		(end 150.0776 67.5776)
+		(width 0.2)
+		(layer "F.Cu")
+		(net 2)
 	)
 	(segment
@@
 	)
 	(segment
+		(start 74.5 85)
+		(end 75.5 85)
+		(width 0.2)
+		(layer "F.Cu")
+		(net 2)
+	)
+	(segment
 		(start 58.9625 85.5)
 		(end 58.9625 88.4625)
@@
 	)
 	(segment
+		(start 71.5772 91)
+		(end 75.5 91)
+		(width 0.2)
+		(layer "F.Cu")
+		(net 2)
+	)
+	(segment
 		(start 65.6125 56.2983)
 		(end 65.65 56.3358)
@@
 	)
 	(segment
+		(start 151.1776 66)
+		(end 154.1 66)
+		(width 0.2)
+		(layer "F.Cu")
+		(net 2)
+	)
+	(segment
+		(start 75.5 87.5)
+		(end 75.5 91)
+		(width 0.2)
+		(layer "F.Cu")
+		(net 2)
+	)
+	(segment
 		(start 163.5 58.5)
 		(end 154.5 58.5)
@@
 	)
 	(segment
+		(start 60 83)
+		(end 72.5 83)
+		(width 0.2)
+		(layer "F.Cu")
+		(net 2)
+	)
+	(segment
 		(start 87.425 68.925)
 		(end 91 68.925)
@@
 	)
 	(segment
-		(start 154.5375 67.5)
-		(end 150.9685 63.931)
-		(width 0.2)
-		(layer "F.Cu")
-		(net 2)
-	)
-	(segment
 		(start 82.3358 63.8358)
 		(end 82.5 64)
@@
 	)
 	(segment
+		(start 58.9625 85.5)
+		(end 58.9625 84.0375)
+		(width 0.2)
+		(layer "F.Cu")
+		(net 2)
+	)
+	(segment
 		(start 82.5 75.5)
 		(end 82.5 80.5)
@@
 	)
 	(segment
+		(start 154.1 66)
+		(end 154.5 65.6)
+		(width 0.2)
+		(layer "F.Cu")
+		(net 2)
+	)
+	(segment
 		(start 103.5 75)
 		(end 105.25 73.25)
@@
 	)
 	(segment
+		(start 150.0776 67.5776)
+		(end 150.5 68)
+		(width 0.2)
+		(layer "F.Cu")
+		(net 2)
+	)
+	(segment
 		(start 78 91)
 		(end 78 93.065686)
@@
 	)
 	(segment
+		(start 58.9625 84.0375)
+		(end 60 83)
+		(width 0.2)
+		(layer "F.Cu")
+		(net 2)
+	)
+	(segment
 		(start 105.25 73.25)
 		(end 105.5 73.5)
@@
 	)
 	(segment
-		(start 150.176 63.931)
-		(end 150.0776 63.8326)
-		(width 0.2)
-		(layer "F.Cu")
-		(net 2)
-	)
-	(segment
-		(start 71.5772 91)
-		(end 78 91)
+		(start 72.5 83)
+		(end 74.5 85)
 		(width 0.2)
 		(layer "F.Cu")
@@
 	)
 	(segment
+		(start 150.0776 63.25)
+		(end 150.0776 65.4224)
+		(width 0.2)
+		(layer "F.Cu")
+		(net 2)
+	)
+	(segment
 		(start 160 67)
 		(end 159.5 67)
@@
 	)
 	(segment
+		(start 75.5 91)
+		(end 78 91)
+		(width 0.2)
+		(layer "F.Cu")
+		(net 2)
+	)
+	(segment
 		(start 112.5 75)
 		(end 117 75)
@@
 	)
 	(segment
-		(start 150.0776 63.8326)
-		(end 150.0776 63.25)
-		(width 0.2)
-		(layer "F.Cu")
-		(net 2)
-	)
-	(segment
 		(start 159 67.5)
 		(end 154.5375 67.5)
@@
 	)
 	(segment
-		(start 150.9685 63.931)
-		(end 150.176 63.931)
-		(width 0.2)
-		(layer "F.Cu")
-		(net 2)
-	)
-	(segment
 		(start 80.434314 95.5)
 		(end 85.5 95.5)
@@
 		(width 0.2)
 		(layer "F.Cu")
+		(net 2)
+	)
+	(via
+		(at 151.1776 66)
+		(size 0.6)
+		(drill 0.3)
+		(layers "F.Cu" "B.Cu")
 		(net 2)
 	)
@@
 	)
 	(via
+		(at 75.5 87.5)
+		(size 0.6)
+		(drill 0.3)
+		(layers "F.Cu" "B.Cu")
+		(net 2)
+	)
+	(via
 		(at 103.02 75)
 		(size 0.6)
@@
 	)
 	(via
+		(at 75.5 85)
+		(size 0.6)
+		(drill 0.3)
+		(layers "F.Cu" "B.Cu")
+		(net 2)
+	)
+	(via
 		(at 154.5 65.6)
+		(size 0.6)
+		(drill 0.3)
+		(layers "F.Cu" "B.Cu")
+		(net 2)
+	)
+	(via
+		(at 150.5 68)
 		(size 0.6)
 		(drill 0.3)
@@
 	)
 	(segment
+		(start 150.5 68)
+		(end 151.1776 67.3224)
+		(width 0.2)
+		(layer "B.Cu")
+		(net 2)
+	)
+	(segment
+		(start 151.1776 67.3224)
+		(end 151.1776 66)
+		(width 0.2)
+		(layer "B.Cu")
+		(net 2)
+	)
+	(segment
 		(start 154.5 59.9)
 		(end 154.5 65.6)
@@
 		(start 101.5 75)
 		(end 103.02 75)
+		(width 0.2)
+		(layer "B.Cu")
+		(net 2)
+	)
+	(segment
+		(start 75.5 85)
+		(end 75.5 87.5)
 		(width 0.2)
 		(layer "B.Cu")
@@
 	)
 	(segment
+		(start 151.5 67.5)
+		(end 152.4625 67.5)
+		(width 0.2)
+		(layer "F.Cu")
+		(net 7)
+	)
+	(segment
 		(start 111 87.5)
 		(end 110 86.5)
@@
 	)
 	(segment
+		(start 150.5776 63.25)
+		(end 150.5776 66.5776)
+		(width 0.2)
+		(layer "F.Cu")
+		(net 7)
+	)
+	(segment
 		(start 62.5 64)
 		(end 62.5 63.5)
@@
 		(width 0.2)
 		(layer "F.Cu")
+		(net 7)
+	)
+	(segment
+		(start 150.5776 66.5776)
+		(end 151.5 67.5)
+		(width 0.2)
+		(layer "F.Cu")

Commit message: Fixed edge cut
Other:
- board outline added: 119.5 x 65.5 mm
Changed lines of the file:
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@@
 		)
 		(fill none)
-		(layer "F.Cu")
+		(layer "Edge.Cuts")
 	)
 	(gr_text "V 1.0"

Commit message: Update With Tire Temp Sensor
Update With Tire Temp Sensor
Parts:
- added J5: Tire temp, Connector_PinHeader_1.00mm:PinHeader_1x04_P1.00mm_Vertical, F.Cu at (92.0, 89.0)
Connections:
- C2 pad 1: /Wheel Speed -> PA4
- J3 pad 2: /Shock position -> PA6
- R4 pad 2: /Wheel Speed -> PA4
- U2 pad 10: /Strain -> PA7
- U2 pad 11: /Strain -> PA7
Routing:
- net PA7: track 8.38 -> 181.0 mm, vias 0 -> 6
- net PA6: track 8.59 -> 124.3 mm, vias 0 -> 4
- net PA4: track 9.65 -> 120.4 mm, vias 0 -> 4
- net CANH: track 13.4 -> 38.0 mm, vias 0 -> 2
- net CANL: track 12.2 -> 34.1 mm, vias 0 -> 4
- net GND: track 425.8 -> 432.9 mm, vias 12 -> 14
- net /Wheel Speed: track 5.02 -> 0.00 mm
- net +5V: track 388.0 -> 391.5 mm
- net /VrefBG: track 24.7 -> 25.6 mm
Other:
- board outline removed

Commit message: Updated Peripheral Board(Compact)
Parts:
- added REF**: MountingHole_3.5mm, MountingHole:MountingHole_3.5mm, F.Cu at (245.0, 56.5)
- added REF**: MountingHole_3.5mm, MountingHole:MountingHole_3.5mm, F.Cu at (162.0, 56.0)
- added REF**: MountingHole_3.5mm, MountingHole:MountingHole_3.5mm, F.Cu at (162.5, 94.5)
- added REF**: MountingHole_3.5mm, MountingHole:MountingHole_3.5mm, F.Cu at (245.5, 95.0)
- J5: value Tire temp -> Tire temp Sensor
- moved R1 165.0 mm to (229.5, 66.5)
- moved R2 163.9 mm to (229.5, 62.5)
- moved R4 159.3 mm to (234.5, 58.5), turned to -90 degrees
- moved R5 158.8 mm to (229.5, 58.5), turned to -90 degrees
- moved C2 154.4 mm to (234.5, 63.0)
- moved U1 149.4 mm to (221.3, 62.8), turned to 0 degrees
- moved C1 149.0 mm to (213.5, 60.0)
- moved J1 144.9 mm to (205.0, 57.0)
- moved C6 139.6 mm to (200.0, 66.0), turned to -90 degrees
- moved R3 139.5 mm to (209.0, 60.0)
- moved R6 133.8 mm to (214.5, 66.0), turned to -90 degrees
- moved C5 132.4 mm to (191.1, 67.4), turned to 90 degrees
- moved C3 131.1 mm to (210.0, 66.0)
- moved C4 130.6 mm to (205.0, 66.0)
- moved R11 126.5 mm to (187.1, 55.9), turned to 180 degrees
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Connections:
- D1 pad 1: +3.3V -> +3V3
- R14 pad 1: +3.3V -> +3V3
- U2 pad 6: /VIN+ -> /Vin+
- U2 pad 7: /VIN- -> /Vin-
Routing:
- net +5V: track 391.5 -> 227.3 mm, vias 9 -> 12
- net PA7: track 181.0 -> 40.9 mm
- net GND: track 432.9 -> 306.2 mm, vias 14 -> 26
- net PA3/SCK: track 171.6 -> 45.8 mm, vias 2 -> 0
- net PA2: track 169.0 -> 43.6 mm, vias 0 -> 6
- net PA6: track 124.3 -> 16.1 mm, vias 4 -> 0
- net +3V3: track 247.4 -> 142.0 mm, vias 4 -> 12
- net PA1: track 145.4 -> 40.2 mm, vias 4 -> 2
- net PC3: track 118.8 -> 44.9 mm
- net CANL: track 34.1 -> 78.9 mm
- net CANH: track 38.0 -> 81.6 mm, vias 2 -> 4
- net CAN1_RX: track 15.6 -> 45.4 mm, vias 0 -> 2
- net /VrefBG: track 25.6 -> 1.27 mm, vias 4 -> 0
- net CAN1_TX: track 15.1 -> 37.6 mm, vias 0 -> 2
- net Net-(U3-OSC2): track 28.4 -> 12.4 mm, vias 4 -> 0
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
Commit message: peripheral board notes
Other:
- board outline added: 98 x 50.5 mm
Changed lines of the file:
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@@
 			(outputformat 1)
 			(mirror no)
-			(drillshape 1)
+			(drillshape 0)
 			(scaleselection 1)
 			(outputdirectory "")
@@
 		(tags "resistor handsolder")
 		(property "Reference" "R10"
-			(at 0 -1.65 360)
+			(at 0 -1.65 0)
 			(layer "F.SilkS")
 			(effects
@@
 		)
 		(property "Value" "~"
-			(at 0 1.65 360)
+			(at 0 1.65 0)
 			(layer "F.Fab")
 			(effects
@@
 		)
 		(fp_text user "${REFERENCE}"
-			(at 0 0 360)
+			(at 0 0 0)
 			(layer "F.Fab")
 			(effects
@@
 		(tags "resistor handsolder")
 		(property "Reference" "R11"
-			(at 0 -1.65 360)
+			(at 0 -1.65 0)
 			(layer "F.SilkS")
 			(effects
@@
 		)
 		(property "Value" "0.64"
-			(at 0 1.65 360)
+			(at 0 1.65 0)
 			(layer "F.Fab")
 			(effects
@@
 		)
 		(fp_text user "${REFERENCE}"
-			(at 0 0 360)
+			(at 0 0 0)
 			(layer "F.Fab")
 			(effects
@@
 		(tags "Through hole pin header THT 1x10 1.00mm single row")
 		(property "Reference" "H1"
-			(at 0 -1.56 360)
+			(at 0 -1.56 0)
 			(layer "F.SilkS")
 			(effects
@@
 		)
 		(property "Value" "Conn_01x10_MountingPin"
-			(at 0 10.56 360)
+			(at 0 10.56 0)
 			(layer "F.Fab")
 			(effects
@@
 		(tags "capacitor handsolder")
 		(property "Reference" "C15"
-			(at 0 -1.68 360)
+			(at 0 -1.68 0)
 			(layer "F.SilkS")
 			(effects
@@
 		)
 		(property "Value" "100 nF"
-			(at 0 1.68 360)
+			(at 0 1.68 0)
 			(layer "F.Fab")
 			(effects
@@
 		)
 		(fp_text user "${REFERENCE}"
-			(at 0 0 360)
+			(at 0 0 0)
 			(layer "F.Fab")
 			(effects
@@
 		(tags "SOIC SO")
 		(property "Reference" "U3"
-			(at 0 -6.72 360)
+			(at 0 -6.72 0)
 			(layer "F.SilkS")
 			(effects
@@
 		)
 		(property "Value" "MCP2515-I/SO"
-			(at 0 6.72 360)
+			(at 0 6.72 0)
 			(layer "F.Fab")
 			(effects
@@
 		)
 		(fp_text user "${REFERENCE}"
-			(at 0 0 360)
+			(at 0 0 0)
 			(layer "F.Fab")
 			(effects
@@
 		)
 		(property "Footprint" "New Library:105313-1108"
-			(at 0 0 360)
+			(at 0 0 0)
 			(layer "F.Fab")
 			(hide yes)
@@
 		)
 		(property "Datasheet" ""
-			(at 0 0 360)
+			(at 0 0 0)
 			(layer "F.Fab")
 			(hide yes)
@@
 		)
 		(property "Description" ""
-			(at 0 0 360)
+			(at 0 0 0)
 			(layer "F.Fab")
 			(hide yes)
@@
 		)
 		(fp_text user "*"
-			(at -2.6162 -6.1468 360)
+			(at -2.6162 -6.1468 0)
 			(layer "F.SilkS")
 			(effects
@@
 		)
 		(fp_text user "*"
-			(at -2.6162 -6.1468 360)
+			(at -2.6162 -6.1468 0)
 			(layer "F.Fab")
 			(effects
@@
 		(tags "Through hole pin header THT 1x10 1.00mm single row")
 		(property "Reference" "H2"
-			(at 0 -1.56 360)
+			(at 0 -1.56 0)
 			(layer "F.SilkS")
 			(effects
@@
 		)
 		(property "Value" "Conn_01x10_MountingPin"
-			(at 3.5 10.5 360)
+			(at 3.5 10.5 0)
 			(layer "F.Fab")
 			(hide yes)
@@
 		(tags "Through hole pin header THT 1x02 2.00mm single row")
 		(property "Reference" "J4"
-			(at 0 -2.06 360)
+			(at 0 -2.06 0)
 			(layer "F.SilkS")
 			(effects
@@
 		)
 		(property "Value" "Strain Gauge"
-			(at 0 4.06 360)
+			(at 0 4.06 0)
 			(layer "F.Fab")
 			(effects
@@
 		(tags "resistor handsolder")
 		(property "Reference" "R7"
-			(at 0 -1.65 360)
+			(at 0 -1.65 0)
 			(layer "F.SilkS")
 			(effects
@@
 		)
 		(property "Value" "120"
-			(at 0 1.65 360)
+			(at 0 1.65 0)
 			(layer "F.Fab")
 			(effects
@@
 		)
 		(fp_text user "${REFERENCE}"
-			(at 0 0 360)
+			(at 0 0 0)
 			(layer "F.Fab")
 			(effects
@@
 		)
 		(fill none)
-		(layer "F.Cu")
+		(layer "Edge.Cuts")
 	)
 	(gr_text "V 1.0"
