File: Telemetry Main Rev 2/TelemMainV2/TelemMainV2.kicad_pcb (KiCad board)
At the start: 2 copper layers, 121.5 x 113.3 mm, 34 parts, among them J1 8 pin ATM connector, J3 12 pin ATM connector, J4 SD to SPI (Molex nanofit), U1 LM7805_TO220, U2 LM7809_TO220, U3 NUCLEO-F446RE, U4 ISO1050DUB, U6 MCP6004, U8 ISO1050DUB

Commit message: added new components and began creating traces
Parts:
- removed the REF** at (184.2, 152.4)
- removed the REF** at (184.2, 47.5)
- added C11: 1.0 uF, Capacitor_SMD:C_0805_2012Metric_Pad1.18x1.45mm_HandSolder, F.Cu at (206.9, 151.3)
- added C12: 47 pF, Capacitor_SMD:C_0805_2012Metric_Pad1.18x1.45mm_HandSolder, F.Cu at (207.9, 147.8)
- added C15: 1 µF, Capacitor_SMD:C_0805_2012Metric, F.Cu at (139.5, 134.6)
- added C16: 0.1 µF, Capacitor_SMD:C_0805_2012Metric, F.Cu at (139.5, 129.7)
- added C17: 100nF, Capacitor_SMD:C_0805_2012Metric, F.Cu at (134.0, 132.5)
- added C18: 10 µF, Capacitor_SMD:C_0805_2012Metric, F.Cu at (120.4, 129.2)
- added C19: 100nF, Capacitor_SMD:C_0805_2012Metric, F.Cu at (123.1, 134.0)
- added C20: 100nF, Capacitor_SMD:C_0805_2012Metric, F.Cu at (119.2, 134.1)
- added C21: 0.1 µF, Capacitor_SMD:C_0805_2012Metric, F.Cu at (138.0, 142.0)
- added C22: 100 nF, Capacitor_SMD:C_0805_2012Metric, F.Cu at (126.7, 105.4)
- added C23: 1 µF, Capacitor_SMD:C_0805_2012Metric, F.Cu at (120.1, 121.4)
- added C24: 10 µF, Capacitor_SMD:C_0805_2012Metric, F.Cu at (132.6, 102.9)
- added C25: 1 µF, Capacitor_SMD:C_0805_2012Metric, F.Cu at (109.9, 143.9)
- added C26: 1 µF, Capacitor_SMD:C_0805_2012Metric, F.Cu at (109.9, 141.6)
- added D2: 470 mV @ 2A Forward / 40V 2A Reverse, FS_3_Global_Footprint_Library:US2H_TOS, F.Cu at (137.1, 114.1)
- added J2: 40 pin ZIF FPC Connector, FS_3_Global_Footprint_Library:CONN_F32D-1A7Y1-21040_AMP, F.Cu at (128.9, 151.3)
- added JP1: Open, Jumper:SolderJumper-2_P1.3mm_Open_RoundedPad1.0x1.5mm, F.Cu at (132.5, 114.4)
- added L1: 4.7 µH, Inductor_SMD:L_TDK_SLF7045, F.Cu at (106.9, 132.1)
- added R10: 2.49 ±1%, Resistor_SMD:R_0805_2012Metric, F.Cu at (127.1, 117.1)
- added R11: 4.7k, Resistor_SMD:R_0805_2012Metric, F.Cu at (105.3, 121.3)
- added R3: 4.99 ±1%, Resistor_SMD:R_0805_2012Metric, F.Cu at (114.7, 146.1)
- added R4: 33K ±1%, Resistor_SMD:R_0805_2012Metric, F.Cu at (110.1, 150.0)
- added R9: 100K ±1%, Resistor_SMD:R_0805_2012Metric, F.Cu at (125.5, 130.0)
- added U10: ~, Package_TO_SOT_SMD:SOT-23-6_Handsoldering, F.Cu at (116.6, 141.1)
- added U5: XBP9B-DPST-001, FS_3_Global_Footprint_Library:XBP9B-DPST-001, F.Cu at (192.7, 138.9)
- added U7: BT817Q, Package_DFN_QFN:VQFN-64-1EP_9x9mm_P0.5mm_EP7.15x7.15mm, F.Cu at (129.3, 138.3)
- added U9: ~, Package_SO:SOIC-8_5.23x5.23mm_P1.27mm, F.Cu at (129.4, 124.7)
- moved G1 87.4 mm to (207.7, 68.7)
- moved G*** 29.3 mm to (149.4, 61.2), turned to 0 degrees
- moved C10 15.2 mm to (183.5, 80.4)
- moved C6 15.2 mm to (183.4, 64.6)
- moved C7 15.2 mm to (172.7, 64.6)
- moved C8 15.2 mm to (172.7, 80.4)
- moved U4 15.2 mm to (169.9, 72.1)
- moved U8 15.2 mm to (180.7, 72.1)
- moved J1 13.2 mm to (161.5, 61.0)
- moved J3 0.50 mm to (89.9, 43.1)
- moved C1 0.14 mm to (120.0, 64.1)
- moved C3 0.14 mm to (124.0, 64.1)
Connections:
- net SPI2_CS renamed SD CS2
- net SPI2_MISO renamed SD MISO2
- net SPI2_MOSI renamed SD MOSI2
- net SPI2_SCK renamed SD SCK2
- J3 pad 10: Acc Intake Flow Rate -> Acc Intake Pressure
- J3 pad 11: unconnected-(J3-Pin_11-Pad11) -> Acc Intake Flow Rate
- J3 pad 5: Brake Sensor F -> GND
- J3 pad 6: Brake Sensor B -> Brake Sensor F
- J3 pad 7: Acc Intake Temp -> Brake Sensor B
- J3 pad 8: Acc Exhaust Temp -> Acc Intake Temp
- J3 pad 9: Acc Intake Pressure -> Acc Exhaust Temp
- U3 pad CN10_1: CAN1_RX -> unconnected-(U3B-PC9-PadCN10_1)
- U3 pad CN10_11: unconnected-(U3B-PA5-PadCN10_11) -> Radio SCK1
- U3 pad CN10_12: unconnected-(U3B-PA12-PadCN10_12) -> Radio RTS1
- U3 pad CN10_13: Brake Sensor R 3V3 -> Radio MISO1
- U3 pad CN10_14: unconnected-(U3B-PA11-PadCN10_14) -> Radio CTS1
- U3 pad CN10_15: Brake Sensor F 3V3 -> Radio MOSI1
- U3 pad CN10_19: unconnected-(U3B-PC7-PadCN10_19) -> Radio Reset
- U3 pad CN10_21: unconnected-(U3B-PA9-PadCN10_21) -> Radio TX1
- U3 pad CN10_3: unconnected-(U3B-PB8-PadCN10_3) -> CAN1_RX
- U3 pad CN10_33: unconnected-(U3B-PA10-PadCN10_33) -> Radio RX1
- U3 pad CN7_1: unconnected-(U3A-PC10-PadCN7_1) -> Dash SCK3
- U3 pad CN7_13: unconnected-(U3A-PA13-PadCN7_13) -> Radio ATTN
- U3 pad CN7_15: unconnected-(U3A-PA14-PadCN7_15) -> Dash CS3
- U3 pad CN7_17: unconnected-(U3A-PA15-PadCN7_17) -> Radio CS1
- U3 pad CN7_2: unconnected-(U3A-PC11-PadCN7_2) -> Dash MISO3
- U3 pad CN7_21: unconnected-(U3A-PB7-PadCN7_21) -> PD
- U3 pad CN7_23: unconnected-(U3A-PC13-PadCN7_23) -> INT
- U3 pad CN7_3: unconnected-(U3A-PC12-PadCN7_3) -> Dash MOSI3
- U3 pad CN7_36: unconnected-(U3A-PC1/PB9-PadCN7_36) -> Brake Sensor F 3V3
- U3 pad CN7_38: unconnected-(U3A-PC0/PB8-PadCN7_38) -> Brake Sensor R 3V3
Routing:
- net +3V3: track 208.3 -> 272.7 mm
- net GND: track 58.1 -> 83.7 mm
- net INT: track 0.00 -> 11.5 mm, vias 0 -> 1
- net +5V: track 107.1 -> 117.9 mm
- net CAN2_H: track 20.7 -> 28.5 mm
- net CAN2_RX: track 66.0 -> 70.1 mm
- net CAN1_TX: track 29.5 -> 33.5 mm
- net CAN1_RX: track 23.9 -> 27.6 mm
- net CAN2_TX: track 52.1 -> 53.7 mm
- net CAN1_H: track 19.5 -> 17.8 mm, vias 2 -> 1
- net CAN1_L: track 13.9 -> 14.6 mm
Other:
- board size 121.5 x 113.3 mm -> 161 x 113.3 mm

Commit message: dash traces
Parts:
- moved C15 41.5 mm to (133.5, 93.6)
- moved C16 41.5 mm to (133.5, 88.6)
- moved C21 41.5 mm to (132.1, 101.0)
- moved C17 41.5 mm to (128.0, 91.5)
- moved R4 40.6 mm to (149.2, 139.1), turned to -90 degrees
- moved C26 35.6 mm to (145.5, 142.2), turned to -90 degrees
- moved R3 34.1 mm to (141.7, 125.4), turned to -90 degrees
- moved C24 33.7 mm to (134.4, 136.5), turned to -90 degrees
- moved L1 33.5 mm to (140.2, 135.7), turned to 0 degrees
- moved C25 33.4 mm to (143.3, 142.2), turned to -90 degrees
- moved R9 27.0 mm to (149.2, 142.9), turned to -90 degrees
- moved U10 26.3 mm to (140.2, 129.4), turned to 180 degrees
- moved D2 23.5 mm to (146.4, 135.7), turned to 180 degrees
- moved C23 19.4 mm to (132.2, 136.5), turned to -90 degrees
- moved R10 18.2 mm to (144.8, 121.7), turned to -90 degrees
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Connections:
- U3 pad CN10_12: Radio RTS1 -> unconnected-(U3B-PA12-PadCN10_12)
- U3 pad CN10_14: Radio CTS1 -> unconnected-(U3B-PA11-PadCN10_14)
- U3 pad CN10_21: Radio TX1 -> unconnected-(U3B-PA9-PadCN10_21)
- U3 pad CN10_33: Radio RX1 -> unconnected-(U3B-PA10-PadCN10_33)
Routing:
- net Brake Sensor R 3V3: track 78.2 -> 15.2 mm
- net GND: track 83.7 -> 135.1 mm, vias 9 -> 12
- net BL-Low: track 0.00 -> 36.4 mm
- net Brake Sensor F 3V3: track 62.4 -> 26.5 mm
- net BL-High: track 0.00 -> 33.4 mm
- net +3V3: track 272.7 -> 293.3 mm
- net R1: track 0.00 -> 15.1 mm
- net DEN: track 0.00 -> 14.8 mm
- net R2: track 0.00 -> 14.7 mm
- net VSYNC: track 0.00 -> 14.4 mm
- net R3: track 0.00 -> 14.3 mm
- net HSYNC: track 0.00 -> 14.0 mm
- net R4: track 0.00 -> 13.8 mm
- net DISP: track 0.00 -> 13.5 mm
- net R5: track 0.00 -> 13.4 mm
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
Commit message: updated dash traces
Parts:
- moved C17 41.5 mm to (125.5, 133.0)
Connections:
- U3 pad CN10_34: unconnected-(U3B-PC4-PadCN10_34) -> Radio CS1
- U3 pad CN7_17: Radio CS1 -> unconnected-(U3A-PA15-PadCN7_17)
Routing:
- net +3V3: track 293.3 -> 301.7 mm
- net GND: track 135.1 -> 140.2 mm, vias 12 -> 14
- net Brake Sensor R 3V3: track 15.2 -> 14.4 mm

Commit message: almost done with dash traces
Parts:
- moved C16 44.7 mm to (127.9, 133.0), turned to 90 degrees
- moved C15 39.5 mm to (130.0, 133.0), turned to 90 degrees
- moved C21 38.3 mm to (128.4, 139.1), turned to -90 degrees
- moved C22 18.9 mm to (124.8, 124.2), turned to 180 degrees
Connections:
- J3 pad 10: Acc Intake Pressure -> Acc Intake Flow Rate
- J3 pad 11: Acc Intake Flow Rate -> GND
- J3 pad 5: GND -> Brake Sensor F
- J3 pad 6: Brake Sensor F -> Brake Sensor B
- J3 pad 7: Brake Sensor B -> Acc Intake Temp
- J3 pad 8: Acc Intake Temp -> Acc Exhaust Temp
- J3 pad 9: Acc Exhaust Temp -> Acc Intake Pressure
- U3 pad CN10_21: unconnected-(U3B-PA9-PadCN10_21) -> Radio ATTN
- U3 pad CN7_13: Radio ATTN -> unconnected-(U3A-PA13-PadCN7_13)
- U7 pad 3: Dash SCLK3 -> Dash SCK3
Routing:
- net BL-PWM: track 0.00 -> 46.6 mm
- net +3V3: track 301.7 -> 347.9 mm, vias 1 -> 6
- net OV: track 1.99 -> 37.8 mm
- net +9V: track 92.4 -> 126.8 mm, vias 4 -> 2
- net VCC1.2: track 4.32 -> 33.6 mm, vias 0 -> 2
- net R0: track 0.00 -> 16.5 mm
- net GND: track 140.2 -> 156.1 mm, vias 14 -> 18
- net INT: track 11.5 -> 14.3 mm, vias 1 -> 0
- net Net-(JP1-A): track 0.00 -> 2.11 mm
- net G4: track 10.8 -> 12.2 mm
- net G5: track 10.5 -> 11.8 mm
- net G3: track 11.3 -> 12.6 mm
- net Acc Intake Temp: track 93.0 -> 94.3 mm
- net G6: track 10.1 -> 11.4 mm
- net G0: track 12.5 -> 13.7 mm
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
Commit message: almost there please god
Routing:
- net Brake Sensor R 3V3: track 14.4 -> 94.8 mm
- net Brake Sensor F 3V3: track 26.6 -> 96.3 mm
- net BL-PWM: track 46.6 -> 105.6 mm
- net SD CS2: track 22.6 -> 33.6 mm, vias 1 -> 0
- net +3V3: track 347.9 -> 353.2 mm, vias 6 -> 8
- net GND: track 156.1 -> 155.0 mm

Commit message: i can see the light
Parts:
- moved G1 25.0 mm to (201.8, 92.9)
Connections:
- U3 pad CN7_15: Dash CS3 -> unconnected-(U3A-PA14-PadCN7_15)
- U3 pad CN7_4: unconnected-(U3A-PD2-PadCN7_4) -> Dash CS3
Routing:
- net +5V: track 128.8 -> 189.9 mm, vias 1 -> 3
- net Dash SCK3: track 0.00 -> 59.7 mm
- net Dash MOSI3: track 0.00 -> 56.6 mm
- net Dash MISO3: track 0.00 -> 55.4 mm
- net Dash CS3: track 0.00 -> 52.3 mm
- net PD: track 0.00 -> 30.7 mm, vias 0 -> 1
- net INT: track 14.3 -> 37.9 mm, vias 0 -> 2
- net +3V3: track 353.2 -> 376.3 mm, vias 8 -> 10
- net MEM-CS: track 0.00 -> 22.4 mm
- net MEM-IO3: track 10.6 -> 27.6 mm
- net +9V: track 126.8 -> 116.5 mm
- net MEM-MISO: track 0.00 -> 8.65 mm
- net MEM-IO2: track 0.00 -> 7.58 mm
- net GND: track 155.0 -> 149.4 mm, vias 18 -> 19
- net MEM-SCLK: track 8.49 -> 10.1 mm
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
Commit message: i had to delete half of this board and start it over again i am going to go missing soon
Parts:
- removed C10, C6: 100nf, Capacitor_SMD:C_0805_2012Metric_Pad1.18x1.45mm_HandSolder
- removed the REF** at (71.2, 152.4)
- removed the REF** at (71.2, 47.5)
- removed U8: ISO1050DUB, Package_SO:SOP-8_6.62x9.15mm_P2.54mm
- added REF**: MountingHole_3.5mm, MountingHole:MountingHole_3.5mm, F.Cu at (212.6, 28.3)
- added REF**: MountingHole_3.5mm, MountingHole:MountingHole_3.5mm, F.Cu at (78.9, 28.3)
- added REF**: MountingHole_3.5mm, MountingHole:MountingHole_3.5mm, F.Cu at (79.0, 160.9)
- added REF**: MountingHole_3.5mm, MountingHole:MountingHole_3.5mm, F.Cu at (212.7, 161.0)
- moved J3 126.9 mm to (216.8, 45.4), turned to -90 degrees
- moved D1 123.8 mm to (195.7, 41.4), turned to 0 degrees
- moved U5 116.4 mm to (132.7, 39.1), turned to -90 degrees
- moved C9 100.8 mm to (176.7, 48.9), turned to 180 degrees
- moved G1 77.6 mm to (124.3, 97.9)
- moved C7 68.7 mm to (195.8, 129.3), turned to 90 degrees
- moved J1 63.6 mm to (198.8, 112.4), turned to -90 degrees
- moved U4 57.4 mm to (188.3, 126.5), turned to 0 degrees
- moved C8 49.4 mm to (180.1, 129.3), turned to 90 degrees
- moved C11 15.7 mm to (191.4, 153.5)
- moved C12 15.7 mm to (192.4, 150.1)
Connections:
- J1 pad 1: CAN1_H -> CAN1_L
- J1 pad 2: CAN1_H -> CAN1_L
- J1 pad 3: CAN1_L -> CAN1_H
- J1 pad 4: CAN1_L -> CAN1_H
- J1 pad 5: CAN2_H -> unconnected-(J1-Pin_5-Pad5)
- J1 pad 6: CAN2_H -> unconnected-(J1-Pin_6-Pad6)
- J1 pad 7: CAN2_L -> unconnected-(J1-Pin_7-Pad7)
- J1 pad 8: CAN2_L -> unconnected-(J1-Pin_8-Pad8)
- U3 pad CN10_17: CAN2_TX -> unconnected-(U3B-PB6-PadCN10_17)
- U3 pad CN10_29: CAN2_RX -> unconnected-(U3B-PB5-PadCN10_29)
Routing:
- net +12VIN: track 149.3 -> 272.6 mm, vias 1 -> 0
- net Acc Intake Pressure: track 96.2 -> 0.00 mm
- net Acc Intake Flow Rate: track 95.6 -> 0.00 mm
- net Acc Exhaust Temp: track 95.2 -> 0.00 mm
- net Acc Intake Temp: track 94.3 -> 0.00 mm
- net CAN2_RX: track 70.1 -> 0.00 mm, vias 1 -> 0
- net CAN2_TX: track 53.7 -> 0.00 mm, vias 2 -> 0
- net +3V3: track 376.3 -> 325.3 mm, vias 10 -> 9
- net Steering Sensor: track 42.7 -> 0.00 mm, vias 2 -> 0
- net Brake Sensor B: track 36.5 -> 0.00 mm
- net Brake Sensor F: track 34.7 -> 0.00 mm
- net GND: track 149.4 -> 118.9 mm, vias 19 -> 17
- net CAN2_H: track 28.5 -> 0.00 mm, vias 1 -> 0
- net CAN1_RX: track 27.6 -> 0.00 mm, vias 1 -> 0
- net +5V: track 189.9 -> 164.4 mm
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Other:
- board size 161 x 113.3 mm -> 142.3 x 141.3 mm

Commit message: pushing changes from 2/18
Parts:
- moved U5 73.1 mm to (182.9, 92.2), turned to 0 degrees
- moved U6 38.7 mm to (170.1, 70.5), turned to 180 degrees
- moved U1 15.7 mm to (101.3, 58.6)
- moved C8 10.9 mm to (183.9, 119.0), turned to -90 degrees
- moved C7 10.7 mm to (192.8, 119.0), turned to -90 degrees
- moved C2 7.70 mm to (122.8, 61.8)
- moved C4 7.70 mm to (126.8, 61.8)
- moved U2 7.70 mm to (122.2, 58.2)
- moved REF** 5.61 mm to (84.5, 27.8)
- moved REF** 5.08 mm to (84.1, 160.9)
Routing:
- net +3V3: track 325.3 -> 204.8 mm
- net Steering Sensor 3V3: track 59.2 -> 1.27 mm, vias 1 -> 0
- net +5V: track 164.4 -> 120.4 mm
- net CAN1_RX: track 0.00 -> 36.8 mm
- net +12V: track 74.1 -> 48.9 mm, vias 3 -> 1
- net Brake Sensor F: track 0.00 -> 19.8 mm
- net +12VIN: track 272.6 -> 253.8 mm
- net Steering Sensor: track 0.00 -> 17.4 mm
- net Brake Sensor B: track 0.00 -> 15.5 mm
- net GND: track 118.9 -> 106.2 mm
- net Net-(U6B--): track 5.85 -> 1.27 mm
- net Net-(U6A--): track 5.54 -> 1.27 mm
- net CAN1_TX: track 33.5 -> 36.8 mm, vias 1 -> 0
- net +9V: track 115.5 -> 112.9 mm
Other:
- board text added: "FS-3 Main Telemetry Board Formula Slug Shaunak Lal, Slav Miroschenko, Jack Nystrom, Nova Mondal, Njeri Gachoka, Nathan Pham Rev 2.0"
- board text removed: "FS-3 Main Telemetry Board Formula Slug Designed by Shaunak Lal and Slav Miroshnichenko Rev 1.0"
