File: Telemetry Main Rev 2/TelemMainV2/TelemMainV2.kicad_sch (KiCad schematic)
At the start: 21 parts, among them J1 8 pin ATM connector, J3 12 pin ATM connector, J4 SD to SPI (Molex nanofit), U3 NUCLEO-F446RE, U4 ISO1050DUB, U6 MCP6004, U8 ISO1050DUB

Commit message: dash traces
Connections:
- net Radio CTS1: no longer names the net of U3.CN10_14 (PA11)
- net Radio RTS1: no longer names the net of U3.CN10_12 (PA12)
- net Radio RX1: no longer names the net of U3.CN10_33 (PA10)
- net Radio TX1: no longer names the net of U3.CN10_21 (PA9)
- no-connect marks 39 -> 43
Changed lines of the file:
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@@
+	)
+	(no_connect
+		(at 166.37 45.72)
 	)
 	(no_connect
@@
 	)
 	(no_connect
+		(at 201.93 35.56)
+	)
+	(no_connect
 		(at 35.56 100.33)
 	)
@@
 	)
 	(no_connect
+		(at 201.93 33.02)
+	)
+	(no_connect
 		(at 201.93 101.6)
 	)
@@
 	(no_connect
 		(at 166.37 58.42)
+	)
+	(no_connect
+		(at 166.37 60.96)
 	)
 	(no_connect
@@
 		)
 	)
-	(global_label "Radio TX1"
-		(shape output)
-		(at 166.37 45.72 180)
-		(fields_autoplaced yes)
-		(effects
-			(font
-				(size 1.27 1.27)
-			)
-			(justify right)
-		)
-		(property "Intersheetrefs" "${INTERSHEET_REFS}"
-			(at 153.7088 45.72 0)
-			(effects
-				(font
-					(size 1.27 1.27)
-				)
-				(justify right)
-				(hide yes)
-			)
-		)
-	)
 	(global_label "Radio CS1"
 		(shape output)
@@
 		)
 	)
-	(global_label "Radio CTS1"
-		(shape input)
-		(at 201.93 35.56 0)
-		(fields_autoplaced yes)
-		(effects
-			(font
-				(size 1.27 1.27)
-			)
-			(justify left)
-		)
-		(property "Intersheetrefs" "${INTERSHEET_REFS}"
-			(at 215.8612 35.56 0)
-			(effects
-				(font
-					(size 1.27 1.27)
-				)
-				(justify left)
-				(hide yes)
-			)
-		)
-	)
 	(global_label "Acc Exhaust Temp"
 		(shape output)
@@
 		)
 	)
-	(global_label "Radio RX1"
-		(shape input)
-		(at 166.37 60.96 180)
-		(fields_autoplaced yes)
-		(effects
-			(font
-				(size 1.27 1.27)
-			)
-			(justify right)
-		)
-		(property "Intersheetrefs" "${INTERSHEET_REFS}"
-			(at 153.4064 60.96 0)
-			(effects
-				(font
-					(size 1.27 1.27)
-				)
-				(justify right)
-				(hide yes)
-			)
-		)
-	)
 	(global_label "Brake Sensor F"
 		(shape input)
@@
 	)
 	(global_label "Radio ATTN"
-		(shape output)
+		(shape input)
 		(at 166.37 96.52 180)
 		(fields_autoplaced yes)
@@
 				(hide yes)
 			)
-		)
-	)
-	(global_label "Radio RTS1"
-		(shape input)
-		(at 201.93 33.02 0)
-		(fields_autoplaced yes)
-		(effects
-			(font
-				(size 1.27 1.27)
-			)
-			(justify left)
-		)
-		(property "Intersheetrefs" "${INTERSHEET_REFS}"
-			(at 215.8612 33.02 0)
-			(effects
-				(font
-					(size 1.27 1.27)
-				)
-				(justify left)
-				(hide yes)
-			)

Commit message: updated dash traces
Connections:
- net Radio CS1: now also U3.CN10_34 (PC4); no longer U3.CN7_17 (PA15)
Changed lines of the file:
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@@
-	)
-	(no_connect
-		(at 201.93 60.96)
 	)
 	(no_connect
@@
 	(no_connect
 		(at 201.93 91.44)
+	)
+	(no_connect
+		(at 166.37 101.6)
 	)
 	(no_connect
@@
 		)
 	)
+	(global_label "Radio CS1"
+		(shape output)
+		(at 201.93 60.96 0)
+		(fields_autoplaced yes)
+		(effects
+			(font
+				(size 1.27 1.27)
+			)
+			(justify left)
+		)
+		(property "Intersheetrefs" "${INTERSHEET_REFS}"
+			(at 214.8936 60.96 0)
+			(effects
+				(font
+					(size 1.27 1.27)
+				)
+				(justify left)
+				(hide yes)
+			)
+		)
+	)
 	(global_label "Acc Intake Temp"
 		(shape output)
@@
 				(hide yes)
 			)
-		)
-	)
-	(global_label "Radio CS1"
-		(shape output)
-		(at 166.37 101.6 180)
-		(fields_autoplaced yes)
-		(effects
-			(font
-				(size 1.27 1.27)
-			)
-			(justify right)
-		)
-		(property "Intersheetrefs" "${INTERSHEET_REFS}"
-			(at 153.4064 101.6 0)
-			(effects
-				(font
-					(size 1.27 1.27)
-				)
-				(justify right)
-				(hide yes)
-			)

Commit message: almost done with dash traces
Connections:
- net Acc Exhaust Temp: now also J3.8 (Pin_8); no longer J3.9 (Pin_9)
- net Acc Intake Flow Rate: now also J3.10 (Pin_10); no longer J3.11 (Pin_11)
- net Acc Intake Pressure: now also J3.9 (Pin_9); no longer J3.10 (Pin_10)
- net Acc Intake Temp: now also J3.7 (Pin_7); no longer J3.8 (Pin_8)
- net Brake Sensor B: now also J3.6 (Pin_6); no longer J3.7 (Pin_7)
- net Brake Sensor F: now also J3.5 (Pin_5); no longer J3.6 (Pin_6)
- net GND: now also J3.11 (Pin_11); no longer J3.5 (Pin_5)
- net Radio ATTN: now also U3.CN10_21 (PA9); no longer U3.CN7_13 (PA13)

Commit message: i can see the light
Connections:
- net Dash CS3: now also U3.CN7_4 (PD2); no longer U3.CN7_15 (PA14)
Changed lines of the file:
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@@
+	)
+	(no_connect
+		(at 166.37 99.06)
 	)
 	(no_connect
@@
 	(no_connect
 		(at 166.37 48.26)
-	)
-	(no_connect
-		(at 201.93 83.82)
 	)
 	(wire
@@
 	(global_label "Dash CS3"
 		(shape output)
-		(at 166.37 99.06 180)
-		(fields_autoplaced yes)
-		(effects
-			(font
-				(size 1.27 1.27)
-			)
-			(justify right)
-		)
-		(property "Intersheetrefs" "${INTERSHEET_REFS}"
-			(at 154.1321 99.06 0)
-			(effects
-				(font
-					(size 1.27 1.27)
-				)
-				(justify right)
-				(hide yes)
-			)
+		(at 201.93 83.82 0)
+		(fields_autoplaced yes)
+		(effects
+			(font
+				(size 1.27 1.27)
+			)
+			(justify left)
+		)
+		(property "Intersheetrefs" "${INTERSHEET_REFS}"
+			(at 214.1679 83.82 0)
+			(effects
+				(font
+					(size 1.27 1.27)
+				)
+				(justify left)
+				(hide yes)
+			)

Commit message: i had to delete half of this board and start it over again i am going to go missing soon
Parts:
- removed C10, C6: 100nf, Capacitor_SMD:C_0805_2012Metric_Pad1.18x1.45mm_HandSolder, symbol Device:C
- removed U8: ISO1050DUB, Package_SO:SOP-8_6.62x9.15mm_P2.54mm, symbol Interface_CAN_LIN:ISO1050DUB
Connections:
- net CAN1_H: now also J1.3 (Pin_3), J1.4 (Pin_4); no longer J1.1 (Pin_1), J1.2 (Pin_2)
- net CAN1_L: now also J1.1 (Pin_1), J1.2 (Pin_2); no longer J1.3 (Pin_3), J1.4 (Pin_4)
- net CAN2_H: no longer names the net of J1.5 (Pin_5)
- net CAN2_H: no longer J1.6 (Pin_6)
- net CAN2_L: no longer names the net of J1.7 (Pin_7)
- net CAN2_L: no longer J1.8 (Pin_8)
- net CAN2_RX: no longer names the net of U3.CN10_29 (PB5)
- net CAN2_TX: no longer names the net of U3.CN10_17 (PB6)
- no-connect marks 43 -> 49
Other:
- note removed: "CAN2 transceiver"

Commit message: add 10DoF IMU to Telem Main board v2
Parts:
- added U8: ~, FS_3_Global_Footprint_Library:Adafruit_E336755_10DoF_IMU, symbol FS_3_Global_Symbol_Library:Adafruit_E336755_10DoF_IMU
Connections:
- net +5V: now also U8.1 (VIN)
- net GND: now also U8.3 (GND), U8.GND (GND2)
- net IMU SCL: now reaches U3.CN10_25 (PB10)
- net IMU SCL: now also U8.4 (SCL)
- net IMU SDA: now reaches U3.CN10_31 (PB3)
- net IMU SDA: now also U8.5 (SDA)
- net IMU LRDY: now reaches U3.CN7_13 (PA13)
- net IMU LRDY: now also U8.10 (LRDY)
- net IMU LINT2: now reaches U3.CN7_15 (PA14)
- net IMU LINT2: now also U8.9 (LINT2)
- net IMU LINT1: now reaches U3.CN7_17 (PA15)
- net IMU LINT1: now also U8.8 (LINT1)
- net IMU GRDY: now reaches U3.CN7_29 (PH0)
- net IMU GRDY: now also U8.7 (GRDY)
- net IMU GINT: now reaches U3.CN7_31 (PH1)
- net IMU GINT: now also U8.6 (GINT)
- no-connect marks 49 -> 43
Other:
- note added: "<- optional output interrupt/ready pins for the IMU's gyroscope (G) and accelerometer/magnotomer (L1/L2)"

Commit message: i woke up at 6 am and finished the first part and most of it will probably get deleted by later today. for good luck: Our Father, who art in heaven, hallowed be thy Name, thy kingdom come, thy will be done, on earth as it is in heaven. Give us this day our daily bread. And forgive us our trespasses, as we forgive those who trespass against us. And lead us not into temptation, but deliver us from evil.
Connections:
- net Radio CS1: now also U3.CN10_2 (PC8); no longer U3.CN10_34 (PC4)
Changed lines of the file:
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@@
-	)
-	(no_connect
-		(at 201.93 20.32)
 	)
 	(no_connect
@@
 	(no_connect
 		(at 67.31 187.96)
+	)
+	(no_connect
+		(at 201.93 60.96)
 	)
 	(no_connect
@@
 		)
 	)
-	(global_label "Radio CS1"
-		(shape output)
-		(at 201.93 60.96 0)
-		(fields_autoplaced yes)
-		(effects
-			(font
-				(size 1.27 1.27)
-			)
-			(justify left)
-		)
-		(property "Intersheetrefs" "${INTERSHEET_REFS}"
-			(at 214.8936 60.96 0)
-			(effects
-				(font
-					(size 1.27 1.27)
-				)
-				(justify left)
-				(hide yes)
-			)
-		)
-	)
 	(global_label "IMU SDA"
 		(shape input)
@@
 				(hide yes)
 			)
+		)
+	)
+	(global_label "Radio CS1"
+		(shape output)
+		(at 201.93 20.32 0)
+		(fields_autoplaced yes)
+		(effects
+			(font
+				(size 1.27 1.27)
+			)
+			(justify left)
+		)
+		(property "Intersheetrefs" "${INTERSHEET_REFS}"
+			(at 214.8936 20.32 0)
+			(effects
+				(font
+					(size 1.27 1.27)
+				)
+				(justify left)
+				(hide yes)
+			)

Commit message: stopped a micro pin from being blown up at a solid 9V
Parts:
- added R12: 10k, Resistor_SMD:R_0805_2012Metric_Pad1.20x1.40mm_HandSolder, symbol Device:R_US
- added R13: 20k, Resistor_SMD:R_0805_2012Metric_Pad1.20x1.40mm_HandSolder, symbol Device:R_US
Connections:
- net +12VIN: now also R2.2; no longer R1.1
- net GND: now also R1.1, R13.1; no longer R2.1
- net Steering Sensor 3V3: now also R12.2, R13.2; no longer U6.8, U6.9 (-)
- net at R1.2, U3.CN7_35 (PC2): now also R2.1; no longer R2.2
- new net: R12.1, U6.8, U6.9 (-)
