File: Telemetry Main Rev 2/TelemMainV2/dash.kicad_sch (KiCad schematic)
At the start: 9 parts, among them J2 40 pin ZIF FPC Connector, U7 BT817Q

Commit message: updated dash integration
Parts:
- added C22: 100 nF, Capacitor_SMD:C_0805_2012Metric, symbol Device:C
- added C23, C25, C26: 1 µF, Capacitor_SMD:C_0805_2012Metric, symbol Device:C
- added C24: 10 µF, Capacitor_SMD:C_0805_2012Metric, symbol Device:C
- added D2: 470 mV @ 2A Forward / 40V 2A Reverse, FS_3_Global_Footprint_Library:US2H_TOS, symbol Device:D_Schottky
- added JP1: Open, Jumper:SolderJumper-2_P1.3mm_Open_RoundedPad1.0x1.5mm, symbol Jumper:SolderJumper_2_Open
- added L1: 4.7 µH, Inductor_SMD:L_TDK_SLF7045, symbol Device:L
- added R10: 2.49 ±1%, Resistor_SMD:R_0805_2012Metric, symbol Device:R_US
- added R3: 4.99 ±1%, Resistor_SMD:R_0805_2012Metric, symbol Device:R_US
- added R4: 33K ±1%, Resistor_SMD:R_0805_2012Metric, symbol Device:R_US
- added R9: 100K ±1%, Resistor_SMD:R_0805_2012Metric, symbol Device:R_US
- added U10: ~, Package_TO_SOT_SMD:SOT-23-6_Handsoldering, symbol FS_3_Global_Symbol_Library:AP3032KTR-G1
- added U9: ~, Package_SO:SOIC-8_5.23x5.23mm_P1.27mm, symbol FS_3_Global_Symbol_Library:W25Q40CLSNIG_TR
Connections:
- net BL-High: now also C25.1, C26.1, D2.1 (K), R4.1
- net BL-Low: now also JP1.2 (B), R3.2, U10.3 (FB)
- net BL-PWM: now also U10.4 (CTRL)
- net GND: now also C22.1, C23.2, C24.2, C25.2, C26.2, R10.1, R3.1, R9.2, U10.2 (GND), U9.4 (GND)
- net MEM-CS: now also U9.1 (CS)
- net MEM-IO2: now also U9.3 (WP)
- net MEM-IO3: now also U9.7 (Hold)
- net MEM-MISO: now also U9.2 (DO)
- net MEM-MOSI: now also U9.5 (DI)
- net MEM-SCLK: now also U9.6 (CLK)
- net +3.3V renamed +3V3
- net +3V3: now also C22.2, U9.8 (VCC)
- net Host-CS renamed Dash CS3
- net Host-MISO renamed Dash MISO3
- net Host-MOSI renamed Dash MOSI3
- net Host-SCLK renamed Dash SCLK3
- new net: D2.2 (A), L1.2, U10.1 (SW)
- new net: JP1.1 (A), R10.2
- new net +5V: C23.1, C24.1, L1.1, U10.6 (VIN)
- new net OV: R4.2, R9.1, U10.5 (OV)
Other:
- moved on the sheet: C15, C16, C17, C18, C19, C20, C21, J2, U7

Commit message: almost done with dash traces
Connections:
- net Dash SCLK3 renamed Dash SCK3
Changed lines of the file:
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@@
 		)
 	)
-	(global_label "Dash SCLK3"
+	(global_label "Dash SCK3"
 		(shape input)
 		(at 104.14 33.02 180)
@@
 		)
 		(property "Intersheetrefs" "${INTERSHEET_REFS}"
-			(at 89.604 33.02 0)
+			(at 90.6321 33.02 0)
 			(effects
 				(font

Commit message: consistency
Parts:
- C17, C19, C20: value 100nF -> 100nf
- C22: value 100 nF -> 100nf
Changed lines of the file:
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@@
 			)
 		)
-		(property "Value" "100nF"
+		(property "Value" "100nf"
 			(at 83.82 83.566 0)
 			(effects
@@
 			)
 		)
-		(property "Value" "100nF"
+		(property "Value" "100nf"
 			(at 98.298 101.854 0)
 			(effects
@@
 			)
 		)
-		(property "Value" "100nF"
+		(property "Value" "100nf"
 			(at 86.36 50.8001 0)
 			(effects
@@
 			)
 		)
-		(property "Value" "100 nF"
+		(property "Value" "100nf"
 			(at 195.072 32.766 0)
 			(effects
