File: Telemetry peripheral boards/F3 Peripheral Boards V2(CORRECT PCB)/F3 peripheral boards.kicad_pcb (KiCad board)
At the start: 2 copper layers, 130.5 x 48.5 mm, 52 parts, among them J1 ATS668LSM, J2 CAN & Power Supply, J3 Potentiometer, J4 Strain Gauge, J5 Tire temp Sensor, U1 LM2907M/NOPB, U2 INA125U, U3 MCP2515-I/SO, U4 ISO1050DUB, U5 ATtiny1616-S, U6 LM7805CV, U7 LF33CV, Y1 Crystal

Commit message: PCB I HOPE
Routing:
- net GND: track 367.3 -> 55.6 mm, vias 20 -> 22
- net PA6: track 116.8 -> 108.9 mm, vias 12 -> 6
- net Net-(U3-*RESET): track 3.93 -> 11.2 mm
- net +12V: track 20.7 -> 27.2 mm
- net CANL: track 60.8 -> 54.7 mm, vias 8 -> 0
- net CAN1_TX: track 69.3 -> 64.0 mm, vias 10 -> 4
- net PC1: track 41.2 -> 36.1 mm
- net PA7: track 109.4 -> 104.4 mm, vias 6 -> 2
- net PC2: track 45.2 -> 40.2 mm
- net CANH: track 63.4 -> 59.6 mm, vias 8 -> 0
- net PA4: track 112.5 -> 109.3 mm
- net PC3: track 62.9 -> 59.8 mm, vias 8 -> 7
- net PA5: track 88.0 -> 85.0 mm
- net PA2: track 125.6 -> 123.5 mm, vias 6 -> 4
- net Net-(H2-Pin_1): track 36.8 -> 35.2 mm
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Other:
- board text added: "5V"
- board text added: "GND"
- board text added: "PA1"
- board text added: "PA2"
- board text added: "PA3/SCK"
- board text added: "PA4"
- board text added: "PA5"
- board text added: "PA6"
- board text added: "PA7"
- board text added: "PB0"
- board text added: "PB1"
- board text added: "PB4"
- board text added: "PB5"
- board text added: "PC0"
- board text added: "PC1"
- board text added: "PC2"
- board text added: "PC3"
- board text added: "TOSC1/PB3"
- board text added: "TOSC2/PB2"
- board text added: "UPDI"
- board text removed: "pinheaders for attiny"

Commit message: pcb done
Parts:
- moved REF** 7.62 mm to (175.3, 37.5)
- moved REF** 7.62 mm to (175.3, 75.6)
Routing:
- net PA4: track 109.3 -> 94.9 mm, vias 6 -> 4
- net Net-(C4-Pad1): track 15.7 -> 10.2 mm
- net PA2: track 123.5 -> 119.6 mm
- net +5V: track 172.0 -> 175.5 mm, vias 14 -> 12
- net PC3: track 59.8 -> 56.7 mm, vias 7 -> 8
- net PA7: track 104.4 -> 101.4 mm
- net Net-(U1-EMIT): track 34.1 -> 31.8 mm
- net PB5: track 36.6 -> 34.2 mm
- net UPDI: track 39.7 -> 41.9 mm, vias 8 -> 4
- net PA6: track 108.9 -> 107.1 mm
- net Net-(J1-Pin_2): track 24.4 -> 25.7 mm, vias 4 -> 0
- net PC0: track 12.4 -> 13.6 mm
Other:
- board size 130.5 x 48.5 mm -> 121.1 x 48.5 mm

Commit message: Updated Board and Gerbers
Parts:
- removed R8: 200, Resistor_SMD:R_0805_2012Metric_Pad1.20x1.40mm_HandSolder
- added RV1: 200R, Potentiometer_THT:Potentiometer_Bourns_3296W_Vertical, F.Cu at (84.5, 53.2)
- C11: value 330nf -> 330nF
- C12: value 100nf -> 100nF
- H2: value pinheaders for attiny -> Conn_01x10_MountingPin
- J2: value CAN & Power Supply -> Exit Connector
- R10: value ~ -> Extra
- R14: value 100 Ω -> 100R
- R7, R9: value 120 -> 120R
- U4: value ISO1050DUB -> ISO1050
- Y1: value Crystal -> STDCSU1-8M
- moved R9 1.32 mm to (90.1, 57.2)
Connections:
- C1 pad 2: +5V -> GND
- R3 pad 1: Net-(J1-Pin_2) -> +5V
- R3 pad 2: +5V -> Net-(J1-Pin_2)
Routing:
- net /VrefBG: track 27.2 -> 5.99 mm, vias 4 -> 0
- net Net-(U1-EMIT): track 31.8 -> 13.6 mm, vias 4 -> 0
- net /Vin-: track 11.5 -> 17.3 mm
- net /RG2: track 14.1 -> 9.62 mm
- net +5V: track 175.5 -> 179.2 mm, vias 12 -> 10
- net /Vin+: track 22.2 -> 25.8 mm, vias 4 -> 2
- net Net-(J1-Pin_2): track 25.7 -> 29.2 mm
- net CAN1_RX: track 69.3 -> 71.1 mm
- net PA1: track 88.6 -> 87.2 mm
- net GND: track 55.5 -> 55.2 mm, vias 22 -> 23
Other:
- board text added: "3.5mm diameter"
- board text added: "FS-3 Telemetry Peripheral Board V 2.0 Designed by Ruandy Salazar"
- board text removed: "Designed by Ruandy Salazar"
- board text removed: "FS-3 Telemetry Peripheral Board"
- board text removed: "V 2.0"
