File: TSSI/TSSI.kicad_sch (KiCad schematic)
At the start: 134 parts, among them J1 Conn_01x04_Pin, J2 Conn_01x02_Pin, J3 Conn_01x03_Pin, J4 Conn_01x02_Pin, U2 M74VHC1GT32DFT1G, U3 LM555xN, U4 SN74AHC1G02MDCKREP, U5 LD1086DT50TR

Commit message: TSSI_v2.0 Final Commit
Parts:
- removed CR3: BSS806NEH6327XTSA1, Footprints:PG-SOT23-3-5_INF, symbol 2025-02-02_06-48-36:BSS806NEH6327XTSA1
- added C5: 10nF, Capacitor_SMD:C_0805_2012Metric_Pad1.18x1.45mm_HandSolder, symbol Device:C
- C2: value 10nF -> 100nF
- R4: value 10k -> 10M
Connections:
- net +12V: now also CR5.3; no longer CR5.2
- net +5V: now also C2.1, CR2.3, R4.2, U3.8 (VCC); no longer CR2.2
- net GND: now also CR1.2, CR4.2, C5.1; no longer CR1.3, CR4.3
- net GREEN_LIGHTS: now also CR4.3; no longer CR4.2
- net RED_LIGHTS: now also CR1.3; no longer CR1.2
- net RED_LIGHT_LOGIC: now also U3.4 (R)
- net RTDS_BUZZER: now also CR2.2; no longer CR2.3
- net RTML_12V: now also CR5.2; no longer CR5.3
- net at C1.2, U3.2 (TR), U3.6 (THR): now also R3.1; no longer R4.2
- net at U3.5 (CV): now also C5.2; no longer C2.1
- removed net FLASH_ACTIVE: R3.1, U3.4 (R), U3.8 (VCC)
Other:
- note removed: "Switch 5V to Enable 555"
- moved on the sheet: C1, C2, C3, C4, CR1, CR2, CR4, CR5, J2, J4, R1, R3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

Commit message: TSSI v3.0
Parts:
- removed D10, D11, D12, D34, D35, D36, D4, D40, D41, D42, D5, D6, D64, D65, D66, D70, D71, D72, D76, D77, D78, D82, D83, D84: T1681USD-20C000312U1930, Footprints:T1681NG--20C000112U1930, symbol T1681NG--20C000112U1930:T1681USD-20C000312U1930
- removed D19, D20, D21, D25, D26, D27, D49, D50, D51, D55, D56, D57, D61, D62, D63, D67, D68, D69, D73, D74, D75, D79, D80, D81: T1681NG--20C000112U1930, Footprints:T1681NG--20C000112U1930, symbol T1681NG--20C000112U1930:T1681NG--20C000112U1930
- removed R25, R27, R29, R31: 330, Resistor_SMD:R_0805_2012Metric_Pad1.20x1.40mm_HandSolder, symbol Device:R
- removed R26, R28, R30, R32: 470, Resistor_SMD:R_0805_2012Metric_Pad1.20x1.40mm_HandSolder, symbol Device:R
- removed U2: M74VHC1GT32DFT1G, Footprints:SOT65P210X110-5N, symbol 74xGxx:74AHC1G32
- removed U4: SN74AHC1G02MDCKREP, Footprints:SOT65P210X110-5N, symbol 74xGxx:74AHC1G02
- added D10, D11, D12, D34, D35, D36, D4, D40, D41, D42, D5, D6: T1681NG--20C000112U1930, Footprints:T1681NG--20C000112U1930, symbol T1681NG--20C000112U1930:T1681NG--20C000112U1930
- added D19, D20, D21, D25, D26, D27, D49, D50, D51, D55, D56, D57: T1681USD-20C000312U1930, Footprints:T1681NG--20C000112U1930, symbol T1681NG--20C000112U1930:T1681USD-20C000312U1930
- added U1: SN74AHC1G08DCKR, Footprints:SOT65P210X110-5N, symbol 74xGxx:74AHC1G08
- added U2: SN74AHC1G00DCKR, Footprints:SOT65P210X110-5N, symbol 74xGxx:74AHC1G00
- R11, R13, R21, R23: value 330 -> 470
- R16, R18, R6, R8: value 470 -> 330
Connections:
- net BMS_STATUS: now also U1.1, U2.1
- net GND: now also U1.3 (GND), U2.3 (GND)
- net GREEN_LIGHTS: now also D12.1 (K), D12.2 (K), D12.3 (K), D36.1 (K), D36.2 (K), D36.3 (K), D42.1 (K), D42.2 (K), D42.3 (K), D6.1 (K), D6.2 (K), D6.3 (K)
- net GREEN_LIGHT_LOGIC: now also U1.4
- net IMD_STATUS: now also U1.2, U2.2
- net RED_LIGHTS: now also D21.1 (K), D21.2 (K), D21.3 (K), D27.1 (K), D27.2 (K), D27.3 (K), D51.1 (K), D51.2 (K), D51.3 (K), D57.1 (K), D57.2 (K), D57.3 (K)
- net RED_LIGHT_LOGIC: now also U2.4
- net at R16.2: now also D34.4 (A)
- net at R13.2: now also D25.4 (A)
- net at R2.1: now also U2.5 (VCC)
- net at R6.2: now also D4.4 (A)
- net at R18.2: now also D40.4 (A)
- net at R21.2: now also D49.4 (A)
- net at R23.2: now also D55.4 (A)
- net at R8.2: now also D10.4 (A)
- net at R11.2: now also D19.4 (A)
- net at R1.1: now also U1.5 (VCC)
- new net: D41.1 (K), D41.2 (K), D41.3 (K), D42.4 (A)
- new net: D5.1 (K), D5.2 (K), D5.3 (K), D6.4 (A)
- new net: D26.1 (K), D26.2 (K), D26.3 (K), D27.4 (A)
- new net: D25.1 (K), D25.2 (K), D25.3 (K), D26.4 (A)
- new net: D11.1 (K), D11.2 (K), D11.3 (K), D12.4 (A)
- new net: D10.1 (K), D10.2 (K), D10.3 (K), D11.4 (A)
- new net: D49.1 (K), D49.2 (K), D49.3 (K), D50.4 (A)
- new net: D50.1 (K), D50.2 (K), D50.3 (K), D51.4 (A)
- new net: D4.1 (K), D4.2 (K), D4.3 (K), D5.4 (A)
- new net: D35.1 (K), D35.2 (K), D35.3 (K), D36.4 (A)
- new net: D56.1 (K), D56.2 (K), D56.3 (K), D57.4 (A)
- new net: D19.1 (K), D19.2 (K), D19.3 (K), D20.4 (A)
- new net: D55.1 (K), D55.2 (K), D55.3 (K), D56.4 (A)
- new net: D20.1 (K), D20.2 (K), D20.3 (K), D21.4 (A)
- new net: D34.1 (K), D34.2 (K), D34.3 (K), D35.4 (A)
- new net: D40.1 (K), D40.2 (K), D40.3 (K), D41.4 (A)
Other:
- moved on the sheet: CR1, CR2, CR4, CR5, D1, D2, D3, L1, R5

Commit message: edits from feedback and finalizing TSSI_v3
Parts:
- removed R1, R2: 100, Resistor_SMD:R_0805_2012Metric_Pad1.20x1.40mm_HandSolder, symbol Device:R
- added C6, C7: 100nF, Capacitor_SMD:C_0805_2012Metric_Pad1.18x1.45mm_HandSolder, symbol Device:C
- C1: value 22uF -> 22nF
- L1: footprint CPT_1625_80_SMT_TR:XDCR_CPT-1625-80-SMT-TR -> Footprints:XDCR_CPT-1625-80-SMT-TR
- renumbered CR4 to CR3, CR5 to CR4, U5 to U4
Connections:
- net +12V: now also J2.2 (Pin_2), J4.2 (Pin_2); no longer CR4.3
- net +5V: now also L1.P, U1.5 (VCC), U2.5 (VCC), C6.1, C7.1; no longer CR2.3
- net GND: now also CR2.2, CR4.2, C6.2, C7.2; no longer J2.1 (Pin_1), J4.1 (Pin_1), L1.N
- net RTDS_BUZZER: now also CR2.3, L1.N; no longer CR2.2, L1.P
- net RTML_12V: now also CR4.3, J2.1 (Pin_1), J4.1 (Pin_1); no longer CR4.2, J2.2 (Pin_2), J4.2 (Pin_2)
Other:
- note added: "Switch 5V to Buzzer"
- note removed: "Switch 12V to Buzzer"
- moved on the sheet: CR1, CR2, CR3, CR4, L1, U2

Commit message: TSSI 3.2
Changed buzzer to meet volume requirements, added Gate inrush and pulldown resistors.
Parts:
- added R27, R28, R29, R3, R30, R4, R5, R6: 1k, Resistor_SMD:R_0805_2012Metric_Pad1.20x1.40mm_HandSolder, symbol Device:R
- J1: renamed from J3; value Conn_01x03_Pin -> 1053131103
- J2: renamed from J1; value Conn_01x04_Pin -> 1053131104
- J3: renamed from J4; value Conn_01x02_Pin -> 1053131102
- J4: renamed from J2; value Conn_01x02_Pin -> 1053131102
- L1: value XDCR_CPT-1625-80-SMT-TR -> AI-3035-TT-12V-R; footprint Footprints:XDCR_CPT-1625-80-SMT-TR -> FS_3_Global_Footprint_Library:AI-3035-TT-12V-R; Digikey Part Number 458-1071-ND -> 668-1652-ND; Height 9.7 -> 20; MANUFACTURER CUI Inc. -> PUI Audio, Inc; MAXIMUM_PACKAGE_HEIGHT 2.5mm -> 20mm; Manufacturer Mallory -> PUI Audio, Inc
- renumbered C3 to C2, C5 to C3, C2 to C4, C4 to C5, CR2 to CR1, CR1 to CR2, CR4 to CR3, CR3 to CR4, D34 to D10, D35 to D11, D36 to D12, D7 to D13, D8 to D14, D9 to D15, D37 to D16, D38 to D17, D39 to D18, D10 to D19, D11 to D20, D12 to D21, D40 to D22, D41 to D23, D42 to D24, D13 to D25, D14 to D26, D15 to D27, D43 to D28, D44 to D29, D45 to D30, D16 to D31, D17 to D32, D18 to D33, D46 to D34, D47 to D35, D48 to D36, D19 to D37, D20 to D38, D21 to D39, D31 to D4, D49 to D40, D50 to D41, D51 to D42, D22 to D43, D23 to D44, D24 to D45, D52 to D46, D53 to D47, D54 to D48, D25 to D49, D32 to D5, D26 to D50, D27 to D51, D55 to D52, D56 to D53, D57 to D54, D28 to D55, D29 to D56, D30 to D57, D33 to D6, D4 to D7, D5 to D8, D6 to D9, R4 to R1, R16 to R10, R7 to R11, R17 to R12, R8 to R13, R18 to R14, R9 to R15, R19 to R16, R10 to R17, R20 to R18, R11 to R19, R3 to R2, R21 to R20, R12 to R21, R13 to R23, R23 to R24, R14 to R25, R24 to R26, R5 to R7, R15 to R8, R6 to R9, U3 to U1, U4 to U2, U2 to U3, U1 to U4
Connections:
- net +12V: now also L1.P
- net +5V: no longer L1.P
- net FLASH_LEDS: now also R30.1; no longer CR2.1
- net GND: now also R3.1, R4.1, R5.1, R6.1
- net GREEN_LIGHT_LOGIC: now also R29.1; no longer CR4.1
- net RTDS_SIGNAL: now also R27.1; no longer CR1.1
- net RTML_5V: now also R28.1; no longer CR3.1
- new net: CR2.1, R30.2, R4.2
- new net: CR3.1, R28.2, R5.2
- new net: CR1.1, R27.2, R3.2
- new net: CR4.1, R29.2, R6.2
Other:
- moved on the sheet: CR4
