File: BSPD/BSPD.kicad_sch (KiCad schematic)
At the start: 5 parts, among them J1 Conn_01x08, U1 MCP6004, U2 MCP6004, U3 MCP6004, U4 MCP6004

Commit message: finished V1 of bspd
Parts:
- added C1, C2, C3, C4, C5: 100nF, symbol Device:C
- added R1, R11, R12, R17, R18, R2: 10k, symbol Device:R
- added R13, R14, R19, R20, R23, R24, R25, R28: 100k, symbol Device:R
- added R3, R5: 1k, symbol Device:R
- added R4, R6: 20k, symbol Device:R
- added unit 5 of U1
- added unit 4 of U1
- added unit 3 of U1
- added unit 4 of U2
- added unit 2 of U2
- added unit 5 of U2
- added unit 3 of U2
- added unit 2 of U3
- added unit 4 of U3
- added unit 3 of U3
- added unit 5 of U3
- added unit 2 of U4
- added unit 4 of U4
- added unit 3 of U4
- added unit 5 of U4
- added U5: MCP6004, symbol Amplifier_Operational:MCP6004
Connections:
- net +5V: now also C1.2, C2.2, C3.2, C4.2, C5.2, U1.4 (V+), U2.4 (V+), U3.4 (V+), U4.4 (V+), U5.4 (V+)
- net Current_Sensor_Output: now also U1.10 (+); no longer U3.3 (+)
- net Current_Sensor_Output_Buffered: now also U3.3 (+), R25.2, R3.1, U1.8, U1.9 (-), U2.9 (-); no longer U3.1, U3.2 (-)
- net Current_Sensor_VREF: now also U1.12 (+); no longer U4.3 (+)
- net Current_Sensor_VREF_Buffered: now also R28.2, R5.1, U1.13 (-), U1.14, U2.13 (-), U3.12 (+); no longer U4.1, U4.2 (-)
- net Front_Brake_Buffered: now also R17.1, R24.2, U2.6 (-), U3.5 (+)
- net GND: now also C1.1, C2.1, C3.1, C4.1, C5.1, R13.1, R19.1, R23.1, R24.1, R25.1, R28.1, R4.1, U1.11 (V-), U2.11 (V-), U3.11 (V-), U4.11 (V-), U5.11 (V-)
- net Rear_Brake_Buffered: now also U1.6 (-), U1.7, R11.1, R23.2, U3.10 (+); no longer U2.1
- net Rear_Brake_Sensor: now also U1.5 (+); no longer U2.3 (+)
- net Fault renamed BSPD_Fault
- new net: R17.2, R19.2, U5.3 (+)
- new net: R1.1, R2.2, U5.12 (+)
- new net: R11.2, R13.2, U4.12 (+)
- new net: R5.2, R6.1, U4.9 (-)
- new net: R12.2, R14.1, U4.13 (-)
- new net: R18.2, R20.1, U5.2 (-)
- new net: R3.2, R4.2, U4.10 (+)
- new net 0.5V: R12.1, R18.1
- new net average_brake_output: U4.5 (+), U5.13 (-), U5.14
- new net current_VREF_open: U2.14
- new net current_VREF_short: U3.14
- new net current_sensor_open: U2.8
- new net current_sensor_short: U3.1
- new net differential_current_output: R6.2, U4.3 (+), U4.8
- new net differential_front_brake_output: R20.2, U5.1, U5.5 (+)
- new net differential_front_buffered: R1.2, U5.6 (-), U5.7
- new net differential_rear_brake_output: R14.2, U4.14, U5.10 (+)
- new net differential_rear_buffered: R2.1, U5.8, U5.9 (-)
- new net front_brake_open: U2.7
- new net front_brake_short: U3.7
- new net hard_braking: U4.7
- new net hard_braking_threshhold: U4.6 (-)
- new net high_current: U4.1
- new net high_current_threshold: U4.2 (-)
- new net open_circuit_threshhold: U2.10 (+), U2.12 (+), U2.3 (+), U2.5 (+)
- new net rear_brake_open: U2.1
- new net rear_brake_short: U3.8
- new net short_circuit_threshhold: U3.13 (-), U3.2 (-), U3.6 (-), U3.9 (-)
Other:
- added sheet Voltage_Dividers (voltage_dividers.kicad_sch)
- added sheet logic (bspd_logic.kicad_sch)
- added sheet status_lights (status_lights.kicad_sch)
- note added: "Buffers"
- note added: "Differential Amplifiers"
- note added: "Hard braking and high current"
- note added: "Op-amp Power"
- note added: "Opens"
- note added: "Shorts"
- note added: "average between rear and front brake outputs"
- moved on the sheet: J1

Commit message: Finished BSPD
Parts:
- removed J1: Conn_01x08, Connector_Molex:Molex_Nano-Fit_105313-xx08_1x08_P2.50mm_Horizontal, symbol Connector_Generic:Conn_01x08
- removed R1, R11, R12, R17, R18, R2: 10k, symbol Device:R
- removed R13, R14, R19, R20: 100k, symbol Device:R
- removed unit 4 of U4
- removed unit 4 of U5
- removed unit 3 of U5
- added C12: 0.33µF, Capacitor_SMD:C_0805_2012Metric_Pad1.18x1.45mm_HandSolder, symbol Device:C
- added C13: 0.1µF, Capacitor_SMD:C_0805_2012Metric_Pad1.18x1.45mm_HandSolder, symbol Device:C
- added J2: Conn_01x12, Connector_Molex:Molex_Nano-Fit_105310-xx12_2x06_P2.50mm_Vertical, symbol Connector_Generic:Conn_01x12
- added RV1, RV2: 3296W_10K, Potentiometer_THT:Potentiometer_Bourns_3296W_Vertical, symbol Device:R_Potentiometer
- added U7: LD1086DT50TR, Package_TO_SOT_SMD:TO-252-2, symbol Regulator_Linear:LD1086DT50TR
- added U8: MCP6004, Package_SO:SOIC-14_3.9x8.7mm_P1.27mm, symbol Amplifier_Operational:MCP6004
- C1, C2, C3, C4, C5: value 100nF -> 0.1μF; footprint (none) -> Capacitor_SMD:C_0805_2012Metric_Pad1.18x1.45mm_HandSolder; Digikey Link (none) -> https://www.digikey.com/en/products/detail/yageo/CC0805KRX7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; Part Name (none) -> Capacitor
- R23, R24, R25, R28, R3, R4, R5, R6: footprint (none) -> Resistor_SMD:R_0805_2012Metric_Pad1.20x1.40mm_HandSolder; Digikey Link (none) -> https://www.digikey.com/en/products/detail/yageo/RC0805FR-0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; Part Name (none) -> Resistor
- U1, U2, U3, U4, U5: footprint (none) -> Package_SO:SOIC-14_3.9x8.7mm_P1.27mm; Digikey Link (none) -> https://www.digikey.com/en/products/detail/microchip-techno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; Part Name (none) -> OPAMP
Connections:
- net average_brake_output is gone; now on net differential_front_brake_output: U4.5 (+)
- net +5V: now also C13.2, U7.2 (OUT)
- net Current_Sensor_Output: now also U1.12 (+), J2.5 (Pin_5); no longer U1.10 (+)
- net Current_Sensor_Output_Buffered: now also R28.2, U1.13 (-), U1.14, U2.13 (-); no longer R25.2, U1.8, U1.9 (-), U2.9 (-)
- net Current_Sensor_VREF: now also U1.10 (+), J2.6 (Pin_6); no longer U1.12 (+)
- net Current_Sensor_VREF_Buffered: now also R25.2, U1.8, U1.9 (-), U2.9 (-), U3.5 (+); no longer R28.2, U1.13 (-), U1.14, U2.13 (-), U3.12 (+)
- net Front_Brake_Buffered: now also U1.6 (-), U1.7, U3.10 (+), U5.3 (+); no longer U1.1, U1.2 (-), U3.5 (+)
- net Front_Brake_Sensor: now also U1.5 (+), J2.4 (Pin_4); no longer U1.3 (+)
- net GND: now also C12.1, C13.1, J2.2 (Pin_2), RV1.1, RV2.1, U7.1 (ADJ/GND)
- net Rear_Brake_Buffered: now also U1.1, U1.2 (-), U3.12 (+), U8.3 (+); no longer U1.6 (-), U1.7, U3.10 (+)
- net Rear_Brake_Sensor: now also U1.3 (+), J2.3 (Pin_3); no longer U1.5 (+)
- net current_VREF_open: now also U2.8; no longer U2.14
- net current_VREF_short: now also U3.7; no longer U3.14
- net current_sensor_open: now also U2.14; no longer U2.8
- net differential_front_brake_output: now also RV2.3; no longer U5.5 (+)
- net differential_rear_brake_output: now also U5.5 (+), RV1.3, U8.1
- net front_brake_short: now also U3.8; no longer U3.7
- net rear_brake_short: now also U3.14; no longer U3.8
- net at U5.2 (-): now also RV2.2
- net differential_front_buffered renamed rear_braking_threshhold
- net rear_braking_threshhold: no longer U5.7
- net hard_braking renamed front_hard_braking
- net hard_braking_threshhold renamed front_braking_threshhold
- net high_current_threshold renamed high_current_threshhold
- new net: RV1.2, U8.2 (-)
- new net +12V: C12.2, J2.1 (Pin_1), U7.3 (IN)
- new net BSPD_Fault_LOW: J2.9 (Pin_9)
- new net Shutdown_In: J2.7 (Pin_7)
- new net Shutdown_Out: J2.8 (Pin_8)
- new net rear_hard_braking: U5.7
Other:
- added sheet BSPD_timer (BSPD_timer.kicad_sch)
- sheet Voltage_Dividers ports: added front_braking_threshhold, high_current_threshhold, rear_braking_threshhold; removed 0.5V, current_threshhold, hard_braking_threshhold
- sheet logic ports: added BSPD_Fault_HIGH, current_sensor_open, current_sensor_short, front_hard_braking, rear_hard_braking; removed BSPD_Fault, current_sensor_output_open, current_sensor_output_short, hard_braking
- sheet status_lights ports: added BSPD_Fault_LOW, front_hard_braking, high_current, rear_hard_braking; removed none
- note added: "Amplifiers"
- note added: "linear regulator"
- note removed: "Differential Amplifiers"
- note removed: "average between rear and front brake outputs"
- moved on the sheet: U2A, U3A, U3B, U3C, U3D, U5A

Commit message: all BSPD changes
Parts:
- removed RV1, RV2: 3296W_10K, Potentiometer_THT:Potentiometer_Bourns_3296W_Vertical, symbol Device:R_Potentiometer
- added C11: 0.1μF, Capacitor_SMD:C_0805_2012Metric_Pad1.18x1.45mm_HandSolder, symbol Device:C
- added R19, R20, R21, R22: 10k, Resistor_SMD:R_0805_2012Metric_Pad1.20x1.40mm_HandSolder, symbol Device:R
- added unit 5 of U8
Connections:
- net +5V: now also C11.2, U8.4 (V+)
- net GND: now also C11.1, R19.1, R21.1, U8.11 (V-)
- net at U5.2 (-): now also R21.2, R22.1
- net at U8.2 (-): now also R19.2, R20.1
- net differential_front_brake_output renamed non_inv_front_brake_output
- net non_inv_front_brake_output: now also R22.2
- net differential_rear_brake_output renamed non_inv_rear_brake_output
- net non_inv_rear_brake_output: now also R20.2
- no-connect marks 0 -> 3
Other:
- sheet status_lights ports: added BSPD_Fault_HIGH; removed BSPD_Fault_LOW
- note added: "1.0.0"
- note added: "1/15/2025"
- note added: "FS-3 BSPD"
- moved on the sheet: U5A, U8A
