File: BSPD/bspd_logic.kicad_sch (KiCad schematic)
At the start: 4 parts, among them U6 4072, U7 4081

Commit message: Finished BSPD
Parts:
- removed U7: 4081, symbol 4xxx:4081
- added C10: 0.1μF, Capacitor_SMD:C_0805_2012Metric_Pad1.18x1.45mm_HandSolder, symbol Device:C
- added U10: 4072, Package_SO:SOIC-14_3.9x8.7mm_P1.27mm, symbol 4xxx:4072
- added U9: 74HC00, Package_SO:SOIC-14_3.9x8.7mm_P1.27mm, symbol 74xx:74HC00
- C6, C7: value 100nF -> 0.1μF; footprint (none) -> Capacitor_SMD:C_0805_2012Metric_Pad1.18x1.45mm_HandSolder; Digikey Link (none) -> https://www.digikey.com/en/products/detail/yageo/CC0805KRX7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; Part Name (none) -> Capacitor
- U6: footprint (none) -> Package_SO:SOIC-14_3.9x8.7mm_P1.27mm; Digikey Link (none) -> https://www.digikey.com/en/products/detail/texas-instrument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; Part Name (none) -> OR Gate
Connections:
- net +5V: now also C10.2, U10.14 (VDD), U9.14 (VCC)
- net GND: now also C10.1, U10.12, U10.4, U10.5, U10.7 (VSS), U9.7 (GND)
- net current_VREF_open: now also U6.10
- net current_VREF_short: now also U6.9
- net hard_braking: now also U10.1, U9.1
- net high_current: now also U9.2
- net brake_opens_shorts: now reaches U6.1
- net brake_opens_shorts: now also U10.10; no longer U6.10
- net BSPD_Fault renamed current_opens_shorts
- net current_opens_shorts: now also U10.11
- net current_sensor_output_open renamed current_sensor_open
- net current_sensor_output_short renamed current_sensor_short
- new net: U9.12, U9.13, U9.3
- new net BSPD_Fault_HIGH: U10.13
- new net front_hard_braking: U10.2
- new net hard_braking_high_current: U10.9, U9.11
- new net rear_hard_braking: U10.3
- no-connect marks 9 -> 3
Other:
- note added: "Extra NAND gate"
- note added: "NAND gate power supply"
- note removed: "AND gate power supply"
- note removed: "Extra AND gates"
- moved on the sheet: C7, U6A, U6B, U6C

Commit message: all BSPD changes
Changed lines of the file:
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@@
+	(wire
+		(pts
+			(xy 44.45 17.78) (xy 74.93 17.78)
+		)
+		(stroke
+			(width 0)
+			(type default)
+		)
+	)
 	(wire
 		(pts
@@
 		(pts
 			(xy 228.6 26.67) (xy 231.14 26.67)
-		)
-		(stroke
-			(width 0)
-			(type default)
-		)
-	)
-	(wire
-		(pts
-			(xy 44.45 17.78) (xy 74.93 17.78)
 		)
 		(stroke
@@
 		)
 	)
+	(label "front_hard_braking"
+		(at 74.93 17.78 180)
+		(fields_autoplaced yes)
+		(effects
+			(font
+				(size 1.27 1.27)
+			)
+			(justify right bottom)
+		)
+	)
 	(label "current_opens_shorts"
 		(at 132.08 96.52 0)
@@
 		)
 	)
-	(label "front_hard_braking"
-		(at 74.93 17.78 180)
-		(fields_autoplaced yes)
-		(effects
-			(font
-				(size 1.27 1.27)
-				(thickness 0.1588)
-			)
-			(justify right bottom)
-		)
-	)
