File: BSPD/voltage_dividers.kicad_sch (KiCad schematic)
At the start: 10 parts

Commit message: Finished BSPD
Parts:
- removed R29: 12k, symbol Device:R
- removed R30: 82k, symbol Device:R
- removed R31: 330k, symbol Device:R
- removed R32: 22k, symbol Device:R
- removed R33: 3.9k, symbol Device:R
- removed R34: 15k, symbol Device:R
- removed R35: 18k, symbol Device:R
- removed R36: 39k, symbol Device:R
- removed R37: 1.2k, symbol Device:R
- removed R38: 33k, symbol Device:R
- added RV3, RV4, RV5, RV6, RV7: 3296W_10K, Potentiometer_THT:Potentiometer_Bourns_3296W_Vertical, symbol Device:R_Potentiometer
Connections:
- net +5V: now also RV3.1, RV4.1, RV5.1, RV6.1, RV7.1
- net GND: now also RV3.3, RV4.3, RV5.3, RV6.3, RV7.3
- net open_circuit_threshhold: now also RV5.2
- net short_circuit_threshhold: now also RV6.2
- new net front_braking_threshhold: RV3.2
- new net high_current_threshhold: RV4.2
- new net rear_braking_threshhold: RV7.2
Other:
- note removed: "exact value: 0.528V"
- note removed: "ideally: 0.5V"
- note removed: "use in comparison to brake sensors in diff amps"

Commit message: all BSPD changes
Parts:
- removed RV4, RV5, RV6: 3296W_10K, Potentiometer_THT:Potentiometer_Bourns_3296W_Vertical, symbol Device:R_Potentiometer
- added R11: 3.9k, Resistor_SMD:R_0805_2012Metric_Pad1.20x1.40mm_HandSolder, symbol Device:R
- added R12: 33k, Resistor_SMD:R_0805_2012Metric_Pad1.20x1.40mm_HandSolder, symbol Device:R
- added R13: 22k, Resistor_SMD:R_0805_2012Metric_Pad1.20x1.40mm_HandSolder, symbol Device:R
- added R14: 1.2k, Resistor_SMD:R_0805_2012Metric_Pad1.20x1.40mm_HandSolder, symbol Device:R
- added R15: 12k, Resistor_SMD:R_0805_2012Metric_Pad1.20x1.40mm_HandSolder, symbol Device:R
- added R16: 15k, Resistor_SMD:R_0805_2012Metric_Pad1.20x1.40mm_HandSolder, symbol Device:R
- added TP1: rear_braking_threshold, Connector_PinHeader_2.54mm:PinHeader_1x01_P2.54mm_Vertical, symbol Connector:TestPoint
- added TP2: front_braking_threshold, Connector_PinHeader_2.54mm:PinHeader_1x01_P2.54mm_Vertical, symbol Connector:TestPoint
- renumbered RV3 to RV1, RV7 to RV2
Connections:
- net +5V: now also R11.2, R13.2, R15.2
- net GND: now also R12.1, R14.1, R16.1
- net front_braking_threshhold: now also TP2.1
- net high_current_threshhold: now also R15.1, R16.2
- net open_circuit_threshhold: now also R13.1, R14.2
- net rear_braking_threshhold: now also TP1.1
- net short_circuit_threshhold: now also R11.1, R12.2
Other:
- note added: "Set to 1.5V"
- note added: "Set to 2.0V"
- note removed: "exact value: 0.9V"
- note removed: "ideally 0.9V"
- note removed: "threshhold for short circuit"
- moved on the sheet: RV1, RV2
