File: BMS/BMS.kicad_sch (KiCad schematic)
At the start: 55 parts, among them J1 Conn_01x02_Pin, J2 IsoSPI, J3 IsoSPI, Q1 NSV1C201MZ4, SW2 A6H-4101, U2 ADG708, U3 LTC6811IG-2-TRPBF

Commit message: fixed voltage drop issue with parallel fuses
Parts:
- R1: value 10 -> 100
Connections:
- net V-: now also C1.2, C3.2, F9.1; no longer F1.1, R3.2
- new net BB0/B#: F1.1, R3.2
Other:
- note added: "Unkown if R1 10 or 100 ohms, inconsistent in datasheet"
- moved on the sheet: C1, C2, R3

Commit message: Updated fuse values to contain part numbers
Other:
- note added: "Little Fuse LF110•33"
Changed lines of the file:
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@@
 	(wire
 		(pts
-			(xy 104.14 67.31) (xy 104.14 66.04)
+			(xy 105.41 66.04) (xy 105.41 91.44)
 		)
 		(stroke
@@
 	(wire
 		(pts
-			(xy 104.14 66.04) (xy 83.82 66.04)
+			(xy 105.41 66.04) (xy 83.82 66.04)
 		)
 		(stroke
@@
 	(wire
 		(pts
-			(xy 105.41 67.31) (xy 105.41 91.44)
-		)
-		(stroke
-			(width 0)
-			(type default)
-		)
-	)
-	(wire
-		(pts
 			(xy 289.56 116.84) (xy 289.56 121.92)
 		)
@@
 		(pts
 			(xy 170.18 116.84) (xy 175.26 116.84)
-		)
-		(stroke
-			(width 0)
-			(type default)
-		)
-	)
-	(wire
-		(pts
-			(xy 104.14 67.31) (xy 105.41 67.31)
 		)
 		(stroke
@@
 		)
 	)
+	(text "Little Fuse LF110•33"
+		(exclude_from_sim no)
+		(at 80.264 56.896 0)
+		(effects
+			(font
+				(size 1.27 1.27)
+			)
+		)
+	)
