File: BMS/BMS.kicad_pcb (KiCad board)
At the start: 2 copper layers, 57.4 x 171.2 mm, 98 parts, among them J1 Conn_01x02_Pin, J2 IsoSPI, J3 IsoSPI, Q1 NSV1C201MZ4, Q3 BSS308PE, Q4 BSS308PE, Q5 BSS308PE, Q6 BSS308PE, Q7 BSS308PE, Q8 BSS308PE, SW2 A6H-4101, U2 ADG708, U3 LTC6811IG-2-TRPBF

Commit message: moved pos fuse
Parts:
- moved F9 10.2 mm to (50.0, 43.4), turned to 180 degrees
- moved F1 1.58 mm to (50.0, 38.8), turned to 180 degrees
- moved C1 0.50 mm to (52.4, 47.5)
- moved C3 0.50 mm to (50.4, 47.5)
Routing:
- net V-: track 48.9 -> 38.7 mm, vias 12 -> 11
- net Net-(J1-Pin_2): track 23.9 -> 18.2 mm
- net VREG: track 121.3 -> 120.4 mm
- net Net-(C1-Pad1): track 23.7 -> 23.2 mm

Commit message: Minor silkscreen cleanup
Parts:
- moved G*** 2.79 mm to (43.9, 186.5)
Other:
- board text added: "BMS Board V${REVISION} ${COMPANY} FS-3 Designed by Lucas Balbuena, Abhi Chaubey"
- board text removed: "FS-3 BMS Board Formula Slug v2.1 Designed by Lucas Balbuena, Abhi Chaubey Schematic by Abhi Chaubey,"
Changed lines of the file:
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@@
 	(title_block
 		(title "FS-3 Battery Management System Bank Board")
-		(date "2024-10-27")
-		(rev "v1.4")
+		(date "2025-05-02")
+		(rev "3.1")
+		(company "Formula Slug")
 	)
 	(layers
@@
 		(tags "capacitor handsolder")
 		(property "Reference" "C3"
-			(at 0.01 -1.61 -90)
+			(at -0.76 -1.61 -90)
 			(layer "F.SilkS")
 			(effects
@@
 		(tags "fuse handsolder")
 		(property "Reference" "F9"
-			(at 0 -2.65 360)
+			(at 1.74 -2.65 0)
 			(layer "F.SilkS")
 			(effects
@@
 		)
 		(property "Value" "Polyfuse"
-			(at 0 2.65 360)
+			(at 0 2.65 0)
 			(layer "F.Fab")
 			(effects
@@
 		)
 		(fp_text user "${REFERENCE}"
-			(at 0 0 360)
+			(at 0 0 0)
 			(layer "F.Fab")
 			(effects
@@
 		(tags "fuse handsolder")
 		(property "Reference" "F1"
-			(at -3.6865 1.648 90)
+			(at -0.165 2.605 180)
 			(layer "F.SilkS")
 			(effects
@@
 		)
 		(property "Value" "Polyfuse"
-			(at 0 2.65 360)
+			(at 0 2.65 0)
 			(layer "F.Fab")
 			(effects
@@
 		)
 		(fp_text user "${REFERENCE}"
-			(at 0 0 360)
+			(at 0 0 0)
 			(layer "F.Fab")
 			(effects
@@
 		(tags "resistor handsolder")
 		(property "Reference" "R45"
-			(at 1.86 -1.51 0)
+			(at 2.445 -0.09 90)
 			(layer "F.SilkS")
 			(effects
@@
 	(footprint "FS_3_Global_Footprint_Library:FORMULA SLUG"
 		(layer "F.Cu")
-		(at 46.64658 186.494544)
+		(at 43.85258 186.494544)
 		(property "Reference" "G***"
 			(at 0 0 0)
@@
 		(tags "resistor handsolder")
 		(property "Reference" "R44"
-			(at -2.35 -1.4 180)
+			(at -1.165 -1.425 -90)
 			(layer "F.SilkS")
 			(effects
@@
 		)
 	)
-	(gr_text "FS-3 BMS Board\nFormula Slug\nv2.1\nDesigned by Lucas Balbuena, Abhi Chaubey\nSchematic by Abhi Chaubey, "
-		(at 45.466 188.976 0)
+	(gr_text "BMS Board V${REVISION}\n${COMPANY}\nFS-3\nDesigned by Lucas Balbuena, Abhi Chaubey"
+		(at 41.91 188.595 0)
 		(layer "F.SilkS")
 		(effects
 			(font
-				(size 0.5 0.5)
+				(size 0.6 0.6)
 				(thickness 0.125)
 				(bold yes)

Commit message: Final BMS PCB Layout
Shifted top right balance block to better fit the new fuses. Shifted bottom layer to remove islands from ground plane. Removed all 90 degree tracks.
Parts:
- moved Q8 3.45 mm to (60.1, 28.7)
- moved D8 3.45 mm to (52.1, 30.2)
- moved R42 3.45 mm to (55.9, 30.2)
- moved R43 3.45 mm to (53.9, 27.2)
- moved R44 1.71 mm to (56.0, 34.7)
- moved F1 1.21 mm to (51.1, 38.3)
- moved F9 1.21 mm to (51.1, 42.9)
- moved R45 0.93 mm to (59.4, 34.8)
- moved C14 0.85 mm to (58.1, 37.8)
- moved C2 0.85 mm to (58.9, 41.8)
- moved R3 0.85 mm to (56.9, 41.8)
- moved R31 0.45 mm to (63.4, 54.1)
- moved R34 0.30 mm to (60.4, 51.6)
- moved D7 0.20 mm to (63.4, 50.1)
Routing:
- net /C3: track 119.1 -> 122.9 mm
- net /BB0/B#+1: track 22.1 -> 24.8 mm
- net /C0: track 47.1 -> 49.3 mm
- net /S1: track 43.4 -> 45.1 mm
- net Net-(Q8-G): track 3.91 -> 5.59 mm
- net /C1: track 53.6 -> 55.0 mm
- net V-: track 38.7 -> 39.9 mm
- net /BB0/B#: track 17.3 -> 18.6 mm
- net Net-(C1-Pad1): track 23.2 -> 24.2 mm
- net /BB3/B#+1: track 52.8 -> 51.8 mm
- net Net-(J1-Pin_2): track 18.2 -> 19.1 mm
