File: ETC/ETC.kicad_sch (KiCad schematic)
At the start: 36 parts, among them P1 DTM1312PC12PDR008, U1 NUCLEO-F446RE, U2 MCP6004, U3 LM7805_TO220, U4 LM7809_TO220, U5 ISO1050DUB, U6 ISO1050DUB, U7 SSM6N37FU_LF

Commit message: add test points
Parts:
- added BSE1, Cockpit1, HE1, HE2, Reverse1: TestPoint, TestPoint:TestPoint_Plated_Hole_D2.0mm, symbol Connector:TestPoint
- U3, U4: footprint Package_TO_SOT_THT:TO-220-3_Vertical -> Package_TO_SOT_THT:TO-220-3_Horizontal_TabUp
Connections:
- net BSE: now also BSE1.1
- net Cockpit_Signal: now also Cockpit1.1
- net HE1: now also HE1.1
- net HE2: now also HE2.1
- net Reverse_Signal: now also Reverse1.1
Other:
- moved on the sheet: C5, C7, R1, R2, R3, R7, R8, R9, U2A, U2C, U2D, U2E

Commit message: remove 12V power for brake/rtds, move capacitors around
Connections:
- net +12V: no longer P1.C4, P1.D8
- no-connect marks 51 -> 53
Other:
- note removed: "Brake"
- note removed: "RTDS"
Changed lines of the file:
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@@
 	)
 	(no_connect
+		(at 66.04 62.23)
+	)
+	(no_connect
 		(at 387.35 135.89)
 	)
@@
 	)
 	(no_connect
+		(at 35.56 36.83)
+	)
+	(no_connect
 		(at 275.59 135.89)
 	)
@@
 	(wire
 		(pts
-			(xy 66.04 52.07) (xy 76.2 52.07)
-		)
-		(stroke
-			(width 0)
-			(type default)
-		)
-	)
-	(wire
-		(pts
 			(xy 111.76 234.95) (xy 124.46 234.95)
 		)
@@
 	(wire
 		(pts
-			(xy 66.04 59.69) (xy 78.74 59.69)
-		)
-		(stroke
-			(width 0)
-			(type default)
-		)
-	)
-	(wire
-		(pts
 			(xy 142.24 54.61) (xy 142.24 57.15)
 		)
@@
 	(wire
 		(pts
+			(xy 66.04 52.07) (xy 77.47 52.07)
+		)
+		(stroke
+			(width 0)
+			(type default)
+		)
+	)
+	(wire
+		(pts
 			(xy 168.91 119.38) (xy 168.91 120.65)
 		)
@@
 	(wire
 		(pts
-			(xy 27.94 57.15) (xy 35.56 57.15)
+			(xy 22.86 57.15) (xy 35.56 57.15)
 		)
 		(stroke
@@
 	(wire
 		(pts
+			(xy 66.04 59.69) (xy 77.47 59.69)
+		)
+		(stroke
+			(width 0)
+			(type default)
+		)
+	)
+	(wire
+		(pts
 			(xy 76.2 118.11) (xy 72.39 118.11)
 		)
@@
 	(wire
 		(pts
-			(xy 27.94 59.69) (xy 35.56 59.69)
+			(xy 22.86 59.69) (xy 35.56 59.69)
 		)
 		(stroke
@@
 		)
 	)
-	(text "RTDS"
-		(exclude_from_sim no)
-		(at 78.994 62.484 0)
-		(effects
-			(font
-				(size 1.27 1.27)
-			)
-		)
-	)
 	(text "CAN Trancievers"
 		(exclude_from_sim no)
@@
 		)
 	)
-	(text "Brake"
-		(exclude_from_sim no)
-		(at 24.892 36.83 0)
-		(effects
-			(font
-				(size 1.27 1.27)
-			)
-		)
-	)
 	(text "Cockpit"
 		(exclude_from_sim no)
@@
 	)
 	(label "L_CAN"
-		(at 27.94 59.69 0)
+		(at 22.86 59.69 0)
 		(fields_autoplaced yes)
 		(effects
@@
 	)
 	(label "H_CAN"
-		(at 27.94 57.15 0)
+		(at 22.86 57.15 0)
 		(fields_autoplaced yes)
 		(effects
@@
 	)
 	(label "RTDS"
-		(at 78.74 59.69 180)
+		(at 77.47 59.69 180)
 		(fields_autoplaced yes)
 		(effects
@@
 	)
 	(label "BSE_RAW"
-		(at 76.2 52.07 180)
+		(at 77.47 52.07 180)
 		(fields_autoplaced yes)
 		(effects
@@
 	)
 	(symbol
-		(lib_id "power:+12V")
-		(at 35.56 36.83 90)
-		(unit 1)
-		(exclude_from_sim no)
-		(in_bom yes)
-		(on_board yes)
-		(dnp no)
-		(fields_autoplaced yes)
-		(property "Reference" "#PWR030"
-			(at 39.37 36.83 0)
-			(effects
-				(font
-					(size 1.27 1.27)
-				)
-				(hide yes)
-			)
-		)
-		(property "Value" "+12V"
-			(at 31.75 36.8299 90)
-			(effects
-				(font
-					(size 1.27 1.27)
-				)
-				(justify left)
-			)
-		)
-		(property "Footprint" ""
-			(at 35.56 36.83 0)
-			(effects
-				(font
-					(size 1.27 1.27)
-				)
-				(hide yes)
-			)
-		)
-		(property "Datasheet" ""
-			(at 35.56 36.83 0)
-			(effects
-				(font
-					(size 1.27 1.27)
-				)
-				(hide yes)
-			)
-		)
-		(property "Description" "Power symbol creates a global label with name \"+12V\""
-			(at 35.56 36.83 0)
-			(effects
-				(font
-					(size 1.27 1.27)
-				)
-				(hide yes)
-			)
-		)
-		(pin "1"
-		)
-		(instances
-			(project "ETC"
-				(path "/61e913ea-868b-4b77-8707-03788b798f2b"
-					(reference "#PWR030")
-					(unit 1)
-				)
-			)
-		)
-	)
-	(symbol
 		(lib_id "power:GND")
 		(at 233.68 162.56 0)
@@
 	)
 	(symbol
-		(lib_id "power:+12V")
-		(at 66.04 62.23 270)
-		(unit 1)
-		(exclude_from_sim no)
-		(in_bom yes)
-		(on_board yes)
-		(dnp no)
-		(fields_autoplaced yes)
-		(property "Reference" "#PWR04"
-			(at 62.23 62.23 0)
-			(effects
-				(font
-					(size 1.27 1.27)
-				)
-				(hide yes)
-			)
-		)
-		(property "Value" "+12V"
-			(at 69.85 62.2299 90)
-			(effects
-				(font
-					(size 1.27 1.27)
-				)
-				(justify left)
-			)
-		)
-		(property "Footprint" ""
-			(at 66.04 62.23 0)
-			(effects
-				(font
-					(size 1.27 1.27)
-				)
-				(hide yes)
-			)
-		)
-		(property "Datasheet" ""
-			(at 66.04 62.23 0)
-			(effects
-				(font
-					(size 1.27 1.27)
-				)
-				(hide yes)
-			)
-		)
-		(property "Description" "Power symbol creates a global label with name \"+12V\""
-			(at 66.04 62.23 0)
-			(effects
-				(font
-					(size 1.27 1.27)
-				)
-				(hide yes)
-			)
-		)
-		(pin "1"
-		)
-		(instances
-			(project "ETC"
-				(path "/61e913ea-868b-4b77-8707-03788b798f2b"
-					(reference "#PWR04")
-					(unit 1)
-				)
-			)
-		)
-	)
-	(symbol
 		(lib_id "Device:R")
 		(at 168.91 124.46 0)
@@
 		(on_board yes)
 		(dnp no)
-		(fields_autoplaced yes)
 		(property "Reference" "#PWR026"
 			(at 62.23 55.88 0)

Commit message: add additional decoupling caps
Parts:
- added C16, C8, C9: 100 nF, Capacitor_SMD:C_0805_2012Metric_Pad1.18x1.45mm_HandSolder, symbol Device:C
- U2: footprint FS_3_Global_Footprint_Library:N14 -> Package_SO:SOIC-14_3.9x8.7mm_P1.27mm
Connections:
- net +3V3: now also C9.1
- net +5V: now also C8.1
- net +9V: now also C16.1
- net GND: now also C16.2, C8.2, C9.2
Other:
- moved on the sheet: U2D, U2E

Commit message: connect rtds signal to dtm connector
Parts:
- removed U7: SSM6N37FU_LF, Package_TO_SOT_SMD:SOT-363_SC-70-6_Handsoldering, symbol FS_3_Global_Symbol_Library:SSM6N37FU_LF
Connections:
- net RTDS is gone; now on net RTDS_Signal: P1.D9
- net Brake_light: no longer names the net of P1.C3
- no-connect marks 53 -> 54
Other:
- note removed: "Brake Light and RTDS Switching"

Commit message: add mosfet for brake light
Parts:
- added CR1: STS6NF20V, Package_SO:PowerIntegrations_SO-8, symbol FS_3_Global_Symbol_Library:STS6NF20V
- added R10: 1k, Resistor_SMD:R_0805_2012Metric_Pad1.20x1.40mm_HandSolder, symbol Device:R
Connections:
- net Brake_Signal: now also R10.1
- net GND: now also CR1.1 (S), CR1.2 (S), CR1.3 (S)
- net Brake_Light_In: now reaches P1.D8
- net Brake_Light_In: now also CR1.5 (D), CR1.6 (D), CR1.7 (D), CR1.8 (D)
- new net: CR1.4 (G), R10.2
- no-connect marks 54 -> 53
Other:
- note added: "Brake Light MOSFET"

Commit message: no can transciever, switch to L432KC
Parts:
- removed C10, C11: 100nF, Capacitor_SMD:C_0805_2012Metric_Pad1.18x1.45mm_HandSolder, symbol Device:C
- removed R14: 120Ω, Resistor_SMD:R_0805_2012Metric_Pad1.20x1.40mm_HandSolder, symbol Device:R
- removed U1: NUCLEO-F446RE, FS_3_Global_Footprint_Library:NUCLEO-F446RE, symbol FS_3_Global_Symbol_Library:NUCLEO-F446RE
- removed U5: ISO1050DUB, Package_SO:SOP-8_6.62x9.15mm_P2.54mm, symbol Interface_CAN_LIN:ISO1050DUB
- added CN1: NUCLEO-L432KC, FS_3_Global_Footprint_Library:NUCLEO-L432KC, symbol FS_3_Global_Symbol_Library:NUCLEO-L432KC
Connections:
- net +3V3: now also CN1.CN4_14 (3V3)
- net +9V: now also CN1.CN4_1 (VIN)
- net BSE: now also CN1.CN4_8 (PA5)
- net Brake_Signal: now also CN1.CN3_8 (PB6)
- net CAN_RD: now also CN1.CN3_13 (PA11)
- net CAN_TD: now also CN1.CN3_5 (PA12)
- net Cockpit_Signal: now also CN1.CN3_6 (PB0)
- net GND: now also CN1.CN4_2 (GND)
- net HE1: now also CN1.CN4_6 (PA7)
- net HE2: now also CN1.CN4_7 (PA6)
- net RTDS_Signal: now also CN1.CN3_7 (PB7)
- net Reverse_Signal: now also CN1.CN3_9 (PB1)
- net H_Motor_CAN: no longer names the net of P1.D1
- net L_Motor_CAN: no longer names the net of P1.D2
- no-connect marks 53 -> 25
Other:
- note added: "CAN Tranciever"
- note removed: "CAN Trancievers"
- moved on the sheet: C12, C13, C16, C9, R15, U6

Commit message: Revision 3.1 nanofit headers
Parts:
- removed P1: DTM1312PC12PDR008, FS_3_Global_Footprint_Library:TE_DTM1312PC12PDR008, symbol FS_3_Global_Symbol_Library:DTM1312PC12PDR008
- added J1: 1053101212, Connector_Molex:Molex_Nano-Fit_105310-xx12_2x06_P2.50mm_Vertical, symbol FS_Symbols:1053101212
- added J2: 1053101206, Connector_Molex:Molex_Nano-Fit_105310-xx06_2x03_P2.50mm_Vertical, symbol FS_Symbols:1053101206
Connections:
- net +12V: now also J1.5
- net +3V3: now also J1.9
- net +5V: now also J2.3, J2.4
- net BSE_RAW: now also J1.11
- net Brake_Light_In: now also J1.7
- net Cockpit_Raw: now also J1.10
- net GND: now also J1.2, J1.6, J2.5, J2.6
- net HE1_RAW: now also J2.2
- net HE2_RAW: now also J2.1
- net H_CAN: now also J1.3
- net L_CAN: now also J1.4
- net RTDS_Signal: now also J1.8
- net Reverse_Raw: now also J1.1
- no-connect marks 25 -> 19
Other:
- note added: "Nanofit header"
- note removed: "DTM Connector"
- moved on the sheet: BSE1, C1, C12, C13, C14, C15, C16, C2, C3, C4, C5, C6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

Commit message: revision 3.2: Semantic changes, added brake_switch pull down resistor, moved mosfet closer to nanofits, moved lin reg capacitors out from under, switched test point footprints to PinHeader_1x01_P2.54mm_Vertical
Parts:
- added R11: 1k, Resistor_SMD:R_0805_2012Metric_Pad1.20x1.40mm_HandSolder, symbol Device:R
- BSE1, HE1, HE2, Reverse1: footprint TestPoint:TestPoint_Plated_Hole_D2.0mm -> Connector_PinHeader_2.54mm:PinHeader_1x01_P2.54mm_Vertical
- CN1: footprint FS_3_Global_Footprint_Library:NUCLEO-L432KC -> FS_Footprints:NUCLEO-L432KC
- Cockpit1: footprint TestPoint:TestPoint_Plated_Hole_D2.0mm -> Connector_PinHeader_2.54mm:PinHeader_1x01_P2.54mm_Vertical; now left out of the parts list
Connections:
- net GND: now also R11.1
- net Brake_Light_In renamed Brake_Light
- net Brake_Signal renamed Brake_Switch
- net Brake_Switch: now also R11.2
- net RTDS_Signal renamed RTDS_Switch
Other:
- note added: "Brake System Encoder"
- note added: "Hall Effect 1"
- note added: "Hall Effect 2"
Changed lines of the file:
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@@
 		(title "ETC")
 		(date "2025-03-25")
-		(rev "3.1")
+		(rev "3.2")
 		(company "Dustin Wang - Formula Slug")
 	)
@@
 		)
 	)
+	(text "Hall Effect 1"
+		(exclude_from_sim no)
+		(at 59.182 22.098 0)
+		(effects
+			(font
+				(size 1.27 1.27)
+			)
+		)
+	)
+	(text "Hall Effect 2"
+		(exclude_from_sim no)
+		(at 58.928 24.638 0)
+		(effects
+			(font
+				(size 1.27 1.27)
+			)
+		)
+	)
 	(text "Brake Light MOSFET"
 		(exclude_from_sim no)
@@
 		)
 	)
+	(text "Brake System Encoder"
+		(exclude_from_sim no)
+		(at 22.352 47.752 0)
+		(effects
+			(font
+				(size 0.508 0.508)
+			)
+		)
+	)
 	(text "Reverse"
 		(exclude_from_sim no)
@@
 	)
 	(junction
+		(at 39.37 198.12)
+		(diameter 0)
+		(color 0 0 0 0)
+	)
+	(junction
 		(at 250.19 118.11)
 		(diameter 0)
@@
 	(wire
 		(pts
+			(xy 39.37 198.12) (xy 41.91 198.12)
+		)
+		(stroke
+			(width 0)
+			(type default)
+		)
+	)
+	(wire
+		(pts
 			(xy 196.85 116.84) (xy 196.85 119.38)
 		)
@@
 	(wire
 		(pts
-			(xy 27.94 198.12) (xy 41.91 198.12)
+			(xy 27.94 198.12) (xy 39.37 198.12)
 		)
 		(stroke
@@
 		)
 	)
-	(label "Brake_Signal"
+	(label "Brake_Switch"
 		(at 292.1 129.54 0)
 		(effects
@@
 		)
 	)
-	(label "RTDS_Signal"
+	(label "RTDS_Switch"
 		(at 292.1 127 0)
 		(effects
@@
 		)
 	)
-	(label "Brake_Light_In"
+	(label "Brake_Light"
 		(at 105.41 190.5 180)
 		(effects
@@
 		)
 	)
-	(label "Brake_Signal"
+	(label "Brake_Switch"
 		(at 27.94 198.12 0)
 		(effects
@@
 		)
 	)
-	(label "RTDS_Signal"
+	(label "RTDS_Switch"
 		(at 26.67 40.64 0)
 		(effects
@@
 		)
 	)
-	(label "Brake_Light_In"
+	(label "Brake_Light"
 		(at 22.86 38.1 0)
 		(effects
@@
 			)
 		)
-		(property "Footprint" "TestPoint:TestPoint_Plated_Hole_D2.0mm"
+		(property "Footprint" "Connector_PinHeader_2.54mm:PinHeader_1x01_P2.54mm_Vertical"
 			(at 356.87 49.53 0)
 			(effects
@@
 			)
 		)
-		(property "Footprint" "TestPoint:TestPoint_Plated_Hole_D2.0mm"
+		(property "Footprint" "Connector_PinHeader_2.54mm:PinHeader_1x01_P2.54mm_Vertical"
 			(at 201.93 116.84 0)
 			(effects
@@
 		(unit 1)
 		(exclude_from_sim no)
-		(in_bom yes)
+		(in_bom no)
 		(on_board yes)
 		(dnp no)
@@
 			)
 		)
-		(property "Footprint" "TestPoint:TestPoint_Plated_Hole_D2.0mm"
+		(property "Footprint" "Connector_PinHeader_2.54mm:PinHeader_1x01_P2.54mm_Vertical"
 			(at 298.45 49.53 0)
 			(effects
@@
 			)
 		)
-		(property "Footprint" "TestPoint:TestPoint_Plated_Hole_D2.0mm"
+		(property "Footprint" "Connector_PinHeader_2.54mm:PinHeader_1x01_P2.54mm_Vertical"
 			(at 201.93 149.86 0)
 			(effects
@@
 	(symbol
 		(lib_id "power:GND")
+		(at 39.37 205.74 0)
+		(unit 1)
+		(exclude_from_sim no)
+		(in_bom yes)
+		(on_board yes)
+		(dnp no)
+		(fields_autoplaced yes)
+		(property "Reference" "#PWR031"
+			(at 39.37 212.09 0)
+			(effects
+				(font
+					(size 1.27 1.27)
+				)
+				(hide yes)
+			)
+		)
+		(property "Value" "GND"
+			(at 39.37 210.82 0)
+			(effects
+				(font
+					(size 1.27 1.27)
+				)
+			)
+		)
+		(property "Footprint" ""
+			(at 39.37 205.74 0)
+			(effects
+				(font
+					(size 1.27 1.27)
+				)
+				(hide yes)
+			)
+		)
+		(property "Datasheet" ""
+			(at 39.37 205.74 0)
+			(effects
+				(font
+					(size 1.27 1.27)
+				)
+				(hide yes)
+			)
+		)
+		(property "Description" "Power symbol creates a global label with name \"GND\" , ground"
+			(at 39.37 205.74 0)
+			(effects
+				(font
+					(size 1.27 1.27)
+				)
+				(hide yes)
+			)
+		)
+		(pin "1"
+		)
+		(instances
+			(project "ETC"
+				(path "/61e913ea-868b-4b77-8707-03788b798f2b"
+					(reference "#PWR031")
+					(unit 1)
+				)
+			)
+		)
+	)
+	(symbol
+		(lib_id "Device:R")
+		(at 39.37 201.93 180)
+		(unit 1)
+		(exclude_from_sim no)
+		(in_bom yes)
+		(on_board yes)
+		(dnp no)
+		(fields_autoplaced yes)
+		(property "Reference" "R11"
+			(at 41.91 200.6599 0)
+			(effects
+				(font
+					(size 1.27 1.27)
+				)
+				(justify right)
+			)
+		)
+		(property "Value" "1k"
+			(at 41.91 203.1999 0)
+			(effects
+				(font
+					(size 1.27 1.27)
+				)
+				(justify right)
+			)
+		)
+		(property "Footprint" "Resistor_SMD:R_0805_2012Metric_Pad1.20x1.40mm_HandSolder"
+			(at 41.148 201.93 90)
+			(effects
+				(font
+					(size 1.27 1.27)
+				)
+				(hide yes)
+			)
+		)
+		(property "Datasheet" "~"
+			(at 39.37 201.93 0)
+			(effects
+				(font
+					(size 1.27 1.27)
+				)
+				(hide yes)
+			)
+		)
+		(property "Description" "Resistor"
+			(at 39.37 201.93 0)
+			(effects
+				(font
+					(size 1.27 1.27)
+				)
+				(hide yes)
+			)
+		)
+		(pin "2"
+		)
+		(pin "1"
+		)
+		(instances
+			(project "ETC"
+				(path "/61e913ea-868b-4b77-8707-03788b798f2b"
+					(reference "R11")
+					(unit 1)
+				)
+			)
+		)
+	)
+	(symbol
+		(lib_id "power:GND")
 		(at 38.1 25.4 270)
 		(unit 1)
@@
 			)
 		)
-		(property "Footprint" "FS_3_Global_Footprint_Library:NUCLEO-L432KC"
+		(property "Footprint" "FS_Footprints:NUCLEO-L432KC"
 			(at 276.86 121.92 0)
 			(effects
@@
 			)
 		)
-		(property "Footprint" "TestPoint:TestPoint_Plated_Hole_D2.0mm"
+		(property "Footprint" "Connector_PinHeader_2.54mm:PinHeader_1x01_P2.54mm_Vertical"
 			(at 255.27 115.57 0)
 			(effects
