File: Telemetry peripheral boards/FS3 Peripheral V3 ATTINY/F3 peripheral boards.kicad_pcb (KiCad board)
At the start: 2 copper layers, 111.7 x 48.5 mm, 55 parts, among them J1 ATS668LSM, J10 Conn_01x10_Pin, J2 Exit Connector, J3 Potentiometer, J4 Strain Gauge, J5 Tire temp Sensor, J6 1x1 Tire Air Temp Sensor, J7 1x8 Tire Surface Temp Sensor, J8 Conn_01x03, J9 Conn_01x10_Pin, U1 LM2907M/NOPB, U2 INA125U, U3 MCP2515-I/SO, U4 ISO1050DUB, U5 ATtiny1616-S, U6 LM7805CV, U7 LF33CV, Y1 STDCSU1-8M

Commit message: fixed attiny v3
Parts:
- removed J8: Conn_01x03, Connector_PinHeader_2.54mm:PinHeader_1x03_P2.54mm_Vertical
- J10, J9: footprint Connector_PinHeader_2.00mm:PinHeader_1x10_P2.00mm_Vertical -> Connector_PinHeader_2.54mm:PinHeader_1x10_P2.54mm_Vertical
- moved J10 6.92 mm to (159.5, 35.3)
- moved J9 3.00 mm to (155.7, 58.2)
Routing:
- net PA3/SCK: track 47.3 -> 22.1 mm, vias 3 -> 2
- net PA2: track 64.8 -> 41.8 mm, vias 3 -> 2
- net +5V: track 191.9 -> 169.7 mm, vias 12 -> 10
- net PB1: track 39.7 -> 47.1 mm
- net PB2: track 38.3 -> 45.2 mm
- net PA6: track 94.8 -> 101.5 mm
- net PB3: track 36.9 -> 43.2 mm
- net PA7: track 104.2 -> 110.3 mm
- net PB4: track 35.3 -> 41.2 mm
- net PA1: track 97.3 -> 102.9 mm
- net PB5: track 33.9 -> 39.3 mm
- net PA4: track 92.3 -> 96.4 mm
- net PA5: track 29.4 -> 33.5 mm
- net PC3: track 48.1 -> 50.1 mm
- net Net-(U5-~{RESET}/PA0): track 11.3 -> 9.65 mm, vias 3 -> 2
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Other:
- board text added: "1x1 Tire Air Temp Sensor"
- board text added: "1x1 Tire Surface Temp Sensor"
- board text added: "FS-3 Telemetry Peripheral Board V3A Ruandy Salazar, Shaunak Lal"
- board text removed: "FS-3 Telemetry Peripheral Board V 2.5 Designed by Ruandy Salazar"

Commit message: fixed attiny pin headers
Routing:
- net PA3/SCK: track 22.1 -> 51.0 mm, vias 2 -> 4
- net PA2: track 41.8 -> 56.9 mm
Changed lines of the file:
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@@
-	)
-	(segment
-		(start 139.131372 43)
-		(end 141.936129 43)
-		(width 0.2)
-		(layer "F.Cu")
-		(net 37)
 	)
 	(segment
@@
 	)
 	(segment
+		(start 141.732 43)
+		(end 153.088 43)
+		(width 0.2)
+		(layer "F.Cu")
+		(net 37)
+	)
+	(segment
 		(start 128.6 45.72)
 		(end 128.6 48.26853)
@@
 	)
 	(segment
+		(start 141.732 43)
+		(end 141.936129 43)
+		(width 0.2)
+		(layer "F.Cu")
+		(net 37)
+	)
+	(segment
+		(start 153.088 43)
+		(end 155.702 40.386)
+		(width 0.2)
+		(layer "F.Cu")
+		(net 37)
+	)
+	(segment
+		(start 139.131372 43)
+		(end 141.732 43)
+		(width 0.2)
+		(layer "F.Cu")
+		(net 37)
+	)
+	(segment
 		(start 144.5 45.563871)
 		(end 144.5 54)
@@
 	)
 	(segment
+		(start 138.022663 55.118)
+		(end 137.083331 56.057331)
+		(width 0.2)
+		(layer "F.Cu")
+		(net 42)
+	)
+	(segment
 		(start 126.9596 52.69)
 		(end 125.65 52.69)
@@
 	)
 	(segment
-		(start 138.022663 55.118)
-		(end 134.637193 58.50347)
+		(start 148.082 42.164)
+		(end 151.384 42.164)
+		(width 0.2)
+		(layer "F.Cu")
+		(net 42)
+	)
+	(segment
+		(start 137.083331 56.057331)
+		(end 137.083331 51.331925)
+		(width 0.2)
+		(layer "F.Cu")
+		(net 42)
+	)
+	(segment
+		(start 151.384 42.164)
+		(end 155.702 37.846)
 		(width 0.2)
 		(layer "F.Cu")
@@
 	)
 	(segment
+		(start 137.083331 56.057331)
+		(end 134.637193 58.50347)
+		(width 0.2)
+		(layer "F.Cu")
+		(net 42)
+	)
+	(segment
+		(start 142.590056 45.8252)
+		(end 143.9 45.8252)
+		(width 0.2)
+		(layer "F.Cu")
+		(net 42)
+	)
+	(segment
 		(start 133.35 59.0804)
 		(end 126.9596 52.69)
@@
 	)
 	(segment
+		(start 137.083331 51.331925)
+		(end 142.590056 45.8252)
+		(width 0.2)
+		(layer "F.Cu")
+		(net 42)
+	)
+	(segment
 		(start 139.430929 55.118)
 		(end 138.022663 55.118)
@@
 	)
 	(via
+		(at 148.082 42.164)
+		(size 0.6)
+		(drill 0.3)
+		(layers "F.Cu" "B.Cu")
+		(net 42)
+	)
+	(via
 		(at 133.35 59.0804)
 		(size 0.6)
@@
 		(net 42)
 	)
+	(via
+		(at 143.9 45.8252)
+		(size 0.6)
+		(drill 0.3)
+		(layers "F.Cu" "B.Cu")
+		(net 42)
+	)
+	(segment
+		(start 147.5612 42.164)
+		(end 143.9 45.8252)
+		(width 0.2)
+		(layer "B.Cu")
+		(net 42)
+	)
+	(segment
+		(start 148.082 42.164)
+		(end 147.5612 42.164)
+		(width 0.2)
+		(layer "B.Cu")
+		(net 42)
+	)

Commit message: updated attiny board
Routing:
- net +3V3: track 105.4 -> 104.1 mm
Other:
- board text added: "C5"
Changed lines of the file:
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@@
 		(tags "SOP SO")
 		(property "Reference" "U4"
-			(at -2.4 -5.4 0)
+			(at -0.092 5.62 0)
 			(layer "F.SilkS")
 			(effects
@@
 		(tags "INA125U ")
 		(property "Reference" "U2"
-			(at 0 0 0)
+			(at 0 -5.882 0)
 			(unlocked yes)
 			(layer "F.SilkS")
@@
 		(tags "Potentiometer vertical Bourns 3296W")
 		(property "Reference" "RV1"
-			(at 0.1 -3.4 0)
+			(at -0.59 -3.4 0)
 			(layer "F.SilkS")
 			(effects
@@
 		)
 	)
+	(gr_text "C5"
+		(at 90.932 47.752 90)
+		(layer "F.SilkS")
+		(effects
+			(font
+				(size 1 1)
+				(thickness 0.15)
+			)
+		)
+	)
 	(gr_text "FS-3 Telemetry Peripheral Board\nV3A\nRuandy Salazar, Shaunak Lal"
 		(at 123.6 37.6 0)
@@
 		)
 		(height 3.849999)
-		(gr_text "101.610 mm"
+		(gr_text "4.000 in"
 			(at 114.295 76.95 0)
 			(layer "F.SilkS")
@@
 		)
 		(height 1.999999)
-		(gr_text "38.1000 mm"
+		(gr_text "1.5000 in"
 			(at 59.45 56.55 90)
 			(layer "F.SilkS")
@@
 		)
 		(height 6.799999)
-		(gr_text "111.7200 mm"
+		(gr_text "4.3984 in"
 			(at 114.36 23.550001 0)
 			(layer "Eco1.User")
@@
 		)
 		(height 8.074424)
-		(gr_text "48.5255 mm"
+		(gr_text "1.9105 in"
 			(at 51.540084 55.747431 270.0838323)
 			(layer "Eco1.User")
@@
 	)
 	(segment
-		(start 81.534 48.861)
-		(end 81.534 60.034)
-		(width 0.2)
-		(layer "F.Cu")
-		(net 5)
-	)
-	(segment
-		(start 94.3078 44.1922)
-		(end 94.3078 45.125)
-		(width 0.2)
-		(layer "F.Cu")
-		(net 5)
-	)
-	(segment
-		(start 104.5 44.5)
-		(end 103.5 43.5)
+		(start 111.5 44)
+		(end 111 44.5)
 		(width 0.2)
 		(layer "F.Cu")
@@
 	)
 	(segment
-		(start 95.5 44)
-		(end 94.5 44)
+		(start 81.534 48.861)
+		(end 81.534 60.034)
 		(width 0.2)
 		(layer "F.Cu")
@@
 	)
 	(segment
-		(start 96 43.5)
-		(end 95.5 44)
+		(start 94.9328 44.5)
+		(end 94.3078 45.125)
 		(width 0.2)
 		(layer "F.Cu")
@@
 	)
 	(segment
+		(start 111 44.5)
+		(end 94.9328 44.5)
+		(width 0.2)
+		(layer "F.Cu")
+		(net 5)
+	)
+	(segment
 		(start 87.25 44.25)
 		(end 87.25 41.93)
@@
 	)
 	(segment
-		(start 94.5 44)
-		(end 94.3078 44.1922)
-		(width 0.2)
-		(layer "F.Cu")
-		(net 5)
-	)
-	(segment
 		(start 82.5 64)
 		(end 81.5 65)
@@
 	)
 	(segment
-		(start 111 44.5)
-		(end 104.5 44.5)
-		(width 0.2)
-		(layer "F.Cu")
-		(net 5)
-	)
-	(segment
 		(start 136.5 42)
 		(end 135.58 42.92)
@@
 		(width 0.2)
 		(layer "F.Cu")
-		(net 5)
-	)
-	(segment
-		(start 111.5 44)
-		(end 111 44.5)
-		(width 0.2)
-		(layer "F.Cu")
-		(net 5)
-	)
-	(segment
-		(start 103.5 43.5)
-		(end 96 43.5)
-		(width 0.2)
-		(layer "F.Cu")

Commit message: telemP v3.1: added silkscreens, re-added separate updi testpoints
Parts:
- added J8: Conn_01x03, Connector_PinHeader_2.54mm:PinHeader_1x03_P2.54mm_Vertical, F.Cu at (149.0, 52.9)
Routing:
- net +5V: track 169.7 -> 178.8 mm, vias 10 -> 13
Other:
- board text added: "5V"
- board text added: "GND"
- board text added: "PA1"
- board text added: "PA2"
- board text added: "PA3"
- board text added: "PA4"
- board text added: "PA5"
- board text added: "PA6"
- board text added: "PA7"
- board text added: "PB0"
- board text added: "PB1"
- board text added: "PB2"
- board text added: "PB3"
- board text added: "PB4"
- board text added: "PB5"
- board text added: "PC0"
- board text added: "PC1"
- board text added: "PC2"
- board text added: "PC3"
- board text added: "UPDI"
