File: Discharge/Discharge.kicad_sch (KiCad schematic)
At the start: 17 parts, among them J1 TS, J2 Busbar, J3 LV connector, Q1 2N7002-TP, U1 NE555DR, U2 J1021CS312VDC.20, U3 CPC1008NTR, U4 ZXTR2005ZQ-13

Commit message: Add files via upload
Updated On 11/22/2024.

Added the 12V supply for low voltage connectors, Voltage regulator for the Optometry relay control. Additionally, there are tests points (labeled as TP) available for troubleshooting.
Parts:
- added J4: CAN, Connector_Molex:Molex_KK-254_AE-6410-02A_1x02_P2.54mm_Vertical, symbol Connector_Generic:Conn_01x02
- C1, C2: footprint Capacitor_SMD:C_1206_3216Metric_Pad1.33x1.80mm_HandSolder -> Capacitor_SMD:C_0402_1005Metric
- D1: footprint Diode_SMD:D_2114_3652Metric -> Diode_THT:D_A-405_P10.16mm_Horizontal
- J1, J2: footprint (none) -> Connector_Molex:Molex_KK-254_AE-6410-02A_1x02_P2.54mm_Vertical
- J3: footprint (none) -> Connector_Molex:Molex_KK-254_AE-6410-06A_1x06_P2.54mm_Vertical
- R1, R3, R5, R6: footprint (none) -> Resistor_THT:R_Axial_DIN0207_L6.3mm_D2.5mm_P10.16mm_Horizontal
- R2: footprint (none) -> Resistor_SMD:R_0603_1608Metric_Pad0.98x0.95mm_HandSolder
- U4: footprint SOT-89_4P5X2P45_DIO -> Regulator ZXTR2005ZQ_13:SOT-89_4P5X2P45_DIO
- renumbered D3 to D2
Connections:
- net 12v: now also U3.4 (R)
- net CANH: now also J4.2 (Pin_2)
- net CANL: now also J4.1 (Pin_1)
- net GLV: now also Q1.2 (S); no longer U3.4 (R)
- net GND: no longer Q1.2 (S)
- net at C1.2, R2.1, U1.6 (THRES): no longer U1.2 (TRIG)
- net MC: no longer names the net of J3.2 (Pin_2)
- no-connect marks 3 -> 4
Other:
- note added: "4"
- note added: "The following pads were utilized on the PCB: E1 : MSD(HVD) : Manual Service Disconnect E2 : TS+ : Tractive System E3 : TS- : Tractive System E4 : GLV : GROUND LOW VOLTAGE E5 : RTM : Ready To Move Light E6 : MC : Motor Controller (Same as Diode Shunt)"
- note removed: "3"
- note removed: "The following pads were utilized on the PCB: E1 : MSD(HVD) : Manual Service Disconnect E2 : TS+ : Tractive System E3 : TS- : Tractive System E4 : GLV : GROUND LOW VOLTAGE E5 : RTM : Ready To Move Light E6 : MC : Motor Controller"
- moved on the sheet: J1, J3, R2

Commit message: Add files via upload
Parts:
- removed D2: D, Diode_SMD:D_2010_5025Metric, symbol Device:D
- removed R1: 15k, Resistor_THT:R_Axial_DIN0207_L6.3mm_D2.5mm_P10.16mm_Horizontal, symbol Device:R_US
- removed U3: CPC1008NTR, CPC1008NTR:CPC1008N_IXY, symbol Isolator:NSL-32
- removed U4: ZXTR2005ZQ-13, Regulator ZXTR2005ZQ_13:SOT-89_4P5X2P45_DIO, symbol 2024-11-14_03-53-50:ZXTR2005ZQ-13
- added C3: 0.1uF, Capacitor_THT:C_Rect_L7.0mm_W6.0mm_P5.00mm, symbol Device:C
- added C4: 100nf, Capacitor_SMD:C_1206_3216Metric_Pad1.33x1.80mm_HandSolder, symbol Device:C
- added C5: 10uf, Capacitor_SMD:C_1206_3216Metric_Pad1.33x1.80mm_HandSolder, symbol Device:C
- added D2: 24v, Diode_THT:D_A-405_P10.16mm_Horizontal, symbol Device:D_Zener
- added Q2: LD1117V50C, LD1117V50C:TO-220S_STM, symbol 2025-01-18_02-37-27:LD1117V50C
- added R2: 5k, Resistor_THT:R_Axial_DIN0207_L6.3mm_D2.5mm_P10.16mm_Horizontal, symbol Device:R_US
- added R6: 4k, Resistor_THT:R_Axial_DIN0207_L6.3mm_D2.5mm_P10.16mm_Horizontal, symbol Device:R_US
- added U3: J1021CS324VDC.20, RelayJ1021:RELAY6_J1021CS312VDC.20_CRS, symbol 2024-11-03_23-16-05:J1021CS312VDC.20
- added U4: LD1117V50C, LD1117V50C:TO-220S_STM, symbol 2025-02-01_22-29-22:LD1117V50C
- C1, C2: footprint Capacitor_SMD:C_0402_1005Metric -> Capacitor_SMD:C_0805_2012Metric_Pad1.18x1.45mm_HandSolder
- D1: value 60V -> 50v
- J1, J2: footprint Connector_Molex:Molex_KK-254_AE-6410-02A_1x02_P2.54mm_Vertical -> Connector_Molex:Molex_Nano-Fit_105309-xx03_1x03_P2.50mm_Vertical; symbol Connector_Generic:Conn_01x02 -> Connector_Generic:Conn_01x03
- J3: footprint Connector_Molex:Molex_KK-254_AE-6410-06A_1x06_P2.54mm_Vertical -> Connector_Molex:Molex_Nano-Fit_105309-xx06_1x06_P2.50mm_Vertical
- J4: footprint Connector_Molex:Molex_KK-254_AE-6410-02A_1x02_P2.54mm_Vertical -> Connector_Molex:Molex_Nano-Fit_105309-xx02_1x02_P2.50mm_Vertical
- R3: value 1k -> 220
- R5: value 5k -> 4.7k
- renumbered R2 to R1, R6 to R4
Connections:
- net 12v: now also U3.6
- net CANL: now also J3.2 (Pin_2); no longer J3.5 (Pin_5)
- net GLV: now also C2.2, C4.2, C5.2, U4.1 (ADJ/GND); no longer C2.1
- net GND: now also D1.2 (A), J2.1 (Pin_1), U2.7, C3.2, D2.2 (A), R6.2; no longer R3.2, U2.12
- net Shunt Module: now also J2.3 (Pin_3), R2.2; no longer J2.2 (Pin_2), R5.2
- net TS+: now also R5.1, U2.6; no longer D1.1 (K), U2.1
- net TS-: now also J1.3 (Pin_3), R4.1, U3.7; no longer J1.2 (Pin_2), R5.1
- net at C1.2, R1.1, U1.6 (THRES): now also U1.2 (TRIG)
- net at R1.2, U1.4 (RESET), U1.7 (DISCH)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: now also C2.1, C5.1, U4.2 (VOUT); no longer C2.2
- net at R3.1: now also D2.1 (K), Q2.1 (ADJ/GND), R6.1, U3.1; no longer U2.7
- removed net MSD (HVD): J2.1 (Pin_1), R4.2, U2.6
- new net: C4.1, U3.12, U4.3 (VIN)
- new net: C3.1, D1.1 (K), Q2.3 (VIN), R5.2
- new net: Q2.2 (VOUT), R3.2
- new net: R2.1, U2.12
- new net IR Final: J2.2 (Pin_2), R4.2, U2.1
- no-connect marks 4 -> 6
Other:
- note added: "5"
- note added: "5v Regulator"
- note added: "As close as possible from GND for better load regulation"
- note added: "As close as possible from v_out to minimize voltage drop"
- note added: "Regulator; Input: 60v<, output ~24v"
- note added: "The TS+/- need to go the TSP resistor, specified on the TSMp connectors. Thus two resistors are required. LV power from the motor controller and also has to go to where CAN connector/ from the discharge connector. No pin number required, Check for the ESF Tractive System Schematic for more information. Max HV from TS: 130v U4 is a dual diode voltage regulator GND connection pending (Chassis vs Co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"
- note added: "The following pads were utilized on the PCB: E1 : MSD(HVD) : Manual Service Disconnect E2 : TS+ : Tractive System HV+ E3 : TS- : Tractive System HV- (~54W) E4 : GLV : GROUND LOW VOLTAGE E5 : RTM : Ready To Move Light E6 : DS : Discharge Resistor (Same as Diode Shunt)"
- note removed: "4"
- note removed: "THe TS+/- need to go the TSP resistor, specified on the TSMp connectors. Thus two resistors are required. LV power from the motor controller and also has to go to where CAN connector/ from the discharge connector. No pin number required, Check for the ESF Tractive System Schematic for more information. GND connection pending (Chassis vs Connector)."
- note removed: "The following pads were utilized on the PCB: E1 : MSD(HVD) : Manual Service Disconnect E2 : TS+ : Tractive System E3 : TS- : Tractive System E4 : GLV : GROUND LOW VOLTAGE E5 : RTM : Ready To Move Light E6 : MC : Motor Controller (Same as Diode Shunt)"
- moved on the sheet: C1, C2, J3, J4, Q1, R1, R4, U1, U2

Commit message: Add files via upload
Parts:
- removed D2: 24v, Diode_THT:D_A-405_P10.16mm_Horizontal, symbol Device:D_Zener
- removed J3: LV connector, Connector_Molex:Molex_Nano-Fit_105309-xx06_1x06_P2.50mm_Vertical, symbol Connector_Generic:Conn_01x06
- removed Q2: LD1117V50C, LD1117V50C:TO-220S_STM, symbol 2025-01-18_02-37-27:LD1117V50C
- removed R3: 220, Resistor_THT:R_Axial_DIN0207_L6.3mm_D2.5mm_P10.16mm_Horizontal, symbol Device:R_US
- removed R5: 4.7k, Resistor_THT:R_Axial_DIN0207_L6.3mm_D2.5mm_P10.16mm_Horizontal, symbol Device:R_US
- removed R6: 4k, Resistor_THT:R_Axial_DIN0207_L6.3mm_D2.5mm_P10.16mm_Horizontal, symbol Device:R_US
- removed U3: J1021CS324VDC.20, RelayJ1021:RELAY6_J1021CS312VDC.20_CRS, symbol 2024-11-03_23-16-05:J1021CS312VDC.20
- removed U4: LD1117V50C, LD1117V50C:TO-220S_STM, symbol 2025-02-01_22-29-22:LD1117V50C
- added C6: 10uF, symbol Device:C
- added J3: Conn_01x06, symbol Connector_Generic:Conn_01x04
- added U3: ZXTR2005ZQ-13, Package_TO_SOT_THT:TO-220-3_Vertical, symbol Regulator_Linear:LM7809_TO220
- added U4: TLP3122AE, 1FS_2_Global_Footprint_Library:OptoCoupler 6-SOP, symbol FS_3_Global_Symbol_Library:TLP3122AE
- added U5: LD1117V50C, TO-220S_STM, symbol 2025-02-01_22-29-22:LD1117V50C
- C3: value 0.1uF -> 1uF; footprint Capacitor_THT:C_Rect_L7.0mm_W6.0mm_P5.00mm -> Capacitor_SMD:C_0805_2012Metric_Pad1.18x1.45mm_HandSolder
- C4: value 100nf -> 10uF; footprint Capacitor_SMD:C_1206_3216Metric_Pad1.33x1.80mm_HandSolder -> Capacitor_SMD:C_0805_2012Metric_Pad1.18x1.45mm_HandSolder
- C5: value 10uf -> 100nF; footprint Capacitor_SMD:C_1206_3216Metric_Pad1.33x1.80mm_HandSolder -> (none)
- D1: value 50v -> 50V; footprint Diode_THT:D_A-405_P10.16mm_Horizontal -> Diode_SMD:Nexperia_CFP3_SOD-123W
- J2: symbol Connector_Generic:Conn_01x03 -> Connector_Generic:Conn_01x02
- J4: value CAN -> Conn_01x02; footprint Connector_Molex:Molex_Nano-Fit_105309-xx02_1x02_P2.50mm_Vertical -> (none)
Connections:
- net CANH is gone; now on net Discharge+: J4.2 (Pin_2)
- net 12v: now also J3.1 (Pin_1), U4.6
- net GLV: now also U2.1, C6.2, J3.2 (Pin_2), U5.1 (ADJ/GND); no longer C4.2
- net IR Final: now also U2.7, J3.4 (Pin_4); no longer J2.2 (Pin_2), R4.2, U2.1
- net RTM: now also J3.3 (Pin_3)
- net TS+: now also R4.1; no longer U2.6
- net TS-: now also C3.2, C4.2, D1.1 (K), R2.2, U3.2 (GND), U4.3; no longer R4.1
- net at C2.1, R1.2, U1.4 (RESET)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: now also C6.1, U5.2 (VOUT); no longer C5.1
- net at C4.1: now also U3.3 (VO), U4.1
- net at C3.1: now also D1.2 (A), U3.1 (VI); no longer D1.1 (K)
- net Discharge+: now reaches U2.12
- net Discharge+: no longer R2.1
- net CANL renamed Discharge-
- net Discharge-: now also U2.6
- removed net GND: C3.2, D1.2 (A), J2.1 (Pin_1), U2.7
- removed net Shunt Module: J2.3 (Pin_3), R2.2
- new net: C5.1, U4.4, U5.3 (VIN)
- new net TSMP+: J2.1 (Pin_1), R4.2
- new net TSMP-: J2.2 (Pin_2), R2.1
- no-connect marks 6 -> 3
Other:
- note added: "02/08/2025"
- note added: "6"
- note added: "HPZR-C50-QX"
- note added: "High Voltage"
- note added: "LV connectors + 5v regulator"
- note added: "RTM Logic"
- note added: "TS +/- use for controlling lv logic + measuring points outside of tractive box TSMP +/- == TS+/- measuring points Discharge +/- allows HV to flow once indicator has been given Consider: Trace length = 30V/mil."
- note removed: "11/13/2024"
- note removed: "5"
- note removed: "5v Regulator"
- note removed: "As close as possible from GND for better load regulation"
- note removed: "As close as possible from v_out to minimize voltage drop"
- note removed: "Regulator; Input: 60v<, output ~24v"
- note removed: "The TS+/- need to go the TSP resistor, specified on the TSMp connectors. Thus two resistors are required. LV power from the motor controller and also has to go to where CAN connector/ from the discharge connector. No pin number required, Check for the ESF Tractive System Schematic for more information. Max HV from TS: 130v U4 is a dual diode voltage regulator GND connection pending (Chassis vs Co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"
- note removed: "The following pads were utilized on the PCB: E1 : MSD(HVD) : Manual Service Disconnect E2 : TS+ : Tractive System HV+ E3 : TS- : Tractive System HV- (~54W) E4 : GLV : GROUND LOW VOLTAGE E5 : RTM : Ready To Move Light E6 : DS : Discharge Resistor (Same as Diode Shunt)"
- moved on the sheet: J1, R4

Commit message: Add files via upload
Parts:
- C5, C6: footprint (none) -> Capacitor_SMD:C_1210_3225Metric_Pad1.33x2.70mm_HandSolder
- J2: value Busbar -> TSMP; footprint Connector_Molex:Molex_Nano-Fit_105309-xx03_1x03_P2.50mm_Vertical -> Connector_Molex:Molex_Nano-Fit_105309-xx02_1x02_P2.50mm_Vertical
- J3: footprint (none) -> Connector_Molex:Molex_Nano-Fit_105309-xx04_1x04_P2.50mm_Vertical
- J4: footprint (none) -> Connector_Molex:Molex_Nano-Fit_105309-xx02_1x02_P2.50mm_Vertical
- U3: footprint Package_TO_SOT_THT:TO-220-3_Vertical -> Package_TO_SOT_SMD:SOT-89-3_Handsoldering
- U4: footprint 1FS_2_Global_Footprint_Library:OptoCoupler 6-SOP -> Package_SO:SO-5-6_4.55x3.7mm_P1.27mm
- U5: footprint TO-220S_STM -> LD1117V50C:TO-220S_STM
Connections:
- net TS+: now also D1.1 (K), J1.3 (Pin_3), R2.2; no longer J1.1 (Pin_1), R4.1
- net TS-: now also J1.1 (Pin_1), R4.1, U3.1 (GND); no longer D1.1 (K), J1.3 (Pin_3), R2.2, U3.2 (GND)
- net TSMP+: now also J2.2 (Pin_2), R2.1; no longer J2.1 (Pin_1), R4.2
- net TSMP-: now also J2.1 (Pin_1), R4.2; no longer J2.2 (Pin_2), R2.1
- net at C3.1, D1.2 (A): now also U3.2 (VI); no longer U3.1 (VI)

Commit message: Add files via upload
Parts:
- removed U2: J1021CS312VDC.20, RelayJ1021:RELAY6_J1021CS312VDC.20_CRS, symbol 2024-11-03_23-16-05:J1021CS312VDC.20
- added K1: G5V-2, Relay_THT:Relay_DPDT_Omron_G5V-2, symbol Relay:G5V-2
- added TP1: IRF, TestPoint:TestPoint_Loop_D2.50mm_Drill1.0mm, symbol Connector:TestPoint
- added TP2: 5V, TestPoint:TestPoint_Loop_D2.50mm_Drill1.0mm, symbol Connector:TestPoint
- added TP3: RTM, TestPoint:TestPoint_Loop_D2.50mm_Drill1.0mm, symbol Connector:TestPoint
- added TP4: 12V, TestPoint:TestPoint_Loop_D2.50mm_Drill1.0mm, symbol Connector:TestPoint
- added TP5: GLV, TestPoint:TestPoint_Loop_D2.50mm_Drill1.0mm, symbol Connector:TestPoint
- C5, C6: footprint Capacitor_SMD:C_1210_3225Metric_Pad1.33x2.70mm_HandSolder -> Capacitor_SMD:C_0805_2012Metric_Pad1.18x1.45mm_HandSolder
Connections:
- net Discharge+: now also K1.13
- net Discharge-: now also K1.11
- net GLV: now also K1.16, TP5.1
- net IR Final: now also K1.1, TP1.1
- net RTM: now also TP3.1
- net at C2.1, C6.1, R1.2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: now also TP2.1
- net at C5.1, U4.4, U5.3 (VIN): now also TP4.1
- no-connect marks 3 -> 5
Other:
- note added: "Discharge must be normaly closed."

Commit message: Add files via upload
Parts:
- removed U5: LD1117V50C, LD1117V50C:TO-220S_STM, symbol 2025-02-01_22-29-22:LD1117V50C
- added CR1: STS6NF20V, Package_SO:Infineon_PG-DSO-8-24_4x5mm, symbol FS_3_Global_Symbol_Library:STS6NF20V
- added D2: 20v, Diode_SMD:D_0805_2012Metric_Pad1.15x1.40mm_HandSolder, symbol Device:D
- added Q2: 2N7002-TP, 2N7002:2N7002K_ONS, symbol New_Library_2:2N7002-TP
- added U2: ZXTR2005ZQ-13, Package_TO_SOT_SMD:SOT-89-3_Handsoldering, symbol Regulator_Linear:LM7809_TO220
- K1: value G5V-2 -> 1109537
- Q1: value 2N7002-TP -> STS6NF20V; footprint 2N7002:2N7002K_ONS -> STS6NF20V:SO-8_STM
Connections:
- net GLV: now also D2.2 (A), U2.1 (GND)
- net IR Final: now also D2.1 (K)
- net at C2.1, C6.1, R1.2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: now also U2.3 (VO)
- net at C5.1, TP4.1, U4.4: now also U2.2 (VI)
- new net: CR1.1 (S), CR1.2 (S), CR1.3 (S), CR1.4 (G)
- new net: CR1.5 (D), CR1.6 (D), CR1.7 (D), CR1.8 (D)
- no-connect marks 5 -> 10
Other:
- note added: "Better alternative, a 2N7002-TP MOSFET. We don't have the money to ordervthem, so we used a STS6NF20V (we had spares at that time)."
- note added: "JA8"
- note removed: "6"

Commit message: Add files via upload
Parts:
- removed Q1: STS6NF20V, STS6NF20V:SO-8_STM, symbol New_Library_2:2N7002-TP
- D1: value 50V -> HPZR-C50-QX
Connections:
- net RTM: now also U1.3 (OUT)
Other:
- note added: "50V"
- note removed: "HPZR-C50-QX"

Commit message: REV 6 (?)
Parts:
- removed CR1: STS6NF20V, Package_SO:Infineon_PG-DSO-8-24_4x5mm, symbol FS_3_Global_Symbol_Library:STS6NF20V
- removed Q2: 2N7002-TP, 2N7002:2N7002K_ONS, symbol New_Library_2:2N7002-TP
- added R3: 470, Resistor_SMD:R_0603_1608Metric_Pad0.98x0.95mm_HandSolder, symbol Device:R_US
- added TP6: U3Vin, TestPoint:TestPoint_Loop_D2.50mm_Drill1.0mm, symbol Connector:TestPoint
- added TP7: U3Vout, TestPoint:TestPoint_Loop_D2.50mm_Drill1.0mm, symbol Connector:TestPoint
- R2, R4: footprint Resistor_THT:R_Axial_DIN0207_L6.3mm_D2.5mm_P10.16mm_Horizontal -> Resistor_THT:R_Axial_Power_L20.0mm_W6.4mm_P22.40mm
Connections:
- net at C4.1, U3.3 (VO): now also R3.1, TP7.1; no longer U4.1
- net at C3.1, D1.2 (A), U3.2 (VI): now also TP6.1
- new net: R3.2, U4.1
- no-connect marks 10 -> 5
Other:
- note added: "TS +/- use for controlling lv logic + measuring points outside of tractive box TSMP +/- == TS+/- measuring points Discharge +/- allows HV to flow once indicator has been given Consider: Trace length = 30V/mil. All resistor values are in ohms."
- note removed: "Better alternative, a 2N7002-TP MOSFET. We don't have the money to ordervthem, so we used a STS6NF20V (we had spares at that time)."
- note removed: "TS +/- use for controlling lv logic + measuring points outside of tractive box TSMP +/- == TS+/- measuring points Discharge +/- allows HV to flow once indicator has been given Consider: Trace length = 30V/mil."
- moved on the sheet: C3, C4, D1, U3
