File: charger_shutdownboard/charger_shutdownboard.kicad_sch (KiCad schematic)
At the start: 13 parts, among them J1 Conn_01x08_Pin, J2 Conn_01x02_Pin, J3 Conn_01x02_Pin, J4 Conn_01x02_Pin, J5 Conn_01x02_Pin, J6 Conn_01x02_Pin, J7 Conn_01x02_Pin

Commit message: charger shutdown circuit board done!
Parts:
- R1, R2, R3, R4: footprint (none) -> Resistor_SMD:R_0805_2012Metric_Pad1.20x1.40mm_HandSolder
- R5, R6: footprint (none) -> Resistor_THT:R_Axial_DIN0922_L20.0mm_D9.0mm_P25.40mm_Horizontal
Connections:
- net +12V: now also J2.2 (Pin_2), J5.2 (Pin_2); no longer J2.1 (Pin_1), J5.1 (Pin_1)
- net CAN_H: now also J3.2 (Pin_2); no longer J3.1 (Pin_1)
- net CAN_L: now also J3.1 (Pin_1); no longer J3.2 (Pin_2)
- net GND: now also J2.1 (Pin_1); no longer J2.2 (Pin_2)
- net Shutdown_Reset: now also J5.1 (Pin_1); no longer J5.2 (Pin_2)
- net at R6.2: now also J6.1 (Pin_1); no longer J6.2 (Pin_2)
- net at R5.2: now also J6.2 (Pin_2); no longer J6.1 (Pin_1)
Other:
- moved on the sheet: J3, J6, J7, R5, R6

Commit message: value for voltage divider resistors for bspd_fault changed
Changed lines of the file:
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@@
 	(text "Shutdown Button \n"
 		(exclude_from_sim no)
-		(at 66.294 127 0)
+		(at 65.786 139.446 0)
 		(effects
 			(font
@@
 	(text "CAN COTS Charger"
 		(exclude_from_sim no)
-		(at 66.294 112.522 0)
+		(at 65.278 115.062 0)
 		(effects
 			(font
@@
 	(text "12V Power supply"
 		(exclude_from_sim no)
-		(at 65.532 97.028 0)
+		(at 65.786 100.838 0)
 		(effects
 			(font
@@
 	(text "Reset Button \n"
 		(exclude_from_sim no)
-		(at 64.516 142.24 0)
+		(at 64.516 146.304 0)
 		(effects
 			(font

Commit message: Added J1772 negotiation to schematic
Parts:
- added C1, C2, C3, C4, C5: 100nF, symbol Device:C
- added D1: D, symbol Device:D
- added J8: J1772 Negotiation, Connector_Molex:Molex_Nano-Fit_105309-xx02_1x02_P2.50mm_Vertical, symbol Connector:Conn_01x02_Pin
- added R10: 499k, symbol Device:R
- added R11: 120, Resistor_SMD:R_0805_2012Metric_Pad1.20x1.40mm_HandSolder, symbol Device:R
- added R12: 200k, symbol Device:R
- added R13, R9: 330k, symbol Device:R
- added R7: 866, symbol Device:R
- added R8: 330, symbol Device:R
- added U1: NUCLEO-L432KC, NUCLEO-L432KC:MODULE_NUCLEO-L432KC, symbol 1FS_2_Global_Symbol_Library:NUCLEO-L432KC
- added U3: ISO1050DUB, Package_SO:SOP-8_6.62x9.15mm_P2.54mm, symbol Interface_CAN_LIN:ISO1050DUB
- added U4: LM7809_TO220, Package_TO_SOT_THT:TO-220-3_Vertical, symbol Regulator_Linear:LM7809_TO220
- J1: value Conn_01x08_Pin -> Acc SFC
- J2: value Conn_01x02_Pin -> 12V Power supply
- J3: value Conn_01x02_Pin -> CAN COTS Charger
- J4: value Conn_01x02_Pin -> Shutdown Button
- J5: value Conn_01x02_Pin -> Reset Button
- J6: value Conn_01x02_Pin -> TSMP to HV
- J7: value Conn_01x02_Pin -> TSMP to Banana Jacks
Connections:
- net +12V: now also C5.1, U4.1 (VI)
- net CAN_H: now also R11.1, U3.7 (CANH)
- net CAN_L: now also R11.2, U3.6 (CANL)
- net GND: now also C1.2, C2.1, C3.1, C4.2, C5.2, R10.2, R13.2, R7.2, U1.CN3_4 (GND), U1.CN4_2 (GND), U3.4 (GND1), U3.5 (GND2), U4.2 (GND)
- new net +3V3: C2.2, U1.CN4_14 (3V3), U3.1 (VCC1)
- new net +5V: C3.2, R8.1, U1.CN4_4 (5V), U3.8 (VCC2)
- new net +9V: C4.1, U1.CN4_1 (VIN), U4.3 (VO)
- new net CAN_RX: U1.CN3_13 (PA11), U3.2 (RXD)
- new net CAN_TX: U1.CN3_5 (PA12), U3.3 (TXD)
- new net Control Pilot: D1.2 (A), J8.2 (Pin_2)
- new net Control_Pilot_Cutoff: D1.1 (K), R7.1, R9.1
- new net Control_Pilot_Filtered: C1.1, R10.1, R9.2, U1.CN4_6 (PA7)
- new net Proximity Pilot: J8.1 (Pin_1), R12.1, R8.2
- new net Proximity_Pilot_Filtered: R12.2, R13.1, U1.CN4_7 (PA6)
- no-connect marks 0 -> 21
Other:
- note removed: "12V Power supply"
- note removed: "Acc SFC"
- note removed: "CAN COTS Charger"
- note removed: "Reset Button"
- note removed: "Shutdown Button"
- note removed: "TSMP to Banana Jacks"
- note removed: "TSMP to HV"
- company: (none) -> Formula Slug
- title: (none) -> FS-3 Charger Board
- moved on the sheet: J1, J2, J3, J4, J5, J6, J7, R1, R2, R3, R4, R5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

Commit message: Revised PCB for J1772 negotiation
Parts:
- removed R1: 70k, Resistor_SMD:R_0805_2012Metric_Pad1.20x1.40mm_HandSolder, symbol Device:R
- removed R2: 50k, Resistor_SMD:R_0805_2012Metric_Pad1.20x1.40mm_HandSolder, symbol Device:R
- removed R3: 100k, Resistor_SMD:R_0805_2012Metric_Pad1.20x1.40mm_HandSolder, symbol Device:R
- removed R4: 38k, Resistor_SMD:R_0805_2012Metric_Pad1.20x1.40mm_HandSolder, symbol Device:R
- C1, C2, C3, C4, C5: footprint (none) -> Capacitor_SMD:C_0805_2012Metric_Pad1.18x1.45mm_HandSolder
- D1: footprint (none) -> Diode_SMD:D_0805_2012Metric_Pad1.15x1.40mm_HandSolder
- R10, R12, R13, R7, R8, R9: footprint (none) -> Resistor_SMD:R_0805_2012Metric_Pad1.20x1.40mm_HandSolder
- U1: footprint NUCLEO-L432KC:MODULE_NUCLEO-L432KC -> FS_3_Global_Footprint_Library:NUCLEO-L432KC
Connections:
- net BSPD_fault is gone; now on net +5V: J1.5 (Pin_5)
- net Charge_State is gone; now on net +3V3: J1.10 (Pin_10)
- net CAN_H: now also J1.12 (Pin_12); no longer J1.3 (Pin_3)
- net CAN_L: now also J1.11 (Pin_11); no longer J1.4 (Pin_4)
- no-connect marks 21 -> 23
Other:
- note added: "Charger Box Components"
- note added: "High is no fault"
- note added: "J1772 Negotiation"
- note added: "Micro and CAN"
- note added: "Power Block"
- note added: "SFC"
- note added: "TSMPs"
- note added: "Tell the acc board that the charger is connected"
- note added: "Trace + wire must be <150mm to busbars"
- moved on the sheet: C1, C2, C3, C4, C5, D1, J1, J2, J3, J4, J5, J6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

Commit message: added clarification text
Other:
- note added: "Name consistent with the acc pinout -- comes from acc"
- note added: "Shutdown starts here after the charger E-stop, goes to acc"
Changed lines of the file:
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@@
+		)
+	)
+	(text "Shutdown starts here after the charger E-stop, goes to acc"
+		(exclude_from_sim no)
+		(at 42.164 38.354 0)
+		(effects
+			(font
+				(size 1.27 1.27)
+			)
+			(justify left)
+		)
+	)
+	(text "Name consistent with the acc pinout -- comes from acc"
+		(exclude_from_sim no)
+		(at 42.164 41.148 0)
+		(effects
+			(font
+				(size 1.27 1.27)
+			)
+			(justify left)
 		)
 	)
