File: Telemetry peripheral boards/FS3 Peripheral V4 ATTINY/PD.kicad_sch (KiCad schematic)
At the start: 6 parts, among them U6 LF33CV, U7 LM7805CV

Commit message: cleared 3V3 regulator
Parts:
- removed C11: 100nF, Capacitor_SMD:C_0805_2012Metric_Pad1.18x1.45mm_HandSolder, symbol Device:C
- removed C13: 2.2uF, Capacitor_SMD:C_0805_2012Metric_Pad1.18x1.45mm_HandSolder, symbol Device:C
- removed U6: LF33CV, Package_TO_SOT_THT:TO-220-3_Vertical, symbol Regulator_Linear:LM7805_TO220
