File: Telemetry peripheral boards/FS3 Peripheral V4 ATTINY/F3 peripheral boards.kicad_pcb (KiCad board)
At the start: 2 copper layers, 70.7 x 40.3 mm, 55 parts, among them J1 ATS668LSM, J10 Conn_01x10_Pin, J2 Main Connector, J3 Potentiometer, J4 Strain Gauge, J5 Tire temp Sensor, J6 1x1 Tire Air Temp Sensor, J7 1x8 Tire Surface Temp Sensor, J9 Conn_01x10_Pin, U1 LM2907M/NOPB, U2 INA125U, U3 MCP2515-I/SO, U4 ISO1050DUB, U5 ATtiny1616-S, U6 LF33CV, U7 LM7805CV, Y1 STDCSU1-8M

Commit message: cleared 3V3 regulator
Parts:
- removed C11: 100nF, Capacitor_SMD:C_0805_2012Metric_Pad1.18x1.45mm_HandSolder
- removed C13: 2.2uF, Capacitor_SMD:C_0805_2012Metric_Pad1.18x1.45mm_HandSolder
- removed U6: LF33CV, Package_TO_SOT_THT:TO-220-3_Vertical
Routing:
- net GND: track 99.0 -> 69.7 mm, vias 12 -> 13
- net +3V3: track 19.9 -> 0.00 mm
- net +12V: track 31.0 -> 22.1 mm, vias 1 -> 0
Other:
- board text removed: "2.2uf"

Commit message: more stuff and gerbers!
Routing:
- net GND: track 69.7 -> 60.5 mm
- net PA6: track 94.3 -> 97.8 mm, vias 2 -> 1
Changed lines of the file:
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@@
 		(tags "resistor handsolder")
 		(property "Reference" "R15"
-			(at -3.1196 0.3234 360)
+			(at -3.1196 0.3234 0)
 			(layer "F.SilkS")
 			(effects
@@
 		)
 		(property "Value" "4.7k"
-			(at 0 1.65 360)
+			(at 0 1.65 0)
 			(layer "F.Fab")
 			(effects
@@
 		)
 		(fp_text user "${REFERENCE}"
-			(at 0 0 360)
+			(at 0 0 0)
 			(layer "F.Fab")
 			(effects
@@
 		(tags "resistor handsolder")
 		(property "Reference" "R8"
-			(at -2.81 0.2808 360)
+			(at -2.81 0.2808 0)
 			(layer "F.SilkS")
 			(effects
@@
 		)
 		(property "Value" "4.7k"
-			(at 0 1.65 360)
+			(at 0 1.65 0)
 			(layer "F.Fab")
 			(effects
@@
 		)
 		(fp_text user "${REFERENCE}"
-			(at 0 0 360)
+			(at 0 0 0)
 			(layer "F.Fab")
 			(effects
@@
 	)
 	(segment
+		(start 134.5438 78.613001)
+		(end 134.086999 78.613001)
+		(width 0.2)
+		(layer "F.Cu")
+		(net 2)
+	)
+	(segment
 		(start 122.6058 85.830501)
 		(end 122.8383 85.598001)
@@
 	)
 	(segment
+		(start 134.086999 78.613001)
+		(end 132.7 80)
+		(width 0.2)
+		(layer "F.Cu")
+		(net 2)
+	)
+	(segment
 		(start 139.6238 100.105553)
 		(end 141.169047 101.6508)
@@
 	)
 	(segment
-		(start 131.2484 78.588401)
-		(end 134.5192 78.588401)
-		(width 0.2)
-		(layer "F.Cu")
-		(net 2)
-	)
-	(segment
 		(start 125.3783 79.210501)
 		(end 125.3783 77.216001)
@@
 	)
 	(via
-		(at 131.2484 78.588401)
+		(at 93.8022 89.4842)
 		(size 0.6)
 		(drill 0.3)
@@
 	)
 	(via
-		(at 93.8022 89.4842)
+		(at 132.7 80)
 		(size 0.6)
 		(drill 0.3)
@@
 	)
 	(segment
-		(start 132.6788 77.158001)
-		(end 131.2484 78.588401)
-		(width 0.2)
-		(layer "B.Cu")
-		(net 2)
-	)
-	(segment
 		(start 121.7123 85.830501)
 		(end 121.7539 85.788901)
@@
 	)
 	(segment
-		(start 123.227 87.345201)
-		(end 121.7123 85.830501)
-		(width 0.2)
-		(layer "B.Cu")
-		(net 2)
-	)
-	(segment
-		(start 132.6788 72.931001)
-		(end 132.6788 77.158001)
-		(width 0.2)
-		(layer "B.Cu")
-		(net 2)
-	)
-	(segment
 		(start 129.2221 78.613001)
 		(end 128.0508 78.613001)
@@
 	)
 	(segment
-		(start 135.89 87.6808)
-		(end 136.89 88.6808)
-		(width 0.2)
-		(layer "F.Cu")
-		(net 9)
-	)
-	(segment
 		(start 135.579729 94.5388)
 		(end 135.462329 94.6562)
@@
 	)
 	(segment
-		(start 141.389256 89.614201)
-		(end 140.455855 88.6808)
+		(start 137.814201 89.614201)
+		(end 143.8988 89.614201)
+		(width 0.2)
+		(layer "F.Cu")
+		(net 9)
+	)
+	(segment
+		(start 136.89 88.6808)
+		(end 136.89 88.69)
 		(width 0.2)
 		(layer "F.Cu")
@@
 	(segment
 		(start 143.8988 89.614201)
-		(end 141.389256 89.614201)
+		(end 145.2988 88.214201)
 		(width 0.2)
 		(layer "F.Cu")
@@
 	)
 	(segment
-		(start 144.4498 96.393001)
-		(end 143.2981 96.393001)
+		(start 136.89 88.69)
+		(end 137.814201 89.614201)
 		(width 0.2)
 		(layer "F.Cu")
@@
 	)
 	(segment
-		(start 115.5322 90.805001)
-		(end 108.9878 84.260601)
+		(start 144.4498 96.393001)
+		(end 143.2981 96.393001)
 		(width 0.2)
 		(layer "F.Cu")
@@
 	)
 	(segment
-		(start 136.89 88.6808)
-		(end 140.455855 88.6808)
+		(start 115.5322 90.805001)
+		(end 108.9878 84.260601)
 		(width 0.2)
 		(layer "F.Cu")
@@
 	)
 	(segment
-		(start 145.2988 88.214201)
-		(end 143.8988 89.614201)
+		(start 135.89 87.6808)
+		(end 136.89 88.6808)
 		(width 0.2)
 		(layer "F.Cu")
@@
 	)
 	(segment
-		(start 151.5872 76.1492)
-		(end 150.0378 74.5998)
+		(start 147.114623 70.6)
+		(end 151.5872 75.072577)
 		(width 0.2)
 		(layer "F.Cu")
@@
 	)
 	(segment
+		(start 145.784587 70.6)
+		(end 147.114623 70.6)
+		(width 0.2)
+		(layer "F.Cu")
+		(net 10)
+	)
+	(segment
 		(start 115.048771 69.942901)
 		(end 131.9106 69.942901)
@@
 	)
 	(segment
+		(start 151.5872 75.072577)
+		(end 151.5872 76.1492)
+		(width 0.2)
+		(layer "F.Cu")
+		(net 10)
+	)
+	(segment
 		(start 107.6628 73.5154)
 		(end 107.864199 73.314001)
@@
 	)
 	(segment
+		(start 144.8308 71.553787)
+		(end 145.784587 70.6)
+		(width 0.2)
+		(layer "F.Cu")
+		(net 10)
+	)
+	(segment
+		(start 144.8308 73.058001)
+		(end 144.8308 71.553787)
+		(width 0.2)
+		(layer "F.Cu")
+		(net 10)
+	)
+	(segment
 		(start 136.63353 90.014201)
 		(end 150.733544 90.014201)
@@
 		(net 10)
 	)
-	(via
-		(at 150.0378 74.5998)
-		(size 0.6)
-		(drill 0.3)
-		(layers "F.Cu" "B.Cu")
-		(net 10)
-	)
 	(segment
 		(start 132.207 88.9508)
@@
 		(width 0.2)
 		(layer "B.Cu")
-		(net 10)
-	)
-	(segment
-		(start 150.0378 74.5998)
-		(end 146.372599 74.5998)
-		(width 0.2)
-		(layer "B.Cu")
-		(net 10)
-	)
-	(segment
-		(start 146.372599 74.5998)
-		(end 144.8308 73.058001)
-		(width 0.2)
-		(layer "B.Cu")

Commit message: label renames
Parts:
- D1: value D -> TS4148 RBG
Connections:
- net PA1 renamed CAN MOSI
- net PA7 renamed Strain
- net PC3 renamed Wheel Speed
- U3 pad 15: PA2 -> CAN MISO
- U3 pad 16: PA4 -> CAN CS
- U5 pad 18: PA2 -> CAN MISO
- U5 pad 2: PA4 -> CAN CS
