File: Telemetry peripheral boards/FS3 Peripheral V4 ATTINY/F3 peripheral boards.kicad_sch (KiCad schematic)
At the start: 48 parts, among them J1 ATS668LSM, J10 Conn_01x10_Pin, J2 Main Connector, J3 Potentiometer, J4 Strain Gauge, J5 Tire temp Sensor, J6 1x1 Tire Air Temp Sensor, J7 1x8 Tire Surface Temp Sensor, J9 Conn_01x10_Pin, U1 LM2907M/NOPB, U2 INA125U, U3 MCP2515-I/SO, U4 ISO1050DUB, U5 ATtiny1616-S, U6 LM7805CV, Y1 STDCSU1-8M

Commit message: changes
Connections:
- net PC3 renamed Wheel Speed
Other:
- note added: "Attiny1616 Microcontroller"
- note removed: "Attiny1616"
- moved on the sheet: C10, C15, C7, D1, J10, R12, R14, R8, U5

Commit message: label renames
Parts:
- J2, J5, J6, J7: symbol Connector_Generic_MountingPin:Conn_01x04_MountingPin -> Connector_Generic:Conn_01x04
- J4: symbol Connector:Conn_01x02_Pin -> Connector_Generic:Conn_01x02
- renumbered C11 to C12, C12 to C14, U6 to U7
Connections:
- net PA1 renamed CAN MOSI
- net PA2 renamed CAN MISO
- net PA3/SCK renamed ATtiny SCK
- net PA4 renamed CAN CS
- net PA6 renamed Potentiometer
- net PA7 renamed Strain
- net PB0 renamed Tire Temp SCL
- net PB1 renamed Tire Temp SDA
- no-connect marks 9 -> 7
Other:
- note added: "ATtiny1616 SOIC 20-Pin Microcontroller"
- note removed: "Attiny1616 Microcontroller"
- moved on the sheet: J3, R15, R8

Commit message: Updated labels, replaced some wiring with labels, changed symbols,
Parts:
- J10, J9: symbol Connector:Conn_01x10_Pin -> Connector_Generic:Conn_01x10
Connections:
- net IN-: now reaches R4.1, R5.1, U1.10 (IN-), U1.5 (EMIT)
- net CAN1_RX renamed CAN Receive
- net CAN Receive: no longer U4.2 (RXD)
- net CAN1_TX renamed CAN Transmit
- new net CAN Recieve: U4.2 (RXD)
Other:
- moved on the sheet: C10, C15, C2, C7, D1, J3, J6, J7, R13, R14, R15, R4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
