File: TelemetryMainFinal/TelemMainFinal/TelemMainFinal.kicad_sch (KiCad schematic)
At the start: 17 parts, among them J1 8 pin ATM connector, J3 12 pin ATM connector, J4 SD to SPI (Molex nanofit), U3 NUCLEO-F446RE, U4 ISO1050DUB

Commit message: Moved nucleo to its own schematic page, cleaned up power distribution page
Parts:
- removed C5: 100nf, Capacitor_SMD:C_0805_2012Metric_Pad1.18x1.45mm_HandSolder, symbol Device:C
- removed D3, D4: QBLP631-R3A, LED_SMD:LED_0805_2012Metric_Pad1.15x1.40mm_HandSolder, symbol Device:LED
- removed R1: 1 kΩ, Resistor_SMD:R_0805_2012Metric_Pad1.20x1.40mm_HandSolder, symbol Device:R_US
- removed R11: 4.7k, Resistor_SMD:R_0805_2012Metric, symbol Device:R_US
- removed R14, R15: 470R 1/4W, Resistor_SMD:R_0805_2012Metric_Pad1.20x1.40mm_HandSolder, symbol Device:R_US
- removed R2: 3 kΩ, Resistor_SMD:R_0805_2012Metric_Pad1.20x1.40mm_HandSolder, symbol Device:R_US
- removed U3: NUCLEO-F446RE, FS_3_Global_Footprint_Library:NUCLEO-F446RE, symbol FS_3_Global_Symbol_Library:NUCLEO-F446RE
Connections:
- no-connect marks 40 -> 8
Other:
- added sheet Nucleo (Nucleo.kicad_sch)
- note removed: "Voltage check"
- moved on the sheet: U8

Commit message: moved can to its own page
Parts:
- removed C7, C8: 100nf, Capacitor_SMD:C_0805_2012Metric_Pad1.18x1.45mm_HandSolder, symbol Device:C
- removed U4: ISO1050DUB, Package_SO:SOP-8_6.62x9.15mm_P2.54mm, symbol Interface_CAN_LIN:ISO1050DUB
Other:
- added sheet CAN (can.kicad_sch)
- note removed: "CAN1 transceiver"

Commit message: moved sd and imu to own pages, cleaned up root page
Parts:
- removed C13: 100nf, Capacitor_SMD:C_0805_2012Metric_Pad1.18x1.45mm_HandSolder, symbol Device:C
- removed J4: SD to SPI (Molex nanofit), Connector_Molex:Molex_Nano-Fit_105310-xx10_2x05_P2.50mm_Vertical, symbol Connector_Generic:Conn_2Rows-09Pins
- removed U8: ~, FS_3_Global_Footprint_Library:Adafruit_E336755_10DoF_IMU, symbol FS_3_Global_Symbol_Library:Adafruit_E336755_10DoF_IMU
Connections:
- no-connect marks 8 -> 5
Other:
- sheet Dash components renamed Dash
- added sheet IMU (imu.kicad_sch)
- added sheet SD (sd.kicad_sch)
- note removed: "<- optional output interrupt/ready pins for the IMU's gyroscope (G) and accelerometer/magnotomer (L1/L2)"
- moved on the sheet: J1, J3
